File: HARDWARE/ETH1CSMU1/Feedback.sch (KiCad schematic (older format))
At the start: 68 parts

Commit message: Added ADC
Parts:
- added C314: C, symbol Device:C
- added Q301, Q302, Q303, Q304: MMBT6429, symbol Device:Q_NPN_BEC
- added Q305, Q306, Q307: Q_NJFET_DGS, symbol Device:Q_NJFET_DGS
- added R328: 14k7, symbol Device:R
- added R329, R333, R334: 21k5, symbol Device:R
- added R330, R331, R332, R337: 2k/0.1%, symbol Device:R
- added R335: 180k/0.1%, symbol Device:R
- added R336: 18k/0.1%, symbol Device:R
- added R338, R339, R340: R, symbol Device:R
- added R341: 10G, symbol Device:R
- added U309: AD746, symbol opamp_local:AD746
- added U310, U313, U315: AD744, symbol opamp_local:AD744
- added U311, U312, U314: AQY221, symbol relay_local:AQY221
- added U316: REF102CU, symbol Reference_Voltage:REF102CU
- added U317: OPA277, symbol opamp_local:OPA277
- U308: renamed from U?; footprint Package_SO:SOIC-8_3.9x4.9mm_P1.27mm -> (none)
- gave numbers to parts that had none: 59
Connections:
- net +15V: now also U301.8 (V+), Q305.1 (D), U310.7 (V+), U313.7 (V+), U315.7 (V+), U316.2 (Vin), U317.7 (V+); no longer U301.8 (V+)
- net +5V: now also U305.1, U306.1, U307.1, U311.1, U312.1, U314.1; no longer U302.1, U303.1, U304.1
- net -15V: now also U301.4 (V-), U309.4 (V-), U310.4 (V-), U313.4 (V-), U315.4 (V-), U317.4 (V-); no longer U301.4 (V-)
- net CurrentBoostOUT: now also U302.4, U303.4, U304.4, R341.2; no longer U305.4, U306.4, U307.4
- net GND: now also U301.5 (+), C314.2, R337.2, U309.8 (V+), U310.3 (+), U316.4 (GND); no longer U301.3 (+)
- net at C301.1, C302.2, R309.1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: now also U301.2 (-); no longer U301.6 (-)
- net at C301.2, R307.1, R309.2: now also U301.1; no longer U301.7
- net CURRENT_FEEDBACK: now reaches R305.2
- net CURRENT_FEEDBACK: now also U301.7; no longer U301.1
- net at R305.1, R307.2: now also U301.6 (-); no longer U301.2 (-)
- net at C303.1, R310.1, R312.2: now also U301.3 (+); no longer U301.5 (+)
- net at K301.5, K302.5, K303.5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: now also R341.1
- net at C307.2, R316.2: now also U302.3; no longer U305.3
- net at R301.1: now also U302.2; no longer U302.2
- net at R317.2: now also U303.3; no longer U305.3
- net at R302.1: now also U303.2; no longer U302.2
- net at U306.3: now also R320.2; no longer R318.2
- net at R303.1: now also U304.2; no longer U303.2
- net at R319.2: now also U305.3; no longer U306.3
- net at R304.1: now also U305.2; no longer U303.2
- net at U307.3: now also R321.2; no longer R320.2
- net at R306.1: now also U306.2; no longer U304.2
- net at R308.1: now also U307.2; no longer U304.2
- net STIMULUS: now reaches K305.5, K306.5, R322.1, R323.1
- net STIMULUS: now also Q306.2 (G)
- net GUARD1: now reaches U308.2
- new net: R318.2, U304.3
- new net: Q301.1 (B), U309.1
- new net: Q303.2 (E), R331.2, R333.2, U309.2 (-)
- new net: R329.1, R330.2, U309.3 (+), U309.5 (+)
- new net: Q304.2 (E), R332.2, R334.2, U309.6 (-)
- new net: Q302.1 (B), U309.7
- new net: R335.2, R336.1, U312.4
- new net: R336.2, R337.1, U314.4
- new net: Q307.2 (G), U311.3, U312.3, U314.3
- new net: R339.1, U312.2
- new net: R340.1, U314.2
- new net: R338.1, U311.2
- new net: R328.1, R329.2, U310.2 (-)
- new net: R330.1, R331.1, R332.1, U310.6
- new net: R328.2, U317.2 (-), U317.6
- new net: Q302.2 (E), Q304.1 (B), R334.1
- new net: Q302.3 (C), Q304.3 (C), Q307.3 (S), U315.2 (-)
- new net: Q301.2 (E), Q303.1 (B), R333.1
- new net: Q301.3 (C), Q303.3 (C), Q306.3 (S), U313.3 (+), U315.3 (+)
- new net: Q305.2 (G), U313.2 (-), U313.6
- new net: Q305.3 (S), Q306.1 (D), Q307.1 (D)
- new net: C314.1, U316.8 (NR)
- new net: U316.6 (Vout), U317.3 (+)
- new net VOLTAGE_FEEDBACK: R335.1, U311.4, U315.6
- no-connect marks 2 -> 13
Other:
- moved on the sheet: C301, C302, C303, C304, C305, C306, C307, C308, C309, C310, C311, C312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

Commit message: Commit
Parts:
- R320: value 100 -> 100/0.5%/2W
- R321: value 10 -> 10/0.5%/2W
Changed lines of the file:
@@
 P 5650 7050
 F 0 "R320" V 5443 7050 50  0000 C CNN
-F 1 "100" V 5534 7050 50  0000 C CNN
+F 1 "100/0.5%/2W" V 5534 7050 50  0000 C CNN
 F 2 "" V 5580 7050 50  0001 C CNN
 F 3 "~" H 5650 7050 50  0001 C CNN
@@
 P 5650 8100
 F 0 "R321" V 5443 8100 50  0000 C CNN
-F 1 "10" V 5534 8100 50  0000 C CNN
+F 1 "10/0.5%/2W" V 5534 8100 50  0000 C CNN
 F 2 "" V 5580 8100 50  0001 C CNN
 F 3 "~" H 5650 8100 50  0001 C CNN

Commit message: Commit
Parts:
- R310, R312, R318: footprint (none) -> SMD:R_0603_Symbol1
Connections:
- net REF+10V: now reaches R328.2, U317.2 (-), U317.6
Other:
- moved on the sheet: C314, D301, D302, D303, K301, K302, K303, U316, U317

Commit message: Footprints
Parts:
- C301, C302: footprint (none) -> SMD:C_0603_Symbol5
- C303, C304, C305, C308, C309, C310, C312: footprint (none) -> Capacitors_SMD:C_0603
- R305, R307, R309, R311, R317, R324: footprint (none) -> SMD:R_0603_Symbol3
Changed lines of the file:
@@
 F 0 "C305" V 5348 3300 50  0000 C CNN
 F 1 "33p" V 5439 3300 50  0000 C CNN
-F 2 "" H 5638 3150 50  0001 C CNN
+F 2 "Capacitors_SMD:C_0603" H 5638 3150 50  0001 C CNN
 F 3 "~" H 5600 3300 50  0001 C CNN
 	1    5600 3300
@@
 F 0 "R311" V 4143 8300 50  0000 C CNN
 F 1 "100k" V 4234 8300 50  0000 C CNN
-F 2 "" V 4280 8300 50  0001 C CNN
+F 2 "SMD:R_0603_Symbol3" V 4280 8300 50  0001 C CNN
 F 3 "~" H 4350 8300 50  0001 C CNN
 	1    4350 8300
@@
 F 0 "C302" V 4098 8650 50  0000 C CNN
 F 1 "15p" V 4189 8650 50  0000 C CNN
-F 2 "" H 4388 8500 50  0001 C CNN
+F 2 "SMD:C_0603_Symbol5" H 4388 8500 50  0001 C CNN
 F 3 "~" H 4350 8650 50  0001 C CNN
 	1    4350 8650
@@
 F 0 "R309" V 3743 8300 50  0000 C CNN
 F 1 "100k" V 3834 8300 50  0000 C CNN
-F 2 "" V 3880 8300 50  0001 C CNN
+F 2 "SMD:R_0603_Symbol3" V 3880 8300 50  0001 C CNN
 F 3 "~" H 3950 8300 50  0001 C CNN
 	1    3950 8300
@@
 F 0 "C301" V 3698 8650 50  0000 C CNN
 F 1 "15p" V 3789 8650 50  0000 C CNN
-F 2 "" H 3988 8500 50  0001 C CNN
+F 2 "SMD:C_0603_Symbol5" H 3988 8500 50  0001 C CNN
 F 3 "~" H 3950 8650 50  0001 C CNN
 	1    3950 8650
@@
 F 0 "C303" H 4665 9546 50  0000 L CNN
 F 1 "39p" H 4665 9455 50  0000 L CNN
-F 2 "" H 4588 9350 50  0001 C CNN
+F 2 "Capacitors_SMD:C_0603" H 4588 9350 50  0001 C CNN
 F 3 "~" H 4550 9500 50  0001 C CNN
 	1    4550 9500
@@
 F 0 "R307" V 2843 9100 50  0000 C CNN
 F 1 "100k" V 2934 9100 50  0000 C CNN
-F 2 "" V 2980 9100 50  0001 C CNN
+F 2 "SMD:R_0603_Symbol3" V 2980 9100 50  0001 C CNN
 F 3 "~" H 3050 9100 50  0001 C CNN
 	1    3050 9100
@@
 F 0 "R305" V 2193 8800 50  0000 C CNN
 F 1 "100k" V 2284 8800 50  0000 C CNN
-F 2 "" V 2330 8800 50  0001 C CNN
+F 2 "SMD:R_0603_Symbol3" V 2330 8800 50  0001 C CNN
 F 3 "~" H 2400 8800 50  0001 C CNN
 	1    2400 8800
@@
 F 0 "C309" H 6165 3146 50  0000 L CNN
 F 1 "68p" H 6165 3055 50  0000 L CNN
-F 2 "" H 6088 2950 50  0001 C CNN
+F 2 "Capacitors_SMD:C_0603" H 6088 2950 50  0001 C CNN
 F 3 "~" H 6050 3100 50  0001 C CNN
 	1    6050 3100
@@
 F 0 "C310" H 6165 4146 50  0000 L CNN
 F 1 "68p" H 6165 4055 50  0000 L CNN
-F 2 "" H 6088 3950 50  0001 C CNN
+F 2 "Capacitors_SMD:C_0603" H 6088 3950 50  0001 C CNN
 F 3 "~" H 6050 4100 50  0001 C CNN
 	1    6050 4100
@@
 F 0 "R317" V 5443 5700 50  0000 C CNN
 F 1 "100k" V 5534 5700 50  0000 C CNN
-F 2 "" V 5580 5700 50  0001 C CNN
+F 2 "SMD:R_0603_Symbol3" V 5580 5700 50  0001 C CNN
 F 3 "~" H 5650 5700 50  0001 C CNN
 	1    5650 5700
@@
 F 0 "C304" V 5348 2300 50  0000 C CNN
 F 1 "8p" V 5439 2300 50  0000 C CNN
-F 2 "" H 5638 2150 50  0001 C CNN
+F 2 "Capacitors_SMD:C_0603" H 5638 2150 50  0001 C CNN
 F 3 "~" H 5600 2300 50  0001 C CNN
 	1    5600 2300
@@
 F 0 "C308" H 6165 2146 50  0000 L CNN
 F 1 "68p" H 6165 2055 50  0000 L CNN
-F 2 "" H 6088 1950 50  0001 C CNN
+F 2 "Capacitors_SMD:C_0603" H 6088 1950 50  0001 C CNN
 F 3 "~" H 6050 2100 50  0001 C CNN
 	1    6050 2100
@@
 F 0 "R324" H 8220 8746 50  0000 L CNN
 F 1 "100k" H 8220 8655 50  0000 L CNN
-F 2 "" V 8080 8700 50  0001 C CNN
+F 2 "SMD:R_0603_Symbol3" V 8080 8700 50  0001 C CNN
 F 3 "~" H 8150 8700 50  0001 C CNN
 	1    8150 8700
@@
 F 0 "C312" H 8715 8746 50  0000 L CNN
 F 1 "33p" H 8715 8655 50  0000 L CNN
-F 2 "" H 8638 8550 50  0001 C CNN
+F 2 "Capacitors_SMD:C_0603" H 8638 8550 50  0001 C CNN
 F 3 "~" H 8600 8700 50  0001 C CNN
 	1    8600 8700

Commit message: Footprint selection
Parts:
- removed K301, K302, K303, K304, K305, K306: CRR05-1A, symbol relay_local:CRR05-1A
- added C315: 470p, symbol Device:C
- added D307: BAV16W, Diodes_SMD:D_SOD-323_HandSoldering, symbol Device:D
- added K301, K302, K303, K304, K305, K306, K307: MS05-1A87-75D, symbol relay_local:MS05-1A87-75D
- added R342: 51, Resistors_SMD:R_0603, symbol Device:R
- added R343: 10k, SMD:R_0603_Symbol1, symbol Device:R
- added R344: 510, Resistors_SMD:R_0603, symbol Device:R
- added U318: AD744, symbol opamp_local:AD744
- C306, C307: footprint (none) -> Capacitors_SMD:C_0603
- D301, D302, D303, D304, D305, D306: value D -> BAV16W; footprint (none) -> Diodes_SMD:D_SOD-323_HandSoldering
- R325, R335, R336, R337: footprint (none) -> Resistors_SMD:R_0603
Connections:
- net +15V: now also U318.7 (V+)
- net +5V: now also D307.1 (K), K301.2, K302.2, K303.2, K304.2, K305.2, K306.2, K307.2
- net -15V: now also U318.4 (V-)
- net GUARD1: now also R342.2, U318.2 (-), U318.6
- net K100mA: now also K305.3
- net K100nA: now also K302.3
- net K10nA: now also K301.3
- net K10uA-10mA: now also K304.3
- net K1A: now also K306.3
- net K1uA: now also K303.3
- net STIMULUS: now also C315.2, K305.4, K306.4
- net at C305.1, C309.1, R314.1: now also K302.1
- net at R312.1, R326.1, R327.1: now also U318.3 (+)
- net at C304.1, C308.1, R313.1: now also K301.1
- net at R322.2, R341.1: now also K301.4, K302.4, K303.4, K304.4
- net at C306.1, C310.1, R315.1: now also K303.1
- net at C307.1, C311.1, R316.1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: now also K304.1
- net at R320.1: now also K305.1
- net at R321.1: now also K306.1
- new net: U318.5, U318.8
- new net: K307.1, R342.1
- new net: K307.4, R343.2
- new net: C315.1, R344.2
- new net GRD_RLY: D307.2 (A), K307.3
- new net GUARD_OUT: R343.1, R344.1
- no-connect marks 13 -> 14
Other:
- moved on the sheet: C314, D301, D302, D303, D304, D305, D306, U316, U317

Commit message: Redesigned feedback circuit.
Parts:
- removed Q301, Q302, Q303, Q304: MMBT6429, symbol Device:Q_NPN_BEC
- removed Q305, Q306, Q307: Q_NJFET_DGS, symbol Device:Q_NJFET_DGS
- removed R328: 14k7, symbol Device:R
- removed R330, R331, R332: 2k/0.1%, symbol Device:R
- removed R333, R334: 21k5, symbol Device:R
- removed U308: ADA4530-1, symbol Amplifier_Operational:ADA4530-1
- removed U309: AD746, symbol opamp_local:AD746
- removed U310, U318: AD744, symbol opamp_local:AD744
- removed U316: REF102CU, symbol Reference_Voltage:REF102CU
- removed U317: OPA277, symbol opamp_local:OPA277
- added C316, C317, C318, C319, C320, C321, C322, C323: 100n, symbol Device:C
- added Q301, Q302, Q303: BC847, Package_TO_SOT_SMD:SOT-23, symbol Transistor_BJT:BC847
- added U311: AD744, Housings_SOIC:SOIC-8_3.9x4.9mm_Pitch1.27mm, symbol opamp_local:AD744
- added U314: ULN2003, symbol Transistor_Array:ULN2003
- C314: value C -> 22p
- K301, K302, K303, K304, K305, K306, K307: footprint (none) -> THT:MS05-1A87-75D_Socket
- R314: renamed from R341; value 10G -> 10G/0.5%
- R315: renamed from R313; value 1G -> 1G/1%
- R316: renamed from R314; value 100Meg -> 100Meg/1%
- R317: renamed from R315; value 9.88Meg -> 10Meg/0.5%
- R318: renamed from R316; value 988k -> 1Meg/0.5%
- R319: renamed from R317; value 100k -> 100k/0.5%
- R320: renamed from R318; value 10k -> 10k/0.5%; footprint SMD:R_0603_Symbol1 -> (none)
- R321: renamed from R319; value 1k -> 1k/0.5%
- R329: value 21k5 -> 10k
- U301, U313: footprint (none) -> Housings_SOIC:SOIC-8_3.9x4.9mm_Pitch1.27mm
- U302, U303, U304, U305, U306, U307: footprint (none) -> SMD:AQY2
- U308: renamed from U311; footprint (none) -> SMD:AQY2
- U309: renamed from U312; footprint (none) -> SMD:AQY2
- U310: renamed from U314; footprint (none) -> SMD:AQY2
- U312: renamed from U315; footprint (none) -> Housings_SOIC:SOIC-8_3.9x4.9mm_Pitch1.27mm
- renumbered R305 to R302, R302 to R303, R307 to R304, R303 to R305, R304 to R306, R309 to R307, R310 to R308, R306 to R309, R311 to R310, R312 to R311, R308 to R312, R338 to R313, R320 to R322, R321 to R323, R339 to R324, R340 to R325, R322 to R326, R323 to R327, R324 to R328, R325 to R330, R326 to R331, R335 to R332, R336 to R333, R337 to R334, R327 to R335, R342 to R336, R343 to R337, R344 to R338
Connections:
- net +15V: now also C316.1, C317.1, C318.1, C319.1, C320.1, C321.1, C322.1, C323.1, U311.7 (V+)
- net +5V: now also U314.9 (COM)
- net -15V: now also U311.4 (V-)
- net GND: now also C316.2, C317.2, C318.2, C319.2, C320.2, C321.2, C322.2, C323.2, Q301.2 (E), Q302.2 (E), Q303.2 (E), U314.8 (GND); no longer C314.2
- net GUARD1: now also U313.2 (-), U313.6
- net STIMULUS: now also R329.2
- net at R311.1, R331.1, R335.1: now also U313.3 (+)
- net at R329.1: now also U312.3 (+)
- net at U308.3, U309.3, U310.3: now also U312.2 (-)
- net U10uA: now reaches R301.2
- net U10uA: now also U314.11 (O6)
- net U100uA: now reaches R303.2
- net U100uA: now also U314.12 (O5)
- net U1mA: now reaches R305.2
- net U1mA: now also U314.13 (O4)
- net U10mA: now reaches R306.2
- net U10mA: now also U314.14 (O3)
- net U100mA: now reaches R309.2
- net U100mA: now also U314.15 (O2)
- net U1A: now reaches R312.2
- net U1A: now also U314.16 (O1)
- net at R330.1: now also U311.3 (+)
- net at C313.1, R335.2: now also U311.6
- net at C313.2, R331.2: now also U311.2 (-)
- net at U313.5: now also C314.1
- net at U313.8: now also C314.2
- net at R313.2: now also Q301.3 (C)
- net at R324.2: now also Q302.3 (C)
- net at R325.2: now also Q303.3 (C)
- new net MCU_U100mA: U314.2 (I2)
- new net MCU_U100uA: U314.5 (I5)
- new net MCU_U10mA: U314.3 (I3)
- new net MCU_U10uA: U314.6 (I6)
- new net MCU_U1A: U314.1 (I1)
- new net MCU_U1mA: U314.4 (I4)
- new net VF_GAIN1: Q301.1 (B)
- new net VF_GAIN10: Q302.1 (B)
- new net VF_GAIN100: Q303.1 (B)
- no-connect marks 14 -> 9
Other:
- note added: "TE 6-5330808-5 - sockets"
- moved on the sheet: C301, C302, C303, C304, C305, C306, C307, C308, C309, C310, C311, C312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

Commit message: Added MUX schematic
Parts:
- removed U314: ULN2003, symbol Transistor_Array:ULN2003
- added Q304, Q305, Q306, Q307, Q308, Q309: BC847, Package_TO_SOT_SMD:SOT-23, symbol Transistor_BJT:BC847
- added U314: ULN2002, symbol Transistor_Array:ULN2002
- C311, C313, C314, C315: footprint (none) -> Capacitors_SMD:C_0603
- C316, C317, C318, C319, C320, C321, C322, C323: footprint (none) -> SMD:C_0603_Symbol1
Connections:
- net +5V: now also U314.9 (COM)
- net GND: now also Q304.2 (E), Q305.2 (E), Q306.2 (E), Q307.2 (E), Q308.2 (E), Q309.2 (E), U314.8 (GND)
- net K100mA: now also U314.15 (O2)
- net K100nA: now also U314.12 (O5)
- net K10nA: now also U314.11 (O6)
- net K10uA-10mA: now also U314.14 (O3)
- net K1A: now also U314.16 (O1)
- net K1uA: now also U314.13 (O4)
- net MCU_U100mA: now also Q304.1 (B)
- net MCU_U100uA: now also Q309.1 (B)
- net MCU_U10mA: now also Q308.1 (B)
- net MCU_U10uA: now also Q306.1 (B)
- net MCU_U1A: now also Q307.1 (B)
- net MCU_U1mA: now also Q305.1 (B)
- net U100mA: no longer names the net of R309.2
- net U100mA: now also Q304.3 (C)
- net U100uA: no longer names the net of R303.2
- net U100uA: now also Q309.3 (C)
- net U10mA: no longer names the net of R306.2
- net U10mA: now also Q308.3 (C)
- net U10uA: no longer names the net of R301.2
- net U10uA: now also Q306.3 (C)
- net U1A: no longer names the net of R312.2
- net U1A: now also Q307.3 (C)
- net U1mA: no longer names the net of R305.2
- net U1mA: now also Q305.3 (C)
- new net MCU_K100mA: U314.2 (I2)
- new net MCU_K100nA: U314.5 (I5)
- new net MCU_K10nA: U314.6 (I6)
- new net MCU_K10uA-10mA: U314.3 (I3)
- new net MCU_K1A: U314.1 (I1)
- new net MCU_K1uA: U314.4 (I4)
Other:
- moved on the sheet: Q301, Q302, Q303, R301, R303, R305, R306, R309, R312, R313, R324, R325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
