File: HARDWARE/ETH1CSMU1/FGEN.sch (KiCad schematic (older format))
At the start: 35 parts, among them U501 REF5025AD

Commit message: Added ADC
Parts:
- U501: footprint Package_SO:SOIC-8_3.9x4.9mm_P1.27mm -> (none)
- U602: renamed from U?; footprint Package_SO:TSSOP-20_4.4x6.5mm_P0.65mm -> (none)
- gave numbers to parts that had none: 30

Commit message: Commit
Parts:
- C602, C607, C610, C611, C612: footprint (none) -> SMD:C_0603_Symbol1
Changed lines of the file:
@@
 F 0 "C602" H 2185 3754 50  0000 R CNN
 F 1 "100n" H 2185 3845 50  0000 R CNN
-F 2 "" H 2338 3650 50  0001 C CNN
+F 2 "SMD:C_0603_Symbol1" H 2338 3650 50  0001 C CNN
 F 3 "~" H 2300 3800 50  0001 C CNN
 	1    2300 3800
@@
 F 0 "C607" H 5115 7346 50  0000 L CNN
 F 1 "100n" H 5115 7255 50  0000 L CNN
-F 2 "" H 5038 7150 50  0001 C CNN
+F 2 "SMD:C_0603_Symbol1" H 5038 7150 50  0001 C CNN
 F 3 "~" H 5000 7300 50  0001 C CNN
 	1    5000 7300
@@
 F 0 "C610" H 5565 7346 50  0000 L CNN
 F 1 "100n" H 5565 7255 50  0000 L CNN
-F 2 "" H 5488 7150 50  0001 C CNN
+F 2 "SMD:C_0603_Symbol1" H 5488 7150 50  0001 C CNN
 F 3 "~" H 5450 7300 50  0001 C CNN
 	1    5450 7300
@@
 F 0 "C611" H 6015 7346 50  0000 L CNN
 F 1 "100n" H 6015 7255 50  0000 L CNN
-F 2 "" H 5938 7150 50  0001 C CNN
+F 2 "SMD:C_0603_Symbol1" H 5938 7150 50  0001 C CNN
 F 3 "~" H 5900 7300 50  0001 C CNN
 	1    5900 7300
@@
 F 0 "C612" H 6465 7346 50  0000 L CNN
 F 1 "100n" H 6465 7255 50  0000 L CNN
-F 2 "" H 6388 7150 50  0001 C CNN
+F 2 "SMD:C_0603_Symbol1" H 6388 7150 50  0001 C CNN
 F 3 "~" H 6350 7300 50  0001 C CNN
 	1    6350 7300

Commit message: Footprints
Parts:
- C609, C613, C614, C615, C616: footprint (none) -> Capacitors_SMD:C_0603
- R606: footprint (none) -> SMD:R_0603_Symbol3
Changed lines of the file:
@@
 F 0 "C613" H 6765 4746 50  0000 L CNN
 F 1 "1p5" H 6765 4655 50  0000 L CNN
-F 2 "" H 6688 4550 50  0001 C CNN
+F 2 "Capacitors_SMD:C_0603" H 6688 4550 50  0001 C CNN
 F 3 "~" H 6650 4700 50  0001 C CNN
 	1    6650 4700
@@
 F 0 "C614" V 8498 4100 50  0000 C CNN
 F 1 "1p5" V 8589 4100 50  0000 C CNN
-F 2 "" H 8788 3950 50  0001 C CNN
+F 2 "Capacitors_SMD:C_0603" H 8788 3950 50  0001 C CNN
 F 3 "~" H 8750 4100 50  0001 C CNN
 	1    8750 4100
@@
 F 0 "R606" V 5243 1650 50  0000 C CNN
 F 1 "100k" V 5334 1650 50  0000 C CNN
-F 2 "" V 5380 1650 50  0001 C CNN
+F 2 "SMD:R_0603_Symbol3" V 5380 1650 50  0001 C CNN
 F 3 "~" H 5450 1650 50  0001 C CNN
 	1    5450 1650
@@
 F 0 "C609" V 5198 1300 50  0000 C CNN
 F 1 "1000p" V 5289 1300 50  0000 C CNN
-F 2 "" H 5488 1150 50  0001 C CNN
+F 2 "Capacitors_SMD:C_0603" H 5488 1150 50  0001 C CNN
 F 3 "~" H 5450 1300 50  0001 C CNN
 	1    5450 1300
@@
 F 0 "C615" H 9915 5446 50  0000 L CNN
 F 1 "33p" H 9915 5355 50  0000 L CNN
-F 2 "" H 9838 5250 50  0001 C CNN
+F 2 "Capacitors_SMD:C_0603" H 9838 5250 50  0001 C CNN
 F 3 "~" H 9800 5400 50  0001 C CNN
 	1    9800 5400
@@
 F 0 "C616" H 10415 5446 50  0000 L CNN
 F 1 "150p" H 10415 5355 50  0000 L CNN
-F 2 "" H 10338 5250 50  0001 C CNN
+F 2 "Capacitors_SMD:C_0603" H 10338 5250 50  0001 C CNN
 F 3 "~" H 10300 5400 50  0001 C CNN
 	1    10300 5400

Commit message: Footprint selection
Changed lines of the file:
@@
 	2800 1100 3350 1100
 Connection ~ 3350 1650
+Text HLabel 1950 4600 0    50   Input ~ 0
+FGEN_RESET
 $EndSCHEMATC

Commit message: Redesigned feedback circuit.
Parts:
- removed U606, U607: LT1677, symbol opamp_local:LT1677
- added U601: LT1801, Housings_SOIC:SOIC-8_3.9x4.9mm_Pitch1.27mm, symbol opamp_local:LT1801
- R601, R602, R603, R604, R605, R607, R608, R609, R610: footprint (none) -> Resistors_SMD:R_0603
- U501: footprint (none) -> Housings_SOIC:SOIC-8_3.9x4.9mm_Pitch1.27mm
- U603: renamed from U602; footprint (none) -> Housings_SSOP:SSOP-20_4.4x6.5mm_Pitch0.65mm
- U604: renamed from U603; footprint (none) -> Housings_SSOP:MSOP-8_3x3mm_Pitch0.65mm
- U605: renamed from U604; footprint (none) -> Housings_SOIC:SOIC-8_3.9x4.9mm_Pitch1.27mm
- U606: renamed from U605; value AD5452_MSOP -> AD5452; footprint (none) -> Housings_SSOP:MSOP-8_3x3mm_Pitch0.65mm
Connections:
- net +15V: now also U601.8 (V+)
- net -15V: now also U601.4 (V-)
- net GND: now also U601.3 (+), U601.5 (+)
- net at C613.2, U606.1 (IOUT): now also U601.2 (-)
- net at C613.1, R608.2, U606.8 (RFB): now also U601.1
- net at C614.2, R607.1, R608.1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: now also U601.6 (-)
- net at C614.1, R609.1, R610.2: now also U601.7
- no-connect marks 8 -> 6

Commit message: Schematic development
Parts:
- added C509, C511, C513, C514: 100n, SMD:C_0603_Symbol1, symbol Device:C
- renumbered C607 to C501, C501 to C502, C610 to C503, C602 to C504, C503 to C505, C611 to C506, C504 to C507, C612 to C508, C605 to C510, C606 to C512, C608 to C515, C609 to C516, C613 to C517, C614 to C518, C615 to C519, C616 to C520, L601 to L501, R601 to R501, R602 to R502, R603 to R503, R604 to R504, R605 to R505, R606 to R506, R607 to R507, R608 to R508, R609 to R509, R610 to R510, U601 to U501, U501 to U502, U603 to U503, U604 to U504, U605 to U505, U606 to U506, X601 to X501
Connections:
- net +15V: now also C509.1, C511.1, C513.1, C514.1
- net GND: now also C509.2, C511.2, C513.2, C514.2
Other:
- moved on the sheet: C501, C503, C506, C508
