File: HARDWARE/ETH1CSMU1/Feed-ForwardCurrentBooster.sch (KiCad schematic (older format))
At the start: 49 parts, among them Q501 MMBF5486, Q502 MMBT200, Q503 SMBT2222, Q504 SMBT2222, Q505 SMBT2222, Q506 MMBT200, Q507 BCP56-16, Q508 BCP53, Q509 BCP56-16, Q510 BCP53, Q511 BCP56-16, Q512 BCP53, Q513 BCP56-16, Q514 BCP53, U501 AD744

Commit message: Added MUX schematic
Parts:
- R513: footprint (none) -> Resistors_SMD:R_0603
- R515, R516, R517, R518, R519, R520, R521, R522: footprint (none) -> Resistors_SMD:R_2512
Changed lines of the file:
@@
 $Descr A4 11693 8268
 encoding utf-8
-Sheet 5 13
+Sheet 5 14
 Title ""
 Date ""
@@
 F 0 "R515" H 7170 3596 50  0000 L CNN
 F 1 "10/2W" H 7170 3505 50  0000 L CNN
-F 2 "" V 7030 3550 50  0001 C CNN
+F 2 "Resistors_SMD:R_2512" V 7030 3550 50  0001 C CNN
 F 3 "~" H 7100 3550 50  0001 C CNN
 	1    7100 3550
@@
 F 0 "R516" H 7170 3996 50  0000 L CNN
 F 1 "10/2W" H 7170 3905 50  0000 L CNN
-F 2 "" V 7030 3950 50  0001 C CNN
+F 2 "Resistors_SMD:R_2512" V 7030 3950 50  0001 C CNN
 F 3 "~" H 7100 3950 50  0001 C CNN
 	1    7100 3950
@@
 F 0 "R513" V 4993 2900 50  0000 C CNN
 F 1 "33" V 5084 2900 50  0000 C CNN
-F 2 "" V 5130 2900 50  0001 C CNN
+F 2 "Resistors_SMD:R_0603" V 5130 2900 50  0001 C CNN
 F 3 "~" H 5200 2900 50  0001 C CNN
 	1    5200 2900
@@
 F 0 "R517" H 8070 3596 50  0000 L CNN
 F 1 "10/2W" H 8070 3505 50  0000 L CNN
-F 2 "" V 7930 3550 50  0001 C CNN
+F 2 "Resistors_SMD:R_2512" V 7930 3550 50  0001 C CNN
 F 3 "~" H 8000 3550 50  0001 C CNN
 	1    8000 3550
@@
 F 0 "R518" H 8070 3996 50  0000 L CNN
 F 1 "10/2W" H 8070 3905 50  0000 L CNN
-F 2 "" V 7930 3950 50  0001 C CNN
+F 2 "Resistors_SMD:R_2512" V 7930 3950 50  0001 C CNN
 F 3 "~" H 8000 3950 50  0001 C CNN
 	1    8000 3950
@@
 F 0 "R519" H 8970 3596 50  0000 L CNN
 F 1 "10/2W" H 8970 3505 50  0000 L CNN
-F 2 "" V 8830 3550 50  0001 C CNN
+F 2 "Resistors_SMD:R_2512" V 8830 3550 50  0001 C CNN
 F 3 "~" H 8900 3550 50  0001 C CNN
 	1    8900 3550
@@
 F 0 "R520" H 8970 3996 50  0000 L CNN
 F 1 "10/2W" H 8970 3905 50  0000 L CNN
-F 2 "" V 8830 3950 50  0001 C CNN
+F 2 "Resistors_SMD:R_2512" V 8830 3950 50  0001 C CNN
 F 3 "~" H 8900 3950 50  0001 C CNN
 	1    8900 3950
@@
 F 0 "R521" H 9870 3596 50  0000 L CNN
 F 1 "10/2W" H 9870 3505 50  0000 L CNN
-F 2 "" V 9730 3550 50  0001 C CNN
+F 2 "Resistors_SMD:R_2512" V 9730 3550 50  0001 C CNN
 F 3 "~" H 9800 3550 50  0001 C CNN
 	1    9800 3550
@@
 F 0 "R522" H 9870 3996 50  0000 L CNN
 F 1 "10/2W" H 9870 3905 50  0000 L CNN
-F 2 "" V 9730 3950 50  0001 C CNN
+F 2 "Resistors_SMD:R_2512" V 9730 3950 50  0001 C CNN
 F 3 "~" H 9800 3950 50  0001 C CNN
 	1    9800 3950

Commit message: Schematic development
Parts:
- D401: renamed from D501; value 1N4148WS -> BAV16WS
- D402: renamed from D502; value 1N4148WS -> BAV16WS
- renumbered C501 to C401, C502 to C402, C503 to C403, C504 to C404, C505 to C405, C506 to C406, C507 to C407, C508 to C408, C509 to C409, C510 to C410, Q501 to Q401, Q502 to Q402, Q503 to Q403, Q504 to Q404, Q505 to Q405, Q506 to Q406, Q507 to Q407, Q508 to Q408, Q509 to Q409, Q510 to Q410, Q511 to Q411, Q512 to Q412, Q513 to Q413, Q514 to Q414, R501 to R401, R502 to R402, R503 to R403, R504 to R404, R505 to R405, R506 to R406, R507 to R407, R508 to R408, R509 to R409, R510 to R410, R511 to R411, R512 to R412, R513 to R413, R514 to R414, R515 to R415, R516 to R416, R517 to R417, R518 to R418, R519 to R419, R520 to R420, R521 to R421, R522 to R422, U501 to U401
