File: HARDWARE/ETH1CSMU1/ADC.sch (KiCad schematic (older format))
At the start: 25 parts, among them U1201 AD746, U1202 LTC6655-5, U1203 LTC2512-24, U1204 OP07, U1205 ADG5204_TSSOP

Commit message: Commit
Parts:
- C1201, C1204, C1205, C1206, C1207, C1208, C1209, C1210, C1211: footprint (none) -> SMD:C_0603_Symbol1
- R1204, R1205, R1207, R1208: footprint (none) -> SMD:R_0603_Symbol1
Connections:
- net GND: no longer U1205.11 (S3)
- net C_FEEDBACK renamed REF+10V
- net V_FEEDBACK renamed CURRENT_FEEDBACK
- new net VOLTAGE_FEEDBACK: U1205.11 (S3)
Other:
- moved on the sheet: C1201, C1202, C1203, R1202, R1203, R1204, R1205, R1206, R1207, R1208, U1201A, U1201B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

Commit message: Footprints
Parts:
- C1203: footprint (none) -> Capacitors_SMD:C_0603
Changed lines of the file:
@@
 F 0 "C1203" H 5115 2996 50  0000 L CNN
 F 1 "1n2" H 5115 2905 50  0000 L CNN
-F 2 "" H 5038 2800 50  0001 C CNN
+F 2 "Capacitors_SMD:C_0603" H 5038 2800 50  0001 C CNN
 F 3 "~" H 5000 2950 50  0001 C CNN
 	1    5000 2950

Commit message: Footprint selection
Parts:
- R1201, R1202, R1203, R1206: footprint (none) -> Resistors_SMD:R_0603
Changed lines of the file:
@@
 F 0 "R1202" V 5093 2750 50  0000 C CNN
 F 1 "10" V 5184 2750 50  0000 C CNN
-F 2 "" V 5230 2750 50  0001 C CNN
+F 2 "Resistors_SMD:R_0603" V 5230 2750 50  0001 C CNN
 F 3 "~" H 5300 2750 50  0001 C CNN
 	1    5300 2750
@@
 F 0 "R1201" H 1120 1596 50  0000 L CNN
 F 1 "R" H 1120 1505 50  0000 L CNN
-F 2 "" V 980 1550 50  0001 C CNN
+F 2 "Resistors_SMD:R_0603" V 980 1550 50  0001 C CNN
 F 3 "~" H 1050 1550 50  0001 C CNN
 	1    1050 1550
@@
 F 0 "R1203" V 6993 2400 50  0000 C CNN
 F 1 "2k49" V 7084 2400 50  0000 C CNN
-F 2 "" V 7130 2400 50  0001 C CNN
+F 2 "Resistors_SMD:R_0603" V 7130 2400 50  0001 C CNN
 F 3 "~" H 7200 2400 50  0001 C CNN
 	1    7200 2400
@@
 F 0 "R1206" V 7393 3550 50  0000 C CNN
 F 1 "2k49" V 7484 3550 50  0000 C CNN
-F 2 "" V 7530 3550 50  0001 C CNN
+F 2 "Resistors_SMD:R_0603" V 7530 3550 50  0001 C CNN
 F 3 "~" H 7600 3550 50  0001 C CNN
 	1    7600 3550

Commit message: Redesigned feedback circuit.
Parts:
- U1201, U1204: footprint (none) -> Housings_SOIC:SOIC-8_3.9x4.9mm_Pitch1.27mm
- U1202: footprint (none) -> Housings_SSOP:MSOP-8_3x3mm_Pitch0.65mm
- U1203: footprint (none) -> Housings_DFN_QFN:DFN-24-1EP_4x7mm_Pitch0.5mm
- U1205: footprint (none) -> Housings_SSOP:TSSOP-14_4.4x5mm_Pitch0.65mm
Connections:
- net REF+10V: no longer names the net of U1205.4 (S1)
Changed lines of the file:
@@
 F 0 "U1203" H 4400 4450 50  0000 C CNN
 F 1 "LTC2512-24" H 4400 4350 50  0000 C CNN
-F 2 "" H 2900 2650 50  0001 L CNN
+F 2 "Housings_DFN_QFN:DFN-24-1EP_4x7mm_Pitch0.5mm" H 2900 2650 50  0001 L CNN
 F 3 "" H 4050 2550 50  0001 C CNN
 	1    3850 3600
@@
 F 0 "U1201" H 600 7050 50  0000 C CNN
 F 1 "AD746" H 600 6950 50  0000 C CNN
-F 2 "" H 1000 7000 60  0001 C CNN
+F 2 "Housings_SOIC:SOIC-8_3.9x4.9mm_Pitch1.27mm" H 1000 7000 60  0001 C CNN
 F 3 "" H 1000 7000 60  0000 C CNN
 	3    900  7000
@@
 F 0 "U1201" H 6300 3000 50  0000 C CNN
 F 1 "AD746" H 6300 2900 50  0000 C CNN
-F 2 "" H 6150 2750 60  0001 C CNN
+F 2 "Housings_SOIC:SOIC-8_3.9x4.9mm_Pitch1.27mm" H 6150 2750 60  0001 C CNN
 F 3 "" H 6150 2750 60  0000 C CNN
 	2    6050 2750
@@
 F 0 "U1201" H 7150 3100 50  0000 L CNN
 F 1 "AD746" H 7150 3000 50  0000 L CNN
-F 2 "" H 7150 2850 60  0001 C CNN
+F 2 "Housings_SOIC:SOIC-8_3.9x4.9mm_Pitch1.27mm" H 7150 2850 60  0001 C CNN
 F 3 "" H 7150 2850 60  0000 C CNN
 	1    7050 2850
@@
 F 0 "U1202" H 2400 2215 50  0000 C CNN
 F 1 "LTC6655-5" H 2400 2124 50  0000 C CNN
-F 2 "" H 2400 1975 60  0001 C CNN
+F 2 "Housings_SSOP:MSOP-8_3x3mm_Pitch0.65mm" H 2400 1975 60  0001 C CNN
 F 3 "" H 2400 1975 60  0000 C CNN
 	1    2400 1850
@@
 F 0 "U1204" H 8300 3800 50  0000 C CNN
 F 1 "OP07" H 8300 3700 50  0000 C CNN
-F 2 "" H 8200 3600 50  0001 C CNN
+F 2 "Housings_SOIC:SOIC-8_3.9x4.9mm_Pitch1.27mm" H 8200 3600 50  0001 C CNN
 F 3 "http://www.analog.com/media/en/technical-documentation/data-sheets/OP07.pdf" H 8200 3700 50  0001 C CNN
 	1    8150 3550
@@
 F 0 "U1205" H 9800 3915 50  0000 C CNN
 F 1 "ADG5204_TSSOP" H 9800 3824 50  0000 C CNN
-F 2 "" H 9800 3800 50  0001 C CNN
+F 2 "Housings_SSOP:TSSOP-14_4.4x5mm_Pitch0.65mm" H 9800 3800 50  0001 C CNN
 F 3 "" H 9800 3800 50  0001 C CNN
 	1    9800 3300
@@
 Wire Wire Line
 	1050 1750 1050 1800
-Text HLabel 10300 2950 2    50   Input ~ 0
-REF+10V
 Wire Wire Line
 	10250 3250 10350 3250
-Wire Wire Line
-	10300 2950 10250 2950
 $EndSCHEMATC

Commit message: Added MUX schematic
Parts:
- added R1209: 10k, SMD:R_0603_Symbol1, symbol Device:R
Connections:
- net at U1205.4 (S1): now also R1209.1
- net at C1202.1, R1207.1, U1202.6 (VOUT_S)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: now also R1209.2
Changed lines of the file:
@@
 $Descr A4 11693 8268
 encoding utf-8
-Sheet 12 13
+Sheet 12 14
 Title ""
 Date ""
@@
 Wire Wire Line
 	10250 3250 10350 3250
+Wire Wire Line
+	10250 2950 10350 2950
+Wire Wire Line
+	10350 2950 10350 1750
+$Comp
+L Device:R R1209
+U 1 1 5C4660B2
+P 9550 1750
+F 0 "R1209" V 9343 1750 50  0000 C CNN
+F 1 "10k" V 9434 1750 50  0000 C CNN
+F 2 "SMD:R_0603_Symbol1" V 9480 1750 50  0001 C CNN
+F 3 "~" H 9550 1750 50  0001 C CNN
+	1    9550 1750
+	0    1    1    0
+$EndComp
+Wire Wire Line
+	9400 1750 8600 1750
+Connection ~ 8600 1750
+Wire Wire Line
+	9700 1750 10350 1750
 $EndSCHEMATC

Commit message: Schematic development
Parts:
- removed U1201: AD746, Housings_SOIC:SOIC-8_3.9x4.9mm_Pitch1.27mm, symbol opamp_local:AD746
- added C1103, C1104, C1106, C1113, C1114, C1115, C1116, C1118, C1119, C1120: 100n, SMD:C_0603_Symbol1, symbol Device:C
- added C1122: 15p, SMD:C_0603_Symbol5, symbol Device:C
- added R1109, R1110, R1111, R1112: 10k, SMD:R_0603_Symbol1, symbol Device:R
- added U1101, U1102: LT1801, Housings_SOIC:SOIC-8_3.9x4.9mm_Pitch1.27mm, symbol opamp_local:LT1801
- added U1104, U1105: ADG419BN, Package_DIP:DIP-8_W7.62mm, symbol Analog_Switch:ADG419BN
- added U1109: SN74LVC1T45, SMD:SC70-6, symbol logic_local:SN74LVC1T45
- renumbered C1201 to C1101, C1202 to C1102, C1203 to C1105, C1204 to C1107, C1207 to C1108, C1205 to C1109, C1208 to C1110, C1206 to C1111, C1209 to C1112, C1210 to C1117, C1211 to C1121, D1201 to D1101, R1201 to R1101, R1202 to R1102, R1203 to R1103, R1204 to R1104, R1205 to R1105, R1206 to R1106, R1207 to R1107, R1208 to R1108, R1209 to R1113, U1202 to U1103, U1203 to U1106, U1204 to U1107, U1205 to U1108
Connections:
- net +15V: now also C1104.1, C1113.1, C1115.1, U1101.8 (V+), U1102.8 (V+), U1104.4 (V+), U1105.4 (V+)
- net +3V3: now also C1119.1, U1109.1 (VCCA)
- net -15V: now also C1103.1, C1106.1, C1114.1, U1101.4 (V-), U1102.4 (V-), U1104.7 (V-), U1105.7 (V-)
- net GND: now also C1103.2, C1104.2, C1106.2, C1113.2, C1114.2, C1115.2, C1116.2, C1118.2, C1119.2, C1120.2, U1101.3 (+), U1101.5 (+), U1104.3 (GND), U1105.3 (GND), U1109.2 (GND), U1109.5 (DIR)
- net at U1108.6 (D): now also U1105.1; no longer R1105.2
- net at R1102.2: now also U1102.6 (-), U1102.7
- net at R1103.1: now also U1102.1, U1102.5 (+)
- net at R1103.2, R1104.1: now also U1102.2 (-)
- net at R1105.1, R1106.1: now also U1102.3 (+)
- new net: R1105.2, U1104.1
- new net: R1109.1, U1101.7, U1104.2
- new net: U1104.6, U1105.6, U1109.4 (B)
- new net: U1104.8, U1105.8
- new net: R1112.2, U1105.2
- new net: C1122.2, R1111.2, R1112.1, U1101.2 (-)
- new net: C1122.1, R1110.2, R1111.1, U1101.1
- new net: R1109.2, R1110.1, U1101.6 (-)
- new net +5V: C1116.1, C1118.1, C1120.1, U1104.5 (VL), U1105.5 (VL), U1109.6 (VCCB)
- new net ADC_DIS_LPF: U1109.3 (A)
Other:
- moved on the sheet: C1101, C1102, C1105, C1107, C1108, C1109, C1110, C1111, C1112, C1117, C1121, D1101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

Commit message: Changed BUS mux schematic
Other:
- moved on the sheet: C1101, C1102, C1103, C1104, C1105, C1106, C1107, C1108, C1109, C1110, C1111, C1112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
