File: HARDWARE/ETH1CSMU1/ADC.sch (KiCad schematic (older format))
At the start: 45 parts, among them U1101 LT1801, U1102 LT1801, U1103 LTC6655-5, U1104 ADG419BN, U1105 ADG419BN, U1106 LTC2512-24, U1107 OP07, U1108 ADG5204_TSSOP, U1109 SN74LVC1T45

Commit message: Check in
Parts:
- C1102: footprint (none) -> SMD:C_1206_Symbol1
Changed lines of the file:
@@
 F 0 "C1102" H 3515 3696 50  0000 L CNN
 F 1 "10u" H 3515 3605 50  0000 L CNN
-F 2 "" H 3438 3500 50  0001 C CNN
+F 2 "SMD:C_1206_Symbol1" H 3438 3500 50  0001 C CNN
 F 3 "~" H 3400 3650 50  0001 C CNN
 	1    3400 3650

Commit message: Added test circuits, bug fix.
Parts:
- removed U1104, U1105: ADG419BN, Package_DIP:DIP-8_W7.62mm, symbol Analog_Switch:ADG419BN
- added U1102, U1105: ADG419BRM, Package_SO:MSOP-8_3x3mm_P0.65mm, symbol Analog_Switch:ADG419BRM
- renumbered C1122 to C1103, C1105 to C1104, C1103 to C1105, C1108 to C1107, C1110 to C1108, C1112 to C1109, C1114 to C1110, C1117 to C1111, C1119 to C1112, C1104 to C1113, C1107 to C1114, C1109 to C1115, C1111 to C1116, C1113 to C1117, C1115 to C1118, C1116 to C1119, C1118 to C1120, C1120 to C1121, C1121 to C1122, R1113 to R1102, R1109 to R1103, R1103 to R1104, R1104 to R1105, R1111 to R1106, R1112 to R1107, R1102 to R1108, R1110 to R1109, R1105 to R1110, R1107 to R1111, R1106 to R1112, R1108 to R1113, U1103 to U1101, U1102 to U1103, U1101 to U1104, U1108 to U1106, U1106 to U1108
Connections:
- net +15V: now also U1102.4 (V+), U1105.4 (V+)
- net +5V: now also U1102.5 (VL), U1105.5 (VL)
- net -15V: now also U1102.7 (V-), U1105.7 (V-)
- net GND: now also U1102.3 (GND), U1105.3 (GND)
- net at U1106.6 (D): now also U1102.1
- net at R1110.2: now also U1105.1
- net at R1103.1, U1104.7: now also U1105.2
- net at U1109.4 (B): now also U1102.6, U1105.6
- net at R1107.2: now also U1102.2
- new net: U1102.8, U1105.8
