File: HARDWARE/ETH1CSMU1/ETH1CSMU1.kicad_pcb (KiCad board)
At the start: 2 copper layers, 694 parts, among them J1001 C96ABC, J1301 Conn_01x03, J201 Conn_02x05, J601 Conn_02x05, K1301 G6KU-2F-Y, K1302 G6KU-2F-Y, K1303 G6KU-2F-Y, K1304 G6KU-2F-Y, K1401 MS05-1A87-75D, K1402 MS05-1A87-75D, K1403 MS05-1A87-75D, K1404 MS05-1A87-75D, K1405 MS05-1A87-75D, K1406 MS05-1A87-75D, K1407 MS05-1A87-75D, Q1201 IRFR5410, Q1202 Si7456DP, Q1203 SI7850DP, Q1204 FDMC5614P, Q1205 FDMC5614P, Q403 SMBT2222, Q404 SMBT2222, Q405 SMBT2222, Q407 BCP56-16, Q408 BCP53, Q409 BCP56-16, Q410 BCP53, Q411 BCP56-16, Q412 BCP53, Q413 BCP56-16, Q414 BCP53, U1101 LT1801, U1102 LT1801, U1103 LTC6655-5, U1106 LTC2512-24, U1107 OP07, U1108 ADG5204_TSSOP, U1109 SN74LVC1T45, U1201 MAX5902, U1202 TEN 40-2415N, U1203 LT3758, U1204 LT3758, U1205 LTC3864, U1206 LTC3864, U1207 NCP1117-ADJ_TO252, U1208 LM337_TO252, U1209 NCP1117-3.3_TO252, U1210 NCP1117-3.3_TO252, U1211 NCP1117-5.0_TO252, U1301 AQY221, U1302 AQY221, U1303 AQY221, U1304 AQY221, U1305 AQY221, U1306 AQY221, U1307 AQY221, U1308 AQY221, U1309 TCA9534, U1310 ADG3308, U1311 AQY221, U1312 AQY221, U1313 AQY221, U1314 AQY221, U1315 AQY221, U1316 AQY221, U1317 AQY221, U1318 AQY221, U1319 AQY221, U1320 TCA9534, U1321 ADG3308, U1322 AQY221, U1323 TCA9534, U1324 ADG3308, U1325 SN74LVC1T45, U1326 SN74LVC1T45, U1401 AQY221, U1402 AQY221, U1403 AD746, U1404 AQY221, U1405 AQY221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

Commit message: Added test circuits, bug fix.
Parts:
- added C1601: 100n, SMD:C_0603_Symbol1, F.Cu at (208.3, 92.4)
- added C1602: 100n, SMD:C_0603_Symbol1, F.Cu at (208.3, 93.7)
- added C1603: 100n, SMD:C_0603_Symbol1, F.Cu at (211.1, 92.4)
- added C1604: 100n, SMD:C_0603_Symbol1, F.Cu at (208.3, 95.1)
- added C1605: 100n, SMD:C_0603_Symbol1, F.Cu at (211.1, 93.7)
- added C1606: 100n, SMD:C_0603_Symbol1, F.Cu at (214.0, 92.4)
- added C1607: 100n, SMD:C_0603_Symbol1, F.Cu at (211.1, 95.1)
- added C510: 10u, SMD:C_1206_Symbol1, F.Cu at (507.7, 261.8)
- added C512: 100p, Capacitors_SMD:C_0603, F.Cu at (506.7, 267.6)
- added C521: 100n, SMD:C_0603_Symbol1, F.Cu at (509.5, 267.6)
- added C522: 100n, SMD:C_0603_Symbol1, F.Cu at (518.2, 260.4)
- added C523: 100n, SMD:C_0603_Symbol1, F.Cu at (515.2, 261.7)
- added C524: 100n, SMD:C_0603_Symbol1, F.Cu at (506.3, 271.6)
- added C525: 100n, SMD:C_0603_Symbol1, F.Cu at (509.1, 269.0)
- added C526: 100n, SMD:C_0603_Symbol1, F.Cu at (512.4, 266.8)
- added C527: 100n, SMD:C_0603_Symbol1, F.Cu at (506.3, 273.0)
- added C528: 100n, SMD:C_0603_Symbol1, F.Cu at (515.2, 263.1)
- added C529: 100n, SMD:C_0603_Symbol1, F.Cu at (506.7, 266.3)
- added C530: 100n, SMD:C_0603_Symbol1, F.Cu at (515.2, 264.4)
- added C531: 100n, SMD:C_0603_Symbol1, F.Cu at (518.1, 261.7)
- added C532: 100n, SMD:C_0603_Symbol1, F.Cu at (512.4, 264.1)
- added C533: 100n, SMD:C_0603_Symbol1, F.Cu at (518.2, 259.0)
- added C534: 100n, SMD:C_0603_Symbol1, F.Cu at (503.4, 273.0)
- added D1202: VS-30BQ060, Diodes_SMD:D_SMC, F.Cu at (109.7, 135.3)
- added L502: 390n, Resistors_SMD:R_0603, F.Cu at (517.9, 264.6)
- added L503: 470n, Resistors_SMD:R_0603, F.Cu at (517.9, 263.1)
- added Q401: MMBF5486, TO_SOT_Packages_SMD:SOT-23, F.Cu at (464.1, 308.2)
- added Q402: MMBT200, TO_SOT_Packages_SMD:SOT-23, F.Cu at (467.5, 308.2)
- added Q406: BCP56-16, TO_SOT_Packages_SMD:SOT-223-3_TabPin2, F.Cu at (437.8, 313.5)
- added R1226: 100k, SMD:R_0603_Symbol3, F.Cu at (161.9, 113.3)
- added R1228: 0, SMD:R_0603_Symbol2, F.Cu at (142.5, 132.7)
- added R1229: 0, SMD:R_0603_Symbol2, F.Cu at (147.1, 128.0)
- added R1230: 9k53, Resistors_SMD:R_0603, F.Cu at (147.1, 126.5)
- added R1231: 100k, SMD:R_0603_Symbol3, F.Cu at (142.5, 131.2)
- added R1237: 0, SMD:R_0603_Symbol2, F.Cu at (159.3, 114.8)
- added R1238: 0, SMD:R_0603_Symbol2, F.Cu at (159.3, 113.3)
- added R1239: 9k53, Resistors_SMD:R_0603, F.Cu at (156.3, 115.0)
- added R1240: 100k, SMD:R_0603_Symbol3, F.Cu at (140.6, 134.2)
- added R1242: 0, SMD:R_0603_Symbol2, F.Cu at (131.0, 140.1)
- added R511: R, Resistors_SMD:R_0603, F.Cu at (511.8, 269.7)
- added U1104: LT1801, Housings_SOIC:SOIC-8_3.9x4.9mm_Pitch1.27mm, F.Cu at (177.7, 137.6)
- added U1601: OPA2344, Housings_SOIC:SOIC-8_3.9x4.9mm_Pitch1.27mm, F.Cu at (202.9, 89.0)
- added U1602: OPA2344, Housings_SOIC:SOIC-8_3.9x4.9mm_Pitch1.27mm, F.Cu at (210.4, 89.0)
- added U1604: DG408DY, Housings_SOIC:SOIC-16_3.9x9.9mm_Pitch1.27mm, F.Cu at (533.4, 262.3)
- added U1605: OPA344, TO_SOT_Packages_SMD:SOT-23-5, F.Cu at (201.1, 93.5)
- added U1606: ADS1110, TO_SOT_Packages_SMD:SOT-23-6, F.Cu at (204.9, 93.5)
- added U509: SN74LVC1T45, SMD:SC70-6, F.Cu at (513.1, 258.3)
- C1103, C1410: value 100n -> 15p; footprint SMD:C_0603_Symbol1 -> SMD:C_0603_Symbol5
- C1104: value 100n -> 1n2; footprint SMD:C_0603_Symbol1 -> Capacitors_SMD:C_0603
- C1105: value 1n2 -> 100n; footprint Capacitors_SMD:C_0603 -> SMD:C_0603_Symbol1
- C1122, C320: value 15p -> 100n; footprint SMD:C_0603_Symbol5 -> SMD:C_0603_Symbol1
- C1201: value 10u/50V -> 2u2/100V/X7R; footprint Capacitors_SMD:C_1210 -> SMD:C_1206_Symbol3
- C1202: value 4u7/50V -> 2u2/100V/X7R; footprint SMD:C_1210_1 -> SMD:C_1206_Symbol3
- C1203, C1204: value 1000p/2kV -> 4u7/50V; footprint Capacitors_SMD:C_1206 -> SMD:C_1210_1
- C1207, C1208: value 4u7/50V -> 47u; footprint SMD:C_1210_1 -> Capacitors_Tantalum_SMD:CP_Tantalum_Case-X_EIA-7343-43_Hand
- C1209, C1210, C1213, C1215: value 4u7/50V -> 10u; footprint SMD:C_1210_1 -> SMD:C_1206_Symbol1
- C1211, C1212: value 10u/50V -> 10u; footprint Capacitors_SMD:C_1210 -> SMD:C_1206_Symbol1
- C1214, C1216: value 4u7/50V -> 4u7; footprint SMD:C_1210_1 -> SMD:C_1206_Symbol2
- C1217: value 3n3 -> 470n; footprint Capacitors_SMD:C_0603 -> SMD:C_0603_Symbol4
- C1218: value 100p -> 4u7/50V/X7R; footprint Capacitors_SMD:C_0603 -> SMD:C_1210_1
- C1219: value 3n3 -> 10n; footprint Capacitors_SMD:C_0603 -> SMD:C_0603_Symbol2
- C1220: value 100p -> 2u2/100V/X7R; footprint Capacitors_SMD:C_0603 -> SMD:C_1206_Symbol3
- C1221: value 100n -> 1000p/2kV; footprint SMD:C_0603_Symbol1 -> Capacitors_SMD:C_1206
- C1222: value 100n -> 2u2/100V/X7R; footprint SMD:C_0603_Symbol1 -> SMD:C_1206_Symbol3
- C1223, C1224: value 470n -> 4u7/50V; footprint SMD:C_0603_Symbol4 -> SMD:C_1210_1
- C1225, C1226: value 10n -> 4u7/50V; footprint SMD:C_0603_Symbol2 -> SMD:C_1210_1
- C1227, C1228: value 470n -> 47u; footprint SMD:C_0603_Symbol4 -> Capacitors_Tantalum_SMD:CP_Tantalum_Case-X_EIA-7343-43_Hand
- C1229, C1230: value 4u7/50V/X7R -> 10u; footprint SMD:C_1210_1 -> SMD:C_1206_Symbol1
- C1231, C1232: value NC -> 10u; footprint Capacitors_SMD:C_0603 -> SMD:C_1206_Symbol1
- C1233, C1235: value 2u2/100V/X7R -> 10u; footprint SMD:C_1206_Symbol3 -> SMD:C_1206_Symbol1
- C1234, C1236: value 2u2/100V/X7R -> 4u7; footprint SMD:C_1206_Symbol3 -> SMD:C_1206_Symbol2
- C1237: value 47u -> 10u/50V; footprint Capacitors_Tantalum_SMD:CP_Tantalum_Case-X_EIA-7343-43_Hand -> Capacitors_SMD:C_1210
- C1238: value 47u -> 4u7/50V; footprint Capacitors_Tantalum_SMD:CP_Tantalum_Case-X_EIA-7343-43_Hand -> SMD:C_1210_1
- C1239: value 47p -> 1000p/2kV; footprint Capacitors_SMD:C_0603 -> Capacitors_SMD:C_1206
- C1240: value 47p -> 470n; footprint Capacitors_SMD:C_0603 -> SMD:C_0603_Symbol4
- C1241: value 47u -> 4u7/50V/X7R; footprint Capacitors_Tantalum_SMD:CP_Tantalum_Case-X_EIA-7343-43_Hand -> SMD:C_1210_1
- C1242: value 47u -> 10n; footprint Capacitors_Tantalum_SMD:CP_Tantalum_Case-X_EIA-7343-43_Hand -> SMD:C_0603_Symbol2
- C1243: value 10u -> 470n; footprint SMD:C_1206_Symbol1 -> SMD:C_0603_Symbol4
- C1244: value 10u -> 10u/50V; footprint SMD:C_1206_Symbol1 -> Capacitors_SMD:C_1210
- C1245: value 47u -> 4u7/50V; footprint SMD:C_1210_2 -> SMD:C_1210_1
- C1246: value 47u -> 10u; footprint SMD:C_1210_2 -> SMD:C_1206_Symbol1
- C1247, C1258: value 10u -> 4u7; footprint SMD:C_1206_Symbol1 -> SMD:C_1206_Symbol2
- C1249: value 47u -> 4u7; footprint SMD:C_1210_2 -> SMD:C_1206_Symbol2
- C1250: value 47u -> NC; footprint SMD:C_1210_2 -> Capacitors_SMD:C_0603
- C1251, C1265, C505: value 10u -> 100n; footprint SMD:C_1206_Symbol1 -> SMD:C_0603_Symbol1
- C1252, C1266: value 10u -> 3n3; footprint SMD:C_1206_Symbol1 -> Capacitors_SMD:C_0603
- C1253, C1267: value 10u -> 47p; footprint SMD:C_1206_Symbol1 -> Capacitors_SMD:C_0603
- C1254, C1268: value 10u -> 100p; footprint SMD:C_1206_Symbol1 -> Capacitors_SMD:C_0603
- C1255, C1256, C1269: value 10u -> 47u; footprint SMD:C_1206_Symbol1 -> SMD:C_1210_2
- C1261: value 4u7 -> 470n; footprint SMD:C_1206_Symbol2 -> SMD:C_0603_Symbol4
- C1262: value 4u7 -> 10u/50V; footprint SMD:C_1206_Symbol2 -> Capacitors_SMD:C_1210
- C1263: value 4u7 -> 4u7/50V; footprint SMD:C_1206_Symbol2 -> SMD:C_1210_1
- C1264: value 4u7 -> NC; footprint SMD:C_1206_Symbol2 -> Capacitors_SMD:C_0603
- C1270: value 4u7 -> 47u; footprint SMD:C_1206_Symbol2 -> SMD:C_1210_2
- C1271, C1273: value 4u7 -> 10u; footprint SMD:C_1206_Symbol2 -> SMD:C_1206_Symbol1
- C1401, C1403, C1405: value 100n -> 68p; footprint SMD:C_0603_Symbol1 -> Capacitors_SMD:C_0603
- C1402: value 100n -> 8p; footprint SMD:C_0603_Symbol1 -> Capacitors_SMD:C_0603
- C1404, C1411, C513: value 100n -> 33p; footprint SMD:C_0603_Symbol1 -> Capacitors_SMD:C_0603
- C1406: value 15p -> 100p; footprint SMD:C_0603_Symbol5 -> Capacitors_SMD:C_0603
- C1407: value 100n -> 560p; footprint SMD:C_0603_Symbol1 -> Capacitors_SMD:C_0603
- C1408: value 15p -> 270p; footprint SMD:C_0603_Symbol5 -> Capacitors_SMD:C_0603
- C1409: value 39p -> 15p; footprint Capacitors_SMD:C_0603 -> SMD:C_0603_Symbol5
- C1412: value 8p -> 22p
- C1413: value 33p -> 470p
- C1414: value 100p -> 39p
- C1415: value 270p -> 150p
- C1416, C1417, C1418: value 68p -> 100n; footprint Capacitors_SMD:C_0603 -> SMD:C_0603_Symbol1
- C1419: value 560p -> 100n; footprint Capacitors_SMD:C_0603 -> SMD:C_0603_Symbol1
- C1420, C519: value 33p -> 100n; footprint Capacitors_SMD:C_0603 -> SMD:C_0603_Symbol1
- C1421, C520: value 150p -> 100n; footprint Capacitors_SMD:C_0603 -> SMD:C_0603_Symbol1
- C1422: value 22p -> 100n; footprint Capacitors_SMD:C_0603 -> SMD:C_0603_Symbol1
- C1423: value 470p -> 100n; footprint Capacitors_SMD:C_0603 -> SMD:C_0603_Symbol1
- C1502, C201, C504, C601, C608: value 100n -> 1u; footprint SMD:C_0603_Symbol1 -> SMD:C_0603_Symbol6
- C1503, C606: value 1u -> 100n; footprint SMD:C_0603_Symbol6 -> SMD:C_0603_Symbol1
- C202, C203, C602, C603: value 20p -> 2u2; footprint Capacitors_SMD:C_0603 -> SMD:C_0603_Symbol7
- C204, C605: value 1u -> 20p; footprint SMD:C_0603_Symbol6 -> Capacitors_SMD:C_0603
- C205: value 2u2 -> 20p; footprint SMD:C_0603_Symbol7 -> Capacitors_SMD:C_0603
- C206, C607, C609: value 2u2 -> 100n; footprint SMD:C_0603_Symbol7 -> SMD:C_0603_Symbol1
- C304: value 10p -> 15p; footprint Capacitors_SMD:C_0603 -> SMD:C_0603_Symbol5
- C305: value 100n -> 10p; footprint SMD:C_0603_Symbol1 -> Capacitors_SMD:C_0603
- C401: value 10u -> 15p; footprint SMD:C_1206_Symbol1 -> SMD:C_0603_Symbol5
- C402: value 15p -> 10n; footprint SMD:C_0603_Symbol5 -> SMD:C_0603_Symbol2
- C403: value 100u -> 15p; footprint Capacitors_Tantalum_SMD:CP_Tantalum_Case-X_EIA-7343-43_Hand -> SMD:C_0603_Symbol5
- C404: value 10u -> 1n; footprint SMD:C_1206_Symbol1 -> Capacitors_SMD:C_0603
- C405: value 100u -> 10n; footprint Capacitors_Tantalum_SMD:CP_Tantalum_Case-X_EIA-7343-43_Hand -> SMD:C_0603_Symbol2
- C406: value 10n -> 15p; footprint SMD:C_0603_Symbol2 -> SMD:C_0603_Symbol5
- C407: value 10n -> 10u; footprint SMD:C_0603_Symbol2 -> SMD:C_1206_Symbol1
- C408: value 1n -> 100u; footprint Capacitors_SMD:C_0603 -> Capacitors_Tantalum_SMD:CP_Tantalum_Case-X_EIA-7343-43_Hand
- C409: value 15p -> 10u; footprint SMD:C_0603_Symbol5 -> SMD:C_1206_Symbol1
- C410: value 15p -> 100u; footprint SMD:C_0603_Symbol5 -> Capacitors_Tantalum_SMD:CP_Tantalum_Case-X_EIA-7343-43_Hand
- C501: value 100n -> 1000p; footprint SMD:C_0603_Symbol1 -> Capacitors_SMD:C_0603
- C503: value 100n -> 10u; footprint SMD:C_0603_Symbol1 -> SMD:C_1206_Symbol1
- C506: value 100n -> 10n; footprint SMD:C_0603_Symbol1 -> SMD:C_0603_Symbol2
- C507: value 1u -> 10n; footprint SMD:C_0603_Symbol6 -> SMD:C_0603_Symbol2
- C508, C509: value 100n -> 1p5; footprint SMD:C_0603_Symbol1 -> Capacitors_SMD:C_0603
- C511: value 100n -> 150p; footprint SMD:C_0603_Symbol1 -> Capacitors_SMD:C_0603
- C514: value 100n -> 180p; footprint SMD:C_0603_Symbol1 -> Capacitors_SMD:C_0603
- C515: value 10u -> 300p; footprint SMD:C_1206_Symbol1 -> Capacitors_SMD:C_0603
- C516: value 1000p -> 330p
- C517: value 1p5 -> 270p
- C518: value 1p5 -> 100n; footprint Capacitors_SMD:C_0603 -> SMD:C_0603_Symbol1
- C604: value 100n -> 20p; footprint SMD:C_0603_Symbol1 -> Capacitors_SMD:C_0603
- C803: value 47p -> 100n; footprint Capacitors_SMD:C_0603 -> SMD:C_0603_Symbol1
- C808: value 100n -> 47p; footprint SMD:C_0603_Symbol1 -> Capacitors_SMD:C_0603
- C901: value 30p -> 100n; footprint Capacitors_SMD:C_0603 -> SMD:C_0603_Symbol1
- C902: value 30p -> 1000p/2kV; footprint Capacitors_SMD:C_0603 -> Capacitors_SMD:C_1206
- C910: value 100n -> 30p; footprint SMD:C_0603_Symbol1 -> Capacitors_SMD:C_0603
- C911: value 1000p/2kV -> 30p; footprint Capacitors_SMD:C_1206 -> Capacitors_SMD:C_0603
- D1201: value SM6T30AY -> MBRS3100T3G; footprint SMD:DO_214AA_REV -> Diodes_SMD:D_SMC
- D1203: value RED -> SZMMSZ4705T1; footprint LEDs:LED_0603 -> SMD:SOD-323F
- D1204: value SBR3U100LP -> SM6T30AY; footprint SMD:U-DFN3030-8 -> SMD:DO_214AA_REV
- D1205: value SBR3U100LP -> RED; footprint SMD:U-DFN3030-8 -> LEDs:LED_0603
- D1206: value VS-30BQ060 -> SBR3U100LP; footprint Diodes_SMD:D_SMC -> SMD:U-DFN3030-8
- D1207: value MBRS3100T3G -> SBR3U100LP; footprint Diodes_SMD:D_SMC -> SMD:U-DFN3030-8
- D1502, D1504: value MMSZ5227 -> BAV16WS; footprint Diodes_SMD:D_SOD-123 -> Diodes_SMD:D_SOD-323_HandSoldering
- D1505, D1507: value BAV16WS -> MMSZ5227; footprint Diodes_SMD:D_SOD-323_HandSoldering -> Diodes_SMD:D_SOD-123
- D304, D306: value BAT54-02V -> BAT54C; footprint Diodes_SMD:D_SOD-523 -> TO_SOT_Packages_SMD:SOT-23
- D311, D312: value BAT54C -> BAT54-02V; footprint TO_SOT_Packages_SMD:SOT-23 -> Diodes_SMD:D_SOD-523
- D801: value SD36C-01FTG -> SMBJ5.0A; footprint Diodes_SMD:D_SOD-323_HandSoldering -> SMD:DO_214AA_REV
- D802: value SMBJ5.0A -> BAV99; footprint SMD:DO_214AA_REV -> SMD:SOT23
- D803: value BAV99 -> SD36C-01FTG; footprint SMD:SOT23 -> Diodes_SMD:D_SOD-323_HandSoldering
- L501: value 100n -> 270n
- Q1201: value IRFR5410 -> Si7456DP; footprint TO_SOT_Packages_SMD:TO-252-2_Rectifier -> SMD:PowerPAK-SO-8
- Q1202: value Si7456DP -> IRFR5410; footprint SMD:PowerPAK-SO-8 -> TO_SOT_Packages_SMD:TO-252-2_Rectifier
- Q404, Q405: value SMBT2222 -> BCP56-16; footprint TO_SOT_Packages_SMD:SOT-23 -> TO_SOT_Packages_SMD:SOT-223-3_TabPin2
- Q408, Q414: value BCP53 -> SMBT2222; footprint TO_SOT_Packages_SMD:SOT-223-3_TabPin2 -> TO_SOT_Packages_SMD:SOT-23
- Q409, Q411: value BCP56-16 -> BCP53
- Q413: value BCP56-16 -> MMBT200; footprint TO_SOT_Packages_SMD:SOT-223-3_TabPin2 -> TO_SOT_Packages_SMD:SOT-23
- R1102: value 10 -> 10k; footprint Resistors_SMD:R_0603 -> SMD:R_0603_Symbol1
- R1103, R1106: value 2k49 -> 10k; footprint Resistors_SMD:R_0603 -> SMD:R_0603_Symbol1
- R1104, R1112: value 10k -> 2k49; footprint SMD:R_0603_Symbol1 -> Resistors_SMD:R_0603
- R1108: value 10k -> 10; footprint SMD:R_0603_Symbol1 -> Resistors_SMD:R_0603
- R1201: value 100k -> 154k; footprint SMD:R_0603_Symbol3 -> Resistors_SMD:R_0603
- R1203: value R -> 32k4; footprint Resistors_SMD:R_1206 -> Resistors_SMD:R_0603
- R1204, R1205: value NC -> R
- R1206, R1207: value 41k2 -> R
- R1208: value 9k53 -> R
- R1209, R1224: value 0 -> 41k2; footprint SMD:R_0603_Symbol2 -> Resistors_SMD:R_0603
- R1210: value 9k53 -> 10k; footprint Resistors_SMD:R_0603 -> SMD:R_0603_Symbol1
- R1211: value 0 -> 200k; footprint SMD:R_0603_Symbol2 -> Resistors_SMD:R_0603
- R1212: value 154k -> 120
- R1213: value 32k4 -> 100k; footprint Resistors_SMD:R_0603 -> SMD:R_0603_Symbol3
- R1214: value 200k -> R; footprint Resistors_SMD:R_0603 -> Resistors_SMD:R_1206
- R1216: value 100k -> NC; footprint SMD:R_0603_Symbol3 -> Resistors_SMD:R_0603
- R1217: value 100k -> R
- R1218, R601: value 10k -> R; footprint SMD:R_0603_Symbol1 -> Resistors_SMD:R_0603
- R1219: value 10k -> NC; footprint SMD:R_0603_Symbol1 -> Resistors_SMD:R_0603
- R1220, R1221: value 0 -> R
- R1225, R302, R328, R901: value 0 -> 10k; footprint SMD:R_0603_Symbol2 -> SMD:R_0603_Symbol1
- R1232: value 100k -> 422k; footprint SMD:R_0603_Symbol3 -> Resistors_SMD:R_0603
- R1233: value 100k -> 0; footprint SMD:R_0603_Symbol3 -> SMD:R_0603_Symbol2
- R1234: value 422k -> 80k6
- R1235: value 80k6 -> 100k; footprint Resistors_SMD:R_0603 -> SMD:R_0603_Symbol3
- R1243: value 120 -> R
- R1401: value 750 -> 10G/10%; footprint SMD:R_0603_Symbol8 -> Resistors_SMD:R_0805
- R1406: value 100k -> 1G/1%; footprint SMD:R_0603_Symbol3 -> Resistors_SMD:R_1206
- R1407: value 750 -> 100Meg/1%; footprint SMD:R_0603_Symbol8 -> Resistors_SMD:R_1206
- R1408, R1409: value 100k -> 750; footprint SMD:R_0603_Symbol3 -> SMD:R_0603_Symbol8
- R1410: value 10k -> 10Meg/1%; footprint SMD:R_0603_Symbol1 -> Resistors_SMD:R_1206
- R1411: value 100k -> 1Meg/0.5%; footprint SMD:R_0603_Symbol3 -> Resistors_SMD:R_1206
- R1412: value 10k -> 250; footprint SMD:R_0603_Symbol1 -> Resistors_SMD:R_1206
- R1413: value 10G/10% -> 100k/0.5%; footprint Resistors_SMD:R_0805 -> Resistors_SMD:R_1206
- R1414: value 1G/1% -> 180k/0.1%; footprint Resistors_SMD:R_1206 -> Resistors_SMD:R_0603
- R1415: value 100Meg/1% -> 750; footprint Resistors_SMD:R_1206 -> SMD:R_0603_Symbol8
- R1416: value 10Meg/1% -> 750; footprint Resistors_SMD:R_1206 -> SMD:R_0603_Symbol8
- R1417: value 1Meg/0.5% -> 750; footprint Resistors_SMD:R_1206 -> SMD:R_0603_Symbol8
- R1418: value 100k/0.5% -> 10k/0.5%
- R1419: value 10k/0.5% -> 18k/0.1%; footprint Resistors_SMD:R_1206 -> Resistors_SMD:R_0603
- R1421: value 100/0.1%/2W -> 10k; footprint Resistors_SMD:R_1206 -> SMD:R_0603_Symbol1
- R1422: value 10/1%/2W -> 2k/0.1%; footprint Resistors_SMD:R_2512 -> Resistors_SMD:R_0603
- R1423: value 250 -> 100/0.1%/2W
- R1424: value 1k -> 10/1%/2W; footprint SMD:R_0603_Symbol9 -> Resistors_SMD:R_2512
- R1426: value 10k -> 100k; footprint SMD:R_0603_Symbol1 -> SMD:R_0603_Symbol3
- R1427: value 3k9 -> 1k; footprint Resistors_SMD:R_0603 -> SMD:R_0603_Symbol9
- R1428: value 49k9 -> 100k; footprint Resistors_SMD:R_0603 -> SMD:R_0603_Symbol3
- R1429: value 180k/0.1% -> 51
- R1430: value 18k/0.1% -> 10k; footprint Resistors_SMD:R_0603 -> SMD:R_0603_Symbol1
- R1431: value 2k/0.1% -> 100k; footprint Resistors_SMD:R_0603 -> SMD:R_0603_Symbol3
- R1433: value 750 -> 3k9; footprint SMD:R_0603_Symbol8 -> Resistors_SMD:R_0603
- R1434: value 51 -> 510
- R1435: value 750 -> 100k; footprint SMD:R_0603_Symbol8 -> SMD:R_0603_Symbol3
- R1436, R327: value 750 -> 10k; footprint SMD:R_0603_Symbol8 -> SMD:R_0603_Symbol1
- R1438: value 510 -> 49k9
- R201: value 10k -> 200; footprint SMD:R_0603_Symbol1 -> Resistors_SMD:R_0603
- R202: value 4k7 -> 10k; footprint SMD:R_0603_Symbol6 -> SMD:R_0603_Symbol1
- R204: value 200 -> 4k7; footprint Resistors_SMD:R_0603 -> SMD:R_0603_Symbol6
- R301, R330: value 0 -> 2k49; footprint SMD:R_0603_Symbol2 -> SMD:R_0603_Symbol5
- R303: value 12k4 -> 40k
- R304: value 75k -> 10k; footprint Resistors_SMD:R_0603 -> SMD:R_0603_Symbol1
- R305: value 49k9 -> 10k; footprint Resistors_SMD:R_0603 -> SMD:R_0603_Symbol1
- R308, R309, R318, R320: value 10k -> 2k49; footprint SMD:R_0603_Symbol1 -> SMD:R_0603_Symbol5
- R311, R313: value 40k -> 10k; footprint Resistors_SMD:R_0603 -> SMD:R_0603_Symbol1
- R314: value 30k -> 0; footprint SMD:R_0603_Symbol7 -> SMD:R_0603_Symbol2
- R319: value 10k -> 750; footprint SMD:R_0603_Symbol1 -> SMD:R_0603_Symbol8
- R322: value 10k -> 40k; footprint SMD:R_0603_Symbol1 -> Resistors_SMD:R_0603
- R324, R325, R329: value 10k -> 0; footprint SMD:R_0603_Symbol1 -> SMD:R_0603_Symbol2
- R326: value 1k -> 10k; footprint SMD:R_0603_Symbol9 -> SMD:R_0603_Symbol1
- R332: value 10k -> 30k; footprint SMD:R_0603_Symbol1 -> SMD:R_0603_Symbol7
- R335, R336, R337, R340, R346: value 2k49 -> 10k; footprint SMD:R_0603_Symbol5 -> SMD:R_0603_Symbol1
- R339: value 10k -> 1k; footprint SMD:R_0603_Symbol1 -> SMD:R_0603_Symbol9
- R342: value 10k -> 49k9; footprint SMD:R_0603_Symbol1 -> Resistors_SMD:R_0603
- R343: value 2k49 -> 12k4; footprint SMD:R_0603_Symbol5 -> Resistors_SMD:R_0603
- R344: value 10k -> 75k; footprint SMD:R_0603_Symbol1 -> Resistors_SMD:R_0603
- R402: value 10k -> 300; footprint SMD:R_0603_Symbol1 -> Resistors_SMD:R_0603
- R403: value 3k3 -> 3k9
- R404: value 3k9 -> 3k3
- R405: value 30k -> 33; footprint SMD:R_0603_Symbol7 -> Resistors_SMD:R_0603
- R407: value 3k9 -> 1k8
- R408, R411: value 300 -> 10/2W; footprint Resistors_SMD:R_0603 -> Resistors_SMD:R_2512
- R409: value 1k8 -> 10/2W; footprint Resistors_SMD:R_0603 -> Resistors_SMD:R_2512
- R410: value 510 -> 10/2W; footprint Resistors_SMD:R_0603 -> Resistors_SMD:R_2512
- R413, R902, R903: value 33 -> 10k; footprint Resistors_SMD:R_0603 -> SMD:R_0603_Symbol1
- R415: value 10/2W -> 510; footprint Resistors_SMD:R_2512 -> Resistors_SMD:R_0603
- R420: value 10/2W -> 30k; footprint Resistors_SMD:R_2512 -> SMD:R_0603_Symbol7
- R421: value 10/2W -> 3k9; footprint Resistors_SMD:R_2512 -> Resistors_SMD:R_0603
- R422: value 10/2W -> 300; footprint Resistors_SMD:R_2512 -> Resistors_SMD:R_0603
- R501: value 200 -> 33k2
- R502: value 6k81 -> 24k9
- R503: value 33k2 -> 100k; footprint Resistors_SMD:R_0603 -> SMD:R_0603_Symbol3
- R504: value 24k9 -> 17k4
- R505: value 200 -> 17k4
- R506: value 100k -> 511; footprint SMD:R_0603_Symbol3 -> Resistors_SMD:R_0603
- R507: value 17k4 -> 51
- R508: value 511 -> 200
- R509: value 17k4 -> 6k81
- R510: value 34R8 -> 200
- R603: value R -> 10k; footprint Resistors_SMD:R_0603 -> SMD:R_0603_Symbol1
- R701: value 0 -> 120; footprint SMD:R_0603_Symbol2 -> Resistors_SMD:R_1206
- R703: value 120 -> 0; footprint Resistors_SMD:R_1206 -> SMD:R_0603_Symbol2
- R801: value 51R1 -> 10k; footprint Resistors_SMD:R_0603 -> SMD:R_0603_Symbol1
- R802: value 47 -> 255
- R803: value 1k -> NC; footprint SMD:R_0603_Symbol9 -> Resistors_SMD:R_0603
- R804: value 100 -> 1k; footprint Resistors_SMD:R_0603 -> SMD:R_0603_Symbol9
- R805: value 14k7 -> 10k; footprint Resistors_SMD:R_0603 -> SMD:R_0603_Symbol1
- R806: value NC -> 47
- R807: value 10k -> 100; footprint SMD:R_0603_Symbol1 -> Resistors_SMD:R_0603
- R808: value 10k -> 14k7; footprint SMD:R_0603_Symbol1 -> Resistors_SMD:R_0603
- R809: value 255 -> 51R1
- R904, R906, R907: value 10k -> 50; footprint SMD:R_0603_Symbol1 -> SMD:R_0603_Symbol4
- R905: value 33 -> 50; footprint Resistors_SMD:R_0603 -> SMD:R_0603_Symbol4
- R908: value 1k5 -> 33
- R909: value 10k -> 33; footprint SMD:R_0603_Symbol1 -> Resistors_SMD:R_0603
- R911: value 50 -> 33; footprint SMD:R_0603_Symbol4 -> Resistors_SMD:R_0603
- R913: value 50 -> 1k5; footprint SMD:R_0603_Symbol4 -> Resistors_SMD:R_0603
- R914: value 50 -> 75; footprint SMD:R_0603_Symbol4 -> Resistors_SMD:R_0603
- R915: value 270 -> 75
- R916: value 50 -> 10k; footprint SMD:R_0603_Symbol4 -> SMD:R_0603_Symbol1
- R917: value 270 -> 0; footprint Resistors_SMD:R_0603 -> SMD:R_0603_Symbol2
- R919, R920: value 75 -> 270
- U1101: value LT1801 -> LTC6655-5; footprint Housings_SOIC:SOIC-8_3.9x4.9mm_Pitch1.27mm -> Housings_SSOP:MSOP-8_3x3mm_Pitch0.65mm
- U1102: value LT1801 -> ADG419BRM
- U1103: value LTC6655-5 -> LT1801; footprint Housings_SSOP:MSOP-8_3x3mm_Pitch0.65mm -> Housings_SOIC:SOIC-8_3.9x4.9mm_Pitch1.27mm
- U1106: value LTC2512-24 -> ADG5204_TSSOP; footprint Housings_DFN_QFN:DFN-24-1EP_4x7mm_Pitch0.5mm -> Housings_SSOP:TSSOP-14_4.4x5mm_Pitch0.65mm
- U1108: value ADG5204_TSSOP -> LTC2512-24; footprint Housings_SSOP:TSSOP-14_4.4x5mm_Pitch0.65mm -> Housings_DFN_QFN:DFN-24-1EP_4x7mm_Pitch0.5mm
- U1201: value MAX5902 -> NCP1117-ADJ_TO252; footprint SMD:SOT23_6 -> SMD:DPAK
- U1202: value TEN 40-2415N -> LT3758; footprint THT:TEN40 -> Housings_SSOP:MSOP-10-1EP_3x3mm_Pitch0.5mm
- U1203: value LT3758 -> LM337_TO252; footprint Housings_SSOP:MSOP-10-1EP_3x3mm_Pitch0.5mm -> SMD:DPAK
- U1204: value LT3758 -> MAX5902; footprint Housings_SSOP:MSOP-10-1EP_3x3mm_Pitch0.5mm -> SMD:SOT23_6
- U1205: value LTC3864 -> TEN 40-2415N; footprint Housings_SSOP:MSOP-12-1EP_3x4mm_Pitch0.65mm -> THT:TEN40
- U1206: value LTC3864 -> LT3758; footprint Housings_SSOP:MSOP-12-1EP_3x4mm_Pitch0.65mm -> Housings_SSOP:MSOP-10-1EP_3x3mm_Pitch0.5mm
- U1207: value NCP1117-ADJ_TO252 -> NCP1117-3.3_TO252
- U1208: value LM337_TO252 -> LTC3864; footprint SMD:DPAK -> Housings_SSOP:MSOP-12-1EP_3x4mm_Pitch0.65mm
- U1210: value NCP1117-3.3_TO252 -> LTC3864; footprint SMD:DPAK -> Housings_SSOP:MSOP-12-1EP_3x4mm_Pitch0.65mm
- U1403: value AD746 -> AQY221; footprint Housings_SOIC:SOIC-8_3.9x4.9mm_Pitch1.27mm -> SMD:AQY2
- U1405: value AQY221 -> ULN2002; footprint SMD:AQY2 -> SMD:SO16E
- U1406: value AQY221 -> ADG3308; footprint SMD:AQY2 -> Housings_SSOP:SSOP-20_4.4x6.5mm_Pitch0.65mm
- U1407: value AQY221 -> TCA9555_TSSOP; footprint SMD:AQY2 -> Housings_SSOP:TSSOP-24_4.4x7.8mm_Pitch0.65mm
- U1408, U1409, U1414: value AD744 -> AQY221; footprint Housings_SOIC:SOIC-8_3.9x4.9mm_Pitch1.27mm -> SMD:AQY2
- U1410: value TCA9555_TSSOP -> ADG3308; footprint Housings_SSOP:TSSOP-24_4.4x7.8mm_Pitch0.65mm -> Housings_SSOP:SSOP-20_4.4x6.5mm_Pitch0.65mm
- U1411: value AQY221 -> AD744; footprint SMD:AQY2 -> Housings_SOIC:SOIC-8_3.9x4.9mm_Pitch1.27mm
- U1415, U1416: value ADG3308 -> AD744; footprint Housings_SSOP:SSOP-20_4.4x6.5mm_Pitch0.65mm -> Housings_SOIC:SOIC-8_3.9x4.9mm_Pitch1.27mm
- U1417: value ULN2002 -> AD746; footprint SMD:SO16E -> Housings_SOIC:SOIC-8_3.9x4.9mm_Pitch1.27mm
- U201: value 24LC08 -> STM32F746ZGTx; footprint Housings_SSOP:MSOP-8_3x3mm_Pitch0.65mm -> SMD:TQFP-144
- U202: value STM32F746ZGTx -> 24LC08; footprint SMD:TQFP-144 -> Housings_SSOP:MSOP-8_3x3mm_Pitch0.65mm
- U301, U302: value AD746 -> LT1801
- U303: value REF5025AD -> AD746
- U304, U501: value LT1801 -> REF5025AD
- U305: value SN74LVC1T45 -> LT1715; footprint SMD:SC70-6 -> Housings_SSOP:MSOP-10_3x3mm_Pitch0.5mm
- U306: value SN74LVC1T45 -> NC7SZ125; footprint SMD:SC70-6 -> TO_SOT_Packages_SMD:SOT-23-5
- U307: value LT1801 -> DAC80004; footprint Housings_SOIC:SOIC-8_3.9x4.9mm_Pitch1.27mm -> Housings_SSOP:TSSOP-14_4.4x5mm_Pitch0.65mm
- U308: value LT1801 -> AQY221; footprint Housings_SOIC:SOIC-8_3.9x4.9mm_Pitch1.27mm -> SMD:AQY2
- U309: value DAC80004 -> LT1801; footprint Housings_SSOP:TSSOP-14_4.4x5mm_Pitch0.65mm -> Housings_SOIC:SOIC-8_3.9x4.9mm_Pitch1.27mm
- U311: value LT1801 -> AD746
- U312: value OP07 -> SN74LVC1T45; footprint Housings_SOIC:SOIC-8_3.9x4.9mm_Pitch1.27mm -> SMD:SC70-6
- U314, U316: value DG419 -> ADG419BRM
- U315: value LT1715 -> LT1801; footprint Housings_SSOP:MSOP-10_3x3mm_Pitch0.5mm -> Housings_SOIC:SOIC-8_3.9x4.9mm_Pitch1.27mm
- U317: value AQY221 -> SN74LVC1T45; footprint SMD:AQY2 -> SMD:SC70-6
- U319: value NC7SZ125 -> OP07; footprint TO_SOT_Packages_SMD:SOT-23-5 -> Housings_SOIC:SOIC-8_3.9x4.9mm_Pitch1.27mm
- U502: value REF5025AD -> LT1677
- U503: value AD9834 -> DAC8531; footprint Housings_SSOP:SSOP-20_4.4x6.5mm_Pitch0.65mm -> Housings_SSOP:MSOP-8_3x3mm_Pitch0.65mm
- U504: value DAC8531 -> AD9834; footprint Housings_SSOP:MSOP-8_3x3mm_Pitch0.65mm -> Housings_SSOP:SSOP-20_4.4x6.5mm_Pitch0.65mm
- U505: value LT1677 -> AD5452; footprint Housings_SOIC:SOIC-8_3.9x4.9mm_Pitch1.27mm -> Housings_SSOP:MSOP-8_3x3mm_Pitch0.65mm
- U506: value AD5452 -> LT1801; footprint Housings_SSOP:MSOP-8_3x3mm_Pitch0.65mm -> Housings_SOIC:SOIC-8_3.9x4.9mm_Pitch1.27mm
- U802: value 74AHC1G14 -> NXE1S0305MC; footprint SMD:SC-70-5 -> SMD:NXE1
- U803: value NXE1S0305MC -> 74LVC1G14; footprint SMD:NXE1 -> TO_SOT_Packages_SMD:SOT-353_SC-70-5
- U804: value HCPL0710 -> ACPL-214; footprint SMD:SOIC8NB -> SMD:SO4
- U805: value ACPL-214 -> HCPL0710; footprint SMD:SO4 -> SMD:SOIC8NB
- U901: value LAN8742A -> USBLC6-4; footprint Housings_DFN_QFN:QFN-24-1EP_4x4mm_Pitch0.5mm -> TO_SOT_Packages_SMD:SOT-23-6
- U902: value USBLC6-4 -> LC03-3.3; footprint TO_SOT_Packages_SMD:SOT-23-6 -> SMD:SO8E
- U904: value LC03-3.3 -> LAN8742A; footprint SMD:SO8E -> Housings_DFN_QFN:QFN-24-1EP_4x4mm_Pitch0.5mm
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Connections:
- C1101 pad 2: +5V_TRG -> GND
- C1102 pad 2: +5V_TRG -> GND
- C1103 pad 1: -15V -> Net-(C1103-Pad1)
- C1103 pad 2: +5V_TRG -> Net-(C1103-Pad2)
- C1104 pad 1: +15V -> Net-(C1104-Pad1)
- C1104 pad 2: +5V_TRG -> GND
- C1105 pad 1: Net-(C1105-Pad1) -> -15V
- C1105 pad 2: +5V_TRG -> GND
- C1106 pad 2: +5V_TRG -> GND
- C1107 pad 1: +15V -> -15V
- C1107 pad 2: +5V_TRG -> GND
- C1108 pad 2: +5V_TRG -> GND
- C1109 pad 1: +15V -> -15V
- C1109 pad 2: +5V_TRG -> GND
- C1110 pad 2: +5V_TRG -> GND
- C1111 pad 1: +15V -> +3V3
- C1111 pad 2: +5V_TRG -> GND
- C1112 pad 1: -15V -> +3V3
- C1112 pad 2: +5V_TRG -> GND
- C1113 pad 2: +5V_TRG -> GND
- C1114 pad 1: -15V -> +15V
- C1114 pad 2: +5V_TRG -> GND
- C1115 pad 2: +5V_TRG -> GND
- C1116 pad 1: +5V -> +15V
- C1116 pad 2: +5V_TRG -> GND
- C1117 pad 1: +3V3 -> +15V
- C1117 pad 2: +5V_TRG -> GND
- C1118 pad 1: +5V -> +15V
- C1118 pad 2: +5V_TRG -> GND
- C1119 pad 1: +3V3 -> +5V
- C1119 pad 2: +5V_TRG -> GND
- C1120 pad 2: +5V_TRG -> GND
- C1121 pad 1: +2V5 -> +5V
- C1121 pad 2: +5V_TRG -> GND
- C1122 pad 1: Net-(C1122-Pad1) -> +2V5
- C1122 pad 2: Net-(C1122-Pad2) -> GND
- C1201 pad 2: GNDPWR -> Net-(C1201-Pad2)
- C1202 pad 2: GNDPWR -> Net-(C1201-Pad2)
- C1203 pad 1: Net-(C1201-Pad1) -> Net-(C1203-Pad1)
- C1203 pad 2: Net-(C1203-Pad2) -> GND
- C1204 pad 1: GNDPWR -> Net-(C1203-Pad1)
- C1204 pad 2: +5V_TRG -> GND
- C1205 pad 1: Net-(C1203-Pad2) -> Net-(C1203-Pad1)
- C1205 pad 2: +5V_TRG -> GND
- C1206 pad 1: Net-(C1203-Pad2) -> Net-(C1203-Pad1)
- C1206 pad 2: +5V_TRG -> GND
- C1207 pad 1: Net-(C1203-Pad2) -> Net-(C1207-Pad1)
- C1207 pad 2: +5V_TRG -> GND
- C1208 pad 1: Net-(C1203-Pad2) -> Net-(C1207-Pad1)
- C1208 pad 2: +5V_TRG -> GND
- C1209 pad 1: Net-(C1203-Pad2) -> Net-(C1207-Pad1)
- C1209 pad 2: +5V_TRG -> GND
- C1210 pad 1: Net-(C1203-Pad2) -> Net-(C1207-Pad1)
- C1210 pad 2: +5V_TRG -> GND
- C1211 pad 1: Net-(C1203-Pad2) -> Net-(C1207-Pad1)
- C1211 pad 2: +5V_TRG -> GND
- C1212 pad 1: Net-(C1203-Pad2) -> Net-(C1207-Pad1)
- C1212 pad 2: +5V_TRG -> GND
- C1213 pad 1: Net-(C1203-Pad2) -> Net-(C1213-Pad1)
- C1213 pad 2: +5V_TRG -> GND
- C1214 pad 1: Net-(C1203-Pad2) -> Net-(C1213-Pad1)
- C1214 pad 2: +5V_TRG -> GND
- C1215 pad 1: Net-(C1203-Pad2) -> +15V
- C1215 pad 2: +5V_TRG -> GND
- C1216 pad 1: Net-(C1203-Pad2) -> +15V
- C1216 pad 2: +5V_TRG -> GND
- C1217 pad 2: +5V_TRG -> GND
- C1218 pad 2: +5V_TRG -> GND
- C1219 pad 2: +5V_TRG -> GND
- C1220 pad 2: +5V_TRG -> Net-(C1220-Pad2)
- C1221 pad 2: +5V_TRG -> Net-(C1203-Pad1)
- C1222 pad 1: Net-(C1222-Pad1) -> Net-(C1220-Pad1)
- C1222 pad 2: +5V_TRG -> Net-(C1220-Pad2)
- C1223 pad 1: Net-(C1223-Pad1) -> Net-(C1203-Pad1)
- C1223 pad 2: +5V_TRG -> GND
- C1224 pad 1: Net-(C1224-Pad1) -> Net-(C1203-Pad1)
- C1224 pad 2: +5V_TRG -> GND
- C1225 pad 1: Net-(C1225-Pad1) -> Net-(C1203-Pad1)
- C1225 pad 2: +5V_TRG -> GND
- C1226 pad 1: Net-(C1226-Pad1) -> Net-(C1203-Pad1)
- C1226 pad 2: +5V_TRG -> GND
- C1227 pad 1: Net-(C1203-Pad2) -> GND
- C1228 pad 1: Net-(C1203-Pad2) -> GND
- C1228 pad 2: Net-(C1228-Pad2) -> Net-(C1227-Pad2)
- C1229 pad 1: Net-(C1229-Pad1) -> Net-(C1227-Pad2)
- C1229 pad 2: +5V_TRG -> GND
- C1230 pad 1: Net-(C1230-Pad1) -> Net-(C1227-Pad2)
- C1230 pad 2: +5V_TRG -> GND
- C1231 pad 1: Net-(C1203-Pad2) -> Net-(C1227-Pad2)
- C1231 pad 2: Net-(C1231-Pad2) -> GND
- C1232 pad 1: Net-(C1203-Pad2) -> Net-(C1227-Pad2)
- C1232 pad 2: Net-(C1232-Pad2) -> GND
- C1233 pad 2: Net-(C1233-Pad2) -> GND
- C1234 pad 2: Net-(C1233-Pad2) -> GND
- C1235 pad 1: Net-(C1235-Pad1) -> -15V
- C1235 pad 2: Net-(C1235-Pad2) -> GND
- C1236 pad 1: Net-(C1235-Pad1) -> -15V
- C1236 pad 2: Net-(C1235-Pad2) -> GND
- C1237 pad 1: Net-(C1237-Pad1) -> Net-(C1221-Pad1)
- C1237 pad 2: +5V_TRG -> GNDPWR
- C1238 pad 1: +5V_TRG -> Net-(C1221-Pad1)
- C1238 pad 2: Net-(C1238-Pad2) -> GNDPWR
- C1239 pad 1: Net-(C1239-Pad1) -> GNDPWR
- C1239 pad 2: Net-(C1239-Pad2) -> GND
- C1240 pad 2: Net-(C1240-Pad2) -> GND
- C1241 pad 1: Net-(C1237-Pad1) -> Net-(C1241-Pad1)
- C1241 pad 2: +5V_TRG -> GND
- C1242 pad 1: +5V_TRG -> Net-(C1242-Pad1)
- C1242 pad 2: Net-(C1238-Pad2) -> GND
- C1243 pad 1: Net-(C1237-Pad1) -> Net-(C1203-Pad1)
- C1243 pad 2: +5V_TRG -> Net-(C1243-Pad2)
- C1244 pad 1: Net-(C1238-Pad2) -> Net-(C1203-Pad1)
- C1244 pad 2: +5V_TRG -> GND
- C1245 pad 1: Net-(C1239-Pad1) -> Net-(C1203-Pad1)
- C1245 pad 2: +5V_TRG -> GND
- C1246 pad 1: Net-(C1240-Pad1) -> Net-(C1246-Pad1)
- C1246 pad 2: +5V_TRG -> GND
- C1247 pad 1: Net-(C1237-Pad1) -> Net-(C1246-Pad1)
- C1247 pad 2: +5V_TRG -> GND
- C1248 pad 1: Net-(C1238-Pad2) -> MCU1_3V3
- C1248 pad 2: +5V_TRG -> GND
- C1249 pad 1: Net-(C1239-Pad1) -> MCU1_3V3
- C1249 pad 2: +5V_TRG -> GND
- C1250 pad 1: Net-(C1240-Pad1) -> Net-(C1203-Pad1)
- C1250 pad 2: +5V_TRG -> Net-(C1250-Pad2)
- C1251 pad 1: Net-(C1237-Pad1) -> Net-(C1251-Pad1)
- C1251 pad 2: +5V_TRG -> GND
- C1252 pad 1: Net-(C1238-Pad2) -> Net-(C1252-Pad1)
- C1252 pad 2: +5V_TRG -> GND
- C1253 pad 1: Net-(C1237-Pad1) -> Net-(C1253-Pad1)
- C1253 pad 2: +5V_TRG -> Net-(C1253-Pad2)
- C1254 pad 1: Net-(C1238-Pad2) -> Net-(C1254-Pad1)
- C1254 pad 2: +5V_TRG -> GND
- C1255 pad 1: Net-(C1255-Pad1) -> Net-(C1253-Pad1)
- C1255 pad 2: +5V_TRG -> GND
- C1256 pad 1: Net-(C1256-Pad1) -> Net-(C1253-Pad1)
- C1256 pad 2: +5V_TRG -> GND
- C1257 pad 2: +5V_TRG -> GND
- C1258 pad 1: Net-(C1258-Pad1) -> Net-(C1257-Pad1)
- C1258 pad 2: +5V_TRG -> GND
- C1259 pad 1: Net-(C1259-Pad1) -> MCU2_3V3
- C1259 pad 2: +5V_TRG -> GND
- C1260 pad 1: Net-(C1255-Pad1) -> MCU2_3V3
- C1260 pad 2: +5V_TRG -> GND
- C1261 pad 1: Net-(C1256-Pad1) -> Net-(C1203-Pad1)
- C1261 pad 2: +5V_TRG -> Net-(C1261-Pad2)
- C1262 pad 1: Net-(C1257-Pad1) -> Net-(C1203-Pad1)
- C1262 pad 2: +5V_TRG -> GND
- C1263 pad 1: Net-(C1258-Pad1) -> Net-(C1203-Pad1)
- C1263 pad 2: +5V_TRG -> GND
- C1264 pad 1: Net-(C1259-Pad1) -> Net-(C1203-Pad1)
- C1264 pad 2: +5V_TRG -> Net-(C1264-Pad2)
- C1265 pad 1: +15V -> Net-(C1265-Pad1)
- C1265 pad 2: +5V_TRG -> GND
- C1266 pad 1: -15V -> Net-(C1266-Pad1)
- C1266 pad 2: +5V_TRG -> GND
- C1267 pad 1: MCU1_3V3 -> Net-(C1267-Pad1)
- C1267 pad 2: +5V_TRG -> Net-(C1267-Pad2)
- C1268 pad 1: MCU2_3V3 -> Net-(C1268-Pad1)
- C1268 pad 2: +5V_TRG -> GND
- C1269 pad 1: +5V -> Net-(C1267-Pad1)
- C1269 pad 2: +5V_TRG -> GND
- C1270 pad 1: +15V -> Net-(C1267-Pad1)
- C1270 pad 2: +5V_TRG -> GND
- C1271 pad 1: -15V -> Net-(C1271-Pad1)
- C1271 pad 2: +5V_TRG -> GND
- C1272 pad 1: MCU1_3V3 -> Net-(C1271-Pad1)
- C1272 pad 2: +5V_TRG -> GND
- C1273 pad 1: MCU2_3V3 -> +5V
- C1273 pad 2: +5V_TRG -> GND
- C1274 pad 2: +5V_TRG -> GND
- C1301 pad 2: +5V_TRG -> GND
- C1302 pad 2: +5V_TRG -> GND
- C1303 pad 2: +5V_TRG -> GND
- C1304 pad 2: +5V_TRG -> GND
- C1305 pad 2: +5V_TRG -> GND
- C1306 pad 2: +5V_TRG -> GND
- C1307 pad 2: +5V_TRG -> GND
- C1308 pad 2: +5V_TRG -> GND
- C1309 pad 2: +5V_TRG -> GND
- C1310 pad 2: +5V_TRG -> GND
- C1311 pad 2: +5V_TRG -> GND
- C1312 pad 2: +5V_TRG -> GND
- C1313 pad 2: +5V_TRG -> GND
- C1401 pad 1: +15V -> Net-(C1401-Pad1)
- C1401 pad 2: +5V_TRG -> GND
- C1402 pad 1: +15V -> Net-(C1401-Pad1)
- C1402 pad 2: +5V_TRG -> /Feedback/CurrentBoostOUT
- C1403 pad 1: +15V -> Net-(C1403-Pad1)
- C1403 pad 2: +5V_TRG -> GND
- C1404 pad 1: +15V -> Net-(C1403-Pad1)
- C1404 pad 2: +5V_TRG -> /Feedback/CurrentBoostOUT
- C1405 pad 1: +15V -> Net-(C1405-Pad1)
- C1405 pad 2: +5V_TRG -> GND
- C1406 pad 1: Net-(C1406-Pad1) -> Net-(C1405-Pad1)
- C1406 pad 2: Net-(C1406-Pad2) -> /Feedback/CurrentBoostOUT
- C1407 pad 1: +15V -> Net-(C1407-Pad1)
- C1407 pad 2: +5V_TRG -> GND
- C1408 pad 1: /Feedback/CurrentBoostOUT -> Net-(C1407-Pad1)
- C1408 pad 2: Net-(C1406-Pad1) -> Net-(C1408-Pad2)
- C1409 pad 2: +5V_TRG -> Net-(C1409-Pad2)
- C1410 pad 1: +15V -> /Feedback/CurrentBoostOUT
- C1410 pad 2: +5V_TRG -> Net-(C1409-Pad1)
- C1411 pad 1: +15V -> Net-(C1411-Pad1)
- C1411 pad 2: +5V_TRG -> Net-(C1411-Pad2)
- C1412 pad 2: /Feedback/CurrentBoostOUT -> Net-(C1412-Pad2)
- C1413 pad 2: /Feedback/CurrentBoostOUT -> /Feedback/STIMULUS
- C1414 pad 2: /Feedback/CurrentBoostOUT -> GND
- C1416 pad 1: Net-(C1412-Pad1) -> +15V
- C1416 pad 2: +5V_TRG -> GND
- C1417 pad 1: Net-(C1413-Pad1) -> +15V
- C1417 pad 2: +5V_TRG -> GND
- C1418 pad 1: Net-(C1414-Pad1) -> +15V
- C1418 pad 2: +5V_TRG -> GND
- C1419 pad 1: Net-(C1415-Pad1) -> +15V
- C1419 pad 2: +5V_TRG -> GND
- C1420 pad 1: Net-(C1420-Pad1) -> +15V
- C1420 pad 2: Net-(C1420-Pad2) -> GND
- C1421 pad 1: Net-(C1421-Pad1) -> +15V
- C1421 pad 2: Net-(C1421-Pad2) -> GND
- C1422 pad 1: Net-(C1422-Pad1) -> +15V
- C1422 pad 2: Net-(C1422-Pad2) -> GND
- C1423 pad 1: Net-(C1423-Pad1) -> +15V
- C1423 pad 2: /Feedback/STIMULUS -> GND
- C1501 pad 1: Net-(C1501-Pad1) -> /Address/CODE_3V3
- C1501 pad 2: +5V_TRG -> GND
- C1502 pad 2: +5V_TRG -> GND
- C1503 pad 1: /Address/CODE_3V3 -> Net-(C1503-Pad1)
- C1503 pad 2: +5V_TRG -> GND
- C201 pad 1: /MCU Second/SECOND-NRST -> Net-(C201-Pad1)
- C201 pad 2: +5V_TRG -> GND
- C202 pad 2: +5V_TRG -> GND
- C203 pad 1: +5V_TRG -> Net-(C203-Pad1)
- C203 pad 2: Net-(C203-Pad2) -> GND
- C204 pad 2: +5V_TRG -> GND
- C205 pad 1: Net-(C205-Pad1) -> GND
- C205 pad 2: +5V_TRG -> Net-(C205-Pad2)
- C206 pad 1: Net-(C206-Pad1) -> /MCU Second/SECOND-NRST
- C206 pad 2: +5V_TRG -> GND
- C207 pad 2: +5V_TRG -> GND
- C208 pad 2: +5V_TRG -> GND
- C209 pad 2: +5V_TRG -> GND
- C210 pad 2: +5V_TRG -> GND
- C211 pad 2: +5V_TRG -> GND
- C212 pad 2: +5V_TRG -> GND
- C213 pad 2: +5V_TRG -> GND
- C214 pad 2: +5V_TRG -> GND
- C215 pad 2: +5V_TRG -> GND
- C216 pad 2: +5V_TRG -> GND
- C217 pad 2: +5V_TRG -> GND
- C218 pad 2: +5V_TRG -> GND
- C219 pad 2: +5V_TRG -> GND
- C220 pad 2: +5V_TRG -> GND
- C301 pad 2: +5V_TRG -> GND
- C302 pad 2: +5V_TRG -> GND
- C303 pad 2: +5V_TRG -> GND
- C305 pad 1: +5V -> Net-(C305-Pad1)
- C305 pad 2: +5V_TRG -> Net-(C305-Pad2)
- C306 pad 2: +5V_TRG -> GND
- C307 pad 1: +5V -> +3V3
- C307 pad 2: +5V_TRG -> GND
- C308 pad 2: +5V_TRG -> GND
- C309 pad 1: +5V -> +3V3
- C309 pad 2: +5V_TRG -> GND
- C310 pad 2: +5V_TRG -> GND
- C311 pad 1: +5V -> -15V
- C311 pad 2: +5V_TRG -> GND
- C312 pad 1: +3V3 -> -15V
- C312 pad 2: +5V_TRG -> GND
- C313 pad 1: +5V -> -15V
- C313 pad 2: +5V_TRG -> GND
- C314 pad 1: +3V3 -> -15V
- C314 pad 2: +5V_TRG -> GND
- C315 pad 1: +5V -> -15V
- C315 pad 2: +5V_TRG -> GND
- C316 pad 2: +5V_TRG -> GND
- C317 pad 1: +15V -> -15V
- C317 pad 2: +5V_TRG -> GND
- C318 pad 2: +5V_TRG -> GND
- C319 pad 1: +15V -> -15V
- C319 pad 2: +5V_TRG -> GND
- C320 pad 1: Net-(C320-Pad1) -> -15V
- C320 pad 2: Net-(C320-Pad2) -> GND
- C321 pad 1: -15V -> +5V
- C321 pad 2: +5V_TRG -> GND
- C322 pad 1: +15V -> +5V
- C322 pad 2: +5V_TRG -> GND
- C323 pad 1: -15V -> +5V
- C323 pad 2: +5V_TRG -> GND
- C324 pad 1: +15V -> +5V
- C324 pad 2: +5V_TRG -> GND
- C325 pad 1: -15V -> +5V
- C325 pad 2: +5V_TRG -> GND
- C326 pad 1: +15V -> +5V
- C326 pad 2: +5V_TRG -> GND
- C327 pad 1: -15V -> +15V
- C327 pad 2: +5V_TRG -> GND
- C328 pad 2: +5V_TRG -> GND
- C329 pad 1: -15V -> +15V
- C329 pad 2: +5V_TRG -> GND
- C330 pad 2: +5V_TRG -> GND
- C331 pad 1: -15V -> +15V
- C331 pad 2: +5V_TRG -> GND
- C332 pad 2: +5V_TRG -> GND
- C333 pad 1: -15V -> +15V
- C333 pad 2: +5V_TRG -> GND
- C334 pad 2: +5V_TRG -> GND
- C335 pad 1: -15V -> +15V
- C335 pad 2: +5V_TRG -> GND
- C336 pad 2: +5V_TRG -> GND
- C401 pad 1: +15V -> GND
- C401 pad 2: +5V_TRG -> Net-(C401-Pad2)
- C402 pad 1: +5V_TRG -> Net-(C402-Pad1)
- C403 pad 1: +15V -> GND
- C403 pad 2: +5V_TRG -> Net-(C403-Pad2)
- C404 pad 1: -15V -> Net-(C402-Pad1)
- C404 pad 2: +5V_TRG -> Net-(C404-Pad2)
- C405 pad 1: +5V_TRG -> Net-(C404-Pad2)
- C405 pad 2: -15V -> Net-(C402-Pad2)
- C406 pad 1: Net-(C406-Pad1) -> GND
- C407 pad 1: Net-(C407-Pad1) -> +15V
- C407 pad 2: Net-(C406-Pad2) -> GND
- C408 pad 1: Net-(C406-Pad1) -> +15V
- C408 pad 2: Net-(C407-Pad1) -> GND
- C409 pad 1: +5V_TRG -> -15V
- C409 pad 2: Net-(C409-Pad2) -> GND
- C410 pad 1: +5V_TRG -> GND
- C410 pad 2: Net-(C410-Pad2) -> -15V
- C501 pad 1: +3V3 -> Net-(C501-Pad1)
- C501 pad 2: +5V_TRG -> Net-(C501-Pad2)
- C502 pad 2: +5V_TRG -> GND
- C503 pad 1: +3V3 -> Net-(C503-Pad1)
- C503 pad 2: +5V_TRG -> GND
- C504 pad 1: +5V_TRG -> Net-(C503-Pad1)
- C504 pad 2: Net-(C504-Pad2) -> GND
- C505 pad 1: Net-(C505-Pad1) -> GND
- C505 pad 2: +5V_TRG -> Net-(C505-Pad2)
- C506 pad 1: +3V3 -> Net-(C506-Pad1)
- C506 pad 2: +5V_TRG -> +5V
- C507 pad 1: Net-(C505-Pad1) -> Net-(C507-Pad1)
- C507 pad 2: +5V_TRG -> GND
- C508 pad 1: +3V3 -> Net-(C508-Pad1)
- C508 pad 2: +5V_TRG -> Net-(C508-Pad2)
- C509 pad 1: +15V -> Net-(C509-Pad1)
- C509 pad 2: +5V_TRG -> Net-(C509-Pad2)
- C511 pad 1: +15V -> Net-(C511-Pad1)
- C511 pad 2: +5V_TRG -> Net-(C511-Pad2)
- C513 pad 1: +15V -> Net-(C513-Pad1)
- C513 pad 2: +5V_TRG -> Net-(C512-Pad1)
- C514 pad 1: +15V -> Net-(C511-Pad2)
- C514 pad 2: +5V_TRG -> GND
- C515 pad 1: Net-(C515-Pad1) -> Net-(C511-Pad1)
- C515 pad 2: Net-(C515-Pad2) -> GND
- C516 pad 1: Net-(C516-Pad1) -> Net-(C512-Pad1)
- C516 pad 2: Net-(C516-Pad2) -> GND
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Other:
- board outline added: 160 x 100 mm
