File: HARDWARE/ETH1CSMU1/Ethernet.sch (KiCad schematic (older format))
At the start: 41 parts, among them U901 LAN8742A, U902 USBLC6-4, U903 LC03-3.3, U904 LC03-3.3, X901 7M-25.000MAAJ-T

Commit message: Check in
Parts:
- C904: footprint (none) -> SMD:C_0603_Symbol6
- C909: footprint (none) -> SMD:C_1206_Symbol1
Changed lines of the file:
@@
 F 0 "C904" H 5915 3696 50  0000 L CNN
 F 1 "1u" H 5915 3605 50  0000 L CNN
-F 2 "" H 5838 3500 50  0001 C CNN
+F 2 "SMD:C_0603_Symbol6" H 5838 3500 50  0001 C CNN
 F 3 "~" H 5800 3650 50  0001 C CNN
 	1    5800 3650
@@
 F 0 "C909" H 8165 3696 50  0000 L CNN
 F 1 "10u" H 8165 3605 50  0000 L CNN
-F 2 "" H 8088 3500 50  0001 C CNN
+F 2 "SMD:C_1206_Symbol1" H 8088 3500 50  0001 C CNN
 F 3 "~" H 8050 3650 50  0001 C CNN
 	1    8050 3650

Commit message: Added test circuits, bug fix.
Parts:
- renumbered C910 to C901, C912 to C902, C901 to C910, C902 to C911, C911 to C912, R906 to R901, R907 to R902, R910 to R903, R911 to R904, R913 to R905, R914 to R906, R916 to R907, R902 to R908, R903 to R909, R904 to R910, R905 to R911, R908 to R913, R919 to R914, R920 to R915, R909 to R916, R901 to R917, R915 to R919, R917 to R920, U902 to U901, U903 to U902, U904 to U903, U901 to U904
