File: HARDWARE/ETH1CSMU1/Power.sch (KiCad schematic (older format))
At the start: 150 parts, among them Q1201 IRFR5410, Q1202 Si7456DP, Q1203 SI7850DP, Q1204 FDMC5614P, Q1205 FDMC5614P, U1201 MAX5902, U1202 TEN 40-2415N, U1203 LT3758, U1204 LT3758, U1205 LTC3864, U1206 LTC3864, U1207 NCP1117-ADJ_TO252, U1208 LM337_TO252, U1209 NCP1117-3.3_TO252, U1210 NCP1117-3.3_TO252, U1211 NCP1117-5.0_TO252

Commit message: check in
Parts:
- C1201: footprint (none) -> Capacitors_SMD:C_1210
- D1204, D1205: footprint (none) -> SMD:U-DFN3030-8
- D1206, D1207: footprint (none) -> Diodes_SMD:D_SMC
- L1201, L1202: value L_Coupled -> DRQ127-220; footprint (none) -> SMD:DRQ127
- L1203, L1204: footprint (none) -> SMD:DEM8045C
- Q1202, Q1203, Q1204, Q1205: footprint (none) -> SMD:PowerPAK-SO-8
- R1202: footprint (none) -> SMD:R_0603_Symbol2
- R1204, R1205: value R -> NC; footprint (none) -> Resistors_SMD:R_0603
- U1203, U1204: footprint (none) -> Housings_SSOP:MSOP-10-1EP_3x3mm_Pitch0.5mm
- U1205, U1206: footprint (none) -> Housings_SSOP:MSOP-12-1EP_3x4mm_Pitch0.65mm
Connections:
- net GND: now also L1201.3; no longer L1202.2
- net at C1203.2, C1205.1, C1206.1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: now also L1202.1; no longer L1201.3
- net at C1233.1, C1234.1, D1207.2 (A): now also L1201.4; no longer L1202.1
- net at C1235.2, C1236.2, Q1203.1 (D): now also L1202.2; no longer L1201.4
Other:
- moved on the sheet: L1201B, L1202A
Changed lines of the file:
@@
 F 0 "R1202" H 4820 5996 50  0000 L CNN
 F 1 "R" H 4820 5905 50  0000 L CNN
-F 2 "" V 4680 5950 50  0001 C CNN
+F 2 "SMD:R_0603_Symbol2" V 4680 5950 50  0001 C CNN
 F 3 "~" H 4750 5950 50  0001 C CNN
 	1    4750 5950
@@
 P 8300 5850
 F 0 "R1204" H 8370 5896 50  0000 L CNN
-F 1 "R" H 8370 5805 50  0000 L CNN
-F 2 "" V 8230 5850 50  0001 C CNN
+F 1 "NC" H 8370 5805 50  0000 L CNN
+F 2 "Resistors_SMD:R_0603" V 8230 5850 50  0001 C CNN
 F 3 "~" H 8300 5850 50  0001 C CNN
 	1    8300 5850
@@
 P 8300 6150
 F 0 "R1205" H 8370 6196 50  0000 L CNN
-F 1 "R" H 8370 6105 50  0000 L CNN
-F 2 "" V 8230 6150 50  0001 C CNN
+F 1 "NC" H 8370 6105 50  0000 L CNN
+F 2 "Resistors_SMD:R_0603" V 8230 6150 50  0001 C CNN
 F 3 "~" H 8300 6150 50  0001 C CNN
 	1    8300 6150
@@
 F 0 "C1201" H 5865 6046 50  0000 L CNN
 F 1 "10u/50V" H 5865 5955 50  0000 L CNN
-F 2 "" H 5788 5850 50  0001 C CNN
+F 2 "Capacitors_SMD:C_1210" H 5788 5850 50  0001 C CNN
 F 3 "~" H 5750 6000 50  0001 C CNN
 	1    5750 6000
@@
 F 0 "U1203" H 12400 3350 50  0000 C CNN
 F 1 "LT3758" H 12400 3250 50  0000 C CNN
-F 2 "" H 13900 2550 50  0001 C CNN
+F 2 "Housings_SSOP:MSOP-10-1EP_3x3mm_Pitch0.5mm" H 13900 2550 50  0001 C CNN
 F 3 "" H 13900 2550 50  0001 C CNN
 	1    12150 2500
@@
 F 0 "Q1202" H 13255 1946 50  0000 L CNN
 F 1 "Si7456DP" H 13255 1855 50  0000 L CNN
-F 2 "" H 13250 2000 50  0001 C CNN
+F 2 "SMD:PowerPAK-SO-8" H 13250 2000 50  0001 C CNN
 F 3 "~" H 13050 1900 50  0001 C CNN
 	1    13050 1900
@@
 P 12650 1500
 F 0 "L1201" H 12650 1750 50  0000 C CNN
-F 1 "L_Coupled" H 12650 1650 50  0000 C CNN
-F 2 "" H 12650 1650 50  0001 C CNN
+F 1 " DRQ127-220" H 12650 1650 50  0000 C CNN
+F 2 "SMD:DRQ127" H 12650 1650 50  0001 C CNN
 F 3 "" H 12650 1650 50  0001 C CNN
 	1    12650 1500
@@
 L passive_local:L_Coupled L1202
 U 1 1 5BFE8699
-P 14050 1750
-F 0 "L1202" V 14000 2100 50  0000 C CNN
-F 1 "L_Coupled" V 14100 2100 50  0000 C CNN
-F 2 "" H 14050 1900 50  0001 C CNN
-F 3 "" H 14050 1900 50  0001 C CNN
-	1    14050 1750
-	0    1    1    0
-$EndComp
-Wire Wire Line
-	14050 1550 14050 1500
+P 12650 5250
+F 0 "L1202" H 12650 5500 50  0000 C CNN
+F 1 " DRQ127-220" H 12650 5400 50  0000 C CNN
+F 2 "SMD:DRQ127" H 12650 5400 50  0001 C CNN
+F 3 "" H 12650 5400 50  0001 C CNN
+	1    12650 5250
+	1    0    0    -1
+$EndComp
+Wire Wire Line
+	14050 1650 14050 1500
 Connection ~ 14050 1500
 $Comp
@@
 F 0 "D1207" H 14450 1284 50  0000 C CNN
 F 1 "MBRS3100T3G" H 14450 1375 50  0000 C CNN
-F 2 "" H 14450 1500 50  0001 C CNN
+F 2 "Diodes_SMD:D_SMC" H 14450 1500 50  0001 C CNN
 F 3 "~" H 14450 1500 50  0001 C CNN
 	1    14450 1500
@@
 	12550 4050 14050 4050
 Wire Wire Line
-	14050 4050 14050 1950
+	14050 4050 14050 2050
 Connection ~ 12550 4050
 Wire Wire Line
@@
 F 0 "U1204" H 12400 7100 50  0000 C CNN
 F 1 "LT3758" H 12400 7000 50  0000 C CNN
-F 2 "" H 13900 6300 50  0001 C CNN
+F 2 "Housings_SSOP:MSOP-10-1EP_3x3mm_Pitch0.5mm" H 13900 6300 50  0001 C CNN
 F 3 "" H 13900 6300 50  0001 C CNN
 	1    12150 6250
@@
 F 0 "Q1203" H 13255 5696 50  0000 L CNN
 F 1 "SI7850DP" H 13255 5605 50  0000 L CNN
-F 2 "" H 13250 5750 50  0001 C CNN
+F 2 "SMD:PowerPAK-SO-8" H 13250 5750 50  0001 C CNN
 F 3 "~" H 13050 5650 50  0001 C CNN
 	1    13050 5650
@@
 L passive_local:L_Coupled L1201
 U 2 1 5C08C6B9
-P 12650 5250
-F 0 "L1201" H 12650 5500 50  0000 C CNN
-F 1 "L_Coupled" H 12650 5400 50  0000 C CNN
-F 2 "" H 12650 5400 50  0001 C CNN
-F 3 "" H 12650 5400 50  0001 C CNN
-	2    12650 5250
-	1    0    0    -1
+P 14050 1850
+F 0 "L1201" H 14050 2100 50  0000 C CNN
+F 1 " DRQ127-220" H 14050 2000 50  0000 C CNN
+F 2 "SMD:DRQ127" H 14050 2000 50  0001 C CNN
+F 3 "" H 14050 2000 50  0001 C CNN
+	2    14050 1850
+	0    -1   -1   0
 $EndComp
 Wire Wire Line
@@
 F 0 "D1206" V 14100 5300 50  0000 R CNN
 F 1 "VS-30BQ060" V 14005 5421 50  0000 R CNN
-F 2 "" H 14050 5500 50  0001 C CNN
+F 2 "Diodes_SMD:D_SMC" H 14050 5500 50  0001 C CNN
 F 3 "~" H 14050 5500 50  0001 C CNN
 	1    14050 5500
@@
 P 14450 5250
 F 0 "L1202" H 14450 5500 50  0000 C CNN
-F 1 "L_Coupled" H 14450 5400 50  0000 C CNN
-F 2 "" H 14450 5400 50  0001 C CNN
+F 1 " DRQ127-220" H 14450 5400 50  0000 C CNN
+F 2 "SMD:DRQ127" H 14450 5400 50  0001 C CNN
 F 3 "" H 14450 5400 50  0001 C CNN
 	2    14450 5250
@@
 F 0 "U1205" H 12450 11000 50  0000 C CNN
 F 1 "LTC3864" H 12450 10900 50  0000 C CNN
-F 2 "" H 10550 10800 50  0001 C CNN
+F 2 "Housings_SSOP:MSOP-12-1EP_3x4mm_Pitch0.65mm" H 10550 10800 50  0001 C CNN
 F 3 "" H 10550 10800 50  0001 C CNN
 	1    12150 9950
@@
 F 0 "Q1204" H 13705 9754 50  0000 L CNN
 F 1 "FDMC5614P" H 13705 9845 50  0000 L CNN
-F 2 "" H 13700 9900 50  0001 C CNN
+F 2 "SMD:PowerPAK-SO-8" H 13700 9900 50  0001 C CNN
 F 3 "~" H 13500 9800 50  0001 C CNN
 	1    13500 9800
@@
 F 0 "D1204" V 13550 10400 50  0000 L CNN
 F 1 " SBR3U100LP" V 13645 10229 50  0000 L CNN
-F 2 "" H 13600 10150 50  0001 C CNN
+F 2 "SMD:U-DFN3030-8" H 13600 10150 50  0001 C CNN
 F 3 "~" H 13600 10150 50  0001 C CNN
 	1    13600 10150
@@
 F 0 "L1203" V 14790 10000 50  0000 C CNN
 F 1 "1217AS-H-100M" V 14699 10000 50  0000 C CNN
-F 2 "" H 14600 10000 50  0001 C CNN
+F 2 "SMD:DEM8045C" H 14600 10000 50  0001 C CNN
 F 3 "~" H 14600 10000 50  0001 C CNN
 	1    14600 10000
@@
 F 0 "U1206" H 12450 14300 50  0000 C CNN
 F 1 "LTC3864" H 12450 14200 50  0000 C CNN
-F 2 "" H 10550 14100 50  0001 C CNN
+F 2 "Housings_SSOP:MSOP-12-1EP_3x4mm_Pitch0.65mm" H 10550 14100 50  0001 C CNN
 F 3 "" H 10550 14100 50  0001 C CNN
 	1    12150 13250
@@
 F 0 "Q1205" H 13705 13054 50  0000 L CNN
 F 1 "FDMC5614P" H 13705 13145 50  0000 L CNN
-F 2 "" H 13700 13200 50  0001 C CNN
+F 2 "SMD:PowerPAK-SO-8" H 13700 13200 50  0001 C CNN
 F 3 "~" H 13500 13100 50  0001 C CNN
 	1    13500 13100
@@
 F 0 "D1205" V 13550 13700 50  0000 L CNN
 F 1 " SBR3U100LP" V 13645 13529 50  0000 L CNN
-F 2 "" H 13600 13450 50  0001 C CNN
+F 2 "SMD:U-DFN3030-8" H 13600 13450 50  0001 C CNN
 F 3 "~" H 13600 13450 50  0001 C CNN
 	1    13600 13450
@@
 F 0 "L1204" V 14790 13300 50  0000 C CNN
 F 1 "1217AS-H-100M" V 14699 13300 50  0000 C CNN
-F 2 "" H 14600 13300 50  0001 C CNN
+F 2 "SMD:DEM8045C" H 14600 13300 50  0001 C CNN
 F 3 "~" H 14600 13300 50  0001 C CNN
 	1    14600 13300

Commit message: Check in
Parts:
- removed C1237, C1238, C1241, C1242: 47u, symbol Device:C
- added C1237, C1238, C1241, C1242: 47u, Capacitors_Tantalum_SMD:CP_Tantalum_Case-X_EIA-7343-43_Hand, symbol Device:CP
- C1211, C1212: value 12u/50V -> 10u/50V; footprint (none) -> Capacitors_SMD:C_1210
- C1233, C1234, C1235, C1236: footprint Capacitors_SMD:C_1206_HandSoldering -> SMD:C_1206_Symbol3
- C1243, C1244, C1247, C1248, C1251, C1252, C1253, C1254, C1255, C1256, C1257, C1258, C1259, C1265, C1266, C1267, C1268, C1269: footprint (none) -> SMD:C_1206_Symbol1
- C1245, C1246, C1249, C1250: footprint (none) -> SMD:C_1210_2
- C1260, C1261, C1262, C1263, C1264, C1270, C1271, C1272, C1273, C1274: footprint (none) -> SMD:C_1206_Symbol2
- D1202: value D_Zener -> SZMMSZ4705T1; footprint (none) -> SMD:SOD-323F
- R1202: footprint SMD:R_0603_Symbol2 -> Resistors_SMD:R_0603
- R1203: footprint (none) -> Resistors_SMD:R_1206
Connections:
- net GND: now also C1237.2, C1238.1, C1241.2, C1242.1
- net at C1244.1, C1248.1, C1252.1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: now also C1238.2, C1242.2
- net at C1243.1, C1247.1, C1251.1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: now also C1237.1, C1241.1
Other:
- moved on the sheet: D1201, F1201, Q1201, R1201, U1201

Commit message: Added test circuits, bug fix.
Parts:
- renumbered C1233 to C1201, C1234 to C1202, C1205 to C1203, C1207 to C1204, C1209 to C1205, C1213 to C1206, C1237 to C1207, C1241 to C1208, C1243 to C1209, C1247 to C1210, C1251 to C1211, C1253 to C1212, C1255 to C1213, C1260 to C1214, C1265 to C1215, C1270 to C1216, C1223 to C1217, C1229 to C1218, C1225 to C1219, C1235 to C1220, C1203 to C1221, C1236 to C1222, C1206 to C1223, C1208 to C1224, C1210 to C1225, C1214 to C1226, C1238 to C1227, C1242 to C1228, C1244 to C1229, C1248 to C1230, C1252 to C1231, C1254 to C1232, C1256 to C1233, C1261 to C1234, C1266 to C1235, C1271 to C1236, C1201 to C1237, C1202 to C1238, C1204 to C1239, C1224 to C1240, C1230 to C1241, C1226 to C1242, C1227 to C1243, C1211 to C1244, C1215 to C1245, C1257 to C1246, C1262 to C1247, C1267 to C1248, C1272 to C1249, C1231 to C1250, C1221 to C1251, C1217 to C1252, C1239 to C1253, C1218 to C1254, C1245 to C1255, C1249 to C1256, C1258 to C1257, C1263 to C1258, C1268 to C1259, C1273 to C1260, C1228 to C1261, C1212 to C1262, C1216 to C1263, C1232 to C1264, C1222 to C1265, C1219 to C1266, C1240 to C1267, C1220 to C1268, C1246 to C1269, C1250 to C1270, C1259 to C1271, C1264 to C1272, C1269 to C1273, D1207 to D1201, D1206 to D1202, D1202 to D1203, D1201 to D1204, D1203 to D1205, D1204 to D1206, D1205 to D1207, Q1202 to Q1201, Q1201 to Q1202, R1212 to R1201, R1242 to R1202, R1213 to R1203, R1241 to R1204, R1222 to R1205, R1238 to R1206, R1228 to R1207, R1229 to R1208, R1206 to R1209, R1218 to R1210, R1214 to R1211, R1243 to R1212, R1201 to R1213, R1203 to R1214, R1204 to R1216, R1239 to R1217, R1202 to R1218, R1205 to R1219, R1223 to R1220, R1240 to R1221, R1230 to R1222, R1231 to R1223, R1207 to R1224, R1219 to R1225, R1216 to R1226, R1226 to R1227, R1224 to R1228, R1220 to R1229, R1208 to R1230, R1232 to R1231, R1234 to R1232, R1209 to R1233, R1235 to R1234, R1217 to R1235, R1227 to R1236, R1225 to R1237, R1221 to R1238, R1210 to R1239, R1233 to R1240, R1236 to R1241, R1211 to R1242, R1237 to R1243, U1207 to U1201, U1203 to U1202, U1208 to U1203, U1201 to U1204, U1202 to U1205, U1204 to U1206, U1209 to U1207, U1205 to U1208, U1210 to U1209, U1206 to U1210
