File: hardware/project/ETH1CSMU1BASE/Ethernet.sch (KiCad schematic (older format))
At the start: 43 parts, among them U401 LC03-3.3, U402 LAN8742A, U403 LC03-3.3, Y401 NX5032GA-25.000M-LN-CD-1

Commit message: Schematic developement, new footprints.
Parts:
- U401, U403: footprint ETH6C20MUX:SO8E -> ETH1CSMU1:SO8E
- Y401: footprint ETH6C20MUX:NX5032GA -> ETH1CSMU1:NX5032GA
Changed lines of the file:
@@
 $Descr A4 11693 8268
 encoding utf-8
-Sheet 3 6
+Sheet 3 7
 Title "Ethernet"
 Date ""
@@
 F 0 "U401" H 10450 3287 60  0000 C CNN
 F 1 "LC03-3.3" H 10450 3181 60  0000 C CNN
-F 2 "ETH6C20MUX:SO8E" H 10450 2850 60  0001 C CNN
+F 2 "ETH1CSMU1:SO8E" H 10450 2850 60  0001 C CNN
 F 3 "" H 10450 2850 60  0000 C CNN
 	1    10450 2850
@@
 F 0 "U403" H 10450 4087 60  0000 C CNN
 F 1 "LC03-3.3" H 10450 3981 60  0000 C CNN
-F 2 "ETH6C20MUX:SO8E" H 10450 3650 60  0001 C CNN
+F 2 "ETH1CSMU1:SO8E" H 10450 3650 60  0001 C CNN
 F 3 "" H 10450 3650 60  0000 C CNN
 	1    10450 3650
@@
 F 0 "Y401" H 1900 4482 50  0000 C CNN
 F 1 "NX5032GA-25.000M-LN-CD-1" H 1900 4573 50  0000 C CNN
-F 2 "ETH6C20MUX:NX5032GA" H 1900 4750 50  0001 C CNN
+F 2 "ETH1CSMU1:NX5032GA" H 1900 4750 50  0001 C CNN
 F 3 "~" H 1900 4750 50  0001 C CNN
 	1    1900 4750
