File: hardware/project/ETH1CSMU1BASE/MCU.sch (KiCad schematic (older format))
At the start: 0 parts

Commit message: Base board schematic.
Parts:
- added C301, C307, C308, C309, C310, C311, C312, C313, C314, C315, C316, C317, C318, C?: 100n, symbol Device:C
- added C302, C303: 8p, symbol Device:C
- added C304, C305: 2u2, symbol Device:C
- added C306, C319: 1u, symbol Device:C
- added FB301: 742792031, symbol Device:Ferrite_Bead
- added J301: Conn_02x05, symbol Connector_Generic:Conn_02x05_Odd_Even
- added J302: Conn_02x01, symbol Connector_Generic:Conn_02x01
- added R301, R302, R303: 10k, symbol Device:R
- added R? (x2): 4k7, symbol Device:R
- added U?: STM32F765ZGT6, symbol ETH1CSMU1:STM32F765ZGT6
- added U?: 24LC08, symbol Memory_EEPROM:24LC08
- added Y301: NX3225GD-8MHZ-STD-CRA-3, symbol Device:Crystal
Connections:
- new net: R302.1, U?.138 (BOOT0)
- new net: C305.1, U?.106 (VCAP_2)
- new net: C304.1, U?.71 (VCAP_1)
- new net: C302.1, U?.23 (PH0,EVENTOUT,OSC_IN), Y301.1
- new net: C303.1, U?.24 (PH1,EVENTOUT,OSC_OUT), Y301.2
- new net +3V3: C306.1, C307.1, C308.1, C309.1, C310.1, C311.1, C312.1, C313.1, C314.1, C315.1, C316.1, C317.1, C318.1, C?.1, FB301.2, J301.1 (Pin_1), R301.1, R303.2, R?.1, R?.1, U?.108 (VDD), U?.121 (VDDSDMMC), U?.131 (VDD), U?.143 (PDR_ON), U?.144 (VDD), U?.17 (VDD), U?.30 (VDD), U?.39 (VDD), U?.52 (VDD), U?.6 (VBAT), U?.62 (VDD), U?.72 (VDD), U?.8 (VCC), U?.84 (VDD), U?.95 (VDDUSB)
- new net BASE_GPIO_OUT1: U?.7 (PC13,EVENTOUT,RTC_TAMP2,RTC_TS,WKUP5)
- new net BASE_GPIO_OUT2: U?.8 (PC14,EVENTOUT,OSC32_IN)
- new net BASE_MCLK: U?.19 (PF7,TIM11_CH1,SPI5_SCK,SAI1_MCLK_B,UART7_TX,QUADSPI_BK1_IO2,EVENTOUT,ADC3_IN5)
- new net BASE_MISO: U?.20 (PF8,SPI5_MISO,SAI1_SCK_B,UART7_RTS,TIM13_CH1,QUADSPI_BK1_IO0,EVENTOUT,ADC3_IN6)
- new net BASE_MOSI: U?.21 (PF9,SPI5_MOSI,SAI1_FS_B,UART7_CTS,TIM14_CH1,QUADSPI_BK1_IO1,EVENTOUT,ADC3_IN7)
- new net BASE_STATUS_IN: U?.9 (PC15,EVENTOUT,OSC32_OUT)
- new net BASE_~MSS: U?.18 (PF6,TIM10_CH1,SPI5_NSS,SAI1_SD_B,UART7_RX,QUADSPI_BK1_IO3,EVENTOUT,ADC3_IN4)
- new net EEPROM_SCL: R?.2, U?.54 (PF14,I2C4_SCL,DFSDM1_CKIN6,FMC_A8,EVENTOUT), U?.6 (SCL)
- new net EEPROM_SDA: R?.2, U?.5 (SDA), U?.55 (PF15,I2C4_SDA,FMC_A9,EVENTOUT)
- new net EEPROM_WP: U?.53 (PF13,I2C4_SMBA,DFSDM1_DATIN6,FMC_A7,EVENTOUT), U?.7 (WP)
- new net GND: C301.2, C302.2, C303.2, C304.2, C305.2, C306.2, C307.2, C308.2, C309.2, C310.2, C311.2, C312.2, C313.2, C314.2, C315.2, C316.2, C317.2, C318.2, C319.2, C?.2, J301.3 (Pin_3), J301.5 (Pin_5), J302.2 (Pin_2), R302.2, U?.1 (A0), U?.107 (VSS), U?.120 (VSS), U?.130 (VSS), U?.16 (VSS), U?.2 (A1), U?.3 (A2), U?.31 (VSSA), U?.38 (VSS), U?.4 (GND), U?.51 (VSS), U?.61 (VSS), U?.83 (VSS), U?.94 (VSS)
- new net MCU_DEFAULT: J302.1 (Pin_1), R303.1
- new net MCU_VDDA: C319.1, FB301.1, U?.32 (VREF+), U?.33 (VDDA)
- new net NRST: C301.1, J301.10 (Pin_10), R301.2, U?.25 (NRST)
- new net REF_CLK: U?.35 (PA1,TIM2_CH2,TIM5_CH2,UART2_RTS,UART4_RX,QUADSPI_BK1_IO3,SAI2_MCLK_B,ETH_MII_RX_CLK,ETH_RMII_REF_CLK,LCD_R2,EVENTOUT,ADC1_IN1,ADC2_IN1,ADC3_IN1)
- new net RMII_CRS_DV: U?.43 (PA7,TIM1_CH1N,TIM3_CH2,TIM8_CH1N,SPI1_MOSI,I2S1_SD,SPI6_MOSI,TIM14_CH1,ETH_MII_RX_DV,ETH_RMII_CRS_DV,FMC_SDNWE,EVENTOUT,ADC1_IN7,ADC2_IN7)
- new net RMII_MDC: U?.27 (PC1,TRACED0,_DFSDM1_DATIN0,SPI2_MOSI,I2S2_SD,SAI1_SD_A,DFSDM1_CKIN4,ETH_MDC,MDIOS_MDC,EVENTOUT,ADC1_IN11,ADC2_IN11,ADC3_IN11,RTC_TAMP3,WKUP3)
- new net RMII_MDIO: U?.36 (PA2,TIM2_CH3,TIM5_CH3,TIM9_CH1,USART2_TX,SAI2_SCK_B,ETH_MDIO,MDIOS_MDIO,LCD_R1,EVENTOUT,ADC1_IN2,ADC2_IN2,ADC3_IN2,WKUP2)
- new net RMII_RXD0: U?.44 (PC4,DFSDM1_CKIN2,I2S1_MCK,SPDIF_RX2,ETH_MII_RXD0,ETH_RMII_RXD0,FMC_SDNE0,EVENTOUT,ADC1_IN14,ADC2_IN14)
- new net RMII_RXD1: U?.45 (PC5,DFSDM1_DATIN2,SPDIF_RX3,ETH_MII_RXD1,ETH_RMII_RXD1,FMC_SDCKE0,EVENTOUT,ADC1_IN15,ADC2_IN15)
- new net RMII_TXD0: U?.128 (PG13,TRACED0,LPTIM1_OUT,SPI6_SCK,USART6_CTS,ETH_MII_TXD0,ETH_RMII_TXD0,FMC_A24,LCD_R0,EVENTOUT)
- new net RMII_TXD1: U?.129 (PG14,TRACED1,LPTIM1_ETR,SPI6_MOSI,USART6_TX,QUADSPI_BK2_IO3,ETH_MII_TXD1,ETH_RMII_TXD1,FMC_A25,LCD_B0,EVENTOUT)
- new net RMII_TXEN: U?.126 (PG11,SPI1_SCK,I2S1_CK,SPDIF_RX0,SDMMC2_D2,ETH_MII_TX_EN,ETH_RMII_TX_EN,DCMI_D3,LCD_B3,EVENTOUT)
- new net SPI3_MISO: U?.112 (PC11,DFSDM1_DATIN5,SPI3_MISO,USART3_RX,UART4_RX,QUADSPI_BK2_NCS,SDMMC1_D3,DCMI_D4,EVENTOUT)
- new net SPI3_MOSI: U?.113 (PC12,TRACED3,SPI3_MOSI,I2S3_SD,USART3_CK,UART5_TX,SDMMC1_CK,DCMI_D9,EVENTOUT)
- new net SPI3_SCLK: U?.111 (PC10,DFSDM1_CKIN5,SPI3_SCK,I2S3_CK,USART3_TX,UART4_TX,QUADSPI_BK1_IO1,SDMMC1_D2,DCMI_D8,LCD_R2,EVENTOUT)
- new net TCK_SWCLK: J301.4 (Pin_4), U?.109 (PA14,JTCK-SWCLK,EVENTOUT)
- new net TDI: J301.8 (Pin_8), U?.110 (PA15,JTDI,TIM2_CH1,TIM2_ETR,HDMI_CEC,SPI1_NSS,I2S1_WS,SPI3_NSS,I2S3_WS,SPI6_NSS,UART4_RTS,CAN3_TX,UART7_TX,EVENTOUT)
- new net TDO: J301.6 (Pin_6), U?.133 (PB3,JTDO,TRACESWO,TIM2_CH2,SPI1_SCK,I2S1_CK,SPI3_SCK,I2S3_CK,SPI6_SCK,SDMMC2_D2,CAN3_RX,UART7_RX,EVENTOUT)
- new net TMS_SWDIO: J301.2 (Pin_2), U?.105 (PA13,JTMS-SWDIO,EVENTOUT)
- new net TRIG_EN: U?.74 (PB13,TIM1_CH1N,SPI2_SCK,I2S2_CK,DFSDM1_CKIN1,USART3_CTS,UART5_TX,CAN2_TX,OTG_HS_ULPI_D6,ETH_MII_TXD1,ETH_RMII_TXD1,EVENTOUT,OTG_HS_VBUS)
- new net TRIG_IN: U?.76 (PB15,RTC_REFIN,TIM1_CH3N,TIM8_CH3N,USART1_RX,SPI2_MOSI,I2S2_SD,DFSDM1_CKIN2,UART4_CTS,TIM12_CH2,SDMMC2_D1,OTG_HS_DP,EVENTOUT)
- new net TRIG_OUT: U?.75 (PB14,TIM1_CH2N,TIM8_CH2N,USART1_TX,SPI2_MISO,DFSDM1_DATIN2,USART3_RTS,UART4_RTS,TIM12_CH1,SDMMC2_D0,OTG_HS_DM,EVENTOUT)
- no-connect marks 0 -> 2
Other:
- note added: "PROGRAMMING CONNECTOR\nDESIGNED FOR JLINK"

Commit message: Schematic developement, new footprints.
Parts:
- C201: renamed from C?; footprint (none) -> Capacitor_SMD:C_0603_1608Metric_Pad1.05x0.95mm_HandSolder
- C301, C302, C303, C307, C308, C309, C310, C311, C312, C313, C314, C315, C316, C317, C318: footprint (none) -> Capacitor_SMD:C_0603_1608Metric_Pad1.05x0.95mm_HandSolder
- FB301: footprint (none) -> Resistor_SMD:R_0805_2012Metric_Pad1.15x1.40mm_HandSolder
- R201, R202: renamed from R?; footprint (none) -> Resistor_SMD:R_0603_1608Metric_Pad1.05x0.95mm_HandSolder
- R301, R302, R303: footprint (none) -> Resistor_SMD:R_0603_1608Metric_Pad1.05x0.95mm_HandSolder
- U201: renamed from U?; footprint (none) -> ETH1CSMU1:TQFP-144_20x20mm_P0.5mm
- gave numbers to parts that had none: 1
Changed lines of the file:
@@
 $Descr A3 16535 11693
 encoding utf-8
-Sheet 2 6
+Sheet 2 7
 Title ""
 Date ""
@@
 F 0 "R302" H 14720 8896 50  0000 L CNN
 F 1 "10k" H 14720 8805 50  0000 L CNN
-F 2 "" V 14580 8850 50  0001 C CNN
+F 2 "Resistor_SMD:R_0603_1608Metric_Pad1.05x0.95mm_HandSolder" V 14580 8850 50  0001 C CNN
 F 3 "~" H 14650 8850 50  0001 C CNN
 	1    14650 8850
@@
 F 0 "R301" H 15320 8096 50  0000 L CNN
 F 1 "10k" H 15320 8005 50  0000 L CNN
-F 2 "" V 15180 8050 50  0001 C CNN
+F 2 "Resistor_SMD:R_0603_1608Metric_Pad1.05x0.95mm_HandSolder" V 15180 8050 50  0001 C CNN
 F 3 "~" H 15250 8050 50  0001 C CNN
 	1    15250 8050
@@
 F 0 "C301" H 15365 8496 50  0000 L CNN
 F 1 "100n" H 15365 8405 50  0000 L CNN
-F 2 "" H 15288 8300 50  0001 C CNN
+F 2 "Capacitor_SMD:C_0603_1608Metric_Pad1.05x0.95mm_HandSolder" H 15288 8300 50  0001 C CNN
 F 3 "~" H 15250 8450 50  0001 C CNN
 	1    15250 8450
@@
 F 0 "C307" H 815 10746 50  0000 L CNN
 F 1 "100n" H 815 10655 50  0000 L CNN
-F 2 "" H 738 10550 50  0001 C CNN
+F 2 "Capacitor_SMD:C_0603_1608Metric_Pad1.05x0.95mm_HandSolder" H 738 10550 50  0001 C CNN
 F 3 "~" H 700 10700 50  0001 C CNN
 	1    700  10700
@@
 F 0 "C308" H 1315 10746 50  0000 L CNN
 F 1 "100n" H 1315 10655 50  0000 L CNN
-F 2 "" H 1238 10550 50  0001 C CNN
+F 2 "Capacitor_SMD:C_0603_1608Metric_Pad1.05x0.95mm_HandSolder" H 1238 10550 50  0001 C CNN
 F 3 "~" H 1200 10700 50  0001 C CNN
 	1    1200 10700
@@
 F 0 "C309" H 1815 10746 50  0000 L CNN
 F 1 "100n" H 1815 10655 50  0000 L CNN
-F 2 "" H 1738 10550 50  0001 C CNN
+F 2 "Capacitor_SMD:C_0603_1608Metric_Pad1.05x0.95mm_HandSolder" H 1738 10550 50  0001 C CNN
 F 3 "~" H 1700 10700 50  0001 C CNN
 	1    1700 10700
@@
 F 0 "C310" H 2315 10746 50  0000 L CNN
 F 1 "100n" H 2315 10655 50  0000 L CNN
-F 2 "" H 2238 10550 50  0001 C CNN
+F 2 "Capacitor_SMD:C_0603_1608Metric_Pad1.05x0.95mm_HandSolder" H 2238 10550 50  0001 C CNN
 F 3 "~" H 2200 10700 50  0001 C CNN
 	1    2200 10700
@@
 F 0 "C311" H 2815 10746 50  0000 L CNN
 F 1 "100n" H 2815 10655 50  0000 L CNN
-F 2 "" H 2738 10550 50  0001 C CNN
+F 2 "Capacitor_SMD:C_0603_1608Metric_Pad1.05x0.95mm_HandSolder" H 2738 10550 50  0001 C CNN
 F 3 "~" H 2700 10700 50  0001 C CNN
 	1    2700 10700
@@
 F 0 "C312" H 3315 10746 50  0000 L CNN
 F 1 "100n" H 3315 10655 50  0000 L CNN
-F 2 "" H 3238 10550 50  0001 C CNN
+F 2 "Capacitor_SMD:C_0603_1608Metric_Pad1.05x0.95mm_HandSolder" H 3238 10550 50  0001 C CNN
 F 3 "~" H 3200 10700 50  0001 C CNN
 	1    3200 10700
@@
 F 0 "C313" H 3815 10746 50  0000 L CNN
 F 1 "100n" H 3815 10655 50  0000 L CNN
-F 2 "" H 3738 10550 50  0001 C CNN
+F 2 "Capacitor_SMD:C_0603_1608Metric_Pad1.05x0.95mm_HandSolder" H 3738 10550 50  0001 C CNN
 F 3 "~" H 3700 10700 50  0001 C CNN
 	1    3700 10700
@@
 F 0 "C314" H 4315 10746 50  0000 L CNN
 F 1 "100n" H 4315 10655 50  0000 L CNN
-F 2 "" H 4238 10550 50  0001 C CNN
+F 2 "Capacitor_SMD:C_0603_1608Metric_Pad1.05x0.95mm_HandSolder" H 4238 10550 50  0001 C CNN
 F 3 "~" H 4200 10700 50  0001 C CNN
 	1    4200 10700
@@
 F 0 "C315" H 4815 10746 50  0000 L CNN
 F 1 "100n" H 4815 10655 50  0000 L CNN
-F 2 "" H 4738 10550 50  0001 C CNN
+F 2 "Capacitor_SMD:C_0603_1608Metric_Pad1.05x0.95mm_HandSolder" H 4738 10550 50  0001 C CNN
 F 3 "~" H 4700 10700 50  0001 C CNN
 	1    4700 10700
@@
 F 0 "C316" H 5315 10746 50  0000 L CNN
 F 1 "100n" H 5315 10655 50  0000 L CNN
-F 2 "" H 5238 10550 50  0001 C CNN
+F 2 "Capacitor_SMD:C_0603_1608Metric_Pad1.05x0.95mm_HandSolder" H 5238 10550 50  0001 C CNN
 F 3 "~" H 5200 10700 50  0001 C CNN
 	1    5200 10700
@@
 F 0 "C317" H 5815 10746 50  0000 L CNN
 F 1 "100n" H 5815 10655 50  0000 L CNN
-F 2 "" H 5738 10550 50  0001 C CNN
+F 2 "Capacitor_SMD:C_0603_1608Metric_Pad1.05x0.95mm_HandSolder" H 5738 10550 50  0001 C CNN
 F 3 "~" H 5700 10700 50  0001 C CNN
 	1    5700 10700
@@
 F 0 "C318" H 6315 10746 50  0000 L CNN
 F 1 "100n" H 6315 10655 50  0000 L CNN
-F 2 "" H 6238 10550 50  0001 C CNN
+F 2 "Capacitor_SMD:C_0603_1608Metric_Pad1.05x0.95mm_HandSolder" H 6238 10550 50  0001 C CNN
 F 3 "~" H 6200 10700 50  0001 C CNN
 	1    6200 10700
@@
 F 0 "FB301" V 6726 10500 50  0000 C CNN
 F 1 "742792031" V 6817 10500 50  0000 C CNN
-F 2 "" V 6930 10500 50  0001 C CNN
+F 2 "Resistor_SMD:R_0805_2012Metric_Pad1.15x1.40mm_HandSolder" V 6930 10500 50  0001 C CNN
 F 3 "~" H 7000 10500 50  0001 C CNN
 	1    7000 10500
@@
 F 0 "R303" H 7980 10154 50  0000 R CNN
 F 1 "10k" H 7980 10245 50  0000 R CNN
-F 2 "" V 7980 10200 50  0001 C CNN
+F 2 "Resistor_SMD:R_0603_1608Metric_Pad1.05x0.95mm_HandSolder" V 7980 10200 50  0001 C CNN
 F 3 "~" H 8050 10200 50  0001 C CNN
 	1    8050 10200
@@
 F 0 "C303" H 1915 1646 50  0000 L CNN
 F 1 "8p" H 1915 1555 50  0000 L CNN
-F 2 "" H 1838 1450 50  0001 C CNN
+F 2 "Capacitor_SMD:C_0603_1608Metric_Pad1.05x0.95mm_HandSolder" H 1838 1450 50  0001 C CNN
 F 3 "~" H 1800 1600 50  0001 C CNN
 	1    1800 1600
@@
 F 0 "C302" H 1415 1646 50  0000 L CNN
 F 1 "8p" H 1415 1555 50  0000 L CNN
-F 2 "" H 1338 1450 50  0001 C CNN
+F 2 "Capacitor_SMD:C_0603_1608Metric_Pad1.05x0.95mm_HandSolder" H 1338 1450 50  0001 C CNN
 F 3 "~" H 1300 1600 50  0001 C CNN
 	1    1300 1600
@@
 PROGRAMMING CONNECTOR\nDESIGNED FOR JLINK
 $Comp
-L ETH1CSMU1:STM32F765ZGT6 U?
+L ETH1CSMU1:STM32F765ZGT6 U201
 U 1 1 5DC8ECD0
 P 8900 4900
-F 0 "U?" H 3450 8800 50  0000 C CNN
+F 0 "U201" H 3450 8800 50  0000 C CNN
 F 1 "STM32F765ZGT6" H 14050 8800 50  0000 C CNN
-F 2 "" H 24800 6400 50  0001 C CNN
+F 2 "ETH1CSMU1:TQFP-144_20x20mm_P0.5mm" H 24800 6400 50  0001 C CNN
 F 3 "" H 24800 6400 50  0001 C CNN
 	1    8900 4900
@@
 NRST
 $Comp
-L Memory_EEPROM:24LC08 U?
+L Memory_EEPROM:24LC08 U202
 U 1 1 5E082698
 P 1050 4950
-F 0 "U?" H 1250 5300 50  0000 C CNN
+F 0 "U202" H 1250 5300 50  0000 C CNN
 F 1 "24LC08" H 1250 5200 50  0000 C CNN
 F 2 "" H 1050 4950 50  0001 C CNN
@@
 $EndComp
 $Comp
-L power:+3.3V #PWR?
+L power:+3.3V #PWR0101
 U 1 1 5E08AE5B
 P 1050 4650
-F 0 "#PWR?" H 1050 4500 50  0001 C CNN
+F 0 "#PWR0101" H 1050 4500 50  0001 C CNN
 F 1 "+3.3V" H 1065 4823 50  0000 C CNN
 F 2 "" H 1050 4650 50  0001 C CNN
@@
 $EndComp
 $Comp
-L power:GND #PWR?
+L power:GND #PWR0102
 U 1 1 5E08CDE4
 P 1050 5250
-F 0 "#PWR?" H 1050 5000 50  0001 C CNN
+F 0 "#PWR0102" H 1050 5000 50  0001 C CNN
 F 1 "GND" H 1055 5077 50  0000 C CNN
 F 2 "" H 1050 5250 50  0001 C CNN
@@
 	600  5050 650  5050
 $Comp
-L power:GND #PWR?
+L power:GND #PWR0103
 U 1 1 5E096BB8
 P 600 5250
-F 0 "#PWR?" H 600 5000 50  0001 C CNN
+F 0 "#PWR0103" H 600 5000 50  0001 C CNN
 F 1 "GND" H 605 5077 50  0000 C CNN
 F 2 "" H 600 5250 50  0001 C CNN
@@
 EEPROM_SDA
 $Comp
-L Device:R R?
+L Device:R R201
 U 1 1 5E0F3906
 P 2000 4650
-F 0 "R?" H 2070 4696 50  0000 L CNN
+F 0 "R201" H 2070 4696 50  0000 L CNN
 F 1 "4k7" H 2070 4605 50  0000 L CNN
-F 2 "" V 1930 4650 50  0001 C CNN
+F 2 "Resistor_SMD:R_0603_1608Metric_Pad1.05x0.95mm_HandSolder" V 1930 4650 50  0001 C CNN
 F 3 "~" H 2000 4650 50  0001 C CNN
 	1    2000 4650
@@
 $EndComp
 $Comp
-L Device:R R?
+L Device:R R202
 U 1 1 5E0F3C03
 P 2350 4650
-F 0 "R?" H 2420 4696 50  0000 L CNN
+F 0 "R202" H 2420 4696 50  0000 L CNN
 F 1 "4k7" H 2420 4605 50  0000 L CNN
-F 2 "" V 2280 4650 50  0001 C CNN
+F 2 "Resistor_SMD:R_0603_1608Metric_Pad1.05x0.95mm_HandSolder" V 2280 4650 50  0001 C CNN
 F 3 "~" H 2350 4650 50  0001 C CNN
 	1    2350 4650
@@
 	2350 4450 2350 4500
 $Comp
-L power:+3.3V #PWR?
+L power:+3.3V #PWR0104
 U 1 1 5E117FC1
 P 2350 4400
-F 0 "#PWR?" H 2350 4250 50  0001 C CNN
+F 0 "#PWR0104" H 2350 4250 50  0001 C CNN
 F 1 "+3.3V" H 2365 4573 50  0000 C CNN
 F 2 "" H 2350 4400 50  0001 C CNN
@@
 	3200 2850 2700 2850
 $Comp
-L Device:C C?
+L Device:C C201
 U 1 1 5E17592C
 P 700 9800
-F 0 "C?" H 815 9846 50  0000 L CNN
+F 0 "C201" H 815 9846 50  0000 L CNN
 F 1 "100n" H 815 9755 50  0000 L CNN
-F 2 "" H 738 9650 50  0001 C CNN
+F 2 "Capacitor_SMD:C_0603_1608Metric_Pad1.05x0.95mm_HandSolder" H 738 9650 50  0001 C CNN
 F 3 "~" H 700 9800 50  0001 C CNN
 	1    700  9800
@@
 $EndComp
 $Comp
-L power:+3.3V #PWR?
+L power:+3.3V #PWR0105
 U 1 1 5E176017
 P 700 9550
-F 0 "#PWR?" H 700 9400 50  0001 C CNN
+F 0 "#PWR0105" H 700 9400 50  0001 C CNN
 F 1 "+3.3V" H 715 9723 50  0000 C CNN
 F 2 "" H 700 9550 50  0001 C CNN
@@
 $EndComp
 $Comp
-L power:GND #PWR?
+L power:GND #PWR0106
 U 1 1 5E1764D7
 P 700 10050
-F 0 "#PWR?" H 700 9800 50  0001 C CNN
+F 0 "#PWR0106" H 700 9800 50  0001 C CNN
 F 1 "GND" H 705 9877 50  0000 C CNN
 F 2 "" H 700 10050 50  0001 C CNN

Commit message: Power supply design
Parts:
- U201: symbol ETH1CSMU1:STM32F765ZGT6 -> ETH1CSMU1BASE-rescue:STM32F765ZGT6-ETH1CSMU1
Changed lines of the file:
@@
 EESchema Schematic File Version 4
-LIBS:ETH1CSMU1BASE-cache
 EELAYER 30 0
 EELAYER END
@@
 PROGRAMMING CONNECTOR\nDESIGNED FOR JLINK
 $Comp
-L ETH1CSMU1:STM32F765ZGT6 U201
+L ETH1CSMU1BASE-rescue:STM32F765ZGT6-ETH1CSMU1 U201
 U 1 1 5DC8ECD0
 P 8900 4900
+AR Path="/5DC8ECD0" Ref="U201"  Part="1"
+AR Path="/5D98FDB4/5DC8ECD0" Ref="U201"  Part="1"
 F 0 "U201" H 3450 8800 50  0000 C CNN
 F 1 "STM32F765ZGT6" H 14050 8800 50  0000 C CNN

Commit message: Footprint assigment
Parts:
- C304, C305, C306, C319: footprint (none) -> Capacitor_SMD:C_0603_1608Metric_Pad1.05x0.95mm_HandSolder
- J301: footprint (none) -> Connector_PinHeader_1.27mm:PinHeader_2x05_P1.27mm_Vertical
- U202: footprint (none) -> Package_SO:MSOP-8_3x3mm_P0.65mm
Changed lines of the file:
@@
 F 0 "J301" H 9900 10867 50  0000 C CNN
 F 1 "Conn_02x05" H 9900 10776 50  0000 C CNN
-F 2 "" H 9850 10450 50  0001 C CNN
+F 2 "Connector_PinHeader_1.27mm:PinHeader_2x05_P1.27mm_Vertical" H 9850 10450 50  0001 C CNN
 F 3 "~" H 9850 10450 50  0001 C CNN
 	1    9850 10450
@@
 F 0 "C306" H 3265 8946 50  0000 L CNN
 F 1 "1u" H 3265 8855 50  0000 L CNN
-F 2 "" H 3188 8750 50  0001 C CNN
+F 2 "Capacitor_SMD:C_0603_1608Metric_Pad1.05x0.95mm_HandSolder" H 3188 8750 50  0001 C CNN
 F 3 "~" H 3150 8900 50  0001 C CNN
 	1    3150 8900
@@
 F 0 "C319" H 7365 10746 50  0000 L CNN
 F 1 "1u" H 7365 10655 50  0000 L CNN
-F 2 "" H 7288 10550 50  0001 C CNN
+F 2 "Capacitor_SMD:C_0603_1608Metric_Pad1.05x0.95mm_HandSolder" H 7288 10550 50  0001 C CNN
 F 3 "~" H 7250 10700 50  0001 C CNN
 	1    7250 10700
@@
 F 0 "C305" H 2565 8096 50  0000 L CNN
 F 1 "2u2" H 2565 8005 50  0000 L CNN
-F 2 "" H 2488 7900 50  0001 C CNN
+F 2 "Capacitor_SMD:C_0603_1608Metric_Pad1.05x0.95mm_HandSolder" H 2488 7900 50  0001 C CNN
 F 3 "~" H 2450 8050 50  0001 C CNN
 	1    2450 8050
@@
 F 0 "C304" H 2115 8096 50  0000 L CNN
 F 1 "2u2" H 2115 8005 50  0000 L CNN
-F 2 "" H 2038 7900 50  0001 C CNN
+F 2 "Capacitor_SMD:C_0603_1608Metric_Pad1.05x0.95mm_HandSolder" H 2038 7900 50  0001 C CNN
 F 3 "~" H 2000 8050 50  0001 C CNN
 	1    2000 8050
@@
 F 0 "U202" H 1250 5300 50  0000 C CNN
 F 1 "24LC08" H 1250 5200 50  0000 C CNN
-F 2 "" H 1050 4950 50  0001 C CNN
+F 2 "Package_SO:MSOP-8_3x3mm_P0.65mm" H 1050 4950 50  0001 C CNN
 F 3 "http://ww1.microchip.com/downloads/en/DeviceDoc/21710J.pdf" H 1050 4950 50  0001 C CNN
 	1    1050 4950
