File: hardware/project/ETH1CSMU1BASE/Trigger.sch (KiCad schematic (older format))
At the start: 21 parts

Commit message: Schematic developement, new footprints.
Parts:
- gave numbers to parts that had none: 17
Connections:
- net GND: now also D602.3 (A); no longer D602.1 (A)
- net at R603.2, R604.1, U601.3 (O)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: now also D602.1 (A), D602.2 (K); no longer D602.3 (A), D602.3 (K)
- net at D601.1 (K), R601.2: now also D602.3 (K); no longer D602.2 (K)

Commit message: Power supply design
Parts:
- added C607: 1u, ETH1CJTAG:C_0603_T_Pad1.05x0.95mm_HandSolder, symbol Device:C
- added C608, C609: 100n, ETH1CJTAG:C_0603_A_Pad1.05x0.95mm_HandSolder, symbol Device:C
- added R606: 10k, symbol Device:R
- added U603: TXB0104PW, Package_SO:TSSOP-14_4.4x5mm_P0.65mm, symbol Logic_LevelTranslator:TXB0104PW
- D602: symbol Diode:BAV99 -> ETH1CSMU1BASE-rescue:BAV99-Diode
Connections:
- net +3V3: now also C607.1, C608.1, R606.1, U603.1 (VCCA); no longer C601.1, C602.1, U602.1 (VDD1)
- net +5V_TRIG: now also U601.1 (EN); no longer U601.13 (EN)
- net EXT_TRIG_SIGN: now also U601.3 (O); no longer U601.11 (O)
- net GND: now also C607.2, C608.2, C609.2, U603.7 (GND)
- net TRIG_EN: now also U603.2 (A1); no longer U602.3 (VIA)
- net TRIG_IN: now also U603.4 (A3); no longer U602.5 (VOC)
- net TRIG_OUT: now also U603.3 (A2); no longer U602.4 (VIB)
- net TRIG_OUT_EN: now also U601.13 (EN); no longer U601.1 (EN)
- net TRIG_OUT_SIGN: now also U601.12 (D); no longer U601.2 (D)
- net at D602.1 (A), D602.2 (K), R603.2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: now also U601.11 (O); no longer U601.3 (O)
- net at R602.2, R603.1: now also U601.2 (D); no longer U601.12 (D)
- new net: U602.3 (VIA), U603.13 (B1)
- new net: U602.4 (VIB), U603.12 (B2)
- new net: U602.5 (VOC), U603.11 (B3)
- new net: R606.2, U603.8 (OE)
- new net +5V: C601.1, C602.1, C609.1, U602.1 (VDD1), U603.14 (VCCB)
- no-connect marks 3 -> 5
Other:
- moved on the sheet: C601, C602, C603, C604, C605, U601A, U601B, U601C, U601D

Commit message: Footprint assigment
Parts:
- R601: footprint ETH1CJTAG:R_0603_P_Pad1.05x0.95mm_HandSolder -> Resistor_SMD:R_0603_1608Metric_Pad1.05x0.95mm_HandSolder
- R606: footprint (none) -> Resistor_SMD:R_0603_1608Metric_Pad1.05x0.95mm_HandSolder
Changed lines of the file:
@@
 F 0 "R601" H 8020 4446 50  0000 L CNN
 F 1 "1k" H 8020 4355 50  0000 L CNN
-F 2 "ETH1CJTAG:R_0603_P_Pad1.05x0.95mm_HandSolder" V 7880 4400 50  0001 C CNN
+F 2 "Resistor_SMD:R_0603_1608Metric_Pad1.05x0.95mm_HandSolder" V 7880 4400 50  0001 C CNN
 F 3 "~" H 7950 4400 50  0001 C CNN
 	1    7950 4400
@@
 F 0 "R606" H 2770 2646 50  0000 L CNN
 F 1 "10k" H 2770 2555 50  0000 L CNN
-F 2 "" V 2630 2600 50  0001 C CNN
+F 2 "Resistor_SMD:R_0603_1608Metric_Pad1.05x0.95mm_HandSolder" V 2630 2600 50  0001 C CNN
 F 3 "~" H 2700 2600 50  0001 C CNN
 	1    2700 2600
