File: hardware/project/ETH1CSMU1BASE/ETH1CSMU1BASE.sch (KiCad schematic (older format))
At the start: 0 parts

Commit message: Base board schematic.
Changed lines of the file:
@@
 $Descr A4 11693 8268
 encoding utf-8
-Sheet 1 4
+Sheet 1 6
 Title ""
 Date ""
@@
 $EndDescr
 $Sheet
-S 4250 2250 2550 1900
+S 4250 1350 1300 3000
 U 5D98FDB4
 F0 "MCU" 50
 F1 "MCU.sch" 50
+F2 "RMII_TXD1" B R 5550 1450 50
+F3 "RMII_TXD0" B R 5550 1550 50
+F4 "RMII_TXEN" B R 5550 1650 50
+F5 "RMII_RXD0" B R 5550 1750 50
+F6 "RMII_RXD1" B R 5550 1850 50
+F7 "RMII_CRS_DV" B R 5550 1950 50
+F8 "RMII_MDIO" B R 5550 2050 50
+F9 "RMII_MDC" B R 5550 2150 50
+F10 "REF_CLK" B R 5550 2350 50
+F11 "NRST" B R 5550 2250 50
+F12 "BASE_MCLK" O R 5550 3300 50
+F13 "BASE_MOSI" O R 5550 3400 50
+F14 "BASE_MISO" I R 5550 3500 50
+F15 "BASE_~MSS" O R 5550 3600 50
+F16 "TRIG_EN" O R 5550 2800 50
+F17 "TRIG_OUT" O R 5550 2900 50
+F18 "TRIG_IN" I R 5550 3000 50
+F19 "BASE_STATUS_IN" I R 5550 3800 50
+F20 "BASE_GPIO_OUT2" O R 5550 4000 50
+F21 "BASE_GPIO_OUT1" O R 5550 3900 50
 $EndSheet
 $Sheet
-S 4250 4400 2550 1400
-U 5D9881FE
-F0 "Power Digital" 50
-F1 "Power_Digital.sch" 50
+S 5700 1350 900  1100
+U 5D99CDAB
+F0 "Ethernet" 50
+F1 "Ethernet.sch" 50
+F2 "TX+" B R 6600 1450 50
+F3 "TX-" B R 6600 1550 50
+F4 "RX+" B R 6600 1650 50
+F5 "RX-" B R 6600 1750 50
+F6 "RMII_TXD1" B L 5700 1450 50
+F7 "RMII_TXD0" B L 5700 1550 50
+F8 "RMII_TXEN" B L 5700 1650 50
+F9 "RMII_RXD0" B L 5700 1750 50
+F10 "RMII_RXD1" B L 5700 1850 50
+F11 "RMII_CRS_DV" B L 5700 1950 50
+F12 "RMII_MDIO" B L 5700 2050 50
+F13 "RMII_MDC" B L 5700 2150 50
+F14 "NRST" B L 5700 2250 50
+F15 "REF_CLK" B L 5700 2350 50
 $EndSheet
 $Sheet
-S 7000 4400 2150 1400
-U 5D988230
-F0 "Power Analog" 50
-F1 "Power_Analog.sch" 50
+S 4250 4800 2350 800
+U 5DC846AF
+F0 "Power" 50
+F1 "Power.sch" 50
 $EndSheet
+$Sheet
+S 6750 1350 900  4250
+U 5DE8685C
+F0 "Connectors" 50
+F1 "Connectors.sch" 50
+F2 "RX+" B L 6750 1650 50
+F3 "TX+" B L 6750 1450 50
+F4 "RX-" B L 6750 1750 50
+F5 "TX-" B L 6750 1550 50
+F6 "EXT_TRIG" B L 6750 2800 50
+F7 "BASE_MCLK" I L 6750 3300 50
+F8 "BASE_MOSI" I L 6750 3400 50
+F9 "BASE_MISO" I L 6750 3500 50
+F10 "BASE_~MSS" I L 6750 3600 50
+F11 "BASE_STATUS_IN" O L 6750 3800 50
+F12 "BASE_GPIO_OUT2" I L 6750 4000 50
+F13 "BASE_GPIO_OUT1" I L 6750 3900 50
+$EndSheet
+Wire Wire Line
+	6750 1550 6600 1550
+Wire Wire Line
+	6600 1450 6750 1450
+Wire Wire Line
+	6750 1650 6600 1650
+Wire Wire Line
+	6600 1750 6750 1750
+Wire Wire Line
+	5700 1450 5550 1450
+Wire Wire Line
+	5550 1550 5700 1550
+Wire Wire Line
+	5700 1650 5550 1650
+Wire Wire Line
+	5550 1750 5700 1750
+Wire Wire Line
+	5550 1850 5700 1850
+Wire Wire Line
+	5700 1950 5550 1950
+Wire Wire Line
+	5550 2050 5700 2050
+Wire Wire Line
+	5550 2150 5700 2150
+Wire Wire Line
+	5700 2250 5550 2250
+Wire Wire Line
+	5550 2350 5700 2350
+$Sheet
+S 5700 2700 900  400
+U 5EB37D57
+F0 "Trigger" 50
+F1 "Trigger.sch" 50
+F2 "TRIG_EN" I L 5700 2800 50
+F3 "TRIG_OUT" I L 5700 2900 50
+F4 "TRIG_IN" O L 5700 3000 50
+F5 "EXT_TRIG" B R 6600 2800 50
+$EndSheet
+Wire Wire Line
+	6750 2800 6600 2800
+Wire Wire Line
+	5700 2800 5550 2800
+Wire Wire Line
+	5700 2900 5550 2900
+Wire Wire Line
+	5700 3000 5550 3000
+Wire Wire Line
+	6750 3300 5550 3300
+Wire Wire Line
+	5550 3400 6750 3400
+Wire Wire Line
+	6750 3500 5550 3500
+Wire Wire Line
+	5550 3600 6750 3600
+Wire Wire Line
+	5550 3800 6750 3800
+Wire Wire Line
+	6750 3900 5550 3900
+Wire Wire Line
+	5550 4000 6750 4000
 $EndSCHEMATC

Commit message: Schematic developement, new footprints.
Changed lines of the file:
@@
 $Descr A4 11693 8268
 encoding utf-8
-Sheet 1 6
+Sheet 1 7
 Title ""
 Date ""
@@
 S 4250 4800 2350 800
 U 5DC846AF
-F0 "Power" 50
-F1 "Power.sch" 50
+F0 "Power base" 50
+F1 "Power_base.sch" 50
 $EndSheet
 $Sheet
@@
 Wire Wire Line
 	5550 4000 6750 4000
+$Sheet
+S 2300 4800 1850 800
+U 5DCE1F8B
+F0 "Power isolation" 50
+F1 "Power_isolation.sch" 50
+$EndSheet
 $EndSCHEMATC

Commit message: Schematic design.
Changed lines of the file:
@@
 $Descr A4 11693 8268
 encoding utf-8
-Sheet 1 7
+Sheet 1 9
 Title ""
 Date ""
@@
 F1 "Power_isolation.sch" 50
 $EndSheet
+$Sheet
+S 2300 6000 1850 600
+U 5DCF3979
+F0 "Power High Voltage" 50
+F1 "Power_High_Voltage.sch" 50
+$EndSheet
+$Sheet
+S 2200 3250 1700 1200
+U 5DCD9B8B
+F0 "Output module" 50
+F1 "Output_Module.sch" 50
+$EndSheet
 $EndSCHEMATC

Commit message: Footprint assignment
Changed lines of the file:
@@
 $Descr A4 11693 8268
 encoding utf-8
-Sheet 1 9
+Sheet 1 6
 Title ""
 Date ""
@@
 $EndDescr
 $Sheet
-S 4250 1350 1300 3000
-U 5D98FDB4
-F0 "MCU" 50
-F1 "MCU.sch" 50
-F2 "RMII_TXD1" B R 5550 1450 50
-F3 "RMII_TXD0" B R 5550 1550 50
-F4 "RMII_TXEN" B R 5550 1650 50
-F5 "RMII_RXD0" B R 5550 1750 50
-F6 "RMII_RXD1" B R 5550 1850 50
-F7 "RMII_CRS_DV" B R 5550 1950 50
-F8 "RMII_MDIO" B R 5550 2050 50
-F9 "RMII_MDC" B R 5550 2150 50
-F10 "REF_CLK" B R 5550 2350 50
-F11 "NRST" B R 5550 2250 50
-F12 "BASE_MCLK" O R 5550 3300 50
-F13 "BASE_MOSI" O R 5550 3400 50
-F14 "BASE_MISO" I R 5550 3500 50
-F15 "BASE_~MSS" O R 5550 3600 50
-F16 "TRIG_EN" O R 5550 2800 50
-F17 "TRIG_OUT" O R 5550 2900 50
-F18 "TRIG_IN" I R 5550 3000 50
-F19 "BASE_STATUS_IN" I R 5550 3800 50
-F20 "BASE_GPIO_OUT2" O R 5550 4000 50
-F21 "BASE_GPIO_OUT1" O R 5550 3900 50
-$EndSheet
-$Sheet
-S 5700 1350 900  1100
-U 5D99CDAB
-F0 "Ethernet" 50
-F1 "Ethernet.sch" 50
-F2 "TX+" B R 6600 1450 50
-F3 "TX-" B R 6600 1550 50
-F4 "RX+" B R 6600 1650 50
-F5 "RX-" B R 6600 1750 50
-F6 "RMII_TXD1" B L 5700 1450 50
-F7 "RMII_TXD0" B L 5700 1550 50
-F8 "RMII_TXEN" B L 5700 1650 50
-F9 "RMII_RXD0" B L 5700 1750 50
-F10 "RMII_RXD1" B L 5700 1850 50
-F11 "RMII_CRS_DV" B L 5700 1950 50
-F12 "RMII_MDIO" B L 5700 2050 50
-F13 "RMII_MDC" B L 5700 2150 50
-F14 "NRST" B L 5700 2250 50
-F15 "REF_CLK" B L 5700 2350 50
-$EndSheet
-$Sheet
-S 4250 4800 2350 800
+S 5250 3400 1300 800
 U 5DC846AF
 F0 "Power base" 50
@@
 $EndSheet
 $Sheet
-S 6750 1350 900  4250
+S 6700 1950 1250 3300
 U 5DE8685C
 F0 "Connectors" 50
 F1 "Connectors.sch" 50
-F2 "RX+" B L 6750 1650 50
-F3 "TX+" B L 6750 1450 50
-F4 "RX-" B L 6750 1750 50
-F5 "TX-" B L 6750 1550 50
-F6 "EXT_TRIG" B L 6750 2800 50
-F7 "BASE_MCLK" I L 6750 3300 50
-F8 "BASE_MOSI" I L 6750 3400 50
-F9 "BASE_MISO" I L 6750 3500 50
-F10 "BASE_~MSS" I L 6750 3600 50
-F11 "BASE_STATUS_IN" O L 6750 3800 50
-F12 "BASE_GPIO_OUT2" I L 6750 4000 50
-F13 "BASE_GPIO_OUT1" I L 6750 3900 50
 $EndSheet
-Wire Wire Line
-	6750 1550 6600 1550
-Wire Wire Line
-	6600 1450 6750 1450
-Wire Wire Line
-	6750 1650 6600 1650
-Wire Wire Line
-	6600 1750 6750 1750
-Wire Wire Line
-	5700 1450 5550 1450
-Wire Wire Line
-	5550 1550 5700 1550
-Wire Wire Line
-	5700 1650 5550 1650
-Wire Wire Line
-	5550 1750 5700 1750
-Wire Wire Line
-	5550 1850 5700 1850
-Wire Wire Line
-	5700 1950 5550 1950
-Wire Wire Line
-	5550 2050 5700 2050
-Wire Wire Line
-	5550 2150 5700 2150
-Wire Wire Line
-	5700 2250 5550 2250
-Wire Wire Line
-	5550 2350 5700 2350
 $Sheet
-S 5700 2700 900  400
-U 5EB37D57
-F0 "Trigger" 50
-F1 "Trigger.sch" 50
-F2 "TRIG_EN" I L 5700 2800 50
-F3 "TRIG_OUT" I L 5700 2900 50
-F4 "TRIG_IN" O L 5700 3000 50
-F5 "EXT_TRIG" B R 6600 2800 50
-$EndSheet
-Wire Wire Line
-	6750 2800 6600 2800
-Wire Wire Line
-	5700 2800 5550 2800
-Wire Wire Line
-	5700 2900 5550 2900
-Wire Wire Line
-	5700 3000 5550 3000
-Wire Wire Line
-	6750 3300 5550 3300
-Wire Wire Line
-	5550 3400 6750 3400
-Wire Wire Line
-	6750 3500 5550 3500
-Wire Wire Line
-	5550 3600 6750 3600
-Wire Wire Line
-	5550 3800 6750 3800
-Wire Wire Line
-	6750 3900 5550 3900
-Wire Wire Line
-	5550 4000 6750 4000
-$Sheet
-S 2300 4800 1850 800
+S 3850 3400 1300 800
 U 5DCE1F8B
 F0 "Power isolation" 50
@@
 $EndSheet
 $Sheet
-S 2300 6000 1850 600
+S 3850 4450 2700 800
 U 5DCF3979
 F0 "Power High Voltage" 50
@@
 $EndSheet
 $Sheet
-S 2200 3250 1700 1200
+S 3850 1950 2700 1200
 U 5DCD9B8B
 F0 "Output module" 50
