File: hardware/project/ETH1CSMU1BASE/Power_isolation.sch (KiCad schematic (older format))
At the start: 98 parts, among them U701 LM317EMP/NOPB, U702 LT8331EMSE#PBF, U703 LM1117IMP-3.3/NOPB, U704 TSR1-2450, U705 TEL10-2415, U706 LM337IMPX/NOPB, U707 LT8331EMSE#PBF, U708 LM317EMP/NOPB, U709 TEL10-2415, U710 LT8331EMSE#PBF, U711 LM337IMPX/NOPB, U712 LT8331EMSE#PBF

Commit message: Schematic design.
Parts:
- removed C701, C708, C722, C732, C733, C739: 1u, symbol Device:C
- removed C702, C716, C726, C727, C734: 10u/50V, symbol Device:C
- removed C703, C717, C735: 10p, symbol Device:C
- removed C704, C719: 1u/25V, symbol Device:C
- removed C705, C720: 22u/25V, symbol Device:C
- removed C707: 100n, Capacitor_SMD:C_0603_1608Metric_Pad1.05x0.95mm_HandSolder, symbol Device:C
- removed C715: 4u7, symbol Device:C
- removed C721: 100, symbol Device:C
- removed C723, C730: 100p/2kV, symbol Device:C
- removed C724, C725: 4u7/50V, symbol Device:C
- removed C728, C729, C736, C737: 1u/50V, symbol Device:C
- removed C731: 100n, symbol Device:C
- removed C738: 220n, Capacitor_SMD:C_0603_1608Metric_Pad1.05x0.95mm_HandSolder, symbol Device:C
- removed D701: RB578VAM100TR, symbol Device:D_Schottky
- removed D702: BAV21W, symbol Device:D_Schottky
- removed D703, D704, D705: D_Schottky, symbol Device:D_Schottky
- removed FB701, FB702: 742792031, Resistor_SMD:R_0805_2012Metric_Pad1.15x1.40mm_HandSolder, symbol Device:Ferrite_Bead_Small
- removed L701: DRQ74-330, symbol ETH1CSMU1:DRQ74-330
- removed L704, L705: 120u, symbol Device:L
- removed L706: 100u, symbol Device:L
- removed L707: 744273222, ETH1CSMU1:744273222, symbol Device:L_Core_Ferrite_Coupled
- removed L708: 330u, symbol Device:L
- removed R701, R704, R706, R708, R711, R714, R718, R721, R722, R725, R728, R731: R, symbol Device:R
- removed R702, R703, R709, R710, R717, R726, R727: 1M, symbol Device:R
- removed R705, R712: 59k, symbol Device:R
- removed R707, R715, R723: 63k4, symbol Device:R
- removed R713, R730: 0, symbol Device:R
- removed R716: 100, symbol Device:R
- removed R719: 2k7, symbol Device:R
- removed R720: 249k, symbol Device:R
- removed R724: 10, symbol Device:R
- removed R729: 215k, symbol Device:R
- removed R732: 154k, symbol Device:R
- removed U701, U708: LM317EMP/NOPB, Package_TO_SOT_SMD:SOT-223-3_TabPin2, symbol Regulator_Linear:LM317_3PinPackage
- removed U702, U707, U710, U712: LT8331EMSE#PBF, ETH1CSMU1:MSE-16, symbol ETH1CSMU1:LT8331
- removed U706, U711: LM337IMPX/NOPB, Package_TO_SOT_SMD:SOT-223-3_TabPin2, symbol Regulator_Linear:LM337_TO252
- removed U709: TEL10-2415, symbol ETH1CSMU1:TEL10-2415
- added C?: 4u7/50V, symbol Device:C
- added C?: 33u/50V, symbol Device:C
- added C? (x2): 10u/50V, symbol Device:C
- added C?: 10n, symbol Device:C
- added C?: 1n, symbol Device:C
- added C?: 1u, symbol Device:C
- added C?: 4p7, symbol Device:C
- added C? (x4): 100n/100V, symbol Device:C
- added D?: DFLS260, symbol Device:D_Schottky
- added L?: 74479876147, symbol Device:L
- added L?: 74437324068, symbol Device:L
- added L?: 742792040, symbol Device:L
- added R?: 100k, symbol Device:R
- added R?: 20k, symbol Device:R
- added R?: 22k1, symbol Device:R
- added R?: 34k8, symbol Device:R
- added R?: 1M, symbol Device:R
- added U?: LT8362, symbol ETH1CSMU1:LT8362
Connections:
- net labels added: +24VF, +3.3VF, +48VF, +5VF, GNDF
- net labels removed: +15V, +3.3V, +3.3VP, +5V, +5VL, +HV, -15V, -HV, GNDA, GNDHV, GNDS
- wire segments 372 -> 133
Other:
- note removed: "+18V"
- note removed: "+HV set 35V"
- note removed: "-18V"
- moved on the sheet: C706, C709, C710, C711, C712, C713, C714, C718, L702, L703, U703, U704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

Commit message: Power supply design
Parts:
- removed C718: 100p/2kV, symbol Device:C
- removed C?: 4u7/50V, symbol Device:C
- removed C?: 33u/50V, symbol Device:C
- removed C? (x2): 10u/50V, symbol Device:C
- removed C?: 10n, symbol Device:C
- removed C?: 1n, symbol Device:C
- removed C?: 1u, symbol Device:C
- removed C?: 4p7, symbol Device:C
- removed C? (x4): 100n/100V, symbol Device:C
- removed D?: DFLS260, symbol Device:D_Schottky
- removed L703: 744273222, ETH1CSMU1:744273222, symbol Device:L_Core_Ferrite_Coupled
- removed L?: 74479876147, symbol Device:L
- removed L?: 74437324068, symbol Device:L
- removed L?: 742792040, symbol Device:L
- removed R?: 100k, symbol Device:R
- removed R?: 20k, symbol Device:R
- removed R?: 22k1, symbol Device:R
- removed R?: 34k8, symbol Device:R
- removed R?: 1M, symbol Device:R
- removed U705: TEL10-2415, symbol ETH1CSMU1:TEL10-2415
- removed U?: LT8362, symbol ETH1CSMU1:LT8362
- added C701, C723, C745, C750, C756, C768, C790, C794, C797, C? (x2): 4u7/50V, symbol Device:C
- added C702: 33u/50V, symbol Device:C
- added C703, C719, C760, C764, C800: 10u/50V, symbol Device:C
- added C704, C724, C728: 10n, symbol Device:C
- added C705: 1n, symbol Device:C
- added C707, C739, C787: 4p7, symbol Device:C
- added C708, C715, C716: 100n/100V, symbol Device:C
- added C720, C722: 2u2/100V, symbol Device:C
- added C727, C734, C740, C774: 1u, symbol Device:C
- added C731, C733: 2u2, symbol Device:C
- added C732, C780: 1u/HC, symbol Device:C
- added C744: 10u, symbol Device:C
- added C746, C749, C751, C753, C757, C765, C769, C775, C781, C798: 4u7/100V, symbol Device:C
- added C761, C801: 10u/100V, symbol Device:C
- added C? (x2): 100p/2kV, symbol Device:C
- added D701: DFLS260, symbol Device:D_Schottky
- added D704, D710: PMEG6010EP,115, symbol Device:D_Schottky
- added D705: RB558VA150TR, symbol Device:D_Schottky
- added D706: MBRS1100, symbol Device:D_Schottky
- added L701: 74479876147, symbol Device:L
- added L703: 74437324068, symbol Device:L
- added L704: 742792040, symbol Device:L
- added L706, L709, L713, L716: 74489440068, symbol ETH1CSMU1:74489440068
- added L708: DRQ127-101, symbol ETH1CSMU1:DRQ127-101
- added L717: DRQ127-221, symbol ETH1CSMU1:DRQ127-221
- added L?: 744273222, ETH1CSMU1:744273222, symbol Device:L_Core_Ferrite_Coupled
- added R701: 100k, symbol Device:R
- added R702: 20k, symbol Device:R
- added R703: 22k1, symbol Device:R
- added R704, R711, R713, R715, R722, R725, R727, R740, R749: 1M, symbol Device:R
- added R705: 34k8, symbol Device:R
- added R712, R741: 287k, symbol Device:R
- added R714, R716: 59k, symbol Device:R
- added R717, R724: 63k4, symbol Device:R
- added R723: 97k6, symbol Device:R
- added R726: 48k, symbol Device:R
- added R730, R753: 5k62, symbol Device:R
- added R732, R754: 243, symbol Device:R
- added R742: 24k, symbol Device:R
- added R750: 46k4, symbol Device:R
- added U701: LT8362, symbol ETH1CSMU1:LT8362
- added U706, U715: LT8330_S6, symbol ETH1CSMU1:LT8330_S6
- added U707, U708: LT8331, symbol ETH1CSMU1:LT8331
- added U711: MC7815BD2TG, symbol Regulator_Linear:L7815
- added U712: LM317MBDTRKG, symbol Regulator_Linear:LM317_3PinPackage
- added U718: MC7915BD2TG, Package_TO_SOT_SMD:TO-252-2, symbol Regulator_Linear:MC79M15_TO252
- added U719: LM337KVURG3, Package_TO_SOT_SMD:TO-252-2, symbol Regulator_Linear:LM337_TO252
- added U?: TEL10-2415, symbol ETH1CSMU1:TEL10-2415
- C706: value 100p/2kV -> 1u
- C709: value 4u7/50V -> 100n/100V
- C710: value 4u7/50V -> 10u/100V
Connections:
- net +24VF: now also C701.1, C719.1, C723.1, C764.1, C768.1, L701.1, L706.3, L713.3, R711.1, R740.1, U706.6 (VIN), U715.6 (VIN), U?.9 (+VOUT)
- net +48VF: now also C716.1, C720.1, C722.1, L704.2, L708.1, L717.1, R713.1, R715.1, U707.3 (Vin), U708.3 (Vin)
- net GND: now also C?.2, C?.2, L?.3; no longer C709.2, C710.2
- net GNDF: now also C706.2, C709.2, C710.2, C701.2, C702.2, C703.2, C704.2, C705.2, C708.2, C715.2, C716.2, C719.2, C720.2, C722.2, C723.2, C724.2, C727.2, C728.2, C734.2, C740.2, C744.2, C745.2, C746.2, C749.2, C750.2, C751.2, C753.2, C756.2, C757.2, C760.2, C761.2, C764.2, C765.2, C768.2, C769.2, C774.2, C775.2, C781.2, C790.2, C794.2, C797.2, C798.2, C800.2, C801.2, C?.1, C?.1, D705.1 (K), D710.1 (K), L709.1, L717.2, R701.2, R702.2, R705.2, R712.2, R714.2, R716.2, R717.2, R723.2, R724.2, R726.2, R730.2, R741.2, R742.2, R750.2, R753.2, U701.17 (GND), U701.7 (BIAS), U706.2 (GND), U707.12 (SYNC/MODE), U707.17 (GND), U707.7 (BIAS), U708.12 (SYNC/MODE), U708.17 (GND), U711.2 (GND), U715.2 (GND), U718.1 (GND), U?.10 (-VOUT); no longer C706.1
- net +24VDD: no longer names the net of C709.1, C710.1
- net +24VDD: now also C707.1, C708.1, C715.1, D701.1 (K), L704.1, R704.1
- new net: C732.2, L706.2, U706.1 (SW)
- new net: C739.2, R722.2, R723.1, U706.3 (FBX)
- new net: R711.2, R712.1, U706.4 (EN/UVLO)
- new net: C727.1, U706.5 (INTVCC)
- new net: C732.1, D704.2 (A), L709.4
- new net: C739.1, C745.1, C750.1, D704.1 (K), R722.1, U711.1 (IN)
- new net: C780.2, L713.2, U715.1 (SW)
- new net: C787.2, R749.2, R750.1, U715.3 (FBX)
- new net: R740.2, R741.1, U715.4 (EN/UVLO)
- new net: C774.1, U715.5 (INTVCC)
- new net: C780.1, D710.2 (A), L716.4
- new net: C787.1, C790.1, C794.1, L716.1, R749.1, U718.2 (VI)
- new net: C757.1, R730.1, R732.2, U712.1 (ADJ)
- new net: C798.1, R753.1, R754.2, U719.1 (ADJ)
- new net: C744.1, C746.1, C751.1, C765.1, C775.1, L708.2, R727.1, U719.2 (VI)
- new net: C749.1, C753.1, C769.1, C781.1, D706.1 (K), R725.1, U708.7 (BIAS), U712.3 (VI)
- new net: C702.1, C703.1, L701.2, L703.1, U701.1 (EN/UVLO), U701.3 (Vin)
- new net: R702.1, U701.10 (RT)
- new net: C704.1, U701.11 (SS)
- new net: R701.1, U701.12 (SYNC/MODE)
- new net: D701.2 (A), L703.2, U701.14 (SW2), U701.16 (SW1)
- new net: C706.1, U701.5 (INTVcc)
- new net: R703.1, U701.8 (Vc)
- new net: C707.2, R704.2, R705.1, U701.9 (FBX)
- new net: C705.1, R703.2
- new net: R715.2, R716.1, U708.1 (EN/UVLO)
- new net: R724.1, U708.10 (RT)
- new net: C728.1, U708.11 (SS)
- new net: C733.2, L717.3, U708.14 (SW2), U708.16 (SW1)
- new net: C740.1, U708.5 (INTVcc)
- new net: R725.2, R726.1, U708.9 (FBX)
- new net: C733.1, D706.2 (A), L717.4
- new net: R713.2, R714.1, U707.1 (EN/UVLO)
- new net: R717.1, U707.10 (RT)
- new net: C724.1, U707.11 (SS)
- new net: C731.2, L708.3, U707.14 (SW2), U707.16 (SW1)
- new net: C734.1, U707.5 (INTVcc)
- new net: R727.2, R742.1, U707.9 (FBX)
- new net: C731.1, D705.2 (A), L708.4
- new net: C?.2, L?.2, U?.16 (+VIN)
- new net: C?.2, L?.4, U?.1 (-VIN)
- new net +15VF: C756.1, C760.1, U711.3 (OUT)
- new net +24V: C?.1, C?.1, L?.1
- new net +30VF: C761.1, R732.1, U712.2 (VO)
- new net -15VF: C797.1, C800.1, U718.3 (VO)
- new net -30VF: C801.1, R754.1, U719.3 (VO)
Other:
- moved on the sheet: C711, C712, C713, C714, L702, U703, U704

Commit message: Footprint assigment
Parts:
- C701, C703, C708, C709, C711, C715, C716, C719, C723, C732, C745, C750, C756, C760, C764, C768, C790, C794, C797, C800: footprint (none) -> Capacitor_SMD:C_1206_3216Metric_Pad1.42x1.75mm_HandSolder
- C702, C710, C761, C801: footprint (none) -> Capacitor_SMD:C_2220_5650Metric_Pad1.97x5.40mm_HandSolder
- C704, C705, C706, C707, C724, C727, C728, C734, C739, C740, C774, C787: footprint (none) -> Capacitor_SMD:C_0603_1608Metric_Pad1.05x0.95mm_HandSolder
- C717, C718: renamed from C?; footprint (none) -> Capacitor_SMD:C_1206_3216Metric_Pad1.42x1.75mm_HandSolder
- D704, D710: footprint (none) -> Diode_SMD:D_SOD-128
- L706, L709, L713, L716: footprint (none) -> ETH1CSMU1:74489440068
- R701, R702, R703, R704, R705, R711, R712, R713, R714, R715, R716, R717, R722, R723, R724, R725, R726, R727, R730, R732, R740, R741, R742, R749, R750, R753, R754: footprint (none) -> Resistor_SMD:R_0603_1608Metric_Pad1.05x0.95mm_HandSolder
- U701, U707, U708: footprint (none) -> Package_SO:MSOP-12-16-1EP_3x4mm_P0.5mm_EP1.65x2.85mm
- U704: footprint (none) -> ETH1CSMU1:TSR1
- U706, U715: footprint (none) -> Package_TO_SOT_SMD:TSOT-23-6_HandSoldering
- U711: footprint (none) -> Package_TO_SOT_SMD:TO-263-2
- U712: value LM317MBDTRKG -> LM317KTTR; footprint (none) -> Package_TO_SOT_SMD:TO-263-3
- U718: footprint Package_TO_SOT_SMD:TO-252-2 -> Package_TO_SOT_SMD:TO-263-2
- U719: value LM337KVURG3 -> LM337KTTR; footprint Package_TO_SOT_SMD:TO-252-2 -> Package_TO_SOT_SMD:TO-263-3
- gave numbers to parts that had none: 4
Connections:
- net +24VF: now also L709.1, L716.1; no longer L706.3, L713.3
- net GNDF: now also L706.3; no longer L709.1
- net at C732.2, U706.1 (SW): now also L709.4; no longer L706.2
- net at C732.1, D704.2 (A): now also L706.2; no longer L709.4
- net at C780.2, U715.1 (SW): now also L716.4; no longer L713.2
- net at C780.1, D710.2 (A): now also L713.2; no longer L716.4
- net at C787.1, C790.1, C794.1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: now also L713.3; no longer L716.1
Other:
- moved on the sheet: L706B, L709A, L713B, L716A

Commit message: Footprint assignment
Parts:
- added C401, C402: 10u/50V, Capacitor_SMD:C_1206_3216Metric_Pad1.42x1.75mm_HandSolder, symbol Device:C
- added C403, C404: 22u/16V, Capacitor_SMD:C_1206_3216Metric_Pad1.42x1.75mm_HandSolder, symbol Device:C
- added L401: TCK-141, ETH1CSMU1:TCK-141, symbol Device:L
- added U401: TSR1-2450, ETH1CSMU1:TSR1, symbol ETH1CSMU1:TSR1-2450
- added U402: LM1117IMP-3.3/NOPB, Package_TO_SOT_SMD:SOT-223-3_TabPin2, symbol Regulator_Linear:LM1117-3.3
- C501: renamed from C720; footprint (none) -> Capacitor_SMD:C_1206_3216Metric_Pad1.42x1.75mm_HandSolder
- C504: renamed from C722; footprint (none) -> Capacitor_SMD:C_1206_3216Metric_Pad1.42x1.75mm_HandSolder
- C511: renamed from C731; footprint (none) -> Capacitor_SMD:C_1206_3216Metric_Pad1.42x1.75mm_HandSolder
- C512: renamed from C733; footprint (none) -> Capacitor_SMD:C_1206_3216Metric_Pad1.42x1.75mm_HandSolder
- C518: renamed from C744; value 10u -> 10u/100V; footprint (none) -> Capacitor_SMD:C_2220_5650Metric_Pad1.97x5.40mm_HandSolder
- C521: renamed from C749; footprint (none) -> Capacitor_SMD:C_1210_3225Metric_Pad1.42x2.65mm_HandSolder
- C522: renamed from C746; footprint (none) -> Capacitor_SMD:C_1210_3225Metric_Pad1.42x2.65mm_HandSolder
- C525: renamed from C753; footprint (none) -> Capacitor_SMD:C_1210_3225Metric_Pad1.42x2.65mm_HandSolder
- C526: renamed from C751; footprint (none) -> Capacitor_SMD:C_1210_3225Metric_Pad1.42x2.65mm_HandSolder
- C529: renamed from C769; footprint (none) -> Capacitor_SMD:C_1210_3225Metric_Pad1.42x2.65mm_HandSolder
- C530: renamed from C765; footprint (none) -> Capacitor_SMD:C_1210_3225Metric_Pad1.42x2.65mm_HandSolder
- C533: renamed from C781; footprint (none) -> Capacitor_SMD:C_1210_3225Metric_Pad1.42x2.65mm_HandSolder
- C534: renamed from C775; footprint (none) -> Capacitor_SMD:C_1210_3225Metric_Pad1.42x2.65mm_HandSolder
- C537: renamed from C757; footprint (none) -> Capacitor_SMD:C_1210_3225Metric_Pad1.42x2.65mm_HandSolder
- C538: renamed from C798; footprint (none) -> Capacitor_SMD:C_1210_3225Metric_Pad1.42x2.65mm_HandSolder
- C546: renamed from C780; footprint (none) -> Capacitor_SMD:C_1206_3216Metric_Pad1.42x1.75mm_HandSolder
- C552: renamed from C712; footprint Capacitor_SMD:C_2220_5650Metric_Pad1.97x5.40mm_HandSolder -> Capacitor_SMD:C_1206_3216Metric_Pad1.42x1.75mm_HandSolder
- C554: renamed from C713; footprint Capacitor_SMD:C_2220_5650Metric_Pad1.97x5.40mm_HandSolder -> Capacitor_SMD:C_1206_3216Metric_Pad1.42x1.75mm_HandSolder
- C555: renamed from C721; footprint (none) -> Capacitor_SMD:C_1210_3225Metric_Pad1.42x2.65mm_HandSolder
- C556: renamed from C725; footprint (none) -> Capacitor_SMD:C_1210_3225Metric_Pad1.42x2.65mm_HandSolder
- C558: renamed from C714; footprint Capacitor_SMD:C_2220_5650Metric_Pad1.97x5.40mm_HandSolder -> Capacitor_SMD:C_1206_3216Metric_Pad1.42x1.75mm_HandSolder
- D501: renamed from D705; value RB558VA150TR -> RB558VAM150; footprint (none) -> ETH1CSMU1:D_SOD-323HE
- D502: renamed from D706; footprint (none) -> Diode_SMD:D_SMB
- D503: renamed from D704; footprint Diode_SMD:D_SOD-128 -> ETH1CSMU1:D_SOD-128
- D504: renamed from D701; footprint (none) -> ETH1CSMU1:PowerDI-123
- D505: renamed from D710; footprint Diode_SMD:D_SOD-128 -> ETH1CSMU1:D_SOD-128
- L501: renamed from L701; footprint (none) -> Inductor_SMD:L_0805_2012Metric_Pad1.15x1.40mm_HandSolder
- L502: renamed from L708; footprint (none) -> ETH1CSMU1:DRQ127
- L503: renamed from L717; footprint (none) -> ETH1CSMU1:DRQ127
- L505: renamed from L703; footprint (none) -> ETH1CSMU1:74437324068
- L507: renamed from L704; footprint (none) -> Inductor_SMD:L_0805_2012Metric_Pad1.15x1.40mm_HandSolder
- U506: renamed from U712; footprint Package_TO_SOT_SMD:TO-263-3 -> Package_TO_SOT_SMD:TO-263-3_TabPin2
- U507: renamed from U719; footprint Package_TO_SOT_SMD:TO-263-3 -> Package_TO_SOT_SMD:TO-263-3_TabPin2
- U511: renamed from U702; footprint (none) -> ETH1CSMU1:TEL10
- renumbered C719 to C502, C701 to C503, C723 to C505, C702 to C506, C703 to C507, C724 to C508, C727 to C509, C728 to C510, C734 to C513, C740 to C514, C732 to C515, C704 to C516, C705 to C517, C706 to C519, C739 to C520, C745 to C523, C707 to C524, C750 to C527, C708 to C528, C709 to C531, C756 to C532, C760 to C535, C710 to C536, C715 to C539, C764 to C540, C761 to C541, C801 to C542, C768 to C543, C716 to C544, C774 to C545, C717 to C547, C711 to C548, C787 to C549, C718 to C550, C790 to C551, C794 to C553, C797 to C557, C800 to C559, L709 to L504, L706 to L506, L716 to L508, L713 to L509, L702 to L510, L705 to L511, R713 to R501, R714 to R502, R715 to R503, R716 to R504, R711 to R505, R712 to R506, R717 to R507, R724 to R508, R701 to R509, R702 to R510, R703 to R511, R722 to R512, R723 to R513, R725 to R514, R726 to R515, R727 to R516, R742 to R517, R704 to R518, R705 to R519, R730 to R520, R753 to R521, R732 to R522, R754 to R523, R740 to R524, R741 to R525, R749 to R526, R750 to R527, U707 to U501, U708 to U502, U706 to U503, U701 to U504, U711 to U505, U715 to U508, U704 to U509, U718 to U510, U703 to U512
Connections:
- net +24VF: now also C401.1, L401.1
- net GNDF: now also C401.2, C402.2, C403.2, C404.2, U401.2 (GND), U402.1 (GND)
- new net: C402.1, L401.2, U401.1 (VI)
- new net +3.3DVF: C404.1, U402.2 (VO)
- new net +5VD: C403.1, U401.3 (VO), U402.3 (VI)
Other:
- moved on the sheet: C522, C526, C530, C534, C538, C542, L510, R516, R517, R521, R523, U507
