File: hardware/project/ETH1CSMU1ANALOG/MCU.sch (KiCad schematic (older format))
At the start: 0 parts

Commit message: Footprint assigment
Parts:
- added U?: STM32H743ZI, symbol ETH1CSMU1:STM32H743ZI
Changed lines of the file:
@@
 EESchema Schematic File Version 4
-LIBS:ETH1CSMU1ANALOG-cache
 EELAYER 30 0
 EELAYER END
-$Descr A4 11693 8268
+$Descr A3 16535 11693
 encoding utf-8
-Sheet 1 6
+Sheet 5 7
 Title ""
 Date ""
@@
 Comment4 ""
 $EndDescr
+$Comp
+L ETH1CSMU1:STM32H743ZI U?
+U 1 1 5EC81AA4
+P 8400 5550
+F 0 "U?" H 8400 1411 50  0000 C CNN
+F 1 "STM32H743ZI" H 8400 1320 50  0000 C CNN
+F 2 "" H 24300 7050 50  0001 C CNN
+F 3 "" H 24300 7050 50  0001 C CNN
+	1    8400 5550
+	1    0    0    -1
+$EndComp
 $EndSCHEMATC
