File: hardware/project/ETH1CSMU1ANALOG/Ethernet.sch (KiCad schematic (older format))
At the start: 43 parts, among them U201 LAN8742A, U202 LC03-3.3, U203 LC03-3.3, Y201 NX5032GA-25.000M-LN-CD-1

Commit message: Footprint assignment
Parts:
- renumbered C203 to C?, C206 to C?, C212 to C?, C214 to C?, C213 to C?, C202 to C?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
