File: hardware/project/ETH1CSMU1ANALOG/MCU1.sch (KiCad schematic (older format))
At the start: 31 parts, among them J801 Conn_02x01, J802 Conn_02x05, U801 24LC08, U802 STM32F765ZGT6, Y801 NX3225GD-8MHZ-STD-CRA-3

Commit message: Footprint assignment
Parts:
- U802: symbol ETH1CSMU1BASE-rescue:STM32F765ZGT6-ETH1CSMU1 -> ETH1CSMU1:STM32F765ZGT6
- renumbered C820 to C?, C811 to C?, C802 to C?, C803 to C?, C805 to C?, C808 to C?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
