File: hardware/project/ETH1CSMU1ANALOG/Trigger.sch (KiCad schematic (older format))
At the start: 22 parts, among them U901 TXB0104PW, U902 ADuM5402, U903 74AC125

Commit message: Footprint assignment
Parts:
- renumbered C909 to C?, C904 to C?, C905 to C?, C907 to C?, C908 to C?, C906 to C?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
