File: HARDWARE/BASE/HV_Power.sch (KiCad schematic (older format))
At the start: 77 parts, among them U1001 TEL10-2415, U1002 LT8330_S6, U1003 LT8330_S6, U1004 LM317_TO-263, U1006 LT8330_S6, U1007 LT8330_S6, U1008 MC7815BD2TG, U1009 MC7915BD2TG

Commit message: Schematic design
Parts:
- removed C1022, C1023, C1038, C1039: 10u/50V, Capacitor_SMD:C_1206_3216Metric_Pad1.42x1.75mm_HandSolder, symbol Device:C
- removed C1024, C1025, C1032, C1033, C1034, C1035, C1036, C1037: 4u7/50V, Capacitor_SMD:C_1206_3216Metric_Pad1.42x1.75mm_HandSolder, symbol Device:C
- removed C1026, C1027: 1u, Capacitor_SMD:C_0603_1608Metric_Pad1.05x0.95mm_HandSolder, symbol Device:C
- removed C1028, C1029: 1u/HC, Capacitor_SMD:C_1206_3216Metric_Pad1.42x1.75mm_HandSolder, symbol Device:C
- removed C1030, C1031: 4p7, Capacitor_SMD:C_0603_1608Metric_Pad1.05x0.95mm_HandSolder, symbol Device:C
- removed D1003, D1004: PMEG6010EP,115, ETH1CSMU1:D_SOD-128, symbol Device:D_Schottky
- removed L1004, L1005: 74489440068, ETH1CSMU1:74489440068, symbol ETH1CSMU1:74489440068
- removed R1011, R1013, R1015, R1017: 1M, Resistor_SMD:R_0603_1608Metric_Pad1.05x0.95mm_HandSolder, symbol Device:R
- removed R1012, R1014: 287k, Resistor_SMD:R_0603_1608Metric_Pad1.05x0.95mm_HandSolder, symbol Device:R
- removed R1016: 97k6, Resistor_SMD:R_0603_1608Metric_Pad1.05x0.95mm_HandSolder, symbol Device:R
- removed R1018: 46k4, Resistor_SMD:R_0603_1608Metric_Pad1.05x0.95mm_HandSolder, symbol Device:R
- removed U1006, U1007: LT8330_S6, Package_TO_SOT_SMD:TSOT-23-6_HandSoldering, symbol ETH1CSMU1:LT8330_S6
- removed U1008: MC7815BD2TG, symbol Regulator_Linear:L7815
- removed U1009: MC7915BD2TG, symbol Regulator_Linear:MC79M15_TO252
- added C613, C632, C633: 100n, Capacitor_SMD:C_0603_1608Metric_Pad1.08x0.95mm_HandSolder, symbol Device:C
- added C616: 10u, Capacitor_SMD:C_0603_1608Metric_Pad1.08x0.95mm_HandSolder, symbol Device:C
- added C618, C619, C625, C626: 4u7, Capacitor_SMD:C_0603_1608Metric_Pad1.08x0.95mm_HandSolder, symbol Device:C
- added C621, C622, C623, C624, C629, C630: 1u, Capacitor_SMD:C_0603_1608Metric_Pad1.08x0.95mm_HandSolder, symbol Device:C
- added D602, D603, D604, D605, D607, D608, D609, D610, D611, D612: MBR0530, Diode_SMD:D_SOD-123, symbol Diode:MBR0530
- added FB601, FB602: BLM18AG102, Inductor_SMD:L_0603_1608Metric_Pad1.05x0.95mm_HandSolder, symbol Device:Ferrite_Bead_Small
- added L603: SRF0905-202Y, ETH1CSMU1:SRF0905, symbol Device:L_Core_Ferrite_Coupled_1423
- added TR601: Wuerth_750315371, Transformer_SMD:Transformer_Wuerth_750315371, symbol Transformer:Wuerth_750315371
- added U604: SN6505BDBV, Package_TO_SOT_SMD:SOT-23-6, symbol Power_Management:SN6505BDBV
- added U607: L78L15_SO8, Package_SO:SOIC-8_3.9x4.9mm_P1.27mm, symbol Regulator_Linear:L78L15_SO8
- added U608: L79L15_SO8, Package_SO:SOIC-8_3.9x4.9mm_P1.27mm, symbol Regulator_Linear:L79L15_SO8
- C601: renamed from C1002; footprint Capacitor_SMD:C_1206_3216Metric_Pad1.42x1.75mm_HandSolder -> Capacitor_SMD:C_1206_3216Metric_Pad1.33x1.80mm_HandSolder
- C602: renamed from C1001; footprint Capacitor_SMD:C_1206_3216Metric_Pad1.42x1.75mm_HandSolder -> Capacitor_SMD:C_1206_3216Metric_Pad1.33x1.80mm_HandSolder
- C603: renamed from C1005; footprint Capacitor_SMD:C_1206_3216Metric_Pad1.42x1.75mm_HandSolder -> Capacitor_SMD:C_1206_3216Metric_Pad1.33x1.80mm_HandSolder
- C604: renamed from C1004; footprint Capacitor_SMD:C_1206_3216Metric_Pad1.42x1.75mm_HandSolder -> Capacitor_SMD:C_1206_3216Metric_Pad1.33x1.80mm_HandSolder
- C605: renamed from C1007; footprint Capacitor_SMD:C_0603_1608Metric_Pad1.05x0.95mm_HandSolder -> Capacitor_SMD:C_0603_1608Metric_Pad1.08x0.95mm_HandSolder
- C606: renamed from C1009; footprint Capacitor_SMD:C_1210_3225Metric_Pad1.42x2.65mm_HandSolder -> Capacitor_SMD:C_1210_3225Metric_Pad1.33x2.70mm_HandSolder
- C607: renamed from C1010; footprint Capacitor_SMD:C_1210_3225Metric_Pad1.42x2.65mm_HandSolder -> Capacitor_SMD:C_1210_3225Metric_Pad1.33x2.70mm_HandSolder
- C608: renamed from C1012; footprint Capacitor_SMD:C_0603_1608Metric_Pad1.05x0.95mm_HandSolder -> Capacitor_SMD:C_0603_1608Metric_Pad1.08x0.95mm_HandSolder
- C609: renamed from C1013; footprint Capacitor_SMD:C_1206_3216Metric_Pad1.42x1.75mm_HandSolder -> Capacitor_SMD:C_1210_3225Metric_Pad1.33x2.70mm_HandSolder
- C610: renamed from C1015; footprint Capacitor_SMD:C_1206_3216Metric_Pad1.42x1.75mm_HandSolder -> Capacitor_SMD:C_1210_3225Metric_Pad1.33x2.70mm_HandSolder
- C611: renamed from C1018; footprint Capacitor_SMD:C_1206_3216Metric_Pad1.42x1.75mm_HandSolder -> Capacitor_SMD:C_1210_3225Metric_Pad1.33x2.70mm_HandSolder
- C612: renamed from C1020; footprint Capacitor_SMD:C_1206_3216Metric_Pad1.42x1.75mm_HandSolder -> Capacitor_SMD:C_1210_3225Metric_Pad1.33x2.70mm_HandSolder
- C614: renamed from C1003; footprint Capacitor_SMD:C_1206_3216Metric_Pad1.42x1.75mm_HandSolder -> Capacitor_SMD:C_1206_3216Metric_Pad1.33x1.80mm_HandSolder
- C615: renamed from C1006; footprint Capacitor_SMD:C_1206_3216Metric_Pad1.42x1.75mm_HandSolder -> Capacitor_SMD:C_1206_3216Metric_Pad1.33x1.80mm_HandSolder
- C627: renamed from C1014; footprint Capacitor_SMD:C_0603_1608Metric_Pad1.05x0.95mm_HandSolder -> Capacitor_SMD:C_0603_1608Metric_Pad1.08x0.95mm_HandSolder
- C628: renamed from C1016; footprint Capacitor_SMD:C_1206_3216Metric_Pad1.42x1.75mm_HandSolder -> Capacitor_SMD:C_1206_3216Metric_Pad1.33x1.80mm_HandSolder
- C631: renamed from C1017; footprint Capacitor_SMD:C_1206_3216Metric_Pad1.42x1.75mm_HandSolder -> Capacitor_SMD:C_1206_3216Metric_Pad1.33x1.80mm_HandSolder
- C634, C635: renamed from C?; footprint Capacitor_SMD:C_1206_3216Metric_Pad1.42x1.75mm_HandSolder -> Capacitor_SMD:C_1210_3225Metric_Pad1.33x2.70mm_HandSolder
- R601: renamed from R1001; footprint Resistor_SMD:R_0603_1608Metric_Pad1.05x0.95mm_HandSolder -> Resistor_SMD:R_0603_1608Metric_Pad0.98x0.95mm_HandSolder
- R602: renamed from R1002; footprint Resistor_SMD:R_0603_1608Metric_Pad1.05x0.95mm_HandSolder -> Resistor_SMD:R_0603_1608Metric_Pad0.98x0.95mm_HandSolder
- R603: renamed from R1005; footprint Resistor_SMD:R_0603_1608Metric_Pad1.05x0.95mm_HandSolder -> Resistor_SMD:R_0603_1608Metric_Pad0.98x0.95mm_HandSolder
- R604: renamed from R1006; footprint Resistor_SMD:R_0603_1608Metric_Pad1.05x0.95mm_HandSolder -> Resistor_SMD:R_0603_1608Metric_Pad0.98x0.95mm_HandSolder
- R605: renamed from R1009; footprint (none) -> Resistor_SMD:R_0603_1608Metric_Pad0.98x0.95mm_HandSolder
- R606: renamed from R1010; footprint (none) -> Resistor_SMD:R_0603_1608Metric_Pad0.98x0.95mm_HandSolder
- R607: renamed from R1003; footprint Resistor_SMD:R_0603_1608Metric_Pad1.05x0.95mm_HandSolder -> Resistor_SMD:R_0603_1608Metric_Pad0.98x0.95mm_HandSolder
- R608: renamed from R1004; footprint Resistor_SMD:R_0603_1608Metric_Pad1.05x0.95mm_HandSolder -> Resistor_SMD:R_0603_1608Metric_Pad0.98x0.95mm_HandSolder
- R609: renamed from R1007; footprint Resistor_SMD:R_0603_1608Metric_Pad1.05x0.95mm_HandSolder -> Resistor_SMD:R_0603_1608Metric_Pad0.98x0.95mm_HandSolder
- R610: renamed from R1008; footprint Resistor_SMD:R_0603_1608Metric_Pad1.05x0.95mm_HandSolder -> Resistor_SMD:R_0603_1608Metric_Pad0.98x0.95mm_HandSolder
- R611, R612: renamed from R?; footprint (none) -> Resistor_SMD:R_0603_1608Metric_Pad0.98x0.95mm_HandSolder
- gave numbers to parts that had none: 1
- renumbered C1008 to C617, C1011 to C620, D1001 to D601, D1002 to D606, L1001 to L601, L1002 to L602, L1003 to L604, U1002 to U601, U1001 to U602, U1004 to U603, U1003 to U605
Connections:
- net GND: now also L603.2
- net GNDHV: now also C618.1, C619.2, C625.2, C626.1, C629.2, C630.1, C632.2, C633.1, D608.2 (A), D609.1 (K), TR601.5, U607.2 (GND), U607.3 (GND), U607.6 (GND), U607.7 (GND), U608.5 (GND)
- net +24V renamed +24VF
- new net: TR601.1, U604.1 (D1)
- new net: TR601.3, U604.3 (D2)
- new net: C613.2, C616.2, L603.3, U604.4 (GND), U604.6 (CLK)
- new net: C621.2, C624.2, D604.2 (A), D605.1 (K), TR601.4
- new net: C622.2, C623.2, D602.2 (A), D603.1 (K), TR601.6
- new net: C629.1, FB601.1, U607.8 (IN)
- new net: C630.2, FB602.1, U608.2 (IN), U608.3 (IN), U608.6 (IN), U608.7 (IN)
- new net: C625.1, D611.1 (K), FB601.2
- new net: C626.2, D612.2 (A), FB602.2
- new net: C622.1, D607.2 (A), D608.1 (K)
- new net: C623.1, D609.2 (A), D610.1 (K)
- new net: C621.1, D607.1 (K), D611.2 (A)
- new net: C624.1, D610.2 (A), D612.1 (K)
- new net: C619.1, D603.2 (A), D605.2 (A)
- new net: C618.2, D602.1 (K), D604.1 (K)
- new net +15VF: C632.1, U607.1 (OUT)
- new net +5V: L603.1
- new net -15VF: C633.2, U608.1 (OUT)
- new net VDD: C613.1, C616.1, L603.4, TR601.2, U604.2 (VCC), U604.5 (EN)
Other:
- moved on the sheet: C601, C602, C603, C604, C605, C606, C607, C608, C609, C610, C611, C612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

Commit message: Schematic design
Parts:
- renumbered C620 to C601, C608 to C602, C627 to C603, C601 to C604, C603 to C605, C609 to C606, C610 to C607, C611 to C608, C612 to C609, C614 to C610, C615 to C611, C628 to C612, C631 to C613, C634 to C614, C635 to C615, C605 to C616, C606 to C618, C602 to C619, C604 to C620, C618 to C621, C607 to C622, C621 to C623, C622 to C624, C629 to C626, C632 to C627, C626 to C628, C630 to C629, C633 to C630, C613 to C631, C616 to C632, C623 to C633, C624 to C634, C619 to C635, D606 to D602, D602 to D603, D611 to D605, D607 to D606, D608 to D607, D609 to D608, D610 to D609, D612 to D610, D603 to D611, D605 to D612, L602 to L601, L604 to L602, L601 to L603, L603 to L604, R606 to R601, R612 to R602, R601 to R603, R603 to R604, R607 to R605, R609 to R606, R605 to R607, R611 to R608, R602 to R609, R608 to R610, R604 to R611, R610 to R612, U603 to U601, U606 to U602, U601 to U603, U605 to U604, U602 to U605, U607 to U606, U604 to U607
