File: HARDWARE/BASE/Analog.sch (KiCad schematic (older format))
At the start: 0 parts

Commit message: Schematic design.
Parts:
- added C1001, C1002, C1003: 15p, symbol Device:C
- added C1004: 150p/500V, symbol Device:C
- added C1005: 22p/500V, symbol Device:C
- added C1006: 1000p, symbol Device:C
- added C1007: 100p, symbol Device:C
- added C1008, C1009, C1010: 270p, symbol Device:C
- added D1001, D1002: BAV99, Package_TO_SOT_SMD:SOT-23, symbol Diode:BAV99
- added R1001, R1002, R1003, R1004, R1010, R1011: 10k/.1%, symbol Device:R
- added R1005, R1006, R1009: 20k/.1%, symbol Device:R
- added R1007, R1008: 15k, symbol Device:R
- added R1012: 4k99, symbol Device:R
- added R1013: 1k/500V, symbol Device:R
- added R1014: 200k/500V, symbol Device:R
- added R1015, R1016, R1017: 10k, symbol Device:R
- added R1018: 5Meg/25ppm/.1%, symbol Device:R
- added R1019: 560k/.1%, symbol Device:R
- added R1020: 49k9/.1%, symbol Device:R
- added R1021: 4k99/.1%, symbol Device:R
- added R1022: 499/.25W/.1%, symbol Device:R
- added R1023, R1024: 100/1W/.1%, symbol Device:R
- added U1001, U1003, U1005: OPA2140, symbol ETH1CSMU1:OPA2140
- added U1002: LM393, symbol Comparator:LM393
- added U1004, U1006, U1007: DG444DY+, symbol ETH1CSMU1:DG444DY+
Connections:
- new net: U1003.5 (+), U1004.14, U1004.3
- new net: C1006.1, R1015.2, U1005.1
- new net: R1016.1, R1017.2, U1005.2 (-)
- new net: C1004.1, C1005.1, R1014.1, R1015.1, U1005.5 (+)
- new net: D1001.1 (K), D1002.2 (A), R1005.1, R1006.1, R1009.1, R1012.1, R1016.2
- new net: C1006.2, R1017.1
- new net: C1004.2, R1013.1
- new net: C1007.2, R1018.2, U1006.11, U1006.14, U1006.3, U1006.6, U1007.10
- new net: C1010.2, R1021.2, U1006.15
- new net: C1008.2, R1019.2, U1006.10
- new net: C1009.2, R1020.2, U1006.7
- new net: C1007.1, C1008.1, C1009.1, C1010.1, R1018.1, R1019.1, R1020.1, R1021.1, R1022.1, R1023.1, R1024.1
- new net: U1007.11, U1007.3, U1007.6
- new net: R1001.1, R1002.1, U1001.3 (+)
- new net: R1003.1, R1004.1, U1001.5 (+)
- new net: C1001.2, D1001.3 (K), U1001.1, U1002.3 (+)
- new net: C1001.1, D1001.2 (A), R1005.2, U1001.2 (-)
- new net: C1002.1, D1002.1 (K), R1006.2, U1001.6 (-)
- new net: C1002.2, D1002.3 (K), U1001.7, U1002.6 (_)
- new net: R1008.2, U1002.1, U1002.7
- new net: R1010.1, R1011.1, U1003.3 (+)
- new net: C1003.2, R1012.2, U1003.1
- new net: C1003.1, R1009.2, U1003.2 (-)
- new net +15V: U1001.8 (V+), U1002.8 (V+), U1003.8 (V+), U1005.8 (V+)
- new net +5V: R1007.1
- new net -15V: U1001.4 (V-), U1002.4 (V-), U1003.4 (V-), U1005.4 (V-)
- new net 100mA: R1023.2, R1024.2, U1007.2
- new net 10mA: R1022.2, U1006.2, U1007.7
- new net AMPIN: U1005.6 (-), U1005.7
- new net CL+: R1001.2
- new net CL-: R1003.2
- new net CLM: R1002.2, R1004.2, U1004.11, U1004.6
- new net FDACN: R1010.2
- new net FM: R1011.2, U1003.6 (-), U1003.7
- new net GND: U1002.2 (-), U1002.5 (+), U1005.3 (+)
- new net IM: U1004.10, U1004.15
- new net OCOM: C1005.2, R1013.2, R1014.2
- new net VM: U1004.2, U1004.7
- new net ~100uA: U1006.8
- new net ~10mA: U1006.1, U1007.8
- new net ~10uA: U1006.9
- new net ~1mA: U1006.16
- new net ~ICLAMP: R1007.2, R1008.1
- new net ~IMODE: U1004.16, U1004.8
- new net ~LT10mA: U1007.9
- new net ~VMODE: U1004.1, U1004.9
