File: HARDWARE/BASE/Analog.sch (KiCad schematic (older format))
At the start: 43 parts, among them U1001 OPA2140, U1002 LM393, U1003 OPA2140, U1004 DG444DY+, U1005 OPA2140, U1006 DG444DY+, U1007 DG444DY+

Commit message: Schematic design.
Parts:
- added C1005, C1009: 270p/500V, symbol Device:C
- added C1013: 150p, symbol Device:C
- added C1014: 22p/100V, symbol Device:C
- added C1015: 22p, symbol Device:C
- added C1016, C1017, C1018, C1019, C1020, C1021, C1022, C1023, C1024, C1025, C1026, C1027, C1028, C1029, C1030, C1031, C1032, C1033, C1034, C1035: 100n, symbol Device:C
- added C1036, C1037: 10p, symbol Device:C
- added D1001, D1003: 1N4148W, symbol Device:D
- added D1005, D1006, D1007, D1008: BAV99, Package_TO_SOT_SMD:SOT-23, symbol Diode:BAV99
- added K1001, K1002: EE2-5NU, Relay_SMD:Relay_DPDT_Kemet_EE2_NU, symbol Relay:EE2-5NU
- added Q1001, Q1002: MMBT3904, Package_TO_SOT_SMD:SOT-23, symbol Transistor_BJT:MMBT3904
- added R1013, R1014, R1019, R1024, R1025, R1030, R1036, R1039, R1046: 10k/.1%, symbol Device:R
- added R1016, R1035: 4k99/.1%, symbol Device:R
- added R1026: 22k1/.1%, symbol Device:R
- added R1027: 300k/.1%, symbol Device:R
- added R1034, R1042, R1043: 2k, symbol Device:R
- added R1037, R1038: 2/1W/.1%, symbol Device:R
- added R1040, R1041, R1044, R1045: 100k/.1%, symbol Device:R
- added R1047: 1k/.1%, symbol Device:R
- added R1048, R1049: 10k, symbol Device:R
- added TP1001: TP+OUT, symbol Connector:TestPoint
- added TP1002: TP+GUA, symbol Connector:TestPoint
- added TP1003: TP-OUT, symbol Connector:TestPoint
- added TP1004: TP-SEN, symbol Connector:TestPoint
- added TP1005: TPVM, symbol Connector:TestPoint
- added TP1006: TP+SEN, symbol Connector:TestPoint
- added TP1007: TPIM, symbol Connector:TestPoint
- added U1004, U1011: OPA140, symbol ETH1CSMU1:OPA140_REV
- added U1006, U1013: OPA2140, symbol ETH1CSMU1:OPA2140
- added U1009, U1012: OPA2140, symbol ETH1CSMU1:AQY221R2SZ
- added U1014: TL071, symbol Amplifier_Operational:TL071
- R1015: renamed from R1007; value 15k -> 4k99
- R1031: renamed from R1012; value 4k99 -> 4k99/.1%
- renumbered C1004 to C1001, C1007 to C1002, C1005 to C1003, C1008 to C1004, C1001 to C1006, C1006 to C1007, C1009 to C1008, C1002 to C1011, C1003 to C1012, D1001 to D1002, D1002 to D1004, R1013 to R1001, R1018 to R1002, R1014 to R1003, R1005 to R1004, R1015 to R1005, R1016 to R1006, R1019 to R1007, R1001 to R1008, R1017 to R1009, R1002 to R1010, R1020 to R1011, R1006 to R1012, R1021 to R1017, R1003 to R1018, R1008 to R1020, R1004 to R1021, R1009 to R1022, R1022 to R1023, R1010 to R1028, R1023 to R1029, R1011 to R1032, R1024 to R1033, U1005 to U1001, U1006 to U1002, U1001 to U1003, U1007 to U1005, U1002 to U1007, U1003 to U1008, U1004 to U1010
Connections:
- net labels added: +15VH, +GUA, +GUARD, +OUT, +SEN, -15VH, -OUT, -SEN, INT_GUARD, REL1, REL1_CTR, REL2, REL2_CTR, ~100mA, ~1A
- wire segments 203 -> 515
- no-connect marks 0 -> 4
Other:
- moved on the sheet: C1002, C1004, C1008, C1010, R1002, R1007, R1011, R1017, R1023, R1029, R1033, U1001C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

Commit message: Schematic design
Parts:
- added R1033: 2k, Resistor_SMD:R_0603_1608Metric_Pad0.98x0.95mm_HandSolder, symbol Device:R
- added U1009: TLP170D, Package_SO:SO-4_4.4x3.9mm_P2.54mm, symbol ETH1CSMU1:TLP170D
- C1001, C1003, C1005, C1009, C1014: footprint (none) -> Capacitor_SMD:C_0805_2012Metric_Pad1.18x1.45mm_HandSolder
- C1002, C1004, C1006, C1007, C1008, C1010, C1011, C1012, C1013, C1015, C1016, C1017, C1018, C1019, C1020, C1021, C1022, C1023, C1024, C1025, C1026, C1027, C1028, C1029, C1030, C1031, C1032, C1033, C1034, C1035, C1036, C1037: footprint (none) -> Capacitor_SMD:C_0603_1608Metric_Pad1.08x0.95mm_HandSolder
- D1001, D1003: footprint (none) -> Diode_SMD:D_SOD-123
- R1001, R1002, R1003: footprint (none) -> Resistor_SMD:R_1206_3216Metric_Pad1.30x1.75mm_HandSolder
- R1004, R1007, R1008, R1010, R1011, R1012, R1013, R1014, R1016, R1017, R1018, R1019, R1021, R1022, R1023, R1024, R1025, R1026, R1027, R1028, R1030, R1031, R1032: footprint (none) -> Resistor_SMD:R_0805_2012Metric_Pad1.20x1.40mm_HandSolder
- R1005, R1006, R1009: value 10k -> 10k/.1%; footprint (none) -> Resistor_SMD:R_0805_2012Metric_Pad1.20x1.40mm_HandSolder
- R1015, R1020: footprint (none) -> Resistor_SMD:R_0603_1608Metric_Pad0.98x0.95mm_HandSolder
- R1029: value 100/1W/.1% -> 100/1W/.5%; footprint (none) -> Resistor_SMD:R_2512_6332Metric_Pad1.40x3.35mm_HandSolder
- R1034: renamed from R1033; value 100/1W/.1% -> 100/1W/.5%; footprint (none) -> Resistor_SMD:R_2512_6332Metric_Pad1.40x3.35mm_HandSolder
- R1035: renamed from R1034; footprint (none) -> Resistor_SMD:R_0805_2012Metric_Pad1.20x1.40mm_HandSolder
- R1036: renamed from R1035; footprint (none) -> Resistor_SMD:R_0805_2012Metric_Pad1.20x1.40mm_HandSolder
- R1037: renamed from R1036; footprint (none) -> Resistor_SMD:R_0805_2012Metric_Pad1.20x1.40mm_HandSolder
- R1038: renamed from R1037; value 2/1W/.1% -> 2/1W/.5%; footprint (none) -> Resistor_SMD:R_2512_6332Metric_Pad1.40x3.35mm_HandSolder
- R1039: renamed from R1038; value 2/1W/.1% -> 2/1W/.5%; footprint (none) -> Resistor_SMD:R_2512_6332Metric_Pad1.40x3.35mm_HandSolder
- R1040: renamed from R1039; footprint (none) -> Resistor_SMD:R_0805_2012Metric_Pad1.20x1.40mm_HandSolder
- R1041: renamed from R1040; footprint (none) -> Resistor_SMD:R_0805_2012Metric_Pad1.20x1.40mm_HandSolder
- R1042: renamed from R1041; footprint (none) -> Resistor_SMD:R_0805_2012Metric_Pad1.20x1.40mm_HandSolder
- R1043: renamed from R1042; footprint (none) -> Resistor_SMD:R_0603_1608Metric_Pad0.98x0.95mm_HandSolder
- R1044: renamed from R1043; footprint (none) -> Resistor_SMD:R_0603_1608Metric_Pad0.98x0.95mm_HandSolder
- R1045: renamed from R1044; footprint (none) -> Resistor_SMD:R_0805_2012Metric_Pad1.20x1.40mm_HandSolder
- R1046: renamed from R1045; footprint (none) -> Resistor_SMD:R_0805_2012Metric_Pad1.20x1.40mm_HandSolder
- R1047: renamed from R1046; footprint (none) -> Resistor_SMD:R_0805_2012Metric_Pad1.20x1.40mm_HandSolder
- R1048: renamed from R1047; footprint (none) -> Resistor_SMD:R_0603_1608Metric_Pad0.98x0.95mm_HandSolder
- R1049: renamed from R1048; footprint (none) -> Resistor_SMD:R_0603_1608Metric_Pad0.98x0.95mm_HandSolder
- R1050: renamed from R1049; footprint (none) -> Resistor_SMD:R_0603_1608Metric_Pad0.98x0.95mm_HandSolder
- TP1001, TP1002, TP1003, TP1004, TP1005, TP1006, TP1007: footprint (none) -> TestPoint:TestPoint_Loop_D2.60mm_Drill1.6mm_Beaded
- U1001, U1003, U1004, U1006, U1007, U1008: footprint (none) -> Package_SO:SOIC-8_3.9x4.9mm_P1.27mm
- U1002, U1005: footprint (none) -> Package_SO:SOIC-16_3.9x9.9mm_P1.27mm
- U1010: renamed from U1009; value OPA2140 -> AQY221R2SZ; footprint (none) -> ETH1CSMU1:AQY212GS
- U1011: renamed from U1010; footprint (none) -> Package_SO:SOIC-16_3.9x9.9mm_P1.27mm
- U1012: renamed from U1011; footprint (none) -> Package_SO:SOIC-8_3.9x4.9mm_P1.27mm
- U1013: renamed from U1012; value OPA2140 -> AQY221R2SZ; footprint (none) -> ETH1CSMU1:AQY212GS
- U1014: renamed from U1013; footprint (none) -> Package_SO:SOIC-8_3.9x4.9mm_P1.27mm
- U1015: renamed from U1014; footprint (none) -> Package_SO:SOIC-8_3.9x4.9mm_P1.27mm
Connections:
- net labels added: ~VRANGE
- wire segments 515 -> 530
Other:
- moved on the sheet: C1036, Q1001, R1049

Commit message: PCB layout
Parts:
- removed K1001, K1002: EE2-5NU, Relay_SMD:Relay_DPDT_Kemet_EE2_NU, symbol Relay:EE2-5NU
- added K1001, K1002: TQ2SA-5V, ETH1CSMU1:SA, symbol ETH1CSMU1:TQ2SA-5V
Changed lines of the file:
@@
 $Descr A3 16535 11693
 encoding utf-8
-Sheet 10 13
+Sheet 10 12
 Title ""
 Date ""
@@
 Wire Wire Line
 	12650 7200 12900 7200
-$Comp
-L Relay:EE2-5NU K1001
-U 1 1 6150797E
-P 13850 2050
-F 0 "K1001" V 13083 2050 50  0000 C CNN
-F 1 "EE2-5NU" V 13174 2050 50  0000 C CNN
-F 2 "Relay_SMD:Relay_DPDT_Kemet_EE2_NU" H 13850 2050 50  0001 C CNN
-F 3 "https://content.kemet.com/datasheets/KEM_R7002_EC2_EE2.pdf" H 13850 2050 50  0001 C CNN
-	1    13850 2050
-	0    1    1    0
-$EndComp
 Wire Wire Line
 	13550 2050 13000 2050
 Connection ~ 9000 2050
-$Comp
-L power:+5V #PWR01002
-U 1 1 6153E1A3
-P 14250 1650
-F 0 "#PWR01002" H 14250 1500 50  0001 C CNN
-F 1 "+5V" V 14250 1800 50  0000 L CNN
-F 2 "" H 14250 1650 50  0001 C CNN
-F 3 "" H 14250 1650 50  0001 C CNN
-	1    14250 1650
-	0    1    1    0
-$EndComp
-$Comp
-L Device:D D1001
-U 1 1 6153F82D
-P 13850 1150
-F 0 "D1001" H 13850 933 50  0000 C CNN
-F 1 "1N4148W" H 13850 1024 50  0000 C CNN
-F 2 "Diode_SMD:D_SOD-123" H 13850 1150 50  0001 C CNN
-F 3 "~" H 13850 1150 50  0001 C CNN
-	1    13850 1150
-	-1   0    0    1
-$EndComp
-Wire Wire Line
-	14000 1150 14200 1150
-Wire Wire Line
-	14200 1150 14200 1650
-Wire Wire Line
-	14200 1650 14150 1650
-Wire Wire Line
-	13700 1150 13500 1150
-Wire Wire Line
-	13500 1150 13500 1650
-Wire Wire Line
-	13500 1650 13550 1650
-Wire Wire Line
-	14250 1650 14200 1650
-Connection ~ 14200 1650
 Wire Wire Line
 	13550 2450 13100 2450
@@
 Wire Wire Line
 	14150 2150 15000 2150
-$Comp
-L Relay:EE2-5NU K1002
-U 1 1 616C30DD
-P 13850 4100
-F 0 "K1002" V 13083 4100 50  0000 C CNN
-F 1 "EE2-5NU" V 13174 4100 50  0000 C CNN
-F 2 "Relay_SMD:Relay_DPDT_Kemet_EE2_NU" H 13850 4100 50  0001 C CNN
-F 3 "https://content.kemet.com/datasheets/KEM_R7002_EC2_EE2.pdf" H 13850 4100 50  0001 C CNN
-	1    13850 4100
-	0    1    1    0
-$EndComp
-$Comp
-L power:+5V #PWR01010
-U 1 1 616C30E4
-P 14250 3700
-F 0 "#PWR01010" H 14250 3550 50  0001 C CNN
-F 1 "+5V" V 14250 3850 50  0000 L CNN
-F 2 "" H 14250 3700 50  0001 C CNN
-F 3 "" H 14250 3700 50  0001 C CNN
-	1    14250 3700
-	0    1    1    0
-$EndComp
-$Comp
-L Device:D D1003
-U 1 1 616C30EA
-P 13850 3200
-F 0 "D1003" H 13850 2983 50  0000 C CNN
-F 1 "1N4148W" H 13850 3074 50  0000 C CNN
-F 2 "Diode_SMD:D_SOD-123" H 13850 3200 50  0001 C CNN
-F 3 "~" H 13850 3200 50  0001 C CNN
-	1    13850 3200
-	-1   0    0    1
-$EndComp
-Wire Wire Line
-	14000 3200 14200 3200
-Wire Wire Line
-	14200 3200 14200 3700
-Wire Wire Line
-	14200 3700 14150 3700
-Wire Wire Line
-	13700 3200 13500 3200
-Wire Wire Line
-	13500 3200 13500 3700
-Wire Wire Line
-	13500 3700 13550 3700
-Wire Wire Line
-	14250 3700 14200 3700
-Connection ~ 14200 3700
 Wire Wire Line
 	14150 4400 14600 4400
 Wire Wire Line
-	14600 4400 14600 2800
-Wire Wire Line
 	14600 2800 13000 2800
 Wire Wire Line
@@
 Wire Wire Line
 	14150 4600 15000 4600
-Wire Wire Line
-	13500 3700 13100 3700
-Connection ~ 13500 3700
-Text Label 13100 3700 0    50   ~ 0
-REL2
-Wire Wire Line
-	13500 1650 13100 1650
-Text Label 13100 1650 0    50   ~ 0
-REL1
-Connection ~ 13500 1650
 $Comp
 L Transistor_BJT:MMBT3904 Q1002
@@
 Wire Wire Line
 	9550 10450 10000 10450
+$Comp
+L ETH1CSMU1:TQ2SA-5V K1001
+U 1 1 605D44CE
+P 13850 2050
+F 0 "K1001" V 13083 2050 50  0000 C CNN
+F 1 "TQ2SA-5V" V 13174 2050 50  0000 C CNN
+F 2 "ETH1CSMU1:SA" H 14700 2000 50  0001 C CNN
+F 3 "" H 14700 2000 50  0001 C CNN
+	1    13850 2050
+	0    1    1    0
+$EndComp
+Connection ~ 14200 1650
+Text Label 14450 1650 2    50   ~ 0
+REL1
+Wire Wire Line
+	14200 1650 14450 1650
+Connection ~ 13500 1650
+Wire Wire Line
+	13450 1650 13500 1650
+Wire Wire Line
+	14200 1650 14150 1650
+Wire Wire Line
+	14200 1150 14200 1650
+Wire Wire Line
+	14000 1150 14200 1150
+Wire Wire Line
+	13500 1650 13550 1650
+Wire Wire Line
+	13500 1150 13500 1650
+Wire Wire Line
+	13700 1150 13500 1150
+$Comp
+L Device:D D1001
+U 1 1 6153F82D
+P 13850 1150
+F 0 "D1001" H 13850 933 50  0000 C CNN
+F 1 "1N4148W" H 13850 1024 50  0000 C CNN
+F 2 "Diode_SMD:D_SOD-123" H 13850 1150 50  0001 C CNN
+F 3 "~" H 13850 1150 50  0001 C CNN
+	1    13850 1150
+	1    0    0    1
+$EndComp
+$Comp
+L power:+5V #PWR01002
+U 1 1 6153E1A3
+P 13450 1650
+F 0 "#PWR01002" H 13450 1500 50  0001 C CNN
+F 1 "+5V" V 13450 1800 50  0000 L CNN
+F 2 "" H 13450 1650 50  0001 C CNN
+F 3 "" H 13450 1650 50  0001 C CNN
+	1    13450 1650
+	0    -1   1    0
+$EndComp
+$Comp
+L ETH1CSMU1:TQ2SA-5V K1002
+U 1 1 606B687F
+P 13850 4100
+F 0 "K1002" V 13083 4100 50  0000 C CNN
+F 1 "TQ2SA-5V" V 13174 4100 50  0000 C CNN
+F 2 "ETH1CSMU1:SA" H 14700 4050 50  0001 C CNN
+F 3 "" H 14700 4050 50  0001 C CNN
+	1    13850 4100
+	0    1    1    0
+$EndComp
+Wire Wire Line
+	14600 4400 14600 2800
+$Comp
+L power:+5V #PWR01010
+U 1 1 616C30E4
+P 13450 3700
+F 0 "#PWR01010" H 13450 3550 50  0001 C CNN
+F 1 "+5V" V 13450 3850 50  0000 L CNN
+F 2 "" H 13450 3700 50  0001 C CNN
+F 3 "" H 13450 3700 50  0001 C CNN
+	1    13450 3700
+	0    -1   1    0
+$EndComp
+$Comp
+L Device:D D1003
+U 1 1 616C30EA
+P 13850 3200
+F 0 "D1003" H 13850 2983 50  0000 C CNN
+F 1 "1N4148W" H 13850 3074 50  0000 C CNN
+F 2 "Diode_SMD:D_SOD-123" H 13850 3200 50  0001 C CNN
+F 3 "~" H 13850 3200 50  0001 C CNN
+	1    13850 3200
+	1    0    0    1
+$EndComp
+Wire Wire Line
+	13700 3200 13500 3200
+Wire Wire Line
+	13500 3200 13500 3700
+Wire Wire Line
+	13500 3700 13550 3700
+Wire Wire Line
+	14000 3200 14200 3200
+Wire Wire Line
+	14200 3200 14200 3700
+Wire Wire Line
+	14200 3700 14150 3700
+Wire Wire Line
+	13450 3700 13500 3700
+Connection ~ 13500 3700
+Wire Wire Line
+	14200 3700 14450 3700
+Connection ~ 14200 3700
+Text Label 14450 3700 2    50   ~ 0
+REL2
 $EndSCHEMATC

Commit message: Design
Other:
- moved on the sheet: U1011C
Changed lines of the file:
@@
-$Comp
-L ETH1CSMU1:DG444DY+ U1011
-U 3 1 60583C66
-P 2050 8650
-F 0 "U1011" H 2050 8917 50  0000 C CNN
-F 1 "DG444DY+" H 2050 8826 50  0000 C CNN
-F 2 "Package_SO:SOIC-16_3.9x9.9mm_P1.27mm" H 2050 8550 50  0001 C CNN
-F 3 "" H 2050 8650 50  0001 C CNN
-	3    2050 8650
-	-1   0    0    -1
-$EndComp
 $Comp
 L ETH1CSMU1:DG444DY+ U1011
@@
 	2050 8150 2050 7900
 Wire Wire Line
-	2350 8650 2400 8650
-Wire Wire Line
-	2400 8650 2400 7600
+	2400 8900 2400 7600
 Wire Wire Line
 	2400 7600 2350 7600
@@
 Wire Wire Line
 	1750 7600 1650 7600
-Text Label 2050 9200 1    50   ~ 0
+Text Label 2050 9450 1    50   ~ 0
 ~VMODE
 Wire Wire Line
@@
 Wire Wire Line
 	3300 2050 3450 2050
-Wire Wire Line
-	2050 8950 2050 9200
-Wire Wire Line
-	1750 8650 1500 8650
 Wire Wire Line
 	2900 6700 2400 6700
@@
 	1650 5800 1750 5800
 Wire Wire Line
-	1500 8650 1500 6700
+	1500 8900 1500 6700
 Connection ~ 1500 6700
 Wire Wire Line
@@
 Text Label 14450 3700 2    50   ~ 0
 REL2
+Text HLabel 2050 8150 3    50   Input ~ 0
+~IMODE
+Wire Wire Line
+	2050 9200 2050 9450
+Wire Wire Line
+	2350 8900 2400 8900
+Wire Wire Line
+	1750 8900 1500 8900
+$Comp
+L ETH1CSMU1:DG444DY+ U1011
+U 3 1 60583C66
+P 2050 8900
+F 0 "U1011" H 2050 9167 50  0000 C CNN
+F 1 "DG444DY+" H 2050 9076 50  0000 C CNN
+F 2 "Package_SO:SOIC-16_3.9x9.9mm_P1.27mm" H 2050 8800 50  0001 C CNN
+F 3 "" H 2050 8900 50  0001 C CNN
+	3    2050 8900
+	-1   0    0    -1
+$EndComp
+Text HLabel 2050 9450 3    50   Input ~ 0
+~VMODE
+Text HLabel 5450 3500 2    50   Output ~ 0
+~ICLAMP
 $EndSCHEMATC

Commit message: PCB and schematic design.
Parts:
- added J1001: Conn_02x12, Connector_PinHeader_2.54mm:PinHeader_2x12_P2.54mm_Vertical, symbol Connector_Generic:Conn_02x12_Odd_Even
- TP1001, TP1002, TP1003, TP1004, TP1005, TP1006, TP1007: footprint TestPoint:TestPoint_Loop_D2.60mm_Drill1.6mm_Beaded -> TestPoint:TestPoint_Pad_2.0x2.0mm
Connections:
- net +15V: now also J1001.3 (Pin_3), J1001.4 (Pin_4)
- net +15VH: now also J1001.15 (Pin_15), J1001.16 (Pin_16)
- net -15V: now also J1001.7 (Pin_7), J1001.8 (Pin_8)
- net -15VH: now also J1001.19 (Pin_19), J1001.20 (Pin_20)
- net AMPIN: now also J1001.10 (Pin_10), J1001.9 (Pin_9)
- net GND: now also J1001.5 (Pin_5), J1001.6 (Pin_6)
- net OCOM: now also J1001.17 (Pin_17), J1001.18 (Pin_18)
- net at C1002.2, R1002.2, U1002.11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: now also J1001.1 (Pin_1), J1001.2 (Pin_2)
- no-connect marks 4 -> 12
Other:
- moved on the sheet: C1002

Commit message: PCB layout
Connections:
- net +15V: now also J1001.21 (Pin_21), J1001.22 (Pin_22); no longer J1001.3 (Pin_3), J1001.4 (Pin_4)
- net +15VH: now also J1001.10 (Pin_10), J1001.9 (Pin_9); no longer J1001.15 (Pin_15), J1001.16 (Pin_16)
- net -15V: now also J1001.17 (Pin_17), J1001.18 (Pin_18); no longer J1001.7 (Pin_7), J1001.8 (Pin_8)
- net -15VH: now also J1001.5 (Pin_5), J1001.6 (Pin_6); no longer J1001.19 (Pin_19), J1001.20 (Pin_20)
- net AMPIN: now also J1001.15 (Pin_15), J1001.16 (Pin_16); no longer J1001.10 (Pin_10), J1001.9 (Pin_9)
- net GND: now also J1001.19 (Pin_19), J1001.20 (Pin_20); no longer J1001.5 (Pin_5), J1001.6 (Pin_6)
- net OCOM: now also J1001.7 (Pin_7), J1001.8 (Pin_8); no longer J1001.17 (Pin_17), J1001.18 (Pin_18)
- net at C1002.2, R1002.2, U1002.11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: now also J1001.23 (Pin_23), J1001.24 (Pin_24); no longer J1001.1 (Pin_1), J1001.2 (Pin_2)
Changed lines of the file:
@@
 AMPIN
-Wire Wire Line
-	6450 600  6450 900
 Wire Wire Line
 	6750 900  6750 850
@@
 L Connector_Generic:Conn_02x12_Odd_Even J1001
 U 1 1 60CB8954
-P 6350 1100
-F 0 "J1001" V 6354 1680 50  0000 L CNN
-F 1 "Conn_02x12" V 6445 1680 50  0000 L CNN
-F 2 "Connector_PinHeader_2.54mm:PinHeader_2x12_P2.54mm_Vertical" H 6350 1100 50  0001 C CNN
-F 3 "~" H 6350 1100 50  0001 C CNN
-	1    6350 1100
-	0    1    1    0
+P 6250 1200
+F 0 "J1001" V 6350 250 50  0000 L CNN
+F 1 "Conn_02x12" V 6250 50  50  0000 L CNN
+F 2 "Connector_PinHeader_2.54mm:PinHeader_2x12_P2.54mm_Vertical" H 6250 1200 50  0001 C CNN
+F 3 "~" H 6250 1200 50  0001 C CNN
+	1    6250 1200
+	0    -1   -1   0
 $EndComp
 NoConn ~ 6250 900
@@
 NoConn ~ 5750 1400
 NoConn ~ 5850 1400
+Wire Wire Line
+	6450 600  6450 900
 $EndSCHEMATC

Commit message: PCB layout
Parts:
- removed J1001: Conn_02x12, Connector_PinHeader_2.54mm:PinHeader_2x12_P2.54mm_Vertical, symbol Connector_Generic:Conn_02x12_Odd_Even
- added J1001: Conn_02x02, Connector_PinHeader_2.54mm:PinHeader_2x02_P2.54mm_Vertical, symbol Connector_Generic:Conn_02x02_Odd_Even
- added J1002: Conn_02x06, Connector_PinHeader_2.54mm:PinHeader_2x06_P2.54mm_Vertical, symbol Connector_Generic:Conn_02x06_Odd_Even
Connections:
- net +15V: now also J1002.10 (Pin_10), J1002.9 (Pin_9)
- net +15VH: now also J1001.4 (Pin_4)
- net -15V: now also J1002.5 (Pin_5), J1002.6 (Pin_6)
- net -15VH: now also J1001.2 (Pin_2)
- net AMPIN: now also J1002.3 (Pin_3), J1002.4 (Pin_4)
- net GND: now also J1002.7 (Pin_7), J1002.8 (Pin_8)
- net OCOM: now also J1001.1 (Pin_1), J1001.3 (Pin_3)
- net at C1002.2, R1002.2, U1002.11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: now also J1002.11 (Pin_11), J1002.12 (Pin_12)
- no-connect marks 12 -> 6
Changed lines of the file:
@@
 L ETH1CSMU1:+15VH #PWR01006
 U 1 1 60A93F21
-P 6150 900
-F 0 "#PWR01006" H 6150 750 50  0001 C CNN
-F 1 "+15VH" V 6150 1150 50  0000 C CNN
-F 2 "" H 6150 900 50  0001 C CNN
-F 3 "" H 6150 900 50  0001 C CNN
-	1    6150 900
+P 5700 900
+F 0 "#PWR01006" H 5700 750 50  0001 C CNN
+F 1 "+15VH" V 5700 1150 50  0000 C CNN
+F 2 "" H 5700 900 50  0001 C CNN
+F 3 "" H 5700 900 50  0001 C CNN
+	1    5700 900
 	1    0    0    -1
-$EndComp
-$Comp
-L ETH1CSMU1:+15VH #PWR01010
-U 1 1 60A95537
-P 6150 1400
-F 0 "#PWR01010" H 6150 1250 50  0001 C CNN
-F 1 "+15VH" V 6150 1650 50  0000 C CNN
-F 2 "" H 6150 1400 50  0001 C CNN
-F 3 "" H 6150 1400 50  0001 C CNN
-	1    6150 1400
-	-1   0    0    1
 $EndComp
 $Comp
 L ETH1CSMU1:OCOM #PWR01005
 U 1 1 60AA1230
-P 6050 900
-F 0 "#PWR01005" H 6050 650 50  0001 C CNN
-F 1 "OCOM" V 6050 650 50  0000 C CNN
-F 2 "" H 6050 900 50  0001 C CNN
-F 3 "" H 6050 900 50  0001 C CNN
-	1    6050 900
-	-1   0    0    1
+P 5600 1400
+F 0 "#PWR01005" H 5600 1150 50  0001 C CNN
+F 1 "OCOM" V 5600 1150 50  0000 C CNN
+F 2 "" H 5600 1400 50  0001 C CNN
+F 3 "" H 5600 1400 50  0001 C CNN
+	1    5600 1400
+	1    0    0    -1
 $EndComp
 $Comp
 L ETH1CSMU1:OCOM #PWR01009
 U 1 1 60AA2A36
-P 6050 1400
-F 0 "#PWR01009" H 6050 1150 50  0001 C CNN
-F 1 "OCOM" V 6050 1150 50  0000 C CNN
-F 2 "" H 6050 1400 50  0001 C CNN
-F 3 "" H 6050 1400 50  0001 C CNN
-	1    6050 1400
+P 5700 1400
+F 0 "#PWR01009" H 5700 1150 50  0001 C CNN
+F 1 "OCOM" V 5700 1150 50  0000 C CNN
+F 2 "" H 5700 1400 50  0001 C CNN
+F 3 "" H 5700 1400 50  0001 C CNN
+	1    5700 1400
 	1    0    0    -1
 $EndComp
@@
 L ETH1CSMU1:-15VH #PWR01004
 U 1 1 60AA6459
-P 5950 900
-F 0 "#PWR01004" H 5950 750 50  0001 C CNN
-F 1 "-15VH" V 5950 1150 50  0000 C CNN
-F 2 "" H 5950 900 50  0001 C CNN
-F 3 "" H 5950 900 50  0001 C CNN
-	1    5950 900
+P 5600 900
+F 0 "#PWR01004" H 5600 750 50  0001 C CNN
+F 1 "-15VH" V 5600 1150 50  0000 C CNN
+F 2 "" H 5600 900 50  0001 C CNN
+F 3 "" H 5600 900 50  0001 C CNN
+	1    5600 900
 	1    0    0    -1
 $EndComp
+Wire Wire Line
+	6450 600  6450 900
 $Comp
-L ETH1CSMU1:-15VH #PWR01008
-U 1 1 60AA7A38
-P 5950 1400
-F 0 "#PWR01008" H 5950 1250 50  0001 C CNN
-F 1 "-15VH" V 5950 1650 50  0000 C CNN
-F 2 "" H 5950 1400 50  0001 C CNN
-F 3 "" H 5950 1400 50  0001 C CNN
-	1    5950 1400
-	-1   0    0    1
+L Connector_Generic:Conn_02x06_Odd_Even J1002
+U 1 1 606616AB
+P 6550 1200
+F 0 "J1002" V 6646 812 50  0000 R CNN
+F 1 "Conn_02x06" V 6555 812 50  0000 R CNN
+F 2 "Connector_PinHeader_2.54mm:PinHeader_2x06_P2.54mm_Vertical" H 6550 1200 50  0001 C CNN
+F 3 "~" H 6550 1200 50  0001 C CNN
+	1    6550 1200
+	0    -1   -1   0
 $EndComp
 $Comp
-L Connector_Generic:Conn_02x12_Odd_Even J1001
-U 1 1 60CB8954
-P 6250 1200
-F 0 "J1001" V 6350 250 50  0000 L CNN
-F 1 "Conn_02x12" V 6250 50  50  0000 L CNN
-F 2 "Connector_PinHeader_2.54mm:PinHeader_2x12_P2.54mm_Vertical" H 6250 1200 50  0001 C CNN
-F 3 "~" H 6250 1200 50  0001 C CNN
-	1    6250 1200
+L Connector_Generic:Conn_02x02_Odd_Even J1001
+U 1 1 60671954
+P 5600 1200
+F 0 "J1001" V 5696 1012 50  0000 R CNN
+F 1 "Conn_02x02" V 5605 1012 50  0000 R CNN
+F 2 "Connector_PinHeader_2.54mm:PinHeader_2x02_P2.54mm_Vertical" H 5600 1200 50  0001 C CNN
+F 3 "~" H 5600 1200 50  0001 C CNN
+	1    5600 1200
 	0    -1   -1   0
 $EndComp
-NoConn ~ 6250 900
-NoConn ~ 6250 1400
-NoConn ~ 5850 900
-NoConn ~ 5750 900
-NoConn ~ 5750 1400
-NoConn ~ 5850 1400
-Wire Wire Line
-	6450 600  6450 900
 $EndSCHEMATC

Commit message: PCB and schematic
Connections:
- net 10-100mA: now reaches J1002.1 (Pin_1)
- net 10-100mA: now also J1002.2 (Pin_2)
- no-connect marks 6 -> 4
Other:
- moved on the sheet: C1001, C1002, C1003, C1004, C1005, C1006, C1007, C1008, C1009, C1010, C1011, C1012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
