File: HARDWARE/BASE/SDRAM.sch (KiCad schematic (older format))
At the start: 8 parts, among them U401 MT48LC16M16A2P-6A

Commit message: Schematic design
Parts:
- C301: renamed from C401; footprint Capacitor_SMD:C_0603_1608Metric_Pad1.05x0.95mm_HandSolder -> Capacitor_SMD:C_0603_1608Metric_Pad1.08x0.95mm_HandSolder
- C302: renamed from C402; footprint Capacitor_SMD:C_0603_1608Metric_Pad1.05x0.95mm_HandSolder -> Capacitor_SMD:C_0603_1608Metric_Pad1.08x0.95mm_HandSolder
- C303: renamed from C403; footprint Capacitor_SMD:C_0603_1608Metric_Pad1.05x0.95mm_HandSolder -> Capacitor_SMD:C_0603_1608Metric_Pad1.08x0.95mm_HandSolder
- C304: renamed from C404; footprint Capacitor_SMD:C_0603_1608Metric_Pad1.05x0.95mm_HandSolder -> Capacitor_SMD:C_0603_1608Metric_Pad1.08x0.95mm_HandSolder
- C305: renamed from C405; footprint Capacitor_SMD:C_0603_1608Metric_Pad1.05x0.95mm_HandSolder -> Capacitor_SMD:C_0603_1608Metric_Pad1.08x0.95mm_HandSolder
- C306: renamed from C406; footprint Capacitor_SMD:C_0603_1608Metric_Pad1.05x0.95mm_HandSolder -> Capacitor_SMD:C_0603_1608Metric_Pad1.08x0.95mm_HandSolder
- C307: renamed from C407; footprint Capacitor_SMD:C_0603_1608Metric_Pad1.05x0.95mm_HandSolder -> Capacitor_SMD:C_0603_1608Metric_Pad1.08x0.95mm_HandSolder
- renumbered U401 to U301
Changed lines of the file:
@@
 $Descr A4 11693 8268
 encoding utf-8
-Sheet 4 10
+Sheet 3 10
 Title "SDRAM"
 Date "2020-03-07"
@@
 D[0..15]
 $Comp
-L Device:C C401
+L Device:C C301
 U 1 1 5F12988C
 P 1000 7250
-F 0 "C401" H 1115 7296 50  0000 L CNN
+F 0 "C301" H 1115 7296 50  0000 L CNN
 F 1 "100n" H 1115 7205 50  0000 L CNN
-F 2 "Capacitor_SMD:C_0603_1608Metric_Pad1.05x0.95mm_HandSolder" H 1038 7100 50  0001 C CNN
+F 2 "Capacitor_SMD:C_0603_1608Metric_Pad1.08x0.95mm_HandSolder" H 1038 7100 50  0001 C CNN
 F 3 "~" H 1000 7250 50  0001 C CNN
 	1    1000 7250
@@
 $EndComp
 $Comp
-L Device:C C402
+L Device:C C302
 U 1 1 5F12BD5A
 P 1500 7250
-F 0 "C402" H 1615 7296 50  0000 L CNN
+F 0 "C302" H 1615 7296 50  0000 L CNN
 F 1 "100n" H 1615 7205 50  0000 L CNN
-F 2 "Capacitor_SMD:C_0603_1608Metric_Pad1.05x0.95mm_HandSolder" H 1538 7100 50  0001 C CNN
+F 2 "Capacitor_SMD:C_0603_1608Metric_Pad1.08x0.95mm_HandSolder" H 1538 7100 50  0001 C CNN
 F 3 "~" H 1500 7250 50  0001 C CNN
 	1    1500 7250
@@
 $EndComp
 $Comp
-L Device:C C403
+L Device:C C303
 U 1 1 5F12CAA5
 P 2000 7250
-F 0 "C403" H 2115 7296 50  0000 L CNN
+F 0 "C303" H 2115 7296 50  0000 L CNN
 F 1 "100n" H 2115 7205 50  0000 L CNN
-F 2 "Capacitor_SMD:C_0603_1608Metric_Pad1.05x0.95mm_HandSolder" H 2038 7100 50  0001 C CNN
+F 2 "Capacitor_SMD:C_0603_1608Metric_Pad1.08x0.95mm_HandSolder" H 2038 7100 50  0001 C CNN
 F 3 "~" H 2000 7250 50  0001 C CNN
 	1    2000 7250
@@
 $EndComp
 $Comp
-L Device:C C404
+L Device:C C304
 U 1 1 5F12CAAB
 P 2500 7250
-F 0 "C404" H 2615 7296 50  0000 L CNN
+F 0 "C304" H 2615 7296 50  0000 L CNN
 F 1 "100n" H 2615 7205 50  0000 L CNN
-F 2 "Capacitor_SMD:C_0603_1608Metric_Pad1.05x0.95mm_HandSolder" H 2538 7100 50  0001 C CNN
+F 2 "Capacitor_SMD:C_0603_1608Metric_Pad1.08x0.95mm_HandSolder" H 2538 7100 50  0001 C CNN
 F 3 "~" H 2500 7250 50  0001 C CNN
 	1    2500 7250
@@
 $EndComp
 $Comp
-L Device:C C405
+L Device:C C305
 U 1 1 5F12F1B4
 P 3000 7250
-F 0 "C405" H 3115 7296 50  0000 L CNN
+F 0 "C305" H 3115 7296 50  0000 L CNN
 F 1 "100n" H 3115 7205 50  0000 L CNN
-F 2 "Capacitor_SMD:C_0603_1608Metric_Pad1.05x0.95mm_HandSolder" H 3038 7100 50  0001 C CNN
+F 2 "Capacitor_SMD:C_0603_1608Metric_Pad1.08x0.95mm_HandSolder" H 3038 7100 50  0001 C CNN
 F 3 "~" H 3000 7250 50  0001 C CNN
 	1    3000 7250
@@
 $EndComp
 $Comp
-L Device:C C406
+L Device:C C306
 U 1 1 5F12F1BA
 P 3500 7250
-F 0 "C406" H 3615 7296 50  0000 L CNN
+F 0 "C306" H 3615 7296 50  0000 L CNN
 F 1 "100n" H 3615 7205 50  0000 L CNN
-F 2 "Capacitor_SMD:C_0603_1608Metric_Pad1.05x0.95mm_HandSolder" H 3538 7100 50  0001 C CNN
+F 2 "Capacitor_SMD:C_0603_1608Metric_Pad1.08x0.95mm_HandSolder" H 3538 7100 50  0001 C CNN
 F 3 "~" H 3500 7250 50  0001 C CNN
 	1    3500 7250
@@
 $EndComp
 $Comp
-L Device:C C407
+L Device:C C307
 U 1 1 5F12F1C0
 P 4000 7250
-F 0 "C407" H 4115 7296 50  0000 L CNN
+F 0 "C307" H 4115 7296 50  0000 L CNN
 F 1 "100n" H 4115 7205 50  0000 L CNN
-F 2 "Capacitor_SMD:C_0603_1608Metric_Pad1.05x0.95mm_HandSolder" H 4038 7100 50  0001 C CNN
+F 2 "Capacitor_SMD:C_0603_1608Metric_Pad1.08x0.95mm_HandSolder" H 4038 7100 50  0001 C CNN
 F 3 "~" H 4000 7250 50  0001 C CNN
 	1    4000 7250
@@
 	2500 7000 2500 7050
 $Comp
-L ETH1CSMU1:MT48LC16M16A2P-6A U401
+L ETH1CSMU1:MT48LC16M16A2P-6A U301
 U 1 1 6032E9DB
 P 5650 3200
-F 0 "U401" H 6450 4550 50  0000 C CNN
+F 0 "U301" H 6450 4550 50  0000 C CNN
 F 1 "MT48LC16M16A2P-6A" H 6450 4450 50  0000 C CNN
 F 2 "ETH1CSMU1:TSSOP-54" H 5650 3200 50  0001 C CNN
@@
 	4600 3400 4500 3500
 $Comp
-L power:GND #PWR0404
+L power:GND #PWR0304
 U 1 1 604E3C92
 P 5650 4700
-F 0 "#PWR0404" H 5650 4450 50  0001 C CNN
+F 0 "#PWR0304" H 5650 4450 50  0001 C CNN
 F 1 "GND" H 5655 4527 50  0000 C CNN
 F 2 "" H 5650 4700 50  0001 C CNN
@@
 $EndComp
 $Comp
-L power:GND #PWR0402
+L power:GND #PWR0302
 U 1 1 604E5A22
 P 2500 7500
-F 0 "#PWR0402" H 2500 7250 50  0001 C CNN
+F 0 "#PWR0302" H 2500 7250 50  0001 C CNN
 F 1 "GND" H 2505 7327 50  0000 C CNN
 F 2 "" H 2500 7500 50  0001 C CNN
@@
 $EndComp
 $Comp
-L power:+3.3V #PWR0401
+L power:+3.3V #PWR0301
 U 1 1 604E6150
 P 2500 7000
-F 0 "#PWR0401" H 2500 6850 50  0001 C CNN
+F 0 "#PWR0301" H 2500 6850 50  0001 C CNN
 F 1 "+3.3V" H 2515 7173 50  0000 C CNN
 F 2 "" H 2500 7000 50  0001 C CNN
@@
 $EndComp
 $Comp
-L power:+3.3V #PWR0403
+L power:+3.3V #PWR0303
 U 1 1 604E7F38
 P 5650 1700
-F 0 "#PWR0403" H 5650 1550 50  0001 C CNN
+F 0 "#PWR0303" H 5650 1550 50  0001 C CNN
 F 1 "+3.3V" H 5665 1873 50  0000 C CNN
 F 2 "" H 5650 1700 50  0001 C CNN
