File: HARDWARE/BASE/SWD_Isolated.sch (KiCad schematic (older format))
At the start: 15 parts, among them J1201 20021111-00010T4LF, U1201 MEE1S0303DC, U1202 Si8606

Commit message: Schematic design.
Parts:
- C1101: renamed from C1201; footprint (none) -> Capacitor_SMD:C_0603_1608Metric_Pad1.08x0.95mm_HandSolder
- C1102: renamed from C1202; footprint (none) -> Capacitor_SMD:C_0603_1608Metric_Pad1.08x0.95mm_HandSolder
- C1103: renamed from C1203; footprint (none) -> Capacitor_SMD:C_0603_1608Metric_Pad1.08x0.95mm_HandSolder
- C1104: renamed from C1204; footprint (none) -> Capacitor_SMD:C_0603_1608Metric_Pad1.08x0.95mm_HandSolder
- C1105: renamed from C1205; footprint (none) -> Capacitor_SMD:C_0603_1608Metric_Pad1.08x0.95mm_HandSolder
- C1106: renamed from C1206; footprint (none) -> Capacitor_SMD:C_0603_1608Metric_Pad1.08x0.95mm_HandSolder
- R1101: renamed from R1201; footprint (none) -> Resistor_SMD:R_0603_1608Metric_Pad0.98x0.95mm_HandSolder
- R1102: renamed from R1202; footprint (none) -> Resistor_SMD:R_0603_1608Metric_Pad0.98x0.95mm_HandSolder
- R1103: renamed from R1203; footprint (none) -> Resistor_SMD:R_0603_1608Metric_Pad0.98x0.95mm_HandSolder
- R1104: renamed from R1204; footprint (none) -> Resistor_SMD:R_0603_1608Metric_Pad0.98x0.95mm_HandSolder
- R1105: renamed from R1205; footprint (none) -> Resistor_SMD:R_0603_1608Metric_Pad0.98x0.95mm_HandSolder
- R1106: renamed from R1206; footprint (none) -> Resistor_SMD:R_0603_1608Metric_Pad0.98x0.95mm_HandSolder
- U1101: renamed from U1201; footprint (none) -> ETH1CSMU1:MEE1_DIP
- U1102: renamed from U1202; value Si8606 -> SI8606AC-B-IS1; footprint (none) -> Package_SO:SOIC-16_3.9x9.9mm_P1.27mm
- renumbered J1201 to J1101
Connections:
- no-connect marks 4 -> 6

Commit message: Schematic design
Parts:
- removed U1101: MEE1S0303DC, ETH1CSMU1:MEE1_DIP, symbol ETH1CSMU1:MEE1S0303DC
- added U1101: NXE1S0303MC, Converter_DCDC:Converter_DCDC_muRata_NXExSxxxxMC_SMD, symbol Regulator_Switching:NXE1S0303MC
Connections:
- wire segments 62 -> 54
Other:
- moved on the sheet: C1101, C1102, C1103, C1104
Changed lines of the file:
@@
 $Descr A4 11693 8268
 encoding utf-8
-Sheet 11 12
+Sheet 11 13
 Title ""
 Date ""
@@
 $EndComp
 $Comp
-L ETH1CSMU1:MEE1S0303DC U1101
-U 1 1 6155D8C0
-P 6300 2900
-F 0 "U1101" H 6300 3267 50  0000 C CNN
-F 1 "MEE1S0303DC" H 6300 3176 50  0000 C CNN
-F 2 "ETH1CSMU1:MEE1_DIP" H 5250 2650 50  0001 L CNN
-F 3 "https://power.murata.com/pub/data/power/ncl/kdc_mee1.pdf" H 7350 2600 50  0001 L CNN
-	1    6300 2900
-	-1   0    0    -1
-$EndComp
-$Comp
 L power:+3.3V #PWR01102
 U 1 1 61560827
-P 7400 2650
-F 0 "#PWR01102" H 7400 2500 50  0001 C CNN
-F 1 "+3.3V" H 7415 2823 50  0000 C CNN
-F 2 "" H 7400 2650 50  0001 C CNN
-F 3 "" H 7400 2650 50  0001 C CNN
-	1    7400 2650
-	1    0    0    -1
-$EndComp
-Wire Wire Line
-	6750 2800 6700 2800
+P 7400 2850
+F 0 "#PWR01102" H 7400 2700 50  0001 C CNN
+F 1 "+3.3V" H 7415 3023 50  0000 C CNN
+F 2 "" H 7400 2850 50  0001 C CNN
+F 3 "" H 7400 2850 50  0001 C CNN
+	1    7400 2850
+	1    0    0    -1
+$EndComp
 $Comp
 L Device:C C1103
 U 1 1 61565069
-P 6900 2900
-F 0 "C1103" H 7015 2946 50  0000 L CNN
-F 1 "100n" H 7015 2855 50  0000 L CNN
-F 2 "Capacitor_SMD:C_0603_1608Metric_Pad1.08x0.95mm_HandSolder" H 6938 2750 50  0001 C CNN
-F 3 "~" H 6900 2900 50  0001 C CNN
-	1    6900 2900
+P 6900 3100
+F 0 "C1103" H 7015 3146 50  0000 L CNN
+F 1 "100n" H 7015 3055 50  0000 L CNN
+F 2 "Capacitor_SMD:C_0603_1608Metric_Pad1.08x0.95mm_HandSolder" H 6938 2950 50  0001 C CNN
+F 3 "~" H 6900 3100 50  0001 C CNN
+	1    6900 3100
 	1    0    0    -1
 $EndComp
@@
 L Device:C C1104
 U 1 1 6156506F
-P 7400 2900
-F 0 "C1104" H 7515 2946 50  0000 L CNN
-F 1 "1u" H 7515 2855 50  0000 L CNN
-F 2 "Capacitor_SMD:C_0603_1608Metric_Pad1.08x0.95mm_HandSolder" H 7438 2750 50  0001 C CNN
-F 3 "~" H 7400 2900 50  0001 C CNN
-	1    7400 2900
-	1    0    0    -1
-$EndComp
-Wire Wire Line
-	6900 2700 6900 2750
-Wire Wire Line
-	7400 2750 7400 2700
-Wire Wire Line
-	6900 2700 6750 2700
-Connection ~ 6900 2700
-Wire Wire Line
-	6750 2700 6750 2800
-Wire Wire Line
-	6700 3000 6750 3000
-Wire Wire Line
-	6750 3000 6750 3100
-Wire Wire Line
-	6750 3100 6900 3100
-Wire Wire Line
-	7400 3100 7400 3050
-Wire Wire Line
-	6900 3050 6900 3100
-Connection ~ 6900 3100
-Wire Wire Line
-	6900 3100 7400 3100
-Wire Wire Line
-	6900 2700 7400 2700
+P 7400 3100
+F 0 "C1104" H 7515 3146 50  0000 L CNN
+F 1 "1u" H 7515 3055 50  0000 L CNN
+F 2 "Capacitor_SMD:C_0603_1608Metric_Pad1.08x0.95mm_HandSolder" H 7438 2950 50  0001 C CNN
+F 3 "~" H 7400 3100 50  0001 C CNN
+	1    7400 3100
+	1    0    0    -1
+$EndComp
+Wire Wire Line
+	6900 2900 6900 2950
+Wire Wire Line
+	7400 2950 7400 2900
+Wire Wire Line
+	6900 2900 6750 2900
+Connection ~ 6900 2900
+Wire Wire Line
+	6750 3300 6900 3300
+Wire Wire Line
+	7400 3300 7400 3250
+Wire Wire Line
+	6900 3250 6900 3300
+Connection ~ 6900 3300
+Wire Wire Line
+	6900 3300 7400 3300
+Wire Wire Line
+	6900 2900 7400 2900
 $Comp
 L power:GND #PWR01104
 U 1 1 61571BF7
-P 7400 3150
-F 0 "#PWR01104" H 7400 2900 50  0001 C CNN
-F 1 "GND" H 7405 2977 50  0000 C CNN
-F 2 "" H 7400 3150 50  0001 C CNN
-F 3 "" H 7400 3150 50  0001 C CNN
-	1    7400 3150
-	1    0    0    -1
-$EndComp
-Wire Wire Line
-	7400 3150 7400 3100
-Connection ~ 7400 3100
-Wire Wire Line
-	7400 2650 7400 2700
-Connection ~ 7400 2700
-Wire Wire Line
-	5850 2800 5900 2800
-Wire Wire Line
-	5550 2700 5550 2750
-Wire Wire Line
-	5050 2750 5050 2700
-Wire Wire Line
-	5550 2700 5850 2700
-Connection ~ 5550 2700
-Wire Wire Line
-	5850 2700 5850 2800
-Wire Wire Line
-	5900 3000 5850 3000
-Wire Wire Line
-	5850 3000 5850 3100
-Wire Wire Line
-	5850 3100 5550 3100
-Wire Wire Line
-	5050 3100 5050 3050
-Wire Wire Line
-	5550 3050 5550 3100
-Connection ~ 5550 3100
-Wire Wire Line
-	5550 3100 5050 3100
-Wire Wire Line
-	5550 2700 5050 2700
-Wire Wire Line
-	5050 3150 5050 3100
-Connection ~ 5050 3100
-Wire Wire Line
-	5050 2650 5050 2700
-Connection ~ 5050 2700
+P 7400 3350
+F 0 "#PWR01104" H 7400 3100 50  0001 C CNN
+F 1 "GND" H 7405 3177 50  0000 C CNN
+F 2 "" H 7400 3350 50  0001 C CNN
+F 3 "" H 7400 3350 50  0001 C CNN
+	1    7400 3350
+	1    0    0    -1
+$EndComp
+Wire Wire Line
+	7400 3350 7400 3300
+Connection ~ 7400 3300
+Wire Wire Line
+	7400 2850 7400 2900
+Connection ~ 7400 2900
+Wire Wire Line
+	5350 2900 5350 2950
+Wire Wire Line
+	4850 2950 4850 2900
+Wire Wire Line
+	5350 2900 5750 2900
+Connection ~ 5350 2900
+Wire Wire Line
+	5750 3300 5350 3300
+Wire Wire Line
+	4850 3300 4850 3250
+Wire Wire Line
+	5350 3250 5350 3300
+Connection ~ 5350 3300
+Wire Wire Line
+	5350 3300 4850 3300
+Wire Wire Line
+	5350 2900 4850 2900
+Wire Wire Line
+	4850 3350 4850 3300
+Connection ~ 4850 3300
+Wire Wire Line
+	4850 2850 4850 2900
+Connection ~ 4850 2900
 $Comp
 L ETH1CSMU1:+3.3VF #PWR01101
 U 1 1 6157C491
-P 5050 2650
-F 0 "#PWR01101" H 5050 2500 50  0001 C CNN
-F 1 "+3.3VF" H 5065 2823 50  0000 C CNN
-F 2 "" H 5050 2650 50  0001 C CNN
-F 3 "" H 5050 2650 50  0001 C CNN
-	1    5050 2650
+P 4850 2850
+F 0 "#PWR01101" H 4850 2700 50  0001 C CNN
+F 1 "+3.3VF" H 4865 3023 50  0000 C CNN
+F 2 "" H 4850 2850 50  0001 C CNN
+F 3 "" H 4850 2850 50  0001 C CNN
+	1    4850 2850
 	1    0    0    -1
 $EndComp
@@
 L ETH1CSMU1:DGNDF #PWR01103
 U 1 1 6157D66F
-P 5050 3150
-F 0 "#PWR01103" H 5050 2900 50  0001 C CNN
-F 1 "DGNDF" H 5055 2977 50  0000 C CNN
-F 2 "" H 5050 3150 50  0001 C CNN
-F 3 "" H 5050 3150 50  0001 C CNN
-	1    5050 3150
+P 4850 3350
+F 0 "#PWR01103" H 4850 3100 50  0001 C CNN
+F 1 "DGNDF" H 4855 3177 50  0000 C CNN
+F 2 "" H 4850 3350 50  0001 C CNN
+F 3 "" H 4850 3350 50  0001 C CNN
+	1    4850 3350
 	1    0    0    -1
 $EndComp
@@
 L Device:C C1101
 U 1 1 6157E6AE
-P 5050 2900
-F 0 "C1101" H 5165 2946 50  0000 L CNN
-F 1 "100n" H 5165 2855 50  0000 L CNN
-F 2 "Capacitor_SMD:C_0603_1608Metric_Pad1.08x0.95mm_HandSolder" H 5088 2750 50  0001 C CNN
-F 3 "~" H 5050 2900 50  0001 C CNN
-	1    5050 2900
+P 4850 3100
+F 0 "C1101" H 4965 3146 50  0000 L CNN
+F 1 "100n" H 4965 3055 50  0000 L CNN
+F 2 "Capacitor_SMD:C_0603_1608Metric_Pad1.08x0.95mm_HandSolder" H 4888 2950 50  0001 C CNN
+F 3 "~" H 4850 3100 50  0001 C CNN
+	1    4850 3100
 	1    0    0    -1
 $EndComp
@@
 L Device:C C1102
 U 1 1 6157EE69
-P 5550 2900
-F 0 "C1102" H 5665 2946 50  0000 L CNN
-F 1 "1u" H 5665 2855 50  0000 L CNN
-F 2 "Capacitor_SMD:C_0603_1608Metric_Pad1.08x0.95mm_HandSolder" H 5588 2750 50  0001 C CNN
-F 3 "~" H 5550 2900 50  0001 C CNN
-	1    5550 2900
+P 5350 3100
+F 0 "C1102" H 5465 3146 50  0000 L CNN
+F 1 "1u" H 5465 3055 50  0000 L CNN
+F 2 "Capacitor_SMD:C_0603_1608Metric_Pad1.08x0.95mm_HandSolder" H 5388 2950 50  0001 C CNN
+F 3 "~" H 5350 3100 50  0001 C CNN
+	1    5350 3100
 	1    0    0    -1
 $EndComp
@@
 NoConn ~ 5900 4550
 NoConn ~ 6700 4550
+$Comp
+L Regulator_Switching:NXE1S0303MC U1101
+U 1 1 60A4F8AC
+P 6250 3100
+F 0 "U1101" H 6250 3567 50  0000 C CNN
+F 1 "NXE1S0303MC" H 6250 3476 50  0000 C CNN
+F 2 "Converter_DCDC:Converter_DCDC_muRata_NXExSxxxxMC_SMD" H 6250 2750 50  0001 C CNN
+F 3 "http://power.murata.com/data/power/ncl/kdc_nxe1.pdf" H 6250 2600 50  0001 C CNN
+	1    6250 3100
+	-1   0    0    -1
+$EndComp
 $EndSCHEMATC
