File: HARDWARE/BASE/Connector.sch (KiCad schematic (older format))
At the start: 1 part, among them J701 C64AC

Commit message: Schematic design.
Parts:
- renumbered J701 to J601
Changed lines of the file:
@@
 $Descr A4 11693 8268
 encoding utf-8
-Sheet 8 12
+Sheet 6 11
 Title "Connector"
 Date "2020-03-07"
@@
 	5350 5050 5400 5050
 $Comp
-L power:Earth #PWR0703
+L power:Earth #PWR0603
 U 1 1 5DECE77F
 P 5350 5050
-F 0 "#PWR0703" H 5350 4800 50  0001 C CNN
+F 0 "#PWR0603" H 5350 4800 50  0001 C CNN
 F 1 "Earth" H 5350 4900 50  0001 C CNN
 F 2 "" H 5350 5050 50  0001 C CNN
@@
 	5450 7100 5400 7100
 $Comp
-L Connector:C64AC J701
+L Connector:C64AC J601
 U 1 1 5DE8758D
 P 5750 4000
-F 0 "J701" H 5930 4096 50  0000 L CNN
+F 0 "J601" H 5930 4096 50  0000 L CNN
 F 1 "C64AC" H 5930 4005 50  0000 L CNN
 F 2 "ETH1CSMU1:Socket_DIN41612-CaseC1-AC-Male-64Pin-2rows" H 5750 4050 50  0001 C CNN
@@
 	5400 4300 5450 4300
 $Comp
-L power:Earth #PWR0702
+L power:Earth #PWR0602
 U 1 1 5DED2C4C
 P 5350 4250
-F 0 "#PWR0702" H 5350 4000 50  0001 C CNN
+F 0 "#PWR0602" H 5350 4000 50  0001 C CNN
 F 1 "Earth" H 5350 4100 50  0001 C CNN
 F 2 "" H 5350 4250 50  0001 C CNN
@@
 	5400 4250 5400 4300
 $Comp
-L power:GNDPWR #PWR0704
+L power:GNDPWR #PWR0604
 U 1 1 607E4852
 P 5350 6150
-F 0 "#PWR0704" H 5350 5950 50  0001 C CNN
+F 0 "#PWR0604" H 5350 5950 50  0001 C CNN
 F 1 "GNDPWR" V 5354 6041 50  0000 R CNN
 F 2 "" H 5350 6100 50  0001 C CNN
@@
 $EndComp
 $Comp
-L power:+24V #PWR0705
+L power:+24V #PWR0605
 U 1 1 607E51D3
 P 5350 6950
-F 0 "#PWR0705" H 5350 6800 50  0001 C CNN
+F 0 "#PWR0605" H 5350 6800 50  0001 C CNN
 F 1 "+24V" V 5365 7078 50  0000 L CNN
 F 2 "" H 5350 6950 50  0001 C CNN
@@
 $EndComp
 $Comp
-L ETH1CSMU1:GND_TRIG #PWR0701
+L ETH1CSMU1:GND_TRIG #PWR0601
 U 1 1 607EBE86
 P 5400 3900
-F 0 "#PWR0701" H 5400 3650 50  0001 C CNN
+F 0 "#PWR0601" H 5400 3650 50  0001 C CNN
 F 1 "GND_TRIG" V 5405 3772 50  0000 R CNN
 F 2 "" H 5400 3900 50  0001 C CNN

Commit message: Schematic design.
Parts:
- added C601: 1u, symbol Device:C
- added K601, K602, K603, K604, K605: HE3621A0510, symbol ETH1CSMU1:HE3621A0510
- added U601: ULN2003A, symbol Transistor_Array:ULN2003A
Connections:
- net A: now reaches J601.A2 (2A)
- net A: now also J601.C2 (2C), K601.4
- net B: now reaches J601.A3 (3A)
- net B: now also J601.C3 (3C), K602.4
- net C: now reaches J601.A4 (4A)
- net C: now also J601.C4 (4C), K603.4
- net D: now reaches J601.A5 (5A)
- net D: now also J601.C5 (5C)
- net E: now reaches J601.A6 (6A)
- net E: now also J601.C6 (6C), K604.4
- net F: now reaches J601.A7 (7A)
- net F: now also J601.C7 (7C), K605.4
- new net: K601.3, U601.12 (O5)
- new net: K602.3, U601.13 (O4)
- new net: K603.3, U601.14 (O3)
- new net: K604.3, U601.15 (O2)
- new net: K605.3, U601.16 (O1)
- new net +5V: C601.1, K601.2, K602.2, K603.2, K604.2, K605.2, U601.9 (COM)
- new net +GUA: K603.1
- new net +OUT: K601.1
- new net +SEN: K604.1
- new net -SEN: K605.1
- new net CXN_REL1: U601.5 (I5)
- new net CXN_REL2: U601.4 (I4)
- new net CXN_REL3: U601.3 (I3)
- new net CXN_REL4: U601.2 (I2)
- new net CXN_REL5: U601.1 (I1)
- new net GND: C601.2, U601.8 (GND)
- new net OCOM: K602.1
Other:
- moved on the sheet: J601

Commit message: Schematic design
Parts:
- C601: footprint (none) -> Capacitor_SMD:C_0603_1608Metric_Pad1.08x0.95mm_HandSolder
- K601, K602, K603, K604, K605: footprint (none) -> ETH1CSMU1:HE360_x-5050462-8
- U601: footprint (none) -> Package_SO:TSSOP-16_4.4x5mm_P0.65mm
Changed lines of the file:
@@
 $Descr A4 11693 8268
 encoding utf-8
-Sheet 6 12
+Sheet 6 13
 Title "Connector"
 Date "2020-03-07"
@@
 	4250 5050 4300 5050
 $Comp
-L power:Earth #PWR0603
+L power:Earth #PWR0609
 U 1 1 5DECE77F
 P 4250 5050
-F 0 "#PWR0603" H 4250 4800 50  0001 C CNN
+F 0 "#PWR0609" H 4250 4800 50  0001 C CNN
 F 1 "Earth" H 4250 4900 50  0001 C CNN
 F 2 "" H 4250 5050 50  0001 C CNN
@@
 	4300 4300 4350 4300
 $Comp
-L power:Earth #PWR0602
+L power:Earth #PWR0608
 U 1 1 5DED2C4C
 P 4250 4250
-F 0 "#PWR0602" H 4250 4000 50  0001 C CNN
+F 0 "#PWR0608" H 4250 4000 50  0001 C CNN
 F 1 "Earth" H 4250 4100 50  0001 C CNN
 F 2 "" H 4250 4250 50  0001 C CNN
@@
 	4300 4250 4300 4300
 $Comp
-L power:GNDPWR #PWR0604
+L power:GNDPWR #PWR0610
 U 1 1 607E4852
 P 4250 6150
-F 0 "#PWR0604" H 4250 5950 50  0001 C CNN
+F 0 "#PWR0610" H 4250 5950 50  0001 C CNN
 F 1 "GNDPWR" V 4254 6041 50  0000 R CNN
 F 2 "" H 4250 6100 50  0001 C CNN
@@
 $EndComp
 $Comp
-L power:+24V #PWR0605
+L power:+24V #PWR0611
 U 1 1 607E51D3
 P 4250 6950
-F 0 "#PWR0605" H 4250 6800 50  0001 C CNN
+F 0 "#PWR0611" H 4250 6800 50  0001 C CNN
 F 1 "+24V" V 4265 7078 50  0000 L CNN
 F 2 "" H 4250 6950 50  0001 C CNN
@@
 $EndComp
 $Comp
-L ETH1CSMU1:GND_TRIG #PWR0601
+L ETH1CSMU1:GND_TRIG #PWR0607
 U 1 1 607EBE86
 P 4300 3900
-F 0 "#PWR0601" H 4300 3650 50  0001 C CNN
+F 0 "#PWR0607" H 4300 3650 50  0001 C CNN
 F 1 "GND_TRIG" V 4305 3772 50  0000 R CNN
 F 2 "" H 4300 3900 50  0001 C CNN
@@
 P 2400 1400
 AR Path="/60575ED4/624C9B97" Ref="#PWR?"  Part="1"
-AR Path="/607E0822/624C9B97" Ref="#PWR0606"  Part="1"
-F 0 "#PWR0606" H 2400 1150 50  0001 C CNN
+AR Path="/607E0822/624C9B97" Ref="#PWR0602"  Part="1"
+F 0 "#PWR0602" H 2400 1150 50  0001 C CNN
 F 1 "OCOM" V 2400 1250 50  0000 R CNN
 F 2 "" H 2400 1400 50  0001 C CNN
@@
 F 0 "K601" V 3065 1050 50  0000 C CNN
 F 1 "HE3621A0510" V 2974 1050 50  0000 C CNN
-F 2 "" H 3100 1000 50  0001 C CNN
+F 2 "ETH1CSMU1:HE360_x-5050462-8" H 3100 1000 50  0001 C CNN
 F 3 "" H 3100 1000 50  0001 C CNN
 	1    2850 1050
@@
 F 0 "K601" H 5278 1646 50  0000 L CNN
 F 1 "HE3621A0510" H 5278 1555 50  0000 L CNN
-F 2 "" H 5450 1550 50  0001 C CNN
+F 2 "ETH1CSMU1:HE360_x-5050462-8" H 5450 1550 50  0001 C CNN
 F 3 "" H 5450 1550 50  0001 C CNN
 	2    5200 1600
@@
 F 0 "K602" V 3065 1400 50  0000 C CNN
 F 1 "HE3621A0510" V 2974 1400 50  0000 C CNN
-F 2 "" H 3100 1350 50  0001 C CNN
+F 2 "ETH1CSMU1:HE360_x-5050462-8" H 3100 1350 50  0001 C CNN
 F 3 "" H 3100 1350 50  0001 C CNN
 	1    2850 1400
@@
 F 0 "K602" H 5978 1646 50  0000 L CNN
 F 1 "HE3621A0510" H 5978 1555 50  0000 L CNN
-F 2 "" H 6150 1550 50  0001 C CNN
+F 2 "ETH1CSMU1:HE360_x-5050462-8" H 6150 1550 50  0001 C CNN
 F 3 "" H 6150 1550 50  0001 C CNN
 	2    5900 1600
@@
 F 0 "K603" V 3065 1750 50  0000 C CNN
 F 1 "HE3621A0510" V 2974 1750 50  0000 C CNN
-F 2 "" H 3100 1700 50  0001 C CNN
+F 2 "ETH1CSMU1:HE360_x-5050462-8" H 3100 1700 50  0001 C CNN
 F 3 "" H 3100 1700 50  0001 C CNN
 	1    2850 1750
@@
 F 0 "K603" H 6678 1646 50  0000 L CNN
 F 1 "HE3621A0510" H 6678 1555 50  0000 L CNN
-F 2 "" H 6850 1550 50  0001 C CNN
+F 2 "ETH1CSMU1:HE360_x-5050462-8" H 6850 1550 50  0001 C CNN
 F 3 "" H 6850 1550 50  0001 C CNN
 	2    6600 1600
@@
 F 0 "K604" V 3065 2100 50  0000 C CNN
 F 1 "HE3621A0510" V 2974 2100 50  0000 C CNN
-F 2 "" H 3100 2050 50  0001 C CNN
+F 2 "ETH1CSMU1:HE360_x-5050462-8" H 3100 2050 50  0001 C CNN
 F 3 "" H 3100 2050 50  0001 C CNN
 	1    2850 2100
@@
 F 0 "K604" H 7378 1646 50  0000 L CNN
 F 1 "HE3621A0510" H 7378 1555 50  0000 L CNN
-F 2 "" H 7550 1550 50  0001 C CNN
+F 2 "ETH1CSMU1:HE360_x-5050462-8" H 7550 1550 50  0001 C CNN
 F 3 "" H 7550 1550 50  0001 C CNN
 	2    7300 1600
@@
 F 0 "K605" V 3065 2450 50  0000 C CNN
 F 1 "HE3621A0510" V 2974 2450 50  0000 C CNN
-F 2 "" H 3100 2400 50  0001 C CNN
+F 2 "ETH1CSMU1:HE360_x-5050462-8" H 3100 2400 50  0001 C CNN
 F 3 "" H 3100 2400 50  0001 C CNN
 	1    2850 2450
@@
 F 0 "K605" H 8078 1646 50  0000 L CNN
 F 1 "HE3621A0510" H 8078 1555 50  0000 L CNN
-F 2 "" H 8250 1550 50  0001 C CNN
+F 2 "ETH1CSMU1:HE360_x-5050462-8" H 8250 1550 50  0001 C CNN
 F 3 "" H 8250 1550 50  0001 C CNN
 	2    8000 1600
@@
 	5900 1400 6600 1400
 $Comp
-L power:+5V #PWR0101
+L power:+5V #PWR0601
 U 1 1 6259093E
 P 6600 1350
-F 0 "#PWR0101" H 6600 1200 50  0001 C CNN
+F 0 "#PWR0601" H 6600 1200 50  0001 C CNN
 F 1 "+5V" H 6615 1523 50  0000 C CNN
 F 2 "" H 6600 1350 50  0001 C CNN
@@
 F 0 "U601" H 9400 2667 50  0000 C CNN
 F 1 "ULN2003A" H 9400 2576 50  0000 C CNN
-F 2 "" H 9450 1450 50  0001 L CNN
+F 2 "Package_SO:TSSOP-16_4.4x5mm_P0.65mm" H 9450 1450 50  0001 L CNN
 F 3 "http://www.ti.com/lit/ds/symlink/uln2003a.pdf" H 9500 1800 50  0001 C CNN
 	1    9400 2000
@@
 $EndComp
 $Comp
-L power:+5V #PWR0102
+L power:+5V #PWR0603
 U 1 1 6259B37C
 P 9000 1600
-F 0 "#PWR0102" H 9000 1450 50  0001 C CNN
+F 0 "#PWR0603" H 9000 1450 50  0001 C CNN
 F 1 "+5V" V 9000 1750 50  0000 L CNN
 F 2 "" H 9000 1600 50  0001 C CNN
@@
 $EndComp
 $Comp
-L power:GND #PWR0103
+L power:GND #PWR0606
 U 1 1 625A0234
 P 9400 2600
-F 0 "#PWR0103" H 9400 2350 50  0001 C CNN
+F 0 "#PWR0606" H 9400 2350 50  0001 C CNN
 F 1 "GND" H 9405 2427 50  0000 C CNN
 F 2 "" H 9400 2600 50  0001 C CNN
@@
 	9850 2200 9800 2200
 $Comp
-L power:GND #PWR0104
+L power:GND #PWR0605
 U 1 1 626006E6
 P 10700 2100
-F 0 "#PWR0104" H 10700 1850 50  0001 C CNN
+F 0 "#PWR0605" H 10700 1850 50  0001 C CNN
 F 1 "GND" H 10705 1927 50  0000 C CNN
 F 2 "" H 10700 2100 50  0001 C CNN
@@
 F 0 "C601" H 10815 1996 50  0000 L CNN
 F 1 "1u" H 10815 1905 50  0000 L CNN
-F 2 "" H 10738 1800 50  0001 C CNN
+F 2 "Capacitor_SMD:C_0603_1608Metric_Pad1.08x0.95mm_HandSolder" H 10738 1800 50  0001 C CNN
 F 3 "~" H 10700 1950 50  0001 C CNN
 	1    10700 1950
@@
 $EndComp
 $Comp
-L power:+5V #PWR0105
+L power:+5V #PWR0604
 U 1 1 626034E9
 P 10700 1800
-F 0 "#PWR0105" H 10700 1650 50  0001 C CNN
+F 0 "#PWR0604" H 10700 1650 50  0001 C CNN
 F 1 "+5V" H 10715 1973 50  0000 C CNN
 F 2 "" H 10700 1800 50  0001 C CNN
