File: HARDWARE/BASE/Ethernet.sch (KiCad schematic (older format))
At the start: 43 parts, among them U501 LAN8742A, U502 LC03-3.3, U503 LC03-3.3, Y501 NX5032GA-25.000M-LN-CD-1

Commit message: Schematic design
Parts:
- C401: renamed from C501; footprint Capacitor_SMD:C_0603_1608Metric_Pad1.05x0.95mm_HandSolder -> Capacitor_SMD:C_0603_1608Metric_Pad1.08x0.95mm_HandSolder
- C402: renamed from C502; footprint Capacitor_SMD:C_0603_1608Metric_Pad1.05x0.95mm_HandSolder -> Capacitor_SMD:C_0603_1608Metric_Pad1.08x0.95mm_HandSolder
- C403: renamed from C503; footprint Capacitor_SMD:C_0603_1608Metric_Pad1.05x0.95mm_HandSolder -> Capacitor_SMD:C_0603_1608Metric_Pad1.08x0.95mm_HandSolder
- C404: renamed from C504; footprint Capacitor_SMD:C_0603_1608Metric_Pad1.05x0.95mm_HandSolder -> Capacitor_SMD:C_0603_1608Metric_Pad1.08x0.95mm_HandSolder
- C405: renamed from C505; footprint Capacitor_SMD:C_0603_1608Metric_Pad1.05x0.95mm_HandSolder -> Capacitor_SMD:C_0603_1608Metric_Pad1.08x0.95mm_HandSolder
- C406: renamed from C506; footprint Capacitor_SMD:C_0603_1608Metric_Pad1.05x0.95mm_HandSolder -> Capacitor_SMD:C_0603_1608Metric_Pad1.08x0.95mm_HandSolder
- C407: renamed from C507; footprint Capacitor_SMD:C_0603_1608Metric_Pad1.05x0.95mm_HandSolder -> Capacitor_SMD:C_0603_1608Metric_Pad1.08x0.95mm_HandSolder
- C408: renamed from C508; footprint Capacitor_SMD:C_0603_1608Metric_Pad1.05x0.95mm_HandSolder -> Capacitor_SMD:C_0603_1608Metric_Pad1.08x0.95mm_HandSolder
- C409: renamed from C509; footprint Capacitor_SMD:C_0603_1608Metric_Pad1.05x0.95mm_HandSolder -> Capacitor_SMD:C_0603_1608Metric_Pad1.08x0.95mm_HandSolder
- C410: renamed from C510; footprint Capacitor_SMD:C_0603_1608Metric_Pad1.05x0.95mm_HandSolder -> Capacitor_SMD:C_0603_1608Metric_Pad1.08x0.95mm_HandSolder
- C411: renamed from C511; footprint Capacitor_SMD:C_0603_1608Metric_Pad1.05x0.95mm_HandSolder -> Capacitor_SMD:C_0603_1608Metric_Pad1.08x0.95mm_HandSolder
- C412: renamed from C512; footprint Capacitor_SMD:C_0603_1608Metric_Pad1.05x0.95mm_HandSolder -> Capacitor_SMD:C_0603_1608Metric_Pad1.08x0.95mm_HandSolder
- C413: renamed from C513; footprint Capacitor_SMD:C_1206_3216Metric_Pad1.42x1.75mm_HandSolder -> Capacitor_SMD:C_1206_3216Metric_Pad1.33x1.80mm_HandSolder
- C414: renamed from C514; footprint Capacitor_SMD:C_1206_3216Metric_Pad1.42x1.75mm_HandSolder -> Capacitor_SMD:C_1206_3216Metric_Pad1.33x1.80mm_HandSolder
- R419: renamed from R519; footprint Resistor_SMD:R_1206_3216Metric_Pad1.42x1.75mm_HandSolder -> Resistor_SMD:R_1206_3216Metric_Pad1.30x1.75mm_HandSolder
- renumbered D501 to D401, D502 to D402, FB501 to FB401, L501 to L401, R501 to R401, R502 to R402, R503 to R403, R504 to R404, R505 to R405, R506 to R406, R507 to R407, R508 to R408, R509 to R409, R510 to R410, R511 to R411, R512 to R412, R513 to R413, R514 to R414, R515 to R415, R516 to R416, R517 to R417, R518 to R418, R520 to R420, R521 to R421, U501 to U401, U502 to U402, U503 to U403, Y501 to Y401

Commit message: Schematic design
Parts:
- renumbered C402 to C401, C405 to C402, C407 to C403, C408 to C404, C409 to C405, C410 to C406, C411 to C407, C403 to C408, C406 to C409, C412 to C410, C414 to C411, C413 to C412, C401 to C413, C404 to C414, R415 to R401, R416 to R402, R417 to R403, R418 to R404, R401 to R405, R402 to R406, R403 to R407, R404 to R408, R412 to R409, R420 to R410, R421 to R411, R405 to R412, R411 to R413, R413 to R414, R414 to R415, R419 to R416, R406 to R417, R407 to R418, R408 to R419, R409 to R420, R410 to R421, U402 to U401, U401 to U402
