File: HARDWARE/BASE/MCU.sch (KiCad schematic (older format))
At the start: 42 parts, among them J601 Conn_02x01, J602 20021111-00010T4LF, U601 HDC1080, U602 STM32H743ZI, U603 24LC08B-E/MS, Y601 NX3225GD-8MHZ-STD-CRA-3

Commit message: Schematic design
Parts:
- C501: renamed from C601; footprint Capacitor_SMD:C_0603_1608Metric_Pad1.05x0.95mm_HandSolder -> Capacitor_SMD:C_0603_1608Metric_Pad1.08x0.95mm_HandSolder
- C502: renamed from C602; footprint Capacitor_SMD:C_0603_1608Metric_Pad1.05x0.95mm_HandSolder -> Capacitor_SMD:C_0603_1608Metric_Pad1.08x0.95mm_HandSolder
- C503: renamed from C603; footprint Capacitor_SMD:C_0603_1608Metric_Pad1.05x0.95mm_HandSolder -> Capacitor_SMD:C_0603_1608Metric_Pad1.08x0.95mm_HandSolder
- C504: renamed from C604; footprint Capacitor_SMD:C_0603_1608Metric_Pad1.05x0.95mm_HandSolder -> Capacitor_SMD:C_0603_1608Metric_Pad1.08x0.95mm_HandSolder
- C505: renamed from C605; footprint Capacitor_SMD:C_0603_1608Metric_Pad1.05x0.95mm_HandSolder -> Capacitor_SMD:C_0603_1608Metric_Pad1.08x0.95mm_HandSolder
- C506: renamed from C606; footprint Capacitor_SMD:C_0603_1608Metric_Pad1.05x0.95mm_HandSolder -> Capacitor_SMD:C_0603_1608Metric_Pad1.08x0.95mm_HandSolder
- C507: renamed from C607; footprint Capacitor_SMD:C_0603_1608Metric_Pad1.05x0.95mm_HandSolder -> Capacitor_SMD:C_0603_1608Metric_Pad1.08x0.95mm_HandSolder
- C508: renamed from C608; footprint Capacitor_SMD:C_0805_2012Metric_Pad1.15x1.40mm_HandSolder -> Capacitor_SMD:C_0603_1608Metric_Pad1.08x0.95mm_HandSolder
- C509: renamed from C609; footprint Capacitor_SMD:C_0603_1608Metric_Pad1.05x0.95mm_HandSolder -> Capacitor_SMD:C_0603_1608Metric_Pad1.08x0.95mm_HandSolder
- C510: renamed from C610; footprint Capacitor_SMD:C_0805_2012Metric_Pad1.15x1.40mm_HandSolder -> Capacitor_SMD:C_0603_1608Metric_Pad1.08x0.95mm_HandSolder
- C511: renamed from C611; footprint Capacitor_SMD:C_0603_1608Metric_Pad1.05x0.95mm_HandSolder -> Capacitor_SMD:C_0603_1608Metric_Pad1.08x0.95mm_HandSolder
- C512: renamed from C612; footprint Capacitor_SMD:C_0603_1608Metric_Pad1.05x0.95mm_HandSolder -> Capacitor_SMD:C_0603_1608Metric_Pad1.08x0.95mm_HandSolder
- C513: renamed from C613; footprint Capacitor_SMD:C_0603_1608Metric_Pad1.05x0.95mm_HandSolder -> Capacitor_SMD:C_0603_1608Metric_Pad1.08x0.95mm_HandSolder
- C514: renamed from C614; footprint Capacitor_SMD:C_0603_1608Metric_Pad1.05x0.95mm_HandSolder -> Capacitor_SMD:C_0603_1608Metric_Pad1.08x0.95mm_HandSolder
- C515: renamed from C615; footprint Capacitor_SMD:C_0603_1608Metric_Pad1.05x0.95mm_HandSolder -> Capacitor_SMD:C_0603_1608Metric_Pad1.08x0.95mm_HandSolder
- C516: renamed from C616; footprint Capacitor_SMD:C_0603_1608Metric_Pad1.05x0.95mm_HandSolder -> Capacitor_SMD:C_0603_1608Metric_Pad1.08x0.95mm_HandSolder
- C517: renamed from C617; footprint Capacitor_SMD:C_0603_1608Metric_Pad1.05x0.95mm_HandSolder -> Capacitor_SMD:C_0603_1608Metric_Pad1.08x0.95mm_HandSolder
- C518: renamed from C618; footprint Capacitor_SMD:C_0603_1608Metric_Pad1.05x0.95mm_HandSolder -> Capacitor_SMD:C_0603_1608Metric_Pad1.08x0.95mm_HandSolder
- C519: renamed from C619; footprint Capacitor_SMD:C_0603_1608Metric_Pad1.05x0.95mm_HandSolder -> Capacitor_SMD:C_0603_1608Metric_Pad1.08x0.95mm_HandSolder
- C520: renamed from C620; footprint Capacitor_SMD:C_0603_1608Metric_Pad1.05x0.95mm_HandSolder -> Capacitor_SMD:C_0603_1608Metric_Pad1.08x0.95mm_HandSolder
- C521: renamed from C621; footprint Capacitor_SMD:C_0603_1608Metric_Pad1.05x0.95mm_HandSolder -> Capacitor_SMD:C_0603_1608Metric_Pad1.08x0.95mm_HandSolder
- C522: renamed from C622; footprint Capacitor_SMD:C_0603_1608Metric_Pad1.05x0.95mm_HandSolder -> Capacitor_SMD:C_0603_1608Metric_Pad1.08x0.95mm_HandSolder
- renumbered D601 to D501, D602 to D502, D603 to D503, FB601 to FB501, J601 to J501, J602 to J502, R601 to R501, R602 to R502, R603 to R503, R604 to R504, R605 to R505, R606 to R506, R607 to R507, R608 to R508, R609 to R509, R610 to R510, U601 to U501, U602 to U502, U603 to U503, Y601 to Y501

Commit message: Schematic design
Parts:
- renumbered C505 to C501, C507 to C502, C508 to C503, C510 to C504, C522 to C505, C512 to C506, C501 to C507, C503 to C508, C502 to C509, C504 to C510, C506 to C511, C509 to C512, C511 to C513, C513 to C514, C514 to C515, C515 to C516, C516 to C517, C517 to C518, C518 to C519, C519 to C520, C520 to C521, C521 to C522, R502 to R501, R503 to R502, R504 to R503, R505 to R504, R506 to R505, R510 to R506, R501 to R507, R509 to R508, R507 to R509, R508 to R510

Commit message: Schematic design
Parts:
- Y501: value NX3225GD-8MHZ-STD-CRA-3 -> NX3225GD-8MHZ
Connections:
- net FPGA_SPI3_NSS: no longer names the net of U502.110 (PA15,JTDI,TIM2_CH1,TIM2_ETR,HDMI_CEC,SPI1_NSS,I2S1_WS,SPI3_NSS,I2S3_WS,SPI6_NSS,UART4_RTS,CAN3_TX,UART7_TX,EVENTOUT)
- no-connect marks 53 -> 54
Other:
- note removed: "PROGRAMMING CONNECTOR\nDESIGNED FOR JLINK"
- moved on the sheet: C501, C502, C503, C504, C505, C506, C507, C508, D501, D502, D503, J501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

Commit message: Schematic design.
Parts:
- renumbered R503 to R501, R504 to R502, R505 to R503, R506 to R504, R508 to R505, R507 to R506, R501 to R507, R502 to R508, U502 to U501, U501 to U502
Connections:
- net TCK_SWCLK renamed SWCLK
- net TMS_SWDIO renamed SWDIO
Changed lines of the file:
@@
 $Descr A3 16535 11693
 encoding utf-8
-Sheet 5 10
+Sheet 5 12
 Title "MCU"
 Date "2020-03-07"
@@
 	9350 9050 9350 9100
 $Comp
-L power:GND #PWR0516
+L power:GND #PWR0511
 U 1 1 5DAA3278
 P 9350 9100
-F 0 "#PWR0516" H 9350 8850 50  0001 C CNN
+F 0 "#PWR0511" H 9350 8850 50  0001 C CNN
 F 1 "GND" H 9355 8927 50  0000 C CNN
 F 2 "" H 9350 9100 50  0001 C CNN
@@
 $EndComp
 $Comp
-L Device:R R508
+L Device:R R505
 U 1 1 5DAA6CE1
 P 15050 8900
-F 0 "R508" H 15120 8946 50  0000 L CNN
+F 0 "R505" H 15120 8946 50  0000 L CNN
 F 1 "10k" H 15120 8855 50  0000 L CNN
 F 2 "Resistor_SMD:R_0603_1608Metric_Pad0.98x0.95mm_HandSolder" V 14980 8900 50  0001 C CNN
@@
 $EndComp
 $Comp
-L Device:R R506
+L Device:R R504
 U 1 1 5DAA8BD1
 P 15500 8500
-F 0 "R506" H 15570 8546 50  0000 L CNN
+F 0 "R504" H 15570 8546 50  0000 L CNN
 F 1 "10k" H 15570 8455 50  0000 L CNN
 F 2 "Resistor_SMD:R_0603_1608Metric_Pad0.98x0.95mm_HandSolder" V 15430 8500 50  0001 C CNN
@@
 Connection ~ 15500 8700
 $Comp
-L power:GND #PWR0511
+L power:GND #PWR0509
 U 1 1 5DAAC0BD
 P 15500 9050
-F 0 "#PWR0511" H 15500 8800 50  0001 C CNN
+F 0 "#PWR0509" H 15500 8800 50  0001 C CNN
 F 1 "GND" H 15505 8877 50  0000 C CNN
 F 2 "" H 15500 9050 50  0001 C CNN
@@
 $EndComp
 $Comp
-L power:GND #PWR0514
+L power:GND #PWR0508
 U 1 1 5DAACD0D
 P 15050 9050
-F 0 "#PWR0514" H 15050 8800 50  0001 C CNN
+F 0 "#PWR0508" H 15050 8800 50  0001 C CNN
 F 1 "GND" H 15055 8877 50  0000 C CNN
 F 2 "" H 15050 9050 50  0001 C CNN
@@
 MCU_VDDA
 $Comp
-L power:GND #PWR0510
+L power:GND #PWR0506
 U 1 1 5DACCD5C
 P 3600 8500
-F 0 "#PWR0510" H 3600 8250 50  0001 C CNN
+F 0 "#PWR0506" H 3600 8250 50  0001 C CNN
 F 1 "GND" V 3605 8372 50  0000 R CNN
 F 2 "" H 3600 8500 50  0001 C CNN
@@
 	3600 8700 3650 8700
 $Comp
-L power:GND #PWR0515
+L power:GND #PWR0510
 U 1 1 5DAD7BE9
 P 3600 9100
-F 0 "#PWR0515" H 3600 8850 50  0001 C CNN
+F 0 "#PWR0510" H 3600 8850 50  0001 C CNN
 F 1 "GND" H 3605 8927 50  0000 C CNN
 F 2 "" H 3600 9100 50  0001 C CNN
@@
 $EndComp
 $Comp
-L power:GND #PWR0513
+L power:GND #PWR0521
 U 1 1 5DB88AAB
 P 4650 10200
-F 0 "#PWR0513" H 4650 9950 50  0001 C CNN
+F 0 "#PWR0521" H 4650 9950 50  0001 C CNN
 F 1 "GND" H 4655 10027 50  0000 C CNN
 F 2 "" H 4650 10200 50  0001 C CNN
@@
 $EndComp
 $Comp
-L Device:R R507
+L Device:R R506
 U 1 1 5DB8FF79
 P 4650 9450
-F 0 "R507" H 4580 9404 50  0000 R CNN
+F 0 "R506" H 4580 9404 50  0000 R CNN
 F 1 "10k" H 4580 9495 50  0000 R CNN
 F 2 "Resistor_SMD:R_0603_1608Metric_Pad0.98x0.95mm_HandSolder" V 4580 9450 50  0001 C CNN
@@
 	2450 7700 2450 7950
 $Comp
-L power:GND #PWR0509
+L power:GND #PWR0504
 U 1 1 5DBC271D
 P 2700 8350
-F 0 "#PWR0509" H 2700 8100 50  0001 C CNN
+F 0 "#PWR0504" H 2700 8100 50  0001 C CNN
 F 1 "GND" H 2705 8177 50  0000 C CNN
 F 2 "" H 2700 8350 50  0001 C CNN
@@
 Connection ~ 7100 10500
 $Comp
-L Device:R R503
+L Device:R R501
 U 1 1 5E648C3B
 P 3250 6550
-F 0 "R503" V 3043 6550 50  0000 C CNN
+F 0 "R501" V 3043 6550 50  0000 C CNN
 F 1 "680" V 3134 6550 50  0000 C CNN
 F 2 "Resistor_SMD:R_0603_1608Metric_Pad0.98x0.95mm_HandSolder" V 3180 6550 50  0001 C CNN
@@
 $EndComp
 $Comp
-L Device:R R504
+L Device:R R502
 U 1 1 5E64A32E
 P 3250 6950
-F 0 "R504" V 3043 6950 50  0000 C CNN
+F 0 "R502" V 3043 6950 50  0000 C CNN
 F 1 "560" V 3134 6950 50  0000 C CNN
 F 2 "Resistor_SMD:R_0603_1608Metric_Pad0.98x0.95mm_HandSolder" V 3180 6950 50  0001 C CNN
@@
 $EndComp
 $Comp
-L Device:R R505
+L Device:R R503
 U 1 1 5E64A698
 P 3250 7350
-F 0 "R505" V 3043 7350 50  0000 C CNN
+F 0 "R503" V 3043 7350 50  0000 C CNN
 F 1 "680" V 3134 7350 50  0000 C CNN
 F 2 "Resistor_SMD:R_0603_1608Metric_Pad0.98x0.95mm_HandSolder" V 3180 7350 50  0001 C CNN
@@
 	2650 6950 2700 6950
 $Comp
-L Sensor_Humidity:HDC1080 U501
+L Sensor_Humidity:HDC1080 U502
 U 1 1 5EF9C579
 P 1250 9900
-F 0 "U501" H 1450 10250 50  0000 R CNN
+F 0 "U502" H 1450 10250 50  0000 R CNN
 F 1 "HDC1080" H 1550 10150 50  0000 R CNN
 F 2 "Package_SON:Texas_PWSON-N6" H 1200 9650 50  0001 L CNN
@@
 $EndComp
 $Comp
-L power:GND #PWR0505
+L power:GND #PWR0520
 U 1 1 5EF9F2A6
 P 1150 10200
-F 0 "#PWR0505" H 1150 9950 50  0001 C CNN
+F 0 "#PWR0520" H 1150 9950 50  0001 C CNN
 F 1 "GND" H 1155 10027 50  0000 C CNN
 F 2 "" H 1150 10200 50  0001 C CNN
@@
 $EndComp
 $Comp
-L Device:R R501
+L Device:R R507
 U 1 1 5E375F7B
 P 1650 9600
-F 0 "R501" H 1720 9646 50  0000 L CNN
+F 0 "R507" H 1720 9646 50  0000 L CNN
 F 1 "4k7" H 1720 9555 50  0000 L CNN
 F 2 "Resistor_SMD:R_0603_1608Metric_Pad0.98x0.95mm_HandSolder" V 1580 9600 50  0001 C CNN
@@
 $EndComp
 $Comp
-L Device:R R502
+L Device:R R508
 U 1 1 5E37B6AD
 P 2050 9600
-F 0 "R502" H 2120 9646 50  0000 L CNN
+F 0 "R508" H 2120 9646 50  0000 L CNN
 F 1 "4k7" H 2120 9555 50  0000 L CNN
 F 2 "Resistor_SMD:R_0603_1608Metric_Pad0.98x0.95mm_HandSolder" V 1980 9600 50  0001 C CNN
@@
 	6150 10200 6150 10100
 $Comp
-L power:GND #PWR0521
+L power:GND #PWR0523
 U 1 1 5EFC3E57
 P 6150 10200
-F 0 "#PWR0521" H 6150 9950 50  0001 C CNN
+F 0 "#PWR0523" H 6150 9950 50  0001 C CNN
 F 1 "GND" H 6155 10027 50  0000 C CNN
 F 2 "" H 6150 10200 50  0001 C CNN
@@
 	5650 10200 5650 10100
 $Comp
-L power:GND #PWR0520
+L power:GND #PWR0522
 U 1 1 5E1764D7
 P 5650 10200
-F 0 "#PWR0520" H 5650 9950 50  0001 C CNN
+F 0 "#PWR0522" H 5650 9950 50  0001 C CNN
 F 1 "GND" H 5655 10027 50  0000 C CNN
 F 2 "" H 5650 10200 50  0001 C CNN
@@
 NoConn ~ 15050 5200
 $Comp
-L ETH1CSMU1:STM32H743ZI U502
+L ETH1CSMU1:STM32H743ZI U501
 U 1 1 60365EFD
 P 9350 4950
-F 0 "U502" H 14050 8850 50  0000 C CNN
+F 0 "U501" H 14050 8850 50  0000 C CNN
 F 1 "STM32H743ZI" H 14550 8850 50  0000 C CNN
 F 2 "ETH1CSMU1:TQFP-144_20x20mm_P0.5mm" H 25250 6450 50  0001 C CNN
@@
 NoConn ~ 15050 6500
 $Comp
-L power:+3.3V #PWR0522
+L power:+3.3V #PWR0518
 U 1 1 605724BF
 P 8250 10150
-F 0 "#PWR0522" H 8250 10000 50  0001 C CNN
+F 0 "#PWR0518" H 8250 10000 50  0001 C CNN
 F 1 "+3.3V" H 8265 10323 50  0000 C CNN
 F 2 "" H 8250 10150 50  0001 C CNN
@@
 $EndComp
 $Comp
-L power:+3.3V #PWR0519
+L power:+3.3V #PWR0517
 U 1 1 60572EDC
 P 11500 9900
-F 0 "#PWR0519" H 11500 9750 50  0001 C CNN
+F 0 "#PWR0517" H 11500 9750 50  0001 C CNN
 F 1 "+3.3V" H 11515 10073 50  0000 C CNN
 F 2 "" H 11500 9900 50  0001 C CNN
@@
 $EndComp
 $Comp
-L power:+3.3V #PWR0523
+L power:+3.3V #PWR0519
 U 1 1 60573E5C
 P 10100 10150
-F 0 "#PWR0523" H 10100 10000 50  0001 C CNN
+F 0 "#PWR0519" H 10100 10000 50  0001 C CNN
 F 1 "+3.3V" H 10115 10323 50  0000 C CNN
 F 2 "" H 10100 10150 50  0001 C CNN
@@
 $EndComp
 $Comp
-L power:+3.3V #PWR0517
+L power:+3.3V #PWR0515
 U 1 1 60574D4E
 P 5650 9700
-F 0 "#PWR0517" H 5650 9550 50  0001 C CNN
+F 0 "#PWR0515" H 5650 9550 50  0001 C CNN
 F 1 "+3.3V" H 5665 9873 50  0000 C CNN
 F 2 "" H 5650 9700 50  0001 C CNN
@@
 $EndComp
 $Comp
-L power:+3.3V #PWR0518
+L power:+3.3V #PWR0516
 U 1 1 60576A4F
 P 6150 9700
-F 0 "#PWR0518" H 6150 9550 50  0001 C CNN
+F 0 "#PWR0516" H 6150 9550 50  0001 C CNN
 F 1 "+3.3V" H 6165 9873 50  0000 C CNN
 F 2 "" H 6150 9700 50  0001 C CNN
@@
 $EndComp
 $Comp
-L power:+3.3V #PWR0508
+L power:+3.3V #PWR0512
 U 1 1 60579750
 P 4650 9300
-F 0 "#PWR0508" H 4650 9150 50  0001 C CNN
+F 0 "#PWR0512" H 4650 9150 50  0001 C CNN
 F 1 "+3.3V" H 4665 9473 50  0000 C CNN
 F 2 "" H 4650 9300 50  0001 C CNN
@@
 $EndComp
 $Comp
-L power:+3.3V #PWR0506
+L power:+3.3V #PWR0503
 U 1 1 6057A4C1
 P 2650 6950
-F 0 "#PWR0506" H 2650 6800 50  0001 C CNN
+F 0 "#PWR0503" H 2650 6800 50  0001 C CNN
 F 1 "+3.3V" V 2650 7100 50  0000 L CNN
 F 2 "" H 2650 6950 50  0001 C CNN
@@
 $EndComp
 $Comp
-L power:+3.3V #PWR0504
+L power:+3.3V #PWR0514
 U 1 1 6057DD2A
 P 1150 9500
-F 0 "#PWR0504" H 1150 9350 50  0001 C CNN
+F 0 "#PWR0514" H 1150 9350 50  0001 C CNN
 F 1 "+3.3V" H 1165 9673 50  0000 C CNN
 F 2 "" H 1150 9500 50  0001 C CNN
@@
 $EndComp
 $Comp
-L power:+3.3V #PWR0503
+L power:+3.3V #PWR0513
 U 1 1 6057FA53
 P 1850 9350
-F 0 "#PWR0503" H 1850 9200 50  0001 C CNN
+F 0 "#PWR0513" H 1850 9200 50  0001 C CNN
 F 1 "+3.3V" H 1865 9523 50  0000 C CNN
 F 2 "" H 1850 9350 50  0001 C CNN
@@
 $EndComp
 $Comp
-L power:+3.3V #PWR0507
+L power:+3.3V #PWR0505
 U 1 1 60583AF5
 P 15500 8350
-F 0 "#PWR0507" H 15500 8200 50  0001 C CNN
+F 0 "#PWR0505" H 15500 8200 50  0001 C CNN
 F 1 "+3.3V" H 15515 8523 50  0000 C CNN
 F 2 "" H 15500 8350 50  0001 C CNN
@@
 NoConn ~ 3650 5900
 $Comp
-L power:+3.3V #PWR0512
+L power:+3.3V #PWR0507
 U 1 1 60600C51
 P 3550 8700
-F 0 "#PWR0512" H 3550 8550 50  0001 C CNN
+F 0 "#PWR0507" H 3550 8550 50  0001 C CNN
 F 1 "+3.3V" V 3550 8950 50  0000 C CNN
 F 2 "" H 3550 8700 50  0001 C CNN
@@
 Wire Bus Line
 	1550 2250 1550 3850
+Text HLabel 3200 4500 0    50   BiDi ~ 0
+SWDIO
+Text HLabel 3200 4600 0    50   Input ~ 0
+SWCLK
 $EndSCHEMATC

Commit message: Schematic design.
Changed lines of the file:
@@
 $Descr A3 16535 11693
 encoding utf-8
-Sheet 5 11
+Sheet 5 12
 Title "MCU"
 Date "2020-03-07"
@@
 Text HLabel 3200 4600 0    50   Input ~ 0
 SWCLK
+Text HLabel 15550 3500 2    50   Output ~ 0
+CXN_REL5
+Text HLabel 15550 3400 2    50   Output ~ 0
+CXN_REL4
+Text HLabel 15550 3300 2    50   Output ~ 0
+CXN_REL3
+Text HLabel 15550 3200 2    50   Output ~ 0
+CXN_REL2
+Text HLabel 15550 3100 2    50   Output ~ 0
+CXN_REL1
 Wire Bus Line
 	1550 4100 1550 5500
