File: HARDWARE/BASE/Control.sch (KiCad schematic (older format))
At the start: 0 parts

Commit message: Schematic design
Parts:
- added C1001, C1007, C1016: 10u, symbol Device:C
- added C1002, C1008, C1014, C1015, C1018, C1020: 1u, symbol Device:C
- added C1003, C1004, C1005, C1010, C1011: 1000p, symbol Device:C
- added C1006, C1021, C1022, C1023, C1024, C1025, C1026, C1027, C1028, C1029, C1030, C1031, C1032, C1033, C1034, C1035, C1036, C1037, C1038, C1039, C1040, C1041, C1042, C1043: 100n, symbol Device:C
- added C1009: 4u7/25V, symbol Device:C
- added C1012, C1013: 330p, symbol Device:C
- added C1017, C1019: 22u, symbol Device:C
- added R1001, R1003, R1007, R1009, R1010, R1012, R1013, R1014, R1015, R1016, R1018, R1019: 10k/.1%, symbol Device:R
- added R1002, R1021, R1022, R1023, R1024: 10k, symbol Device:R
- added R1004: 2k/.1%, symbol Device:R
- added R1005: 2k, symbol Device:R
- added R1006: 20k5/.1%, symbol Device:R
- added R1008, R1011, R1017, R1020: 21k5/.1%, symbol Device:R
- added R1025, R1028, R1029: 0R22, symbol Device:R
- added R1026, R1027: 0, symbol Device:R
- added U1001: OPA2140, symbol ETH1CSMU1:OPA2140
- added U1002: OPA2140, symbol ETH1CSMU1:AD5686RARUZ
- added U1003: TL072, symbol Amplifier_Operational:TL072
- added U1004: DG419LDY, Package_SO:SOIC-8_3.9x4.9mm_P1.27mm, symbol ETH1CSMU1:CPC1018N
- added U1005, U1008, U1009: DG419LDY, Package_SO:SOIC-8_3.9x4.9mm_P1.27mm, symbol Analog_Switch:DG419LDY
- added U1006: ADR431ARZ, symbol ETH1CSMU1:ADR431ARZ
- added U1007: TLC2272, symbol ETH1CSMU1:TLC2272
- added U1010: AD7190RUZ, symbol ETH1CSMU1:AD7190RUZ
- added U1011, U1012: ADS8681PWR, symbol ETH1CSMU1:ADS8681PWR
- added U1013: REF5040ID, Package_SO:SOIC-8_3.9x4.9mm_P1.27mm, symbol Reference_Voltage:REF5040ID
Connections:
- new net: C1002.1, R1002.2, U1002.15 (~RESET)
- new net: R1009.2, U1002.2 (VOUTB)
- new net: R1003.2, U1002.3 (VOUTA)
- new net: R1012.2, U1002.6 (VOUTC)
- new net: C1003.2, R1001.1, R1003.1, R1004.2, R1006.2, U1001.2 (-)
- new net: C1003.1, R1006.1, U1001.1, U1004.3, U1005.2
- new net: R1013.2, R1014.1, U1001.6 (-)
- new net: C1005.2, R1010.1, R1011.2, R1012.1, U1003.2 (-)
- new net: C1004.2, R1007.1, R1008.2, R1009.1, U1003.6 (-)
- new net: R1004.1, U1004.4
- new net: R1005.2, U1004.1
- new net: C1010.1, R1016.1, U1007.1, U1010.11 (AIN1)
- new net: C1010.2, R1015.1, R1016.2, R1017.1, U1007.2 (-)
- new net: C1011.2, R1018.1, R1019.2, R1020.1, U1007.6 (-)
- new net: C1011.1, R1019.1, U1007.7, U1010.12 (AIN2)
- new net: R1020.2, U1009.2
- new net: R1017.2, U1008.2
- new net: R1026.1, U1008.8
- new net: R1027.2, U1009.8
- new net: C1015.1, U1013.5 (Trim/NR)
- new net: C1016.1, R1025.2
- new net: R1022.2, U1011.13 (SDO-0), U1012.10 (SDI)
- new net: C1012.1, R1026.2, U1011.7 (AIN_P)
- new net: R1021.2, U1011.9 (~RST)
- new net: C1013.1, R1027.1, U1012.7 (AIN_P)
- new net: R1023.2, U1012.9 (~RST)
- new net: C1017.1, C1018.1, R1028.2
- new net: C1019.1, C1020.1, R1029.2
- new net +15V: C1027.1, C1028.1, C1029.1, C1030.1, C1031.1, C1032.1, U1001.8 (V+), U1003.8 (V+), U1005.4 (V+), U1007.8 (V+), U1008.4 (V+), U1009.4 (V+)
- new net +2V5: C1008.1, R1014.2, U1002.1 (VREF), U1006.6 (VOUT), U1010.10 (AINCOM), U1010.15 (REFIN1+)
- new net +3V3: C1033.1, C1034.1, C1035.1, C1036.1, R1002.1, R1021.1, R1022.1, R1023.1, R1024.1, U1002.10 (GAIN), U1002.11 (VLOGIC), U1002.16 (RSTSEL), U1010.21 (DVDD), U1011.16 (DVDD), U1012.16 (DVDD)
- new net +4V: R1025.1, U1011.4 (REFIO), U1012.4 (REFIO), U1013.6 (Vout)
- new net +5V: C1001.1, C1006.1, C1007.1, C1014.1, C1037.1, C1038.1, C1039.1, C1040.1, C1041.1, C1042.1, C1043.1, U1002.5 (VDD), U1005.5 (VL), U1006.2 (VIN), U1008.5 (VL), U1009.5 (VL), U1010.20 (AVDD), U1011.2 (AVDD), U1012.2 (AVDD), U1013.2 (Vin)
- new net -15V: C1021.1, C1022.1, C1023.1, C1024.1, C1025.1, C1026.1, U1001.4 (V-), U1003.4 (V-), U1005.7 (V-), U1007.4 (V-), U1008.7 (V-), U1009.7 (V-)
- new net -2V5: C1009.1, R1001.2, R1007.2, R1010.2, R1013.1, R1015.2, R1018.2, U1001.7
- new net ADC_HP_MISO: U1010.23 (DOUT)
- new net ADC_HP_MOSI: U1010.24 (DIN)
- new net ADC_HP_SCLK: U1010.3 (SCLK)
- new net ADC_HP_~CS: U1010.4 (~CS)
- new net ADC_HS_MISO: R1024.2, U1012.13 (SDO-0)
- new net ADC_HS_MOSI: U1011.10 (SDI)
- new net ADC_HS_RVS1: U1011.15 (RVS)
- new net ADC_HS_RVS2: U1012.15 (RVS)
- new net ADC_HS_SCLK: U1011.12 (SCLK), U1012.12 (SCLK)
- new net ADC_HS_~CS: U1011.11 (CONVST/~CS), U1012.11 (CONVST/~CS)
- new net ADC_SELECT: U1008.6, U1009.6
- new net CAP1: R1028.1, U1011.6 (REFCAP)
- new net CAP2: R1029.1, U1012.6 (REFCAP)
- new net CL+: C1004.1, R1008.1, U1003.7
- new net CL-: C1005.1, R1011.1, U1003.1
- new net DAC_MISO: U1002.8 (SDO)
- new net DAC_MOSI: U1002.14 (SDIN)
- new net DAC_SCLK: U1002.12 (SCLK)
- new net DAC_SP: U1002.7 (VOUTD)
- new net DAC_~CS: U1002.13 (~SYNC)
- new net FDACLO: R1005.1
- new net FDACN: U1005.1
- new net FDACN_SELECT: U1005.6
- new net FGEN_AMP: U1005.8
- new net GND: C1001.2, C1002.2, C1006.2, C1007.2, C1008.2, C1009.2, C1012.2, C1013.2, C1014.2, C1015.2, C1016.2, C1017.2, C1018.2, C1019.2, C1020.2, C1021.2, C1022.2, C1023.2, C1024.2, C1025.2, C1026.2, C1027.2, C1028.2, C1029.2, C1030.2, C1031.2, C1032.2, C1033.2, C1034.2, C1035.2, C1036.2, C1037.2, C1038.2, C1039.2, C1040.2, C1041.2, C1042.2, C1043.2, U1001.3 (+), U1001.5 (+), U1002.4 (GND), U1002.9 (~LDAC), U1003.3 (+), U1003.5 (+), U1004.2, U1005.3 (GND), U1006.4 (GND), U1007.3 (+), U1007.5 (+), U1008.3 (GND), U1009.3 (GND), U1010.16 (REFIN1-), U1010.18 (AGND), U1010.19 (DGND), U1010.9 (NC), U1011.1 (DGND), U1011.3 (AGND), U1011.5 (REFGND), U1011.8 (AIN_GND), U1012.1 (DGND), U1012.3 (AGND), U1012.5 (REFGND), U1012.8 (AIN_GND), U1013.4 (GND)
- new net IM: U1009.1
- new net VM: U1008.1
- no-connect marks 0 -> 15

Commit message: Schematic design
Parts:
- added U? (x3): SN74LVC1T45DBV, Package_TO_SOT_SMD:SOT-23-6, symbol Logic_LevelTranslator:SN74LVC1T45DBV
Connections:
- net +3V3: now also U?.6 (VCCB), U?.6 (VCCB), U?.6 (VCCB)
- net +5V: now also U?.1 (VCCA), U?.1 (VCCA), U?.1 (VCCA)
- net ADC_SELECT: now also U?.4 (B); no longer U1008.6, U1009.6
- net FDACLO: now also U?.4 (B); no longer R1005.1
- net FDACN_SELECT: now also U?.4 (B); no longer U1005.6
- net GND: now also U?.2 (GND), U?.2 (GND), U?.2 (GND), U?.5 (DIR), U?.5 (DIR), U?.5 (DIR)
- new net ADC_SEL: U1008.6, U1009.6, U?.3 (A)
- new net FDACLO_SEL: R1005.1, U?.3 (A)
- new net FDACN_SEL: U1005.6, U?.3 (A)

Commit message: Schematic design.
Parts:
- gave numbers to parts that had none: 3
- renumbered C1010 to C1001, C1003 to C1002, C1011 to C1003, C1001 to C1005, C1002 to C1006, C1005 to C1007, C1012 to C1008, C1013 to C1009, C1006 to C1010, C1007 to C1011, C1008 to C1012, C1009 to C1013, C1021 to C1017, C1022 to C1018, C1023 to C1019, C1024 to C1020, C1025 to C1021, C1026 to C1022, C1027 to C1023, C1028 to C1024, C1029 to C1025, C1030 to C1026, C1031 to C1027, C1032 to C1028, C1033 to C1029, C1034 to C1030, C1035 to C1031, C1036 to C1032, C1037 to C1033, C1038 to C1034, C1039 to C1035, C1040 to C1036, C1041 to C1037, C1042 to C1038, C1043 to C1039, C1017 to C1040, C1018 to C1041, C1019 to C1042, C1020 to C1043, R1004 to R1001, R1005 to R1002, R1015 to R1003, R1016 to R1004, R1001 to R1005, R1017 to R1007, R1003 to R1008, R1018 to R1009, R1019 to R1010, R1002 to R1011, R1007 to R1012, R1008 to R1013, R1020 to R1014, R1009 to R1015, R1021 to R1016, R1022 to R1017, R1026 to R1018, R1010 to R1019, R1011 to R1020, R1012 to R1021, R1023 to R1022, R1024 to R1023, R1013 to R1024, R1027 to R1025, R1014 to R1026, R1025 to R1027, U1004 to U1001, U1008 to U1002, U1007 to U1003, U1001 to U1004, U1010 to U1006, U1009 to U1007, U1002 to U1008, U1003 to U1010, U1011 to U1012, U1012 to U1014, U1006 to U1015, U1013 to U1016

Commit message: Schematic design.
Parts:
- C901: renamed from C1001; footprint (none) -> Capacitor_SMD:C_0603_1608Metric_Pad1.08x0.95mm_HandSolder
- C902: renamed from C1002; footprint (none) -> Capacitor_SMD:C_0603_1608Metric_Pad1.08x0.95mm_HandSolder
- C903: renamed from C1003; footprint (none) -> Capacitor_SMD:C_0603_1608Metric_Pad1.08x0.95mm_HandSolder
- C904: renamed from C1004; footprint (none) -> Capacitor_SMD:C_0603_1608Metric_Pad1.08x0.95mm_HandSolder
- C905: renamed from C1005; footprint (none) -> Resistor_SMD:R_0805_2012Metric_Pad1.20x1.40mm_HandSolder
- C906: renamed from C1006; footprint (none) -> Capacitor_SMD:C_0603_1608Metric_Pad1.08x0.95mm_HandSolder
- C907: renamed from C1007; footprint (none) -> Capacitor_SMD:C_0603_1608Metric_Pad1.08x0.95mm_HandSolder
- C908: renamed from C1008; footprint (none) -> Capacitor_SMD:C_0603_1608Metric_Pad1.08x0.95mm_HandSolder
- C909: renamed from C1009; footprint (none) -> Capacitor_SMD:C_0603_1608Metric_Pad1.08x0.95mm_HandSolder
- C910: renamed from C1010; footprint (none) -> Capacitor_SMD:C_0603_1608Metric_Pad1.08x0.95mm_HandSolder
- C911: renamed from C1011; footprint (none) -> Resistor_SMD:R_0805_2012Metric_Pad1.20x1.40mm_HandSolder
- C912: renamed from C1012; footprint (none) -> Capacitor_SMD:C_0603_1608Metric_Pad1.08x0.95mm_HandSolder
- C913: renamed from C1013; footprint (none) -> Capacitor_SMD:C_1206_3216Metric_Pad1.33x1.80mm_HandSolder
- C914: renamed from C1014; footprint (none) -> Capacitor_SMD:C_0603_1608Metric_Pad1.08x0.95mm_HandSolder
- C915: renamed from C1015; footprint (none) -> Capacitor_SMD:C_0603_1608Metric_Pad1.08x0.95mm_HandSolder
- C916: renamed from C1016; footprint (none) -> Resistor_SMD:R_0805_2012Metric_Pad1.20x1.40mm_HandSolder
- C917: renamed from C1017; footprint (none) -> Capacitor_SMD:C_0603_1608Metric_Pad1.08x0.95mm_HandSolder
- C918: renamed from C1018; footprint (none) -> Capacitor_SMD:C_0603_1608Metric_Pad1.08x0.95mm_HandSolder
- C919: renamed from C1019; footprint (none) -> Capacitor_SMD:C_0603_1608Metric_Pad1.08x0.95mm_HandSolder
- C920: renamed from C1020; footprint (none) -> Capacitor_SMD:C_0603_1608Metric_Pad1.08x0.95mm_HandSolder
- C921: renamed from C1021; footprint (none) -> Capacitor_SMD:C_0603_1608Metric_Pad1.08x0.95mm_HandSolder
- C922: renamed from C1022; footprint (none) -> Capacitor_SMD:C_0603_1608Metric_Pad1.08x0.95mm_HandSolder
- C923: renamed from C1023; footprint (none) -> Capacitor_SMD:C_0603_1608Metric_Pad1.08x0.95mm_HandSolder
- C924: renamed from C1024; footprint (none) -> Capacitor_SMD:C_0603_1608Metric_Pad1.08x0.95mm_HandSolder
- C925: renamed from C1025; footprint (none) -> Capacitor_SMD:C_0603_1608Metric_Pad1.08x0.95mm_HandSolder
- C926: renamed from C1026; footprint (none) -> Capacitor_SMD:C_0603_1608Metric_Pad1.08x0.95mm_HandSolder
- C927: renamed from C1027; footprint (none) -> Capacitor_SMD:C_0603_1608Metric_Pad1.08x0.95mm_HandSolder
- C928: renamed from C1028; footprint (none) -> Capacitor_SMD:C_0603_1608Metric_Pad1.08x0.95mm_HandSolder
- C929: renamed from C1029; footprint (none) -> Capacitor_SMD:C_0603_1608Metric_Pad1.08x0.95mm_HandSolder
- C930: renamed from C1030; footprint (none) -> Capacitor_SMD:C_0603_1608Metric_Pad1.08x0.95mm_HandSolder
- C931: renamed from C1031; footprint (none) -> Capacitor_SMD:C_0603_1608Metric_Pad1.08x0.95mm_HandSolder
- C932: renamed from C1032; footprint (none) -> Capacitor_SMD:C_0603_1608Metric_Pad1.08x0.95mm_HandSolder
- C933: renamed from C1033; footprint (none) -> Capacitor_SMD:C_0603_1608Metric_Pad1.08x0.95mm_HandSolder
- C934: renamed from C1034; footprint (none) -> Capacitor_SMD:C_0603_1608Metric_Pad1.08x0.95mm_HandSolder
- C935: renamed from C1035; footprint (none) -> Capacitor_SMD:C_0603_1608Metric_Pad1.08x0.95mm_HandSolder
- C936: renamed from C1036; footprint (none) -> Capacitor_SMD:C_0603_1608Metric_Pad1.08x0.95mm_HandSolder
- C937: renamed from C1037; footprint (none) -> Capacitor_SMD:C_0603_1608Metric_Pad1.08x0.95mm_HandSolder
- C938: renamed from C1038; footprint (none) -> Capacitor_SMD:C_0603_1608Metric_Pad1.08x0.95mm_HandSolder
- C939: renamed from C1039; footprint (none) -> Capacitor_SMD:C_0603_1608Metric_Pad1.08x0.95mm_HandSolder
- C940: renamed from C1040; footprint (none) -> Resistor_SMD:R_0805_2012Metric_Pad1.20x1.40mm_HandSolder
- C941: renamed from C1041; footprint (none) -> Capacitor_SMD:C_0603_1608Metric_Pad1.08x0.95mm_HandSolder
- C942: renamed from C1042; footprint (none) -> Resistor_SMD:R_0805_2012Metric_Pad1.20x1.40mm_HandSolder
- C943: renamed from C1043; footprint (none) -> Capacitor_SMD:C_0603_1608Metric_Pad1.08x0.95mm_HandSolder
- R901: renamed from R1001; footprint (none) -> Resistor_SMD:R_0603_1608Metric_Pad0.98x0.95mm_HandSolder
- R902: renamed from R1002; footprint (none) -> Resistor_SMD:R_0603_1608Metric_Pad0.98x0.95mm_HandSolder
- R903: renamed from R1003; footprint (none) -> Resistor_SMD:R_0603_1608Metric_Pad0.98x0.95mm_HandSolder
- R904: renamed from R1004; footprint (none) -> Resistor_SMD:R_0603_1608Metric_Pad0.98x0.95mm_HandSolder
- R905: renamed from R1005; footprint (none) -> Resistor_SMD:R_0603_1608Metric_Pad0.98x0.95mm_HandSolder
- R906: renamed from R1006; footprint (none) -> Resistor_SMD:R_0603_1608Metric_Pad0.98x0.95mm_HandSolder
- R907: renamed from R1007; footprint (none) -> Resistor_SMD:R_0603_1608Metric_Pad0.98x0.95mm_HandSolder
- R908: renamed from R1008; footprint (none) -> Resistor_SMD:R_0603_1608Metric_Pad0.98x0.95mm_HandSolder
- R909: renamed from R1009; footprint (none) -> Resistor_SMD:R_0603_1608Metric_Pad0.98x0.95mm_HandSolder
- R910: renamed from R1010; footprint (none) -> Resistor_SMD:R_0603_1608Metric_Pad0.98x0.95mm_HandSolder
- R911: renamed from R1011; footprint (none) -> Resistor_SMD:R_0603_1608Metric_Pad0.98x0.95mm_HandSolder
- R912: renamed from R1012; footprint (none) -> Resistor_SMD:R_0603_1608Metric_Pad0.98x0.95mm_HandSolder
- R913: renamed from R1013; footprint (none) -> Resistor_SMD:R_0603_1608Metric_Pad0.98x0.95mm_HandSolder
- R914: renamed from R1014; footprint (none) -> Resistor_SMD:R_0603_1608Metric_Pad0.98x0.95mm_HandSolder
- R915: renamed from R1015; footprint (none) -> Resistor_SMD:R_0603_1608Metric_Pad0.98x0.95mm_HandSolder
- R916: renamed from R1016; footprint (none) -> Resistor_SMD:R_0603_1608Metric_Pad0.98x0.95mm_HandSolder
- R917: renamed from R1017; footprint (none) -> Resistor_SMD:R_0603_1608Metric_Pad0.98x0.95mm_HandSolder
- R918: renamed from R1018; footprint (none) -> Resistor_SMD:R_0603_1608Metric_Pad0.98x0.95mm_HandSolder
- R919: renamed from R1019; footprint (none) -> Resistor_SMD:R_0603_1608Metric_Pad0.98x0.95mm_HandSolder
- R920: renamed from R1020; footprint (none) -> Resistor_SMD:R_0603_1608Metric_Pad0.98x0.95mm_HandSolder
- R921: renamed from R1021; footprint (none) -> Resistor_SMD:R_0603_1608Metric_Pad0.98x0.95mm_HandSolder
- R922: renamed from R1022; footprint (none) -> Resistor_SMD:R_0603_1608Metric_Pad0.98x0.95mm_HandSolder
- R923: renamed from R1023; footprint (none) -> Resistor_SMD:R_0603_1608Metric_Pad0.98x0.95mm_HandSolder
- R924: renamed from R1024; footprint (none) -> Resistor_SMD:R_0603_1608Metric_Pad0.98x0.95mm_HandSolder
- R925: renamed from R1025; footprint (none) -> Resistor_SMD:R_0603_1608Metric_Pad0.98x0.95mm_HandSolder
- R926: renamed from R1026; footprint (none) -> Resistor_SMD:R_0603_1608Metric_Pad0.98x0.95mm_HandSolder
- R927: renamed from R1027; footprint (none) -> Resistor_SMD:R_0603_1608Metric_Pad0.98x0.95mm_HandSolder
- R928: renamed from R1028; footprint (none) -> Resistor_SMD:R_0603_1608Metric_Pad0.98x0.95mm_HandSolder
- R929: renamed from R1029; footprint (none) -> Resistor_SMD:R_0603_1608Metric_Pad0.98x0.95mm_HandSolder
- U903: renamed from U1003; footprint (none) -> Package_SO:SOIC-8_3.9x4.9mm_P1.27mm
- U904: renamed from U1004; footprint (none) -> Package_SO:SOIC-8_3.9x4.9mm_P1.27mm
- U906: renamed from U1006; footprint (none) -> Package_SO:TSSOP-24_4.4x7.8mm_P0.65mm
- U908: renamed from U1008; footprint (none) -> Package_SO:SOIC-8_3.9x4.9mm_P1.27mm
- U910: renamed from U1010; footprint (none) -> Package_SO:SOIC-8_3.9x4.9mm_P1.27mm
- U912: renamed from U1012; footprint (none) -> Package_SO:TSSOP-16_4.4x5mm_P0.65mm
- U914: renamed from U1014; footprint (none) -> Package_SO:TSSOP-16_4.4x5mm_P0.65mm
- U915: renamed from U1015; footprint (none) -> Package_SO:SOIC-8_3.9x4.9mm_P1.27mm
- renumbered U1001 to U901, U1002 to U902, U1005 to U905, U1007 to U907, U1009 to U909, U1011 to U911, U1013 to U913, U1016 to U916

Commit message: Schematic design.
Parts:
- added TP?: TPDAC, symbol Connector:TestPoint
Connections:
- net DAC_SP: no longer names the net of U908.7 (VOUTD)
- net DAC_SP: now also TP?.1
Changed lines of the file:
@@
 $Descr A3 16535 11693
 encoding utf-8
-Sheet 9 11
+Sheet 9 12
 Title ""
 Date ""
@@
 Wire Wire Line
 	3350 3550 3800 3550
-Text HLabel 3400 3650 2    50   Output ~ 0
-DAC_SP
-Wire Wire Line
-	3400 3650 3350 3650
 Wire Wire Line
 	5750 2150 5350 2150
@@
 Text Label 6750 800  2    50   ~ 0
 FDACLO_SEL
+$Comp
+L Connector:TestPoint TP?
+U 1 1 627031F9
+P 3350 3650
+F 0 "TP?" V 3304 3838 50  0000 L CNN
+F 1 "TPDAC" V 3395 3838 50  0000 L CNN
+F 2 "" H 3550 3650 50  0001 C CNN
+F 3 "~" H 3550 3650 50  0001 C CNN
+	1    3350 3650
+	0    1    1    0
+$EndComp
 $EndSCHEMATC

Commit message: Schematic design
Parts:
- R901, R903, R904, R905, R906, R907, R908, R909, R910, R912, R913, R914, R915, R919, R920, R921, R924, R926: footprint Resistor_SMD:R_0603_1608Metric_Pad0.98x0.95mm_HandSolder -> Resistor_SMD:R_0805_2012Metric_Pad1.20x1.40mm_HandSolder
- TP901: renamed from TP?; footprint (none) -> TestPoint:TestPoint_Loop_D2.60mm_Drill1.6mm_Beaded
- U908: value OPA2140 -> AD5686RARUZ; footprint Package_SO:SOIC-8_3.9x4.9mm_P1.27mm -> Package_SO:TSSOP-16_4.4x5mm_P0.65mm
Changed lines of the file:
@@
 $Descr A3 16535 11693
 encoding utf-8
-Sheet 9 12
+Sheet 9 13
 Title ""
 Date ""
@@
 Comment4 ""
 $EndDescr
-$Comp
-L ETH1CSMU1:AD5686RARUZ U908
-U 1 1 60554356
-P 2800 3500
-F 0 "U908" H 3250 4200 50  0000 C CNN
-F 1 "OPA2140" H 3250 4100 50  0000 C CNN
-F 2 "Package_SO:SOIC-8_3.9x4.9mm_P1.27mm" H 4350 3850 50  0001 C CNN
-F 3 "" H 4350 3850 50  0001 C CNN
-	1    2800 3500
-	1    0    0    -1
-$EndComp
 Wire Wire Line
 	2250 3650 2150 3650
@@
 F 0 "R908" V 4143 2050 50  0000 C CNN
 F 1 "10k/.1%" V 4234 2050 50  0000 C CNN
-F 2 "Resistor_SMD:R_0603_1608Metric_Pad0.98x0.95mm_HandSolder" V 4280 2050 50  0001 C CNN
+F 2 "Resistor_SMD:R_0805_2012Metric_Pad1.20x1.40mm_HandSolder" V 4280 2050 50  0001 C CNN
 F 3 "~" H 4350 2050 50  0001 C CNN
 	1    4350 2050
@@
 F 0 "R905" V 4143 1600 50  0000 C CNN
 F 1 "10k/.1%" V 4234 1600 50  0000 C CNN
-F 2 "Resistor_SMD:R_0603_1608Metric_Pad0.98x0.95mm_HandSolder" V 4280 1600 50  0001 C CNN
+F 2 "Resistor_SMD:R_0805_2012Metric_Pad1.20x1.40mm_HandSolder" V 4280 1600 50  0001 C CNN
 F 3 "~" H 4350 1600 50  0001 C CNN
 	1    4350 1600
@@
 F 0 "R906" V 4793 1600 50  0000 C CNN
 F 1 "20k5/.1%" V 4884 1600 50  0000 C CNN
-F 2 "Resistor_SMD:R_0603_1608Metric_Pad0.98x0.95mm_HandSolder" V 4930 1600 50  0001 C CNN
+F 2 "Resistor_SMD:R_0805_2012Metric_Pad1.20x1.40mm_HandSolder" V 4930 1600 50  0001 C CNN
 F 3 "~" H 5000 1600 50  0001 C CNN
 	1    5000 1600
@@
 F 0 "R901" V 4793 800 50  0000 C CNN
 F 1 "2k/.1%" V 4884 800 50  0000 C CNN
-F 2 "Resistor_SMD:R_0603_1608Metric_Pad0.98x0.95mm_HandSolder" V 4930 800 50  0001 C CNN
+F 2 "Resistor_SMD:R_0805_2012Metric_Pad1.20x1.40mm_HandSolder" V 4930 800 50  0001 C CNN
 F 3 "~" H 5000 800 50  0001 C CNN
 	1    5000 800
@@
 F 0 "R915" V 4193 3750 50  0000 C CNN
 F 1 "10k/.1%" V 4284 3750 50  0000 C CNN
-F 2 "Resistor_SMD:R_0603_1608Metric_Pad0.98x0.95mm_HandSolder" V 4330 3750 50  0001 C CNN
+F 2 "Resistor_SMD:R_0805_2012Metric_Pad1.20x1.40mm_HandSolder" V 4330 3750 50  0001 C CNN
 F 3 "~" H 4400 3750 50  0001 C CNN
 	1    4400 3750
@@
 F 0 "R912" V 4193 3300 50  0000 C CNN
 F 1 "10k/.1%" V 4284 3300 50  0000 C CNN
-F 2 "Resistor_SMD:R_0603_1608Metric_Pad0.98x0.95mm_HandSolder" V 4330 3300 50  0001 C CNN
+F 2 "Resistor_SMD:R_0805_2012Metric_Pad1.20x1.40mm_HandSolder" V 4330 3300 50  0001 C CNN
 F 3 "~" H 4400 3300 50  0001 C CNN
 	1    4400 3300
@@
 F 0 "R913" V 4843 3300 50  0000 C CNN
 F 1 "21k5/.1%" V 4934 3300 50  0000 C CNN
-F 2 "Resistor_SMD:R_0603_1608Metric_Pad0.98x0.95mm_HandSolder" V 4980 3300 50  0001 C CNN
+F 2 "Resistor_SMD:R_0805_2012Metric_Pad1.20x1.40mm_HandSolder" V 4980 3300 50  0001 C CNN
 F 3 "~" H 5050 3300 50  0001 C CNN
 	1    5050 3300
@@
 F 0 "R921" V 4193 5500 50  0000 C CNN
 F 1 "10k/.1%" V 4284 5500 50  0000 C CNN
-F 2 "Resistor_SMD:R_0603_1608Metric_Pad0.98x0.95mm_HandSolder" V 4330 5500 50  0001 C CNN
+F 2 "Resistor_SMD:R_0805_2012Metric_Pad1.20x1.40mm_HandSolder" V 4330 5500 50  0001 C CNN
 F 3 "~" H 4400 5500 50  0001 C CNN
 	1    4400 5500
@@
 F 0 "R919" V 4193 5050 50  0000 C CNN
 F 1 "10k/.1%" V 4284 5050 50  0000 C CNN
-F 2 "Resistor_SMD:R_0603_1608Metric_Pad0.98x0.95mm_HandSolder" V 4330 5050 50  0001 C CNN
+F 2 "Resistor_SMD:R_0805_2012Metric_Pad1.20x1.40mm_HandSolder" V 4330 5050 50  0001 C CNN
 F 3 "~" H 4400 5050 50  0001 C CNN
 	1    4400 5050
@@
 F 0 "R920" V 4843 5050 50  0000 C CNN
 F 1 "21k5/.1%" V 4934 5050 50  0000 C CNN
-F 2 "Resistor_SMD:R_0603_1608Metric_Pad0.98x0.95mm_HandSolder" V 4980 5050 50  0001 C CNN
+F 2 "Resistor_SMD:R_0805_2012Metric_Pad1.20x1.40mm_HandSolder" V 4980 5050 50  0001 C CNN
 F 3 "~" H 5050 5050 50  0001 C CNN
 	1    5050 5050
@@
 F 0 "R926" V 3093 6900 50  0000 C CNN
 F 1 "10k/.1%" V 3184 6900 50  0000 C CNN
-F 2 "Resistor_SMD:R_0603_1608Metric_Pad0.98x0.95mm_HandSolder" V 3230 6900 50  0001 C CNN
+F 2 "Resistor_SMD:R_0805_2012Metric_Pad1.20x1.40mm_HandSolder" V 3230 6900 50  0001 C CNN
 F 3 "~" H 3300 6900 50  0001 C CNN
 	1    3300 6900
@@
 F 0 "R924" V 3743 6500 50  0000 C CNN
 F 1 "10k/.1%" V 3834 6500 50  0000 C CNN
-F 2 "Resistor_SMD:R_0603_1608Metric_Pad0.98x0.95mm_HandSolder" V 3880 6500 50  0001 C CNN
+F 2 "Resistor_SMD:R_0805_2012Metric_Pad1.20x1.40mm_HandSolder" V 3880 6500 50  0001 C CNN
 F 3 "~" H 3950 6500 50  0001 C CNN
 	1    3950 6500
@@
 $EndComp
 Wire Wire Line
-	12850 7450 12950 7450
-Connection ~ 12850 7450
-Wire Wire Line
-	12850 7450 12850 7500
-Wire Wire Line
-	12750 7450 12850 7450
+	12950 7450 12950 7500
 Connection ~ 12750 7450
 Wire Wire Line
 	12750 7400 12750 7450
 Wire Wire Line
-	12950 7450 13050 7450
-Connection ~ 12950 7450
-Wire Wire Line
 	12950 7400 12950 7450
 Wire Wire Line
-	13050 7450 13050 7400
-Wire Wire Line
 	12650 7450 12750 7450
 Wire Wire Line
@@
 L power:GND #PWR0957
 U 1 1 60C2DCE4
-P 12850 7500
-F 0 "#PWR0957" H 12850 7250 50  0001 C CNN
-F 1 "GND" H 12855 7327 50  0000 C CNN
-F 2 "" H 12850 7500 50  0001 C CNN
-F 3 "" H 12850 7500 50  0001 C CNN
-	1    12850 7500
+P 12950 7500
+F 0 "#PWR0957" H 12950 7250 50  0001 C CNN
+F 1 "GND" H 12955 7327 50  0000 C CNN
+F 2 "" H 12950 7500 50  0001 C CNN
+F 3 "" H 12950 7500 50  0001 C CNN
+	1    12950 7500
 	1    0    0    -1
 $EndComp
@@
 $EndComp
 Wire Wire Line
-	12850 5600 12950 5600
-Connection ~ 12850 5600
-Wire Wire Line
-	12850 5600 12850 5650
-Wire Wire Line
-	12750 5600 12850 5600
+	12950 5600 12950 5650
 Connection ~ 12750 5600
 Wire Wire Line
 	12750 5550 12750 5600
 Wire Wire Line
-	12950 5600 13050 5600
-Connection ~ 12950 5600
-Wire Wire Line
 	12950 5550 12950 5600
 Wire Wire Line
-	13050 5600 13050 5550
-Wire Wire Line
 	12650 5600 12750 5600
 Wire Wire Line
@@
 L power:GND #PWR0939
 U 1 1 60BC66EB
-P 12850 5650
-F 0 "#PWR0939" H 12850 5400 50  0001 C CNN
-F 1 "GND" H 12855 5477 50  0000 C CNN
-F 2 "" H 12850 5650 50  0001 C CNN
-F 3 "" H 12850 5650 50  0001 C CNN
-	1    12850 5650
+P 12950 5650
+F 0 "#PWR0939" H 12950 5400 50  0001 C CNN
+F 1 "GND" H 12955 5477 50  0000 C CNN
+F 2 "" H 12950 5650 50  0001 C CNN
+F 3 "" H 12950 5650 50  0001 C CNN
+	1    12950 5650
 	1    0    0    -1
 $EndComp
@@
 F 0 "R904" V 12343 1300 50  0000 C CNN
 F 1 "10k/.1%" V 12434 1300 50  0000 C CNN
-F 2 "Resistor_SMD:R_0603_1608Metric_Pad0.98x0.95mm_HandSolder" V 12480 1300 50  0001 C CNN
+F 2 "Resistor_SMD:R_0805_2012Metric_Pad1.20x1.40mm_HandSolder" V 12480 1300 50  0001 C CNN
 F 3 "~" H 12550 1300 50  0001 C CNN
 	1    12550 1300
@@
 F 0 "R903" V 11693 1300 50  0000 C CNN
 F 1 "10k/.1%" V 11784 1300 50  0000 C CNN
-F 2 "Resistor_SMD:R_0603_1608Metric_Pad0.98x0.95mm_HandSolder" V 11830 1300 50  0001 C CNN
+F 2 "Resistor_SMD:R_0805_2012Metric_Pad1.20x1.40mm_HandSolder" V 11830 1300 50  0001 C CNN
 F 3 "~" H 11900 1300 50  0001 C CNN
 	1    11900 1300
@@
 F 0 "R907" V 11693 1750 50  0000 C CNN
 F 1 "21k5/.1%" V 11784 1750 50  0000 C CNN
-F 2 "Resistor_SMD:R_0603_1608Metric_Pad0.98x0.95mm_HandSolder" V 11830 1750 50  0001 C CNN
+F 2 "Resistor_SMD:R_0805_2012Metric_Pad1.20x1.40mm_HandSolder" V 11830 1750 50  0001 C CNN
 F 3 "~" H 11900 1750 50  0001 C CNN
 	1    11900 1750
@@
 F 0 "R910" V 12343 3000 50  0000 C CNN
 F 1 "10k/.1%" V 12434 3000 50  0000 C CNN
-F 2 "Resistor_SMD:R_0603_1608Metric_Pad0.98x0.95mm_HandSolder" V 12480 3000 50  0001 C CNN
+F 2 "Resistor_SMD:R_0805_2012Metric_Pad1.20x1.40mm_HandSolder" V 12480 3000 50  0001 C CNN
 F 3 "~" H 12550 3000 50  0001 C CNN
 	1    12550 3000
@@
 F 0 "R909" V 11693 3000 50  0000 C CNN
 F 1 "10k/.1%" V 11784 3000 50  0000 C CNN
-F 2 "Resistor_SMD:R_0603_1608Metric_Pad0.98x0.95mm_HandSolder" V 11830 3000 50  0001 C CNN
+F 2 "Resistor_SMD:R_0805_2012Metric_Pad1.20x1.40mm_HandSolder" V 11830 3000 50  0001 C CNN
 F 3 "~" H 11900 3000 50  0001 C CNN
 	1    11900 3000
@@
 F 0 "R914" V 11693 3450 50  0000 C CNN
 F 1 "21k5/.1%" V 11784 3450 50  0000 C CNN
-F 2 "Resistor_SMD:R_0603_1608Metric_Pad0.98x0.95mm_HandSolder" V 11830 3450 50  0001 C CNN
+F 2 "Resistor_SMD:R_0805_2012Metric_Pad1.20x1.40mm_HandSolder" V 11830 3450 50  0001 C CNN
 F 3 "~" H 11900 3450 50  0001 C CNN
 	1    11900 3450
@@
 FDACLO_SEL
 $Comp
-L Connector:TestPoint TP?
+L Connector:TestPoint TP901
 U 1 1 627031F9
 P 3350 3650
-F 0 "TP?" V 3304 3838 50  0000 L CNN
+F 0 "TP901" V 3304 3838 50  0000 L CNN
 F 1 "TPDAC" V 3395 3838 50  0000 L CNN
-F 2 "" H 3550 3650 50  0001 C CNN
+F 2 "TestPoint:TestPoint_Loop_D2.60mm_Drill1.6mm_Beaded" H 3550 3650 50  0001 C CNN
 F 3 "~" H 3550 3650 50  0001 C CNN
 	1    3350 3650
 	0    1    1    0
 $EndComp
+$Comp
+L ETH1CSMU1:AD5686RARUZ U908
+U 1 1 62562820
+P 2800 3500
+F 0 "U908" H 3250 4200 50  0000 C CNN
+F 1 "AD5686RARUZ" H 3250 4100 50  0000 C CNN
+F 2 "Package_SO:TSSOP-16_4.4x5mm_P0.65mm" H 4350 3850 50  0001 C CNN
+F 3 "" H 4350 3850 50  0001 C CNN
+	1    2800 3500
+	1    0    0    -1
+$EndComp
+Connection ~ 12950 5600
+Wire Wire Line
+	12750 5600 12950 5600
+Connection ~ 12950 7450
+Wire Wire Line
+	12750 7450 12950 7450
 $EndSCHEMATC

Commit message: Design
Connections:
- net FGEN_AMP renamed SIGN_SEL
Changed lines of the file:
@@
 	6050 3000 6050 2550
 Text HLabel 5700 2350 0    50   Input ~ 0
-FGEN_AMP
+SIGN_SEL
 Wire Wire Line
 	5700 2350 5750 2350
