File: HARDWARE/BASE/GPIO.sch (KiCad schematic (older format))
At the start: 0 parts

Commit message: Design
Parts:
- added C? (x28): 100n, symbol Device:C
- added R?: 1k, symbol Device:R
- added U? (x14): SN74LVC1T45DBV, Package_TO_SOT_SMD:SOT-23-6, symbol Logic_LevelTranslator:SN74LVC1T45DBV
- added U?: MCP23S17_SO, Package_SO:SOIC-28W_7.5x17.9mm_P1.27mm, symbol Interface_Expansion:MCP23S17_SO
Connections:
- new net: R?.1, U?.5 (DIR)
- new net +3V3: C?.1, C?.1, C?.1, C?.1, C?.1, C?.1, C?.1, C?.1, C?.1, C?.1, C?.1, C?.1, C?.1, C?.1, U?.6 (VCCB), U?.6 (VCCB), U?.6 (VCCB), U?.6 (VCCB), U?.6 (VCCB), U?.6 (VCCB), U?.6 (VCCB), U?.6 (VCCB), U?.6 (VCCB), U?.6 (VCCB), U?.6 (VCCB), U?.6 (VCCB), U?.6 (VCCB), U?.6 (VCCB)
- new net +5V: C?.1, C?.1, C?.1, C?.1, C?.1, C?.1, C?.1, C?.1, C?.1, C?.1, C?.1, C?.1, C?.1, C?.1, R?.2, U?.1 (VCCA), U?.1 (VCCA), U?.1 (VCCA), U?.1 (VCCA), U?.1 (VCCA), U?.1 (VCCA), U?.1 (VCCA), U?.1 (VCCA), U?.1 (VCCA), U?.1 (VCCA), U?.1 (VCCA), U?.1 (VCCA), U?.1 (VCCA), U?.1 (VCCA)
- new net 10mA: U?.3 (A)
- new net GND: C?.2, C?.2, C?.2, C?.2, C?.2, C?.2, C?.2, C?.2, C?.2, C?.2, C?.2, C?.2, C?.2, C?.2, C?.2, C?.2, C?.2, C?.2, C?.2, C?.2, C?.2, C?.2, C?.2, C?.2, C?.2, C?.2, C?.2, C?.2, U?.2 (GND), U?.2 (GND), U?.2 (GND), U?.2 (GND), U?.2 (GND), U?.2 (GND), U?.2 (GND), U?.2 (GND), U?.2 (GND), U?.2 (GND), U?.2 (GND), U?.2 (GND), U?.2 (GND), U?.2 (GND), U?.5 (DIR), U?.5 (DIR), U?.5 (DIR), U?.5 (DIR), U?.5 (DIR), U?.5 (DIR), U?.5 (DIR), U?.5 (DIR), U?.5 (DIR), U?.5 (DIR), U?.5 (DIR), U?.5 (DIR), U?.5 (DIR)
- new net GPIO_REL1_CTR: U?.4 (B)
- new net GPIO_REL2_CTR: U?.4 (B)
- new net GPIO_~100mA: U?.4 (B)
- new net GPIO_~100uA: U?.4 (B)
- new net GPIO_~10mA: U?.4 (B)
- new net GPIO_~10uA: U?.4 (B)
- new net GPIO_~1A: U?.4 (B)
- new net GPIO_~1mA: U?.4 (B)
- new net GPIO_~IMODE: U?.4 (B)
- new net GPIO_~LT10mA: U?.4 (B)
- new net GPIO_~VMODE: U?.4 (B)
- new net GPIO_~VRANGE: U?.4 (B)
- new net MCU_10mA: U?.4 (B)
- new net MCU_~ICLAMP: U?.4 (B)
- new net REL1_CTR: U?.3 (A)
- new net REL2_CTR: U?.3 (A)
- new net ~100mA: U?.3 (A)
- new net ~100uA: U?.3 (A)
- new net ~10mA: U?.3 (A)
- new net ~10uA: U?.3 (A)
- new net ~1A: U?.3 (A)
- new net ~1mA: U?.3 (A)
- new net ~ICLAMP: U?.3 (A)
- new net ~IMODE: U?.3 (A)
- new net ~LT10mA: U?.3 (A)
- new net ~VMODE: U?.3 (A)
- new net ~VRANGE: U?.3 (A)
