File: HARDWARE/BASE/GPIO.sch (KiCad schematic (older format))
At the start: 44 parts

Commit message: Design
Parts:
- added C1215: 100n, symbol Device:C
- added R1202: 10k, symbol Device:R
- gave numbers to parts that had none: 44
Connections:
- net +3V3: now also U1215.9 (VDD), C1215.1, R1202.2
- net GND: now also U1215.10 (VSS), U1215.15 (A0), U1215.16 (A1), U1215.17 (A2), C1215.2
- net GPIO_REL1_CTR: now also U1215.3 (GPB2)
- net GPIO_REL2_CTR: now also U1215.2 (GPB1)
- net GPIO_~100mA: now also U1215.8 (GPB7)
- net GPIO_~100uA: now also U1215.25 (GPA4)
- net GPIO_~10mA: now also U1215.23 (GPA2)
- net GPIO_~10uA: now also U1215.24 (GPA3)
- net GPIO_~1A: now also U1215.21 (GPA0)
- net GPIO_~1mA: now also U1215.6 (GPB5)
- net GPIO_~IMODE: now also U1215.7 (GPB6)
- net GPIO_~LT10mA: now also U1215.4 (GPB3)
- net GPIO_~VMODE: now also U1215.5 (GPB4)
- net GPIO_~VRANGE: now also U1215.22 (GPA1)
- net MCU_10mA: now also U1215.1 (GPB0)
- net at U1215.18 (~RESET~): now also R1202.1
- no-connect marks 0 -> 5
Other:
- moved on the sheet: C1201, C1202, C1203, C1204, C1205, C1206, C1207, C1208, C1209, C1210, C1211, C1212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

Commit message: PCB and schematic design.
Parts:
- C1201, C1202, C1203, C1204, C1205, C1206, C1207, C1208, C1209, C1210, C1211, C1212, C1213, C1214, C1215, C1216, C1217, C1218, C1219, C1220, C1221, C1222, C1223, C1224, C1225, C1226, C1227, C1228, C1229: footprint (none) -> Capacitor_SMD:C_0603_1608Metric_Pad1.08x0.95mm_HandSolder
- R1201, R1202: footprint (none) -> Resistor_SMD:R_0603_1608Metric_Pad0.98x0.95mm_HandSolder
Changed lines of the file:
@@
 F 0 "C1216" H 765 7296 50  0000 L CNN
 F 1 "100n" H 765 7205 50  0000 L CNN
-F 2 "" H 688 7100 50  0001 C CNN
+F 2 "Capacitor_SMD:C_0603_1608Metric_Pad1.08x0.95mm_HandSolder" H 688 7100 50  0001 C CNN
 F 3 "~" H 650 7250 50  0001 C CNN
 	1    650  7250
@@
 F 0 "C1217" H 1215 7296 50  0000 L CNN
 F 1 "100n" H 1215 7205 50  0000 L CNN
-F 2 "" H 1138 7100 50  0001 C CNN
+F 2 "Capacitor_SMD:C_0603_1608Metric_Pad1.08x0.95mm_HandSolder" H 1138 7100 50  0001 C CNN
 F 3 "~" H 1100 7250 50  0001 C CNN
 	1    1100 7250
@@
 F 0 "C1218" H 1665 7296 50  0000 L CNN
 F 1 "100n" H 1665 7205 50  0000 L CNN
-F 2 "" H 1588 7100 50  0001 C CNN
+F 2 "Capacitor_SMD:C_0603_1608Metric_Pad1.08x0.95mm_HandSolder" H 1588 7100 50  0001 C CNN
 F 3 "~" H 1550 7250 50  0001 C CNN
 	1    1550 7250
@@
 F 0 "C1219" H 2115 7296 50  0000 L CNN
 F 1 "100n" H 2115 7205 50  0000 L CNN
-F 2 "" H 2038 7100 50  0001 C CNN
+F 2 "Capacitor_SMD:C_0603_1608Metric_Pad1.08x0.95mm_HandSolder" H 2038 7100 50  0001 C CNN
 F 3 "~" H 2000 7250 50  0001 C CNN
 	1    2000 7250
@@
 F 0 "C1220" H 2565 7296 50  0000 L CNN
 F 1 "100n" H 2565 7205 50  0000 L CNN
-F 2 "" H 2488 7100 50  0001 C CNN
+F 2 "Capacitor_SMD:C_0603_1608Metric_Pad1.08x0.95mm_HandSolder" H 2488 7100 50  0001 C CNN
 F 3 "~" H 2450 7250 50  0001 C CNN
 	1    2450 7250
@@
 F 0 "C1221" H 3015 7296 50  0000 L CNN
 F 1 "100n" H 3015 7205 50  0000 L CNN
-F 2 "" H 2938 7100 50  0001 C CNN
+F 2 "Capacitor_SMD:C_0603_1608Metric_Pad1.08x0.95mm_HandSolder" H 2938 7100 50  0001 C CNN
 F 3 "~" H 2900 7250 50  0001 C CNN
 	1    2900 7250
@@
 F 0 "C1222" H 3465 7296 50  0000 L CNN
 F 1 "100n" H 3465 7205 50  0000 L CNN
-F 2 "" H 3388 7100 50  0001 C CNN
+F 2 "Capacitor_SMD:C_0603_1608Metric_Pad1.08x0.95mm_HandSolder" H 3388 7100 50  0001 C CNN
 F 3 "~" H 3350 7250 50  0001 C CNN
 	1    3350 7250
@@
 F 0 "C1223" H 3915 7296 50  0000 L CNN
 F 1 "100n" H 3915 7205 50  0000 L CNN
-F 2 "" H 3838 7100 50  0001 C CNN
+F 2 "Capacitor_SMD:C_0603_1608Metric_Pad1.08x0.95mm_HandSolder" H 3838 7100 50  0001 C CNN
 F 3 "~" H 3800 7250 50  0001 C CNN
 	1    3800 7250
@@
 F 0 "C1224" H 4365 7296 50  0000 L CNN
 F 1 "100n" H 4365 7205 50  0000 L CNN
-F 2 "" H 4288 7100 50  0001 C CNN
+F 2 "Capacitor_SMD:C_0603_1608Metric_Pad1.08x0.95mm_HandSolder" H 4288 7100 50  0001 C CNN
 F 3 "~" H 4250 7250 50  0001 C CNN
 	1    4250 7250
@@
 F 0 "C1225" H 4815 7296 50  0000 L CNN
 F 1 "100n" H 4815 7205 50  0000 L CNN
-F 2 "" H 4738 7100 50  0001 C CNN
+F 2 "Capacitor_SMD:C_0603_1608Metric_Pad1.08x0.95mm_HandSolder" H 4738 7100 50  0001 C CNN
 F 3 "~" H 4700 7250 50  0001 C CNN
 	1    4700 7250
@@
 F 0 "C1226" H 5265 7296 50  0000 L CNN
 F 1 "100n" H 5265 7205 50  0000 L CNN
-F 2 "" H 5188 7100 50  0001 C CNN
+F 2 "Capacitor_SMD:C_0603_1608Metric_Pad1.08x0.95mm_HandSolder" H 5188 7100 50  0001 C CNN
 F 3 "~" H 5150 7250 50  0001 C CNN
 	1    5150 7250
@@
 F 0 "C1227" H 5715 7296 50  0000 L CNN
 F 1 "100n" H 5715 7205 50  0000 L CNN
-F 2 "" H 5638 7100 50  0001 C CNN
+F 2 "Capacitor_SMD:C_0603_1608Metric_Pad1.08x0.95mm_HandSolder" H 5638 7100 50  0001 C CNN
 F 3 "~" H 5600 7250 50  0001 C CNN
 	1    5600 7250
@@
 F 0 "C1228" H 6165 7296 50  0000 L CNN
 F 1 "100n" H 6165 7205 50  0000 L CNN
-F 2 "" H 6088 7100 50  0001 C CNN
+F 2 "Capacitor_SMD:C_0603_1608Metric_Pad1.08x0.95mm_HandSolder" H 6088 7100 50  0001 C CNN
 F 3 "~" H 6050 7250 50  0001 C CNN
 	1    6050 7250
@@
 F 0 "C1201" H 765 6196 50  0000 L CNN
 F 1 "100n" H 765 6105 50  0000 L CNN
-F 2 "" H 688 6000 50  0001 C CNN
+F 2 "Capacitor_SMD:C_0603_1608Metric_Pad1.08x0.95mm_HandSolder" H 688 6000 50  0001 C CNN
 F 3 "~" H 650 6150 50  0001 C CNN
 	1    650  6150
@@
 F 0 "C1202" H 1215 6196 50  0000 L CNN
 F 1 "100n" H 1215 6105 50  0000 L CNN
-F 2 "" H 1138 6000 50  0001 C CNN
+F 2 "Capacitor_SMD:C_0603_1608Metric_Pad1.08x0.95mm_HandSolder" H 1138 6000 50  0001 C CNN
 F 3 "~" H 1100 6150 50  0001 C CNN
 	1    1100 6150
@@
 F 0 "C1203" H 1665 6196 50  0000 L CNN
 F 1 "100n" H 1665 6105 50  0000 L CNN
-F 2 "" H 1588 6000 50  0001 C CNN
+F 2 "Capacitor_SMD:C_0603_1608Metric_Pad1.08x0.95mm_HandSolder" H 1588 6000 50  0001 C CNN
 F 3 "~" H 1550 6150 50  0001 C CNN
 	1    1550 6150
@@
 F 0 "C1204" H 2115 6196 50  0000 L CNN
 F 1 "100n" H 2115 6105 50  0000 L CNN
-F 2 "" H 2038 6000 50  0001 C CNN
+F 2 "Capacitor_SMD:C_0603_1608Metric_Pad1.08x0.95mm_HandSolder" H 2038 6000 50  0001 C CNN
 F 3 "~" H 2000 6150 50  0001 C CNN
 	1    2000 6150
@@
 F 0 "C1205" H 2565 6196 50  0000 L CNN
 F 1 "100n" H 2565 6105 50  0000 L CNN
-F 2 "" H 2488 6000 50  0001 C CNN
+F 2 "Capacitor_SMD:C_0603_1608Metric_Pad1.08x0.95mm_HandSolder" H 2488 6000 50  0001 C CNN
 F 3 "~" H 2450 6150 50  0001 C CNN
 	1    2450 6150
@@
 F 0 "C1206" H 3015 6196 50  0000 L CNN
 F 1 "100n" H 3015 6105 50  0000 L CNN
-F 2 "" H 2938 6000 50  0001 C CNN
+F 2 "Capacitor_SMD:C_0603_1608Metric_Pad1.08x0.95mm_HandSolder" H 2938 6000 50  0001 C CNN
 F 3 "~" H 2900 6150 50  0001 C CNN
 	1    2900 6150
@@
 F 0 "C1207" H 3465 6196 50  0000 L CNN
 F 1 "100n" H 3465 6105 50  0000 L CNN
-F 2 "" H 3388 6000 50  0001 C CNN
+F 2 "Capacitor_SMD:C_0603_1608Metric_Pad1.08x0.95mm_HandSolder" H 3388 6000 50  0001 C CNN
 F 3 "~" H 3350 6150 50  0001 C CNN
 	1    3350 6150
@@
 F 0 "C1208" H 3915 6196 50  0000 L CNN
 F 1 "100n" H 3915 6105 50  0000 L CNN
-F 2 "" H 3838 6000 50  0001 C CNN
+F 2 "Capacitor_SMD:C_0603_1608Metric_Pad1.08x0.95mm_HandSolder" H 3838 6000 50  0001 C CNN
 F 3 "~" H 3800 6150 50  0001 C CNN
 	1    3800 6150
@@
 F 0 "C1209" H 4365 6196 50  0000 L CNN
 F 1 "100n" H 4365 6105 50  0000 L CNN
-F 2 "" H 4288 6000 50  0001 C CNN
+F 2 "Capacitor_SMD:C_0603_1608Metric_Pad1.08x0.95mm_HandSolder" H 4288 6000 50  0001 C CNN
 F 3 "~" H 4250 6150 50  0001 C CNN
 	1    4250 6150
@@
 F 0 "C1210" H 4815 6196 50  0000 L CNN
 F 1 "100n" H 4815 6105 50  0000 L CNN
-F 2 "" H 4738 6000 50  0001 C CNN
+F 2 "Capacitor_SMD:C_0603_1608Metric_Pad1.08x0.95mm_HandSolder" H 4738 6000 50  0001 C CNN
 F 3 "~" H 4700 6150 50  0001 C CNN
 	1    4700 6150
@@
 F 0 "C1211" H 5265 6196 50  0000 L CNN
 F 1 "100n" H 5265 6105 50  0000 L CNN
-F 2 "" H 5188 6000 50  0001 C CNN
+F 2 "Capacitor_SMD:C_0603_1608Metric_Pad1.08x0.95mm_HandSolder" H 5188 6000 50  0001 C CNN
 F 3 "~" H 5150 6150 50  0001 C CNN
 	1    5150 6150
@@
 F 0 "C1212" H 5715 6196 50  0000 L CNN
 F 1 "100n" H 5715 6105 50  0000 L CNN
-F 2 "" H 5638 6000 50  0001 C CNN
+F 2 "Capacitor_SMD:C_0603_1608Metric_Pad1.08x0.95mm_HandSolder" H 5638 6000 50  0001 C CNN
 F 3 "~" H 5600 6150 50  0001 C CNN
 	1    5600 6150
@@
 F 0 "C1213" H 6165 6196 50  0000 L CNN
 F 1 "100n" H 6165 6105 50  0000 L CNN
-F 2 "" H 6088 6000 50  0001 C CNN
+F 2 "Capacitor_SMD:C_0603_1608Metric_Pad1.08x0.95mm_HandSolder" H 6088 6000 50  0001 C CNN
 F 3 "~" H 6050 6150 50  0001 C CNN
 	1    6050 6150
@@
 F 0 "C1214" H 6615 6196 50  0000 L CNN
 F 1 "100n" H 6615 6105 50  0000 L CNN
-F 2 "" H 6538 6000 50  0001 C CNN
+F 2 "Capacitor_SMD:C_0603_1608Metric_Pad1.08x0.95mm_HandSolder" H 6538 6000 50  0001 C CNN
 F 3 "~" H 6500 6150 50  0001 C CNN
 	1    6500 6150
@@
 F 0 "C1229" H 6615 7296 50  0000 L CNN
 F 1 "100n" H 6615 7205 50  0000 L CNN
-F 2 "" H 6538 7100 50  0001 C CNN
+F 2 "Capacitor_SMD:C_0603_1608Metric_Pad1.08x0.95mm_HandSolder" H 6538 7100 50  0001 C CNN
 F 3 "~" H 6500 7250 50  0001 C CNN
 	1    6500 7250
@@
 F 0 "R1201" V 8950 2850 50  0000 C CNN
 F 1 "1k" V 9050 2850 50  0000 C CNN
-F 2 "" V 8980 2850 50  0001 C CNN
+F 2 "Resistor_SMD:R_0603_1608Metric_Pad0.98x0.95mm_HandSolder" V 8980 2850 50  0001 C CNN
 F 3 "~" H 9050 2850 50  0001 C CNN
 	1    9050 2850
@@
 F 0 "C1215" H 7065 6196 50  0000 L CNN
 F 1 "100n" H 7065 6105 50  0000 L CNN
-F 2 "" H 6988 6000 50  0001 C CNN
+F 2 "Capacitor_SMD:C_0603_1608Metric_Pad1.08x0.95mm_HandSolder" H 6988 6000 50  0001 C CNN
 F 3 "~" H 6950 6150 50  0001 C CNN
 	1    6950 6150
@@
 F 0 "R1202" V 8393 5250 50  0000 C CNN
 F 1 "10k" V 8484 5250 50  0000 C CNN
-F 2 "" V 8530 5250 50  0001 C CNN
+F 2 "Resistor_SMD:R_0603_1608Metric_Pad0.98x0.95mm_HandSolder" V 8530 5250 50  0001 C CNN
 F 3 "~" H 8600 5250 50  0001 C CNN
 	1    8600 5250

Commit message: PCB and schematic
Connections:
- net 10mA renamed 10-100mA
- net MCU_10mA renamed GPIO_10-100mA
Changed lines of the file:
@@
 Text HLabel 7000 2650 0    50   Output ~ 0
 ~10mA
-Text HLabel 950  1300 0    50   Output ~ 0
-10mA
 Text HLabel 9200 1300 0    50   Output ~ 0
 ~100uA
@@
 $Comp
 L Logic_LevelTranslator:SN74LVC1T45DBV U?
-U 1 1 60C32408
-P 1400 1300
-AR Path="/608EADFA/60C32408" Ref="U?"  Part="1"
-AR Path="/60E4AF69/60C32408" Ref="U1201"  Part="1"
-F 0 "U1201" H 1900 1750 50  0000 L CNN
-F 1 "SN74LVC1T45DBV" H 1650 1650 50  0000 L CNN
-F 2 "Package_TO_SOT_SMD:SOT-23-6" H 1400 850 50  0001 C CNN
-F 3 "http://www.ti.com/lit/ds/symlink/sn74lvc1t45.pdf" H 500 650 50  0001 C CNN
-	1    1400 1300
-	1    0    0    -1
-$EndComp
-Wire Wire Line
-	1000 1500 950  1500
-Wire Wire Line
-	950  1500 950  1750
-Wire Wire Line
-	950  1750 1400 1750
-Wire Wire Line
-	1400 1750 1400 1700
-$Comp
-L power:+5V #PWR?
-U 1 1 60C32412
-P 1300 900
-AR Path="/608EADFA/60C32412" Ref="#PWR?"  Part="1"
-AR Path="/60E4AF69/60C32412" Ref="#PWR01201"  Part="1"
-F 0 "#PWR01201" H 1300 750 50  0001 C CNN
-F 1 "+5V" H 1300 1050 50  0000 C CNN
-F 2 "" H 1300 900 50  0001 C CNN
-F 3 "" H 1300 900 50  0001 C CNN
-	1    1300 900
-	1    0    0    -1
-$EndComp
-$Comp
-L power:+3.3V #PWR?
-U 1 1 60C32418
-P 1500 900
-AR Path="/608EADFA/60C32418" Ref="#PWR?"  Part="1"
-AR Path="/60E4AF69/60C32418" Ref="#PWR01202"  Part="1"
-F 0 "#PWR01202" H 1500 750 50  0001 C CNN
-F 1 "+3.3V" H 1500 1050 50  0000 C CNN
-F 2 "" H 1500 900 50  0001 C CNN
-F 3 "" H 1500 900 50  0001 C CNN
-	1    1500 900
-	1    0    0    -1
-$EndComp
-$Comp
-L power:GND #PWR?
-U 1 1 60C3241E
-P 1400 1800
-AR Path="/608EADFA/60C3241E" Ref="#PWR?"  Part="1"
-AR Path="/60E4AF69/60C3241E" Ref="#PWR01211"  Part="1"
-F 0 "#PWR01211" H 1400 1550 50  0001 C CNN
-F 1 "GND" H 1405 1627 50  0000 C CNN
-F 2 "" H 1400 1800 50  0001 C CNN
-F 3 "" H 1400 1800 50  0001 C CNN
-	1    1400 1800
-	1    0    0    -1
-$EndComp
-Wire Wire Line
-	1400 1800 1400 1750
-Connection ~ 1400 1750
-Wire Wire Line
-	2400 1300 1800 1300
-$Comp
-L Logic_LevelTranslator:SN74LVC1T45DBV U?
 U 1 1 60C32429
 P 1400 2650
@@
 Wire Wire Line
 	1000 2650 950  2650
-Wire Wire Line
-	1000 1300 950  1300
 Wire Wire Line
 	1000 4050 950  4050
@@
 	1    0    0    -1
 $EndComp
-Text Label 2400 1300 2    50   ~ 0
-MCU_10mA
 Text Label 2400 2650 2    50   ~ 0
 GPIO_REL2_CTR
@@
 $EndComp
 Wire Wire Line
-	10750 4350 10150 4350
-Text Label 10750 4350 2    50   ~ 0
-MCU_10mA
-Wire Wire Line
 	10750 4450 10150 4450
 Text Label 10750 4450 2    50   ~ 0
@@
 Wire Wire Line
 	3350 5950 3800 5950
+Wire Wire Line
+	10750 4350 10150 4350
+Text Label 2450 1300 2    50   ~ 0
+GPIO_10-100mA
+Wire Wire Line
+	1000 1300 950  1300
+Wire Wire Line
+	2450 1300 1800 1300
+$Comp
+L power:GND #PWR?
+U 1 1 60C3241E
+P 1400 1800
+AR Path="/608EADFA/60C3241E" Ref="#PWR?"  Part="1"
+AR Path="/60E4AF69/60C3241E" Ref="#PWR01211"  Part="1"
+F 0 "#PWR01211" H 1400 1550 50  0001 C CNN
+F 1 "GND" H 1405 1627 50  0000 C CNN
+F 2 "" H 1400 1800 50  0001 C CNN
+F 3 "" H 1400 1800 50  0001 C CNN
+	1    1400 1800
+	1    0    0    -1
+$EndComp
+$Comp
+L power:+3.3V #PWR?
+U 1 1 60C32418
+P 1500 900
+AR Path="/608EADFA/60C32418" Ref="#PWR?"  Part="1"
+AR Path="/60E4AF69/60C32418" Ref="#PWR01202"  Part="1"
+F 0 "#PWR01202" H 1500 750 50  0001 C CNN
+F 1 "+3.3V" H 1500 1050 50  0000 C CNN
+F 2 "" H 1500 900 50  0001 C CNN
+F 3 "" H 1500 900 50  0001 C CNN
+	1    1500 900
+	1    0    0    -1
+$EndComp
+$Comp
+L power:+5V #PWR?
+U 1 1 60C32412
+P 1300 900
+AR Path="/608EADFA/60C32412" Ref="#PWR?"  Part="1"
+AR Path="/60E4AF69/60C32412" Ref="#PWR01201"  Part="1"
+F 0 "#PWR01201" H 1300 750 50  0001 C CNN
+F 1 "+5V" H 1300 1050 50  0000 C CNN
+F 2 "" H 1300 900 50  0001 C CNN
+F 3 "" H 1300 900 50  0001 C CNN
+	1    1300 900
+	1    0    0    -1
+$EndComp
+Wire Wire Line
+	1400 1800 1400 1750
+Wire Wire Line
+	1400 1750 1400 1700
+Connection ~ 1400 1750
+Wire Wire Line
+	950  1750 1400 1750
+Wire Wire Line
+	950  1500 950  1750
+Wire Wire Line
+	1000 1500 950  1500
+$Comp
+L Logic_LevelTranslator:SN74LVC1T45DBV U?
+U 1 1 60C32408
+P 1400 1300
+AR Path="/608EADFA/60C32408" Ref="U?"  Part="1"
+AR Path="/60E4AF69/60C32408" Ref="U1201"  Part="1"
+F 0 "U1201" H 1900 1750 50  0000 L CNN
+F 1 "SN74LVC1T45DBV" H 1650 1650 50  0000 L CNN
+F 2 "Package_TO_SOT_SMD:SOT-23-6" H 1400 850 50  0001 C CNN
+F 3 "http://www.ti.com/lit/ds/symlink/sn74lvc1t45.pdf" H 500 650 50  0001 C CNN
+	1    1400 1300
+	1    0    0    -1
+$EndComp
+Text HLabel 950  1300 0    50   Output ~ 0
+10-100mA
+Text Label 10750 4350 2    50   ~ 0
+GPIO_10-100mA
 $EndSCHEMATC

Commit message: Schematic and PCB changes
Parts:
- removed C1213, C1214, C1215, C1216, C1217, C1218, C1219, C1220, C1221, C1222, C1223, C1224, C1225, C1226, C1227, C1228, C1229: 100n, Capacitor_SMD:C_0603_1608Metric_Pad1.08x0.95mm_HandSolder, symbol Device:C
- removed U1202, U1204, U1207, U1208, U1209, U1211, U1212, U1213, U1214: SN74LVC1T45DBV, Package_TO_SOT_SMD:SOT-23-6, symbol Logic_LevelTranslator:SN74LVC1T45DBV
- removed U1215: MCP23S17_SO, Package_SO:SOIC-28W_7.5x17.9mm_P1.27mm, symbol Interface_Expansion:MCP23S17_SO
- added U1202, U1204: 74HCT595, Package_SO:TSSOP-16_4.4x5mm_P0.65mm, symbol 74xx:74HCT595
- R1202: value 10k -> 1k
Connections:
- net +3V3: no longer C1201.1, C1202.1, C1203.1, C1204.1, C1205.1, C1206.1, C1207.1, R1202.2
- net +5V: now also C1201.1, C1202.1, C1203.1, C1204.1, C1205.1, C1206.1, C1207.1, R1202.2, U1202.10 (~SRCLR), U1202.16 (VCC), U1204.10 (~SRCLR), U1204.16 (VCC)
- net 10-100mA: now also U1204.7 (QH); no longer U1201.3 (A)
- net GND: now also U1202.13 (~OE), U1202.8 (GND), U1204.13 (~OE), U1204.8 (GND); no longer U1206.5 (DIR)
- net REL1_CTR: now also U1202.2 (QC)
- net REL2_CTR: now also U1202.3 (QD); no longer U1206.3 (A)
- net ~100mA: now also U1204.4 (QE)
- net ~100uA: now also U1204.1 (QB); no longer U1205.3 (A)
- net ~10mA: now also U1204.3 (QD)
- net ~10uA: now also U1204.15 (QA)
- net ~1A: now also U1204.5 (QF)
- net ~1mA: now also U1204.2 (QC)
- net ~IMODE: now also U1202.15 (QA); no longer U1203.3 (A)
- net ~LT10mA: now also U1204.6 (QG)
- net ~VMODE: now also U1202.1 (QB)
- net ~VRANGE: now also U1202.7 (QH)
- net at R1202.1: now also U1206.5 (DIR)
- net GPIO_10-100mA renamed SPI5_MOSI
- net GPIO_REL2_CTR renamed SPI5_MISO
- net GPIO_~100uA renamed SPI5_NSS
- net GPIO_~IMODE renamed SPI5_SCK
- new net: U1202.11 (SRCLK), U1203.3 (A), U1204.11 (SRCLK)
- new net: U1202.12 (RCLK), U1204.12 (RCLK), U1205.3 (A)
- new net: U1201.3 (A), U1202.14 (SER)
- new net: U1202.9 (QH'), U1204.14 (SER)
- new net: U1204.9 (QH'), U1206.3 (A)
- new net ADC_SELECT: U1202.6 (QG)
- new net FDACLO: U1202.4 (QE)
- new net FDACN_SELECT: U1202.5 (QF)
- no-connect marks 5 -> 0
Other:
- moved on the sheet: R1201, U1210
