File: HARDWARE/BASE/BASE.kicad_pcb (KiCad board)
At the start: 6 copper layers, 160 x 100 mm, 281 parts, among them J1101 20021111-00010T4LF, J501 Conn_02x01, J502 20021111-00010T4LF, J601 C64AC, Q701 IRFR5410, U1101 MEE1S0303DC, U1102 SI8606AC-B-IS1, U201 74AC125, U202 TXB0104PW, U203 ADuM5402, U301 MT48LC16M16A2P-6A, U401 LC03-3.3, U402 LAN8742A, U403 LC03-3.3, U501 STM32H743ZI, U502 HDC1080, U503 24LC08B-E/MS, U701 MAX5902, U702 THL15-2415WI, U801 MC7815BD2TG, U802 LM1117DTX-5.0/NOPB, U803 TSR1-2490, U804 LT8330_S6, U805 MC7915BD2TG, U806 LM1117DTX-3.3/NOPB, U807 TSR1-2450, U808 LT8330_S6, U901 DG419LDY, U902 DG419LDY, U903 TLC2272, U904 OPA2140, U905 DG419LDY, U906 AD7190RUZ, U907 DG419LDY, U908 OPA2140, U909 SN74LVC1T45DBV, U910 TL072, U911 SN74LVC1T45DBV, U912 ADS8681PWR, U913 SN74LVC1T45DBV, U914 ADS8681PWR, U915 ADR431ARZ, U916 REF5040ID, Y401 NX5032GA-25.000M-LN-CD-1, Y501 NX3225GD-8MHZ

Commit message: Schematic design
Parts:
- removed C1101, C1103, C1105, C1106: 100n, Capacitor_SMD:C_0603_1608Metric_Pad1.08x0.95mm_HandSolder
- removed C1102, C1104: 1u, Capacitor_SMD:C_0603_1608Metric_Pad1.08x0.95mm_HandSolder
- removed J1101: 20021111-00010T4LF, Connector_PinHeader_1.27mm:PinHeader_2x05_P1.27mm_Vertical
- removed R1101, R1104: 3k3, Resistor_SMD:R_0603_1608Metric_Pad0.98x0.95mm_HandSolder
- removed R1102, R1105: 10k, Resistor_SMD:R_0603_1608Metric_Pad0.98x0.95mm_HandSolder
- removed R1103, R1106: 4k7, Resistor_SMD:R_0603_1608Metric_Pad0.98x0.95mm_HandSolder
- removed U1101: MEE1S0303DC, ETH1CSMU1:MEE1_DIP
- removed U1102: SI8606AC-B-IS1, Package_SO:SOIC-16_3.9x9.9mm_P1.27mm
- added C1001: 150p/500V, Capacitor_SMD:C_0805_2012Metric_Pad1.18x1.45mm_HandSolder, F.Cu at (-7.89, -40.2)
- added C1002: 100p, Capacitor_SMD:C_0603_1608Metric_Pad1.08x0.95mm_HandSolder, F.Cu at (-11.1, -19.1)
- added C1003: 22p/500V, Capacitor_SMD:C_0805_2012Metric_Pad1.18x1.45mm_HandSolder, F.Cu at (-42.0, -5.69)
- added C1004: 270p, Capacitor_SMD:C_0603_1608Metric_Pad1.08x0.95mm_HandSolder, F.Cu at (-25.4, -1.65)
- added C1005: 270p/500V, Capacitor_SMD:C_0805_2012Metric_Pad1.18x1.45mm_HandSolder, F.Cu at (-36.0, -14.9)
- added C1006: 15p, Capacitor_SMD:C_0603_1608Metric_Pad1.08x0.95mm_HandSolder, F.Cu at (-30.1, 0.86)
- added C1007: 1000p, Capacitor_SMD:C_0603_1608Metric_Pad1.08x0.95mm_HandSolder, F.Cu at (-2.10, -25.7)
- added C1008: 270p, Capacitor_SMD:C_0603_1608Metric_Pad1.08x0.95mm_HandSolder, F.Cu at (-18.5, -8.88)
- added C1009: 270p/500V, Capacitor_SMD:C_0805_2012Metric_Pad1.18x1.45mm_HandSolder, F.Cu at (-21.2, -27.1)
- added C1010: 270p, Capacitor_SMD:C_0603_1608Metric_Pad1.08x0.95mm_HandSolder, F.Cu at (-29.7, -1.65)
- added C1011: 15p, Capacitor_SMD:C_0603_1608Metric_Pad1.08x0.95mm_HandSolder, F.Cu at (2.25, -30.0)
- added C1012: 15p, Capacitor_SMD:C_0603_1608Metric_Pad1.08x0.95mm_HandSolder, F.Cu at (-6.80, -19.1)
- added C1013: 150p, Capacitor_SMD:C_0603_1608Metric_Pad1.08x0.95mm_HandSolder, F.Cu at (-25.8, 0.86)
- added C1014: 22p/100V, Capacitor_SMD:C_0805_2012Metric_Pad1.18x1.45mm_HandSolder, F.Cu at (-26.2, -22.1)
- added C1015: 22p, Capacitor_SMD:C_0603_1608Metric_Pad1.08x0.95mm_HandSolder, F.Cu at (2.25, -27.5)
- added C1016: 100n, Capacitor_SMD:C_0603_1608Metric_Pad1.08x0.95mm_HandSolder, F.Cu at (-18.5, -6.37)
- added C1017: 100n, Capacitor_SMD:C_0603_1608Metric_Pad1.08x0.95mm_HandSolder, F.Cu at (-2.64, -23.2)
- added C1018: 100n, Capacitor_SMD:C_0603_1608Metric_Pad1.08x0.95mm_HandSolder, F.Cu at (-12.8, -14.1)
- added C1019: 100n, Capacitor_SMD:C_0603_1608Metric_Pad1.08x0.95mm_HandSolder, F.Cu at (-9.77, -6.57)
- added C1020: 100n, Capacitor_SMD:C_0603_1608Metric_Pad1.08x0.95mm_HandSolder, F.Cu at (-21.4, 0.86)
- added C1021: 100n, Capacitor_SMD:C_0603_1608Metric_Pad1.08x0.95mm_HandSolder, F.Cu at (-2.45, -18.2)
- added C1022: 100n, Capacitor_SMD:C_0603_1608Metric_Pad1.08x0.95mm_HandSolder, F.Cu at (-14.1, -6.57)
- added C1023: 100n, Capacitor_SMD:C_0603_1608Metric_Pad1.08x0.95mm_HandSolder, F.Cu at (-16.7, -3.86)
- added C1024: 100n, Capacitor_SMD:C_0603_1608Metric_Pad1.08x0.95mm_HandSolder, F.Cu at (-8.41, -11.6)
- added C1025: 100n, Capacitor_SMD:C_0603_1608Metric_Pad1.08x0.95mm_HandSolder, F.Cu at (-21.0, -1.82)
- added C1026: 100n, Capacitor_SMD:C_0603_1608Metric_Pad1.08x0.95mm_HandSolder, F.Cu at (-9.77, -9.08)
- added C1027: 100n, Capacitor_SMD:C_0603_1608Metric_Pad1.08x0.95mm_HandSolder, F.Cu at (-4.06, -14.1)
- added C1028: 100n, Capacitor_SMD:C_0603_1608Metric_Pad1.08x0.95mm_HandSolder, F.Cu at (-17.1, 0.69)
- added C1029: 100n, Capacitor_SMD:C_0603_1608Metric_Pad1.08x0.95mm_HandSolder, F.Cu at (-8.41, -14.1)
- added C1030: 100n, Capacitor_SMD:C_0603_1608Metric_Pad1.08x0.95mm_HandSolder, F.Cu at (1.90, -19.9)
- added C1031: 100n, Capacitor_SMD:C_0603_1608Metric_Pad1.08x0.95mm_HandSolder, F.Cu at (-12.3, -4.06)
- added C1032: 100n, Capacitor_SMD:C_0603_1608Metric_Pad1.08x0.95mm_HandSolder, F.Cu at (-4.06, -11.6)
- added C1033: 100n, Capacitor_SMD:C_0603_1608Metric_Pad1.08x0.95mm_HandSolder, F.Cu at (-5.42, -9.08)
- added C1034: 100n, Capacitor_SMD:C_0603_1608Metric_Pad1.08x0.95mm_HandSolder, F.Cu at (1.90, -17.4)
- added C1035: 100n, Capacitor_SMD:C_0603_1608Metric_Pad1.08x0.95mm_HandSolder, F.Cu at (0.29, -14.9)
- added C1036: 10p, Capacitor_SMD:C_0603_1608Metric_Pad1.08x0.95mm_HandSolder, F.Cu at (-2.10, -28.2)
- added C1037: 10p, Capacitor_SMD:C_0603_1608Metric_Pad1.08x0.95mm_HandSolder, F.Cu at (-34.5, -0.04)
- added C1301: 1p5, Capacitor_SMD:C_0603_1608Metric_Pad1.08x0.95mm_HandSolder, F.Cu at (-43.5, 31.2)
- added C1302: 10n, Capacitor_SMD:C_0603_1608Metric_Pad1.08x0.95mm_HandSolder, F.Cu at (-47.9, 31.2)
- added C1303: 4p7, Capacitor_SMD:C_0603_1608Metric_Pad1.08x0.95mm_HandSolder, F.Cu at (-24.2, 12.4)
- added C1304: 18p, Capacitor_SMD:C_0603_1608Metric_Pad1.08x0.95mm_HandSolder, F.Cu at (-34.8, 25.8)
- added C1305: 12p, Capacitor_SMD:C_0603_1608Metric_Pad1.08x0.95mm_HandSolder, F.Cu at (-41.6, 16.2)
- added C1306: 10u, Capacitor_SMD:C_1206_3216Metric_Pad1.33x1.80mm_HandSolder, F.Cu at (-44.5, 7.80)
- added C1307: 100n, Capacitor_SMD:C_0603_1608Metric_Pad1.08x0.95mm_HandSolder, F.Cu at (-34.8, 23.3)
- added C1308: 10u, Capacitor_SMD:C_0805_2012Metric_Pad1.18x1.45mm_HandSolder, F.Cu at (-70.7, 33.7)
- added C1309: 1u, Capacitor_SMD:C_0603_1608Metric_Pad1.08x0.95mm_HandSolder, F.Cu at (-31.9, 20.4)
- added C1310: 100n, Capacitor_SMD:C_0603_1608Metric_Pad1.08x0.95mm_HandSolder, F.Cu at (-36.2, 10.3)
- added C1311: 22p, Capacitor_SMD:C_0603_1608Metric_Pad1.08x0.95mm_HandSolder, F.Cu at (-52.2, 26.0)
- added C1312: 56p, Capacitor_SMD:C_0603_1608Metric_Pad1.08x0.95mm_HandSolder, F.Cu at (-61.4, 34.3)
- added C1313: 56p, Capacitor_SMD:C_0603_1608Metric_Pad1.08x0.95mm_HandSolder, F.Cu at (-56.6, 29.5)
- added C1314: 22p, Capacitor_SMD:C_0603_1608Metric_Pad1.08x0.95mm_HandSolder, F.Cu at (-34.6, 7.38)
- added C1315: 100n, Capacitor_SMD:C_0603_1608Metric_Pad1.08x0.95mm_HandSolder, F.Cu at (-24.2, 14.9)
- added C1316: 100n, Capacitor_SMD:C_0603_1608Metric_Pad1.08x0.95mm_HandSolder, F.Cu at (-44.0, 33.8)
- added C1317: 5p, Capacitor_SMD:C_0603_1608Metric_Pad1.08x0.95mm_HandSolder, F.Cu at (-61.4, 31.8)
- added C1318: 100n, Capacitor_SMD:C_0603_1608Metric_Pad1.08x0.95mm_HandSolder, F.Cu at (-49.3, 21.0)
- added C1319: 10n, Capacitor_SMD:C_0603_1608Metric_Pad1.08x0.95mm_HandSolder, F.Cu at (-41.6, 13.7)
- added C1320: 100n, Capacitor_SMD:C_0603_1608Metric_Pad1.08x0.95mm_HandSolder, F.Cu at (-49.3, 18.5)
- added C1321: 5p, Capacitor_SMD:C_0603_1608Metric_Pad1.08x0.95mm_HandSolder, F.Cu at (-44.9, 21.2)
- added C1322: 220n, Capacitor_SMD:C_0603_1608Metric_Pad1.08x0.95mm_HandSolder, F.Cu at (-27.5, 17.4)
- added C1323: 1n, Capacitor_SMD:C_0603_1608Metric_Pad1.08x0.95mm_HandSolder, F.Cu at (-39.2, 26.2)
- added C1324: 8p, Capacitor_SMD:C_0603_1608Metric_Pad1.08x0.95mm_HandSolder, F.Cu at (150.1, 82.7)
- added C1325: 8p, Capacitor_SMD:C_0603_1608Metric_Pad1.08x0.95mm_HandSolder, F.Cu at (128.8, 91.7)
- added C1326: 2u2, Capacitor_SMD:C_0603_1608Metric_Pad1.08x0.95mm_HandSolder, F.Cu at (133.2, 91.7)
- added C1327: 100n, Capacitor_SMD:C_0603_1608Metric_Pad1.08x0.95mm_HandSolder, F.Cu at (148.6, 77.2)
- added C1328: 100n, Capacitor_SMD:C_0603_1608Metric_Pad1.08x0.95mm_HandSolder, F.Cu at (-40.6, 10.7)
- added C1329: 100n, Capacitor_SMD:C_0603_1608Metric_Pad1.08x0.95mm_HandSolder, F.Cu at (-43.5, 23.7)
- added C1330: 100n, Capacitor_SMD:C_0603_1608Metric_Pad1.08x0.95mm_HandSolder, F.Cu at (-32.9, 12.8)
- added C1331: 100n, Capacitor_SMD:C_0603_1608Metric_Pad1.08x0.95mm_HandSolder, F.Cu at (-31.9, 9.89)
- added C1332: 10u, Capacitor_SMD:C_0805_2012Metric_Pad1.18x1.45mm_HandSolder, F.Cu at (-53.8, 20.7)
- added C1333: 100n, Capacitor_SMD:C_0603_1608Metric_Pad1.08x0.95mm_HandSolder, F.Cu at (-52.2, 31.0)
- added C1334: 100n, Capacitor_SMD:C_0603_1608Metric_Pad1.08x0.95mm_HandSolder, F.Cu at (-40.6, 18.7)
- added C1335: 100n, Capacitor_SMD:C_0603_1608Metric_Pad1.08x0.95mm_HandSolder, F.Cu at (-52.7, 33.5)
- added C1336: 100n, Capacitor_SMD:C_0603_1608Metric_Pad1.08x0.95mm_HandSolder, F.Cu at (-27.5, 9.89)
- added C1337: 100n, Capacitor_SMD:C_0603_1608Metric_Pad1.08x0.95mm_HandSolder, F.Cu at (-36.2, 20.8)
- added C1338: 100n, Capacitor_SMD:C_0603_1608Metric_Pad1.08x0.95mm_HandSolder, F.Cu at (-43.5, 28.7)
- added C1339: 100n, Capacitor_SMD:C_0603_1608Metric_Pad1.08x0.95mm_HandSolder, F.Cu at (-28.6, 14.9)
- added C1340: 100n, Capacitor_SMD:C_0603_1608Metric_Pad1.08x0.95mm_HandSolder, F.Cu at (-48.4, 33.8)
- added C1341: 100n, Capacitor_SMD:C_0603_1608Metric_Pad1.08x0.95mm_HandSolder, F.Cu at (-31.9, 17.9)
- added C1342: 100n, Capacitor_SMD:C_0603_1608Metric_Pad1.08x0.95mm_HandSolder, F.Cu at (-30.5, 22.9)
- added C1343: 100n, Capacitor_SMD:C_0603_1608Metric_Pad1.08x0.95mm_HandSolder, F.Cu at (-23.2, 9.89)
- added C1344: 100n, Capacitor_SMD:C_0603_1608Metric_Pad1.08x0.95mm_HandSolder, F.Cu at (143.9, 80.2)
- added C1345: 100n, Capacitor_SMD:C_0603_1608Metric_Pad1.08x0.95mm_HandSolder, F.Cu at (145.8, 82.7)
- added C1346: 100n, Capacitor_SMD:C_0603_1608Metric_Pad1.08x0.95mm_HandSolder, F.Cu at (148.2, 80.2)
- added C1347: 100n, Capacitor_SMD:C_0603_1608Metric_Pad1.08x0.95mm_HandSolder, F.Cu at (137.5, 92.7)
- added C1348: 100n, Capacitor_SMD:C_0603_1608Metric_Pad1.08x0.95mm_HandSolder, F.Cu at (145.8, 85.2)
- added C1349: 100n, Capacitor_SMD:C_0603_1608Metric_Pad1.08x0.95mm_HandSolder, F.Cu at (142.7, 90.2)
- added C1350: 1u, Capacitor_SMD:C_0603_1608Metric_Pad1.08x0.95mm_HandSolder, F.Cu at (152.6, 79.7)
- added C1351: 100n, Capacitor_SMD:C_0603_1608Metric_Pad1.08x0.95mm_HandSolder, F.Cu at (138.4, 90.2)
- added C1352: 1u, Capacitor_SMD:C_0603_1608Metric_Pad1.08x0.95mm_HandSolder, F.Cu at (141.9, 92.7)
- added C601: 1u, Capacitor_SMD:C_0603_1608Metric_Pad1.08x0.95mm_HandSolder, F.Cu at (11.7, -21.5)
- added D1001: 1N4148W, Diode_SMD:D_SOD-123, F.Cu at (-13.2, -40.0)
- added D1002: BAV99, Package_TO_SOT_SMD:SOT-23, F.Cu at (-21.9, -12.4)
- added D1003: 1N4148W, Diode_SMD:D_SOD-123, F.Cu at (-41.5, -13.9)
- added D1004: BAV99, Package_TO_SOT_SMD:SOT-23, F.Cu at (-6.50, -27.2)
- added D1005: BAV99, Package_TO_SOT_SMD:SOT-23, F.Cu at (-7.04, -22.7)
- added D1006: BAV99, Package_TO_SOT_SMD:SOT-23, F.Cu at (-22.9, -7.86)
- added D1007: BAV99, Package_TO_SOT_SMD:SOT-23, F.Cu at (-17.2, -14.7)
- added D1008: BAV99, Package_TO_SOT_SMD:SOT-23, F.Cu at (0.73, -33.5)
- added D1301: SD103ATW, Package_TO_SOT_SMD:SOT-363_SC-70-6, F.Cu at (95.8, 62.1)
- added D1302: SD103ATW, Package_TO_SOT_SMD:SOT-363_SC-70-6, F.Cu at (-34.9, 31.5)
- added FB1301: 742792031, Inductor_SMD:L_0805_2012Metric_Pad1.15x1.40mm_HandSolder, F.Cu at (144.1, 77.4)
- added J1301: 20021111-00010T4LF, Connector_PinHeader_1.27mm:PinHeader_2x05_P1.27mm_Vertical, F.Cu at (138.3, 77.6)
- added K1001: EE2-5NU, Relay_SMD:Relay_DPDT_Kemet_EE2_NU, F.Cu at (186.9, 59.1)
- added K1002: EE2-5NU, Relay_SMD:Relay_DPDT_Kemet_EE2_NU, F.Cu at (187.1, 72.8)
- added K601: HE3621A0510, ETH1CSMU1:HE360_x-5050462-8, F.Cu at (206.2, 54.9)
- added K602: HE3621A0510, ETH1CSMU1:HE360_x-5050462-8, F.Cu at (206.2, 60.1)
- added K603: HE3621A0510, ETH1CSMU1:HE360_x-5050462-8, F.Cu at (206.2, 65.3)
- added K604: HE3621A0510, ETH1CSMU1:HE360_x-5050462-8, F.Cu at (206.2, 70.5)
- added K605: HE3621A0510, ETH1CSMU1:HE360_x-5050462-8, F.Cu at (206.2, 75.7)
- added L1301: 4u7, Inductor_SMD:L_0603_1608Metric_Pad1.05x0.95mm_HandSolder, F.Cu at (-39.2, 31.2)
- added L1302: 4u7, Inductor_SMD:L_0603_1608Metric_Pad1.05x0.95mm_HandSolder, F.Cu at (-27.5, 19.9)
- added L1303: 4u7, Inductor_SMD:L_0603_1608Metric_Pad1.05x0.95mm_HandSolder, F.Cu at (-30.5, 25.4)
- added Q1001: MMBT3904, Package_TO_SOT_SMD:SOT-23, F.Cu at (-27.9, -5.18)
- added Q1002: MMBT3904, Package_TO_SOT_SMD:SOT-23, F.Cu at (-15.5, -19.2)
- added R1001: 1k/500V, Resistor_SMD:R_1206_3216Metric_Pad1.30x1.75mm_HandSolder, F.Cu at (-26.2, -30.3)
- added R1002: 5Meg/25ppm/.1%, Resistor_SMD:R_1206_3216Metric_Pad1.30x1.75mm_HandSolder, F.Cu at (-26.2, -33.6)
- added R1003: 200k/500V, Resistor_SMD:R_1206_3216Metric_Pad1.30x1.75mm_HandSolder, F.Cu at (-41.4, -17.2)
- added R1004: 20k/.1%, Resistor_SMD:R_0805_2012Metric_Pad1.20x1.40mm_HandSolder, F.Cu at (-21.8, -16.2)
- added R1005: 10k/.1%, Resistor_SMD:R_0805_2012Metric_Pad1.20x1.40mm_HandSolder, F.Cu at (-3.87, -34.2)
- added R1006: 10k/.1%, Resistor_SMD:R_0805_2012Metric_Pad1.20x1.40mm_HandSolder, F.Cu at (-34.3, -2.77)
- added R1007: 560k/.1%, Resistor_SMD:R_0805_2012Metric_Pad1.20x1.40mm_HandSolder, F.Cu at (-6.35, -31.0)
- added R1008: 10k/.1%, Resistor_SMD:R_0805_2012Metric_Pad1.20x1.40mm_HandSolder, F.Cu at (-27.5, -8.93)
- added R1009: 10k/.1%, Resistor_SMD:R_0805_2012Metric_Pad1.20x1.40mm_HandSolder, F.Cu at (0.88, -37.3)
- added R1010: 10k/.1%, Resistor_SMD:R_0805_2012Metric_Pad1.20x1.40mm_HandSolder, F.Cu at (-11.6, -25.1)
- added R1011: 49k9/.1%, Resistor_SMD:R_0805_2012Metric_Pad1.20x1.40mm_HandSolder, F.Cu at (-32.5, -5.98)
- added R1012: 20k/.1%, Resistor_SMD:R_0805_2012Metric_Pad1.20x1.40mm_HandSolder, F.Cu at (-26.5, -16.2)
- added R1013: 10k/.1%, Resistor_SMD:R_0805_2012Metric_Pad1.20x1.40mm_HandSolder, F.Cu at (-21.2, -24.2)
- added R1014: 10k/.1%, Resistor_SMD:R_0805_2012Metric_Pad1.20x1.40mm_HandSolder, F.Cu at (-11.1, -28.0)
- added R1015: 4k99, Resistor_SMD:R_0603_1608Metric_Pad0.98x0.95mm_HandSolder, F.Cu at (-23.5, -4.33)
- added R1016: 4k99/.1%, Resistor_SMD:R_0805_2012Metric_Pad1.20x1.40mm_HandSolder, F.Cu at (160.0, 67.2)
- added R1017: 4k99/.1%, Resistor_SMD:R_0805_2012Metric_Pad1.20x1.40mm_HandSolder, F.Cu at (-15.8, -28.9)
- added R1018: 10k/.1%, Resistor_SMD:R_0805_2012Metric_Pad1.20x1.40mm_HandSolder, F.Cu at (-16.4, -23.0)
- added R1019: 10k/.1%, Resistor_SMD:R_0805_2012Metric_Pad1.20x1.40mm_HandSolder, F.Cu at (-8.62, -33.9)
- added R1020: 15k, Resistor_SMD:R_0603_1608Metric_Pad0.98x0.95mm_HandSolder, F.Cu at (-14.1, -9.08)
- added R1021: 10k/.1%, Resistor_SMD:R_0805_2012Metric_Pad1.20x1.40mm_HandSolder, F.Cu at (-31.5, -11.9)
- added R1022: 20k/.1%, Resistor_SMD:R_0805_2012Metric_Pad1.20x1.40mm_HandSolder, F.Cu at (-37.2, -5.72)
- added R1023: 499/.25W/.1%, Resistor_SMD:R_0805_2012Metric_Pad1.20x1.40mm_HandSolder, F.Cu at (-20.1, -20.0)
- added R1024: 10k/.1%, Resistor_SMD:R_0805_2012Metric_Pad1.20x1.40mm_HandSolder, F.Cu at (-16.4, -25.9)
- added R1025: 10k/.1%, Resistor_SMD:R_0805_2012Metric_Pad1.20x1.40mm_HandSolder, F.Cu at (-43.8, 0.91)
- added R1026: 22k1/.1%, Resistor_SMD:R_0805_2012Metric_Pad1.20x1.40mm_HandSolder, F.Cu at (-39.0, -2.71)
- added R1027: 300k/.1%, Resistor_SMD:R_0805_2012Metric_Pad1.20x1.40mm_HandSolder, F.Cu at (-32.2, -8.93)
- added R1028: 10k/.1%, Resistor_SMD:R_0805_2012Metric_Pad1.20x1.40mm_HandSolder, F.Cu at (-3.87, -37.2)
- added R1029: 100/1W/.5%, Resistor_SMD:R_2512_6332Metric_Pad1.40x3.35mm_HandSolder, F.Cu at (-29.0, -39.2)
- added R1030: 10k/.1%, Resistor_SMD:R_0805_2012Metric_Pad1.20x1.40mm_HandSolder, F.Cu at (1.64, -40.2)
- added R1031: 4k99/.1%, Resistor_SMD:R_0805_2012Metric_Pad1.20x1.40mm_HandSolder, F.Cu at (-39.0, 0.24)
- added R1032: 10k/.1%, Resistor_SMD:R_0805_2012Metric_Pad1.20x1.40mm_HandSolder, F.Cu at (-11.1, -31.0)
- added R1033: 2k, Resistor_SMD:R_0603_1608Metric_Pad0.98x0.95mm_HandSolder, F.Cu at (-6.80, -16.6)
- added R1034: 100/1W/.5%, Resistor_SMD:R_2512_6332Metric_Pad1.40x3.35mm_HandSolder, F.Cu at (-47.1, -27.8)
- added R1035: 2k, Resistor_SMD:R_0805_2012Metric_Pad1.20x1.40mm_HandSolder, F.Cu at (-24.9, -19.1)
- added R1036: 4k99/.1%, Resistor_SMD:R_0805_2012Metric_Pad1.20x1.40mm_HandSolder, F.Cu at (-3.11, -40.2)
- added R1037: 10k/.1%, Resistor_SMD:R_0805_2012Metric_Pad1.20x1.40mm_HandSolder, F.Cu at (-29.6, -19.1)
- added R1038: 2/1W/.5%, Resistor_SMD:R_2512_6332Metric_Pad1.40x3.35mm_HandSolder, F.Cu at (-39.9, -34.3)
- added R1039: 2/1W/.5%, Resistor_SMD:R_2512_6332Metric_Pad1.40x3.35mm_HandSolder, F.Cu at (-38.1, -39.2)
- added R1040: 10k/.1%, Resistor_SMD:R_0805_2012Metric_Pad1.20x1.40mm_HandSolder, F.Cu at (-37.0, -8.93)
- added R1041: 100k/.1%, Resistor_SMD:R_0805_2012Metric_Pad1.20x1.40mm_HandSolder, F.Cu at (-8.62, -36.9)
- added R1042: 100k/.1%, Resistor_SMD:R_0805_2012Metric_Pad1.20x1.40mm_HandSolder, F.Cu at (-15.8, -31.8)
- added R1043: 2k, Resistor_SMD:R_0603_1608Metric_Pad0.98x0.95mm_HandSolder, F.Cu at (-2.45, -20.7)
- added R1044: 2k, Resistor_SMD:R_0603_1608Metric_Pad0.98x0.95mm_HandSolder, F.Cu at (-11.1, -16.6)
- added R1045: 100k/.1%, Resistor_SMD:R_0805_2012Metric_Pad1.20x1.40mm_HandSolder, F.Cu at (-43.8, -2.04)
- added R1046: 100k/.1%, Resistor_SMD:R_0805_2012Metric_Pad1.20x1.40mm_HandSolder, F.Cu at (-31.3, -14.9)
- added R1047: 10k/.1%, Resistor_SMD:R_0805_2012Metric_Pad1.20x1.40mm_HandSolder, F.Cu at (-36.3, -11.9)
- added R1048: 1k/.1%, Resistor_SMD:R_0603_1608Metric_Pad0.98x0.95mm_HandSolder, F.Cu at (1.90, -22.4)
- added R1049: 10k, Resistor_SMD:R_0603_1608Metric_Pad0.98x0.95mm_HandSolder, F.Cu at (-12.8, -11.6)
- added R1050: 10k, Resistor_SMD:R_0603_1608Metric_Pad0.98x0.95mm_HandSolder, F.Cu at (2.25, -25.0)
- added R1301: 10k, Resistor_SMD:R_0603_1608Metric_Pad0.98x0.95mm_HandSolder, F.Cu at (-47.9, 26.2)
- added R1302: 10k, Resistor_SMD:R_0603_1608Metric_Pad0.98x0.95mm_HandSolder, F.Cu at (-37.3, 15.7)
- added R1303: 0, Resistor_SMD:R_0603_1608Metric_Pad0.98x0.95mm_HandSolder, F.Cu at (-57.1, 34.5)
- added R1304: 1k, Resistor_SMD:R_0603_1608Metric_Pad0.98x0.95mm_HandSolder, F.Cu at (-47.9, 23.7)
- added R1305: 4k22, Resistor_SMD:R_0603_1608Metric_Pad0.98x0.95mm_HandSolder, F.Cu at (-37.3, 13.2)
- added R1306: 0, Resistor_SMD:R_0603_1608Metric_Pad0.98x0.95mm_HandSolder, F.Cu at (-56.6, 27.0)
- added R1307: 3k9, Resistor_SMD:R_0603_1608Metric_Pad0.98x0.95mm_HandSolder, F.Cu at (-54.1, 23.4)
- added R1308: 300, Resistor_SMD:R_0603_1608Metric_Pad0.98x0.95mm_HandSolder, F.Cu at (-30.2, 7.38)
- added R1309: 300, Resistor_SMD:R_0603_1608Metric_Pad0.98x0.95mm_HandSolder, F.Cu at (-44.9, 18.7)
- added R1310: 1k96, Resistor_SMD:R_0603_1608Metric_Pad0.98x0.95mm_HandSolder, F.Cu at (-34.8, 28.3)
- added R1311: 1k96, Resistor_SMD:R_0603_1608Metric_Pad0.98x0.95mm_HandSolder, F.Cu at (-39.2, 23.7)
- added R1312: 1k/.1%, Resistor_SMD:R_0805_2012Metric_Pad1.20x1.40mm_HandSolder, F.Cu at (-46.2, 14.2)
- added R1313: 1k/.1%, Resistor_SMD:R_0805_2012Metric_Pad1.20x1.40mm_HandSolder, F.Cu at (-66.0, 33.7)
- added R1314: 0, Resistor_SMD:R_0603_1608Metric_Pad0.98x0.95mm_HandSolder, F.Cu at (-25.9, 7.38)
- added R1315: 1k/.1%, Resistor_SMD:R_0805_2012Metric_Pad1.20x1.40mm_HandSolder, F.Cu at (-39.1, 7.60)
- added R1316: 9k/.1%, Resistor_SMD:R_0805_2012Metric_Pad1.20x1.40mm_HandSolder, F.Cu at (-45.1, 10.9)
- added R1317: 3k9, Resistor_SMD:R_0603_1608Metric_Pad0.98x0.95mm_HandSolder, F.Cu at (-57.1, 32.0)
- added R1318: 10k, Resistor_SMD:R_0603_1608Metric_Pad0.98x0.95mm_HandSolder, F.Cu at (-39.2, 28.7)
- added R1319: 10k, Resistor_SMD:R_0603_1608Metric_Pad0.98x0.95mm_HandSolder, F.Cu at (-28.6, 12.4)
- added R1320: 0, Resistor_SMD:R_0603_1608Metric_Pad0.98x0.95mm_HandSolder, F.Cu at (-52.2, 28.5)
- added R1321: 1k, Resistor_SMD:R_0603_1608Metric_Pad0.98x0.95mm_HandSolder, F.Cu at (-36.2, 18.3)
- added R1322: 0, Resistor_SMD:R_0603_1608Metric_Pad0.98x0.95mm_HandSolder, F.Cu at (-47.9, 28.7)
- added R1323: 24k9, Resistor_SMD:R_0603_1608Metric_Pad0.98x0.95mm_HandSolder, F.Cu at (-43.5, 26.2)
- added R1324: 100k, Resistor_SMD:R_0603_1608Metric_Pad0.98x0.95mm_HandSolder, F.Cu at (-32.9, 15.3)
- added R1325: 33k2, Resistor_SMD:R_0603_1608Metric_Pad0.98x0.95mm_HandSolder, F.Cu at (-40.6, 21.2)
- added R1326: 10k, Resistor_SMD:R_0603_1608Metric_Pad0.98x0.95mm_HandSolder, F.Cu at (145.8, 87.7)
- added R1327: 10k, Resistor_SMD:R_0603_1608Metric_Pad0.98x0.95mm_HandSolder, F.Cu at (150.1, 85.2)
- added R1328: 4k7, Resistor_SMD:R_0603_1608Metric_Pad0.98x0.95mm_HandSolder, F.Cu at (147.1, 90.2)
- added R1329: 4k7, Resistor_SMD:R_0603_1608Metric_Pad0.98x0.95mm_HandSolder, F.Cu at (146.2, 92.7)
- added TP1001: TP+OUT, TestPoint:TestPoint_Loop_D2.60mm_Drill1.6mm_Beaded, F.Cu at (-53.7, -0.99)
- added TP1002: TP+GUA, TestPoint:TestPoint_Loop_D2.60mm_Drill1.6mm_Beaded, F.Cu at (-48.7, -0.99)
- added TP1003: TP-OUT, TestPoint:TestPoint_Loop_D2.60mm_Drill1.6mm_Beaded, F.Cu at (-13.5, -35.8)
- added TP1004: TP-SEN, TestPoint:TestPoint_Loop_D2.60mm_Drill1.6mm_Beaded, F.Cu at (-34.5, -18.9)
- added TP1005: TPVM, TestPoint:TestPoint_Loop_D2.60mm_Drill1.6mm_Beaded, F.Cu at (-20.7, -32.7)
- added TP1006: TP+SEN, TestPoint:TestPoint_Loop_D2.60mm_Drill1.6mm_Beaded, F.Cu at (-26.1, -26.1)
- added TP1007: TPIM, TestPoint:TestPoint_Loop_D2.60mm_Drill1.6mm_Beaded, F.Cu at (-41.9, -9.72)
- added TP901: TPDAC, TestPoint:TestPoint_Loop_D2.60mm_Drill1.6mm_Beaded, F.Cu at (-14.7, 8.65)
- added U1001: OPA2140, Package_SO:SOIC-8_3.9x4.9mm_P1.27mm, F.Cu at (-48.6, -13.2)
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Connections:
- net /Control/CL+ renamed /Analog/CL+
- net /Control/CL- renamed /Analog/CL-
- J601 pad A2: (no net) -> /Connector/A
- J601 pad A3: (no net) -> /Connector/B
- J601 pad A4: (no net) -> /Connector/C
- J601 pad A5: (no net) -> /Connector/D
- J601 pad A6: (no net) -> /Connector/E
- J601 pad A7: (no net) -> /Connector/F
- J601 pad C2: (no net) -> /Connector/A
- J601 pad C3: (no net) -> /Connector/B
- J601 pad C4: (no net) -> /Connector/C
- J601 pad C5: (no net) -> /Connector/D
- J601 pad C6: (no net) -> /Connector/E
- J601 pad C7: (no net) -> /Connector/F
- U902 pad 1: (no net) -> /Analog/VM
- U905 pad 1: (no net) -> /Analog/FDACN
- U907 pad 1: (no net) -> /Analog/IM
- U908 pad 7: (no net) -> Net-(TP901-Pad1)

Commit message: PCB layout
Parts:
- C201, C202, C203, C204, C205, C206, C207, C208, C401, C402, C403, C404, C406, C407, C409, C411, C412, C413, C414, C701, C704, FB401, R201, R202, R206, R401, R402, R403, R404, R409, R410, R411, R413, R414, R415, R416, R417, R418, R419, R420, R702, R704: moved to B.Cu
- K1001, K1002: value EE2-5NU -> TQ2SA-5V; footprint Relay_SMD:Relay_DPDT_Kemet_EE2_NU -> ETH1CSMU1:SA
- moved C704 246.7 mm to (186.8, 142.1)
- moved R704 241.4 mm to (176.7, 135.1), turned to 270 degrees
- moved D701 231.1 mm to (212.9, 131.8), turned to 90 degrees
- moved U701 229.5 mm to (214.5, 123.3)
- moved R702 228.5 mm to (176.7, 128.8), turned to 270 degrees
- moved R703 219.5 mm to (213.0, 127.4), turned to 90 degrees
- moved D703 215.4 mm to (216.2, 127.4), turned to 90 degrees
- moved R701 209.9 mm to (214.5, 120.3)
- moved C701 205.7 mm to (186.8, 121.8)
- moved U601 202.8 mm to (206.2, 81.7)
- moved R416 193.1 mm to (192.4, 115.8), turned to 180 degrees
- moved R420 190.8 mm to (179.1, 113.9), turned to 90 degrees
- moved R404 187.9 mm to (188.3, 113.7), turned to 180 degrees
- moved C405 187.8 mm to (183.9, 113.9), turned to 270 degrees
- moved C408 187.7 mm to (174.2, 105.7), turned to 180 degrees
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Connections:
- K1001 pad 10: (no net) -> /Analog/REL1
- K1001 pad 3: (no net) -> Net-(C1002-Pad1)
- K1001 pad 4: Net-(C1002-Pad1) -> /Analog/+OUT
- K1001 pad 5: /Analog/+OUT -> (no net)
- K1001 pad 8: /Analog/+GUA -> /Analog/+GUARD
- K1001 pad 9: /Analog/+GUARD -> (no net)
- K1002 pad 10: Net-(C1002-Pad1) -> /Analog/REL2
- K1002 pad 3: OCOM -> Net-(C1014-Pad1)
- K1002 pad 4: Net-(C1014-Pad1) -> /Analog/-SEN
- K1002 pad 5: /Analog/-SEN -> (no net)
- K1002 pad 8: /Analog/+SEN -> Net-(K1002-Pad8)
- K1002 pad 9: Net-(K1002-Pad9) -> Net-(C1002-Pad1)
- R1016 pad 1: Net-(K1002-Pad9) -> Net-(K1002-Pad8)

Commit message: Design
Parts:
- C509, C511, C519, C808, C817, C818, C819, C820: moved to B.Cu
- moved C501 301.0 mm to (138.2, 176.9)
- moved C502 301.0 mm to (130.2, 172.6)
- moved C503 301.0 mm to (132.6, 169.4)
- moved C508 301.0 mm to (141.3, 169.6)
- moved C510 301.0 mm to (134.5, 174.4)
- moved C512 301.0 mm to (141.3, 164.6)
- moved C513 301.0 mm to (131.7, 184.9)
- moved C514 301.0 mm to (145.6, 169.6)
- moved C515 301.0 mm to (131.7, 182.4)
- moved C516 301.0 mm to (127.4, 184.9)
- moved C517 301.0 mm to (145.6, 167.1)
- moved C518 301.0 mm to (127.4, 182.4)
- moved C520 301.0 mm to (135.3, 163.8)
- moved C521 301.0 mm to (118.7, 183.9)
- moved D502 301.0 mm to (132.6, 166.8)
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
Commit message: PCB and schematic design.
Parts:
- removed R1328, R1329: 4k7, Resistor_SMD:R_0603_1608Metric_Pad0.98x0.95mm_HandSolder
- removed U1301: DG419LDY, Package_SO:SOIC-8_3.9x4.9mm_P1.27mm
- removed U1313: 24LC08B-E/MS, Package_SO:MSOP-8_3x3mm_P0.65mm
- removed U1314: TL072, Package_SO:SOIC-8_3.9x4.9mm_P1.27mm
- added C1201: 100n, Capacitor_SMD:C_0603_1608Metric_Pad1.08x0.95mm_HandSolder, F.Cu at (46.9, 12.6)
- added C1202: 100n, Capacitor_SMD:C_0603_1608Metric_Pad1.08x0.95mm_HandSolder, F.Cu at (55.6, 15.5)
- added C1203: 100n, Capacitor_SMD:C_0603_1608Metric_Pad1.08x0.95mm_HandSolder, F.Cu at (63.1, 6.52)
- added C1204: 100n, Capacitor_SMD:C_0603_1608Metric_Pad1.08x0.95mm_HandSolder, F.Cu at (64.1, 4.01)
- added C1205: 100n, Capacitor_SMD:C_0603_1608Metric_Pad1.08x0.95mm_HandSolder, F.Cu at (55.6, 12.9)
- added C1206: 100n, Capacitor_SMD:C_0603_1608Metric_Pad1.08x0.95mm_HandSolder, F.Cu at (68.5, -1.01)
- added C1207: 100n, Capacitor_SMD:C_0603_1608Metric_Pad1.08x0.95mm_HandSolder, F.Cu at (69.0, -3.52)
- added C1208: 100n, Capacitor_SMD:C_0603_1608Metric_Pad1.08x0.95mm_HandSolder, F.Cu at (55.6, 10.4)
- added C1209: 100n, Capacitor_SMD:C_0603_1608Metric_Pad1.08x0.95mm_HandSolder, F.Cu at (50.1, 7.92)
- added C1210: 100n, Capacitor_SMD:C_0603_1608Metric_Pad1.08x0.95mm_HandSolder, F.Cu at (64.6, -3.52)
- added C1211: 100n, Capacitor_SMD:C_0603_1608Metric_Pad1.08x0.95mm_HandSolder, F.Cu at (46.9, 15.1)
- added C1212: 100n, Capacitor_SMD:C_0603_1608Metric_Pad1.08x0.95mm_HandSolder, F.Cu at (54.4, 7.92)
- added C1213: 100n, Capacitor_SMD:C_0603_1608Metric_Pad1.08x0.95mm_HandSolder, F.Cu at (59.8, 1.13)
- added C1214: 100n, Capacitor_SMD:C_0603_1608Metric_Pad1.08x0.95mm_HandSolder, F.Cu at (64.6, -6.03)
- added C1215: 100n, Capacitor_SMD:C_0603_1608Metric_Pad1.08x0.95mm_HandSolder, F.Cu at (59.8, -1.38)
- added C1216: 100n, Capacitor_SMD:C_0603_1608Metric_Pad1.08x0.95mm_HandSolder, F.Cu at (69.0, -6.03)
- added C1217: 100n, Capacitor_SMD:C_0603_1608Metric_Pad1.08x0.95mm_HandSolder, F.Cu at (51.2, 10.4)
- added C1218: 100n, Capacitor_SMD:C_0603_1608Metric_Pad1.08x0.95mm_HandSolder, F.Cu at (59.8, 3.64)
- added C1219: 100n, Capacitor_SMD:C_0603_1608Metric_Pad1.08x0.95mm_HandSolder, F.Cu at (64.1, -1.01)
- added C1220: 100n, Capacitor_SMD:C_0603_1608Metric_Pad1.08x0.95mm_HandSolder, F.Cu at (51.2, 12.9)
- added C1221: 100n, Capacitor_SMD:C_0603_1608Metric_Pad1.08x0.95mm_HandSolder, F.Cu at (58.8, 7.92)
- added C1222: 100n, Capacitor_SMD:C_0603_1608Metric_Pad1.08x0.95mm_HandSolder, F.Cu at (51.2, 15.5)
- added C1223: 100n, Capacitor_SMD:C_0603_1608Metric_Pad1.08x0.95mm_HandSolder, F.Cu at (64.1, 1.50)
- added C1224: 100n, Capacitor_SMD:C_0603_1608Metric_Pad1.08x0.95mm_HandSolder, F.Cu at (68.5, 1.50)
- added C1225: 100n, Capacitor_SMD:C_0603_1608Metric_Pad1.08x0.95mm_HandSolder, F.Cu at (64.3, 11.5)
- added C1226: 100n, Capacitor_SMD:C_0603_1608Metric_Pad1.08x0.95mm_HandSolder, F.Cu at (64.3, 9.03)
- added C1227: 100n, Capacitor_SMD:C_0603_1608Metric_Pad1.08x0.95mm_HandSolder, F.Cu at (59.9, 15.5)
- added C1228: 100n, Capacitor_SMD:C_0603_1608Metric_Pad1.08x0.95mm_HandSolder, F.Cu at (67.5, 6.52)
- added C1229: 100n, Capacitor_SMD:C_0603_1608Metric_Pad1.08x0.95mm_HandSolder, F.Cu at (68.5, 4.01)
- added H101: MountingHole, MountingHole:MountingHole_3.2mm_M3_DIN965_Pad, F.Cu at (89.0, 145.0)
- added H102: MountingHole, MountingHole:MountingHole_3.2mm_M3_DIN965_Pad, F.Cu at (89.0, 55.0)
- added H103: MountingHole, MountingHole:MountingHole_3.2mm_M3_DIN965_Pad, F.Cu at (221.0, 55.0)
- added H104: MountingHole, MountingHole:MountingHole_3.2mm_M3_DIN965_Pad, F.Cu at (167.0, 132.0)
- added J1001: Conn_02x12, Connector_PinHeader_2.54mm:PinHeader_2x12_P2.54mm_Vertical, F.Cu at (100.0, 58.0)
- added J801: Conn_02x06_Odd_Even, Connector_PinHeader_2.54mm:PinHeader_2x06_P2.54mm_Vertical, F.Cu at (110.0, 144.0)
- added M101: 60817-096, ETH1CSMU1:60817-096, F.Cu at (73.7, 144.4)
- added R1201: 1k, Resistor_SMD:R_0603_1608Metric_Pad0.98x0.95mm_HandSolder, F.Cu at (59.9, 12.9)
- added R1202: 10k, Resistor_SMD:R_0603_1608Metric_Pad0.98x0.95mm_HandSolder, F.Cu at (59.9, 10.4)
- added U1201: SN74LVC1T45DBV, Package_TO_SOT_SMD:SOT-23-6, F.Cu at (55.2, 4.34)
- added U1202: SN74LVC1T45DBV, Package_TO_SOT_SMD:SOT-23-6, F.Cu at (42.3, 14.5)
- added U1203: SN74LVC1T45DBV, Package_TO_SOT_SMD:SOT-23-6, F.Cu at (60.0, -4.96)
- added U1204: SN74LVC1T45DBV, Package_TO_SOT_SMD:SOT-23-6, F.Cu at (32.6, 14.5)
- added U1205: SN74LVC1T45DBV, Package_TO_SOT_SMD:SOT-23-6, F.Cu at (45.5, 8.99)
- added U1206: SN74LVC1T45DBV, Package_TO_SOT_SMD:SOT-23-6, F.Cu at (50.3, 4.34)
- added U1207: SN74LVC1T45DBV, Package_TO_SOT_SMD:SOT-23-6, F.Cu at (55.2, -0.31)
- added U1208: SN74LVC1T45DBV, Package_TO_SOT_SMD:SOT-23-6, F.Cu at (37.4, 14.5)
- added U1209: SN74LVC1T45DBV, Package_TO_SOT_SMD:SOT-23-6, F.Cu at (45.5, 4.34)
- added U1210: SN74LVC1T45DBV, Package_TO_SOT_SMD:SOT-23-6, F.Cu at (50.3, -0.31)
- added U1211: SN74LVC1T45DBV, Package_TO_SOT_SMD:SOT-23-6, F.Cu at (45.5, -0.31)
- added U1212: SN74LVC1T45DBV, Package_TO_SOT_SMD:SOT-23-6, F.Cu at (55.2, -4.96)
- added U1213: SN74LVC1T45DBV, Package_TO_SOT_SMD:SOT-23-6, F.Cu at (50.3, -4.96)
- added U1214: SN74LVC1T45DBV, Package_TO_SOT_SMD:SOT-23-6, F.Cu at (45.5, -4.96)
- added U1215: MCP23S17_SO, Package_SO:SOIC-28W_7.5x17.9mm_P1.27mm, F.Cu at (154.2, 96.0)
- C1014, C1036, C801, C805, C806, C807, C809, C810, C811, C813, C816, C821, C822, C823, C824, D1003, D801, D802, Q1001, R1038, R1049, R808, Y501: moved to B.Cu
- R1110: renamed from R1310; value 1k96 -> 1k96/.1%
- R1111: renamed from R1311; value 1k96 -> 1k96/.1%
- R1123: renamed from R1323; value 24k9 -> 24k9/.1%
- R1124: renamed from R1324; value 100k -> 100k/.1%
- R1125: renamed from R1325; value 33k2 -> 33k2/.1%
- TP1001, TP1002, TP1003, TP1004, TP1005, TP1006, TP1007, TP901: footprint TestPoint:TestPoint_Loop_D2.60mm_Drill1.6mm_Beaded -> TestPoint:TestPoint_Pad_2.0x2.0mm
- moved U1009 258.6 mm to (178.7, 80.1)
- moved U1012 247.9 mm to (175.4, 74.2)
- moved D1003 243.9 mm to (189.5, 64.4), turned to 180 degrees
- moved R1026 238.4 mm to (185.0, 78.7)
- moved U1002 237.6 mm to (154.9, 71.4)
- moved R1027 235.3 mm to (185.0, 81.5)
- moved U1006 233.2 mm to (183.9, 74.2)
- moved Q1001 227.1 mm to (189.5, 60.6), turned to 270 degrees
- moved R1037 224.9 mm to (177.2, 69.3), turned to 180 degrees
- moved U1005 224.8 mm to (154.9, 59.4)
- moved C1014 223.0 mm to (177.2, 69.3), turned to 180 degrees
- moved R1039 221.8 mm to (161.8, 57.0), turned to 270 degrees
- moved R1038 221.4 mm to (161.8, 57.0), turned to 270 degrees
- moved D1005 221.3 mm to (194.3, 69.2), turned to 180 degrees
- moved R1019 220.0 mm to (185.7, 69.2), turned to 180 degrees
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- renumbered C1301 to C1101, C1302 to C1102, C1303 to C1103, C1304 to C1104, C1305 to C1105, C1306 to C1106, C1307 to C1107, C1308 to C1108, C1309 to C1109, C1310 to C1110, C1311 to C1111, C1312 to C1112, C1313 to C1113, C1314 to C1114, C1315 to C1115, C1316 to C1116, C1317 to C1117, C1318 to C1118, C1319 to C1119, C1320 to C1120, C1321 to C1121, C1322 to C1122, C1323 to C1123, C1324 to C1124, C1325 to C1125, C1326 to C1126, C1327 to C1127, C1328 to C1128, C1329 to C1129, C1330 to C1130, C1331 to C1131, C1332 to C1132, C1333 to C1133, C1334 to C1134, C1335 to C1135, C1336 to C1136, C1337 to C1137, C1338 to C1138, C1339 to C1139, C1340 to C1140, C1341 to C1141, C1342 to C1142, C1343 to C1143, C1344 to C1144, C1345 to C1145, C1346 to C1146, C1347 to C1147, C1348 to C1148, C1349 to C1149, C1350 to C1150, C1351 to C1151, C1352 to C1152, D1301 to D1101, D1302 to D1102, FB1301 to FB1101, J1301 to J1101, L1301 to L1101, L1302 to L1102, L1303 to L1103, R1301 to R1101, R1302 to R1102, R1303 to R1103, R1304 to R1104, R1305 to R1105, R1306 to R1106, R1307 to R1107, R1308 to R1108, R1309 to R1109, R1312 to R1112, R1313 to R1113, R1314 to R1114, R1315 to R1115, R1316 to R1116, R1317 to R1117, R1318 to R1118, R1319 to R1119, R1320 to R1120, R1321 to R1121, R1322 to R1122, R1326 to R1126, R1327 to R1127, U1315 to U1101, U1302 to U1102, U1303 to U1103, U1304 to U1104, U1305 to U1105, U1306 to U1106, U1307 to U1107, U1308 to U1108, U1309 to U1109, U1310 to U1110, U1311 to U1111, U1312 to U1112, Y1301 to Y1101
Connections:
- net /MCU/SWCLK renamed /MCU/TCK_SWCLK
- net /MCU/SWDIO renamed /MCU/TMS_SWDIO
- C1117 pad 1: Net-(C1317-Pad1) -> Net-(C1117-Pad1)
- R1049 pad 2: (no net) -> /Analog/REL2_CTR
- R1050 pad 2: (no net) -> /Analog/REL1_CTR
- R1102 pad 2: Net-(R1302-Pad2) -> Net-(R1102-Pad2)
- R1113 pad 1: Net-(C1317-Pad1) -> Net-(C1117-Pad1)
- U1002 pad 16: (no net) -> /Analog/~1mA
- U1002 pad 8: (no net) -> /Analog/~100uA
- U1002 pad 9: (no net) -> /Analog/~10uA
- U1005 pad 9: (no net) -> /Analog/~LT10mA
- U1009 pad 2: (no net) -> /Analog/~VRANGE
- U1101 pad 1: (no net) -> Net-(C1117-Pad1)
- U1101 pad 2: (no net) -> Net-(R1102-Pad2)
- U1101 pad 6: (no net) -> /Function generator/ANALOG_SWITCH
- U1102 pad 6: Net-(C1317-Pad1) -> Net-(C1117-Pad1)
- U1108 pad 4: (no net) -> -15V
- U1108 pad 8: (no net) -> +15V
- U1112 pad 50: (no net) -> /Function generator/MCU_NSS
- U1112 pad 51: (no net) -> /Function generator/MCU_SCLK
- U1112 pad 52: (no net) -> /Function generator/MCU_MISO
- U1112 pad 53: (no net) -> /Function generator/MCU_MOSI
- U1112 pad 56: /Function generator/EEPROM_WP -> (no net)
- U1112 pad 58: /Function generator/EEPROM_SCL -> (no net)
- U1112 pad 59: /Function generator/EEPROM_SDA -> (no net)
- U501 pad 1: (no net) -> /Control/ADC_HP_SCLK
- U501 pad 110: (no net) -> /Control/ADC_HS_~CS
- U501 pad 111: (no net) -> /Control/ADC_HS_SCLK
- U501 pad 112: (no net) -> /Control/ADC_HS_MISO
- U501 pad 113: (no net) -> /Control/ADC_HS_MOSI
- U501 pad 116: (no net) -> /Connector/CXN_REL1
- U501 pad 117: (no net) -> /Connector/CXN_REL2
- U501 pad 118: (no net) -> /Connector/CXN_REL3
- U501 pad 119: (no net) -> /Connector/CXN_REL4
- U501 pad 122: (no net) -> /Connector/CXN_REL5
- U501 pad 123: (no net) -> /Function generator/MCU_MOSI
- U501 pad 3: (no net) -> /Control/ADC_HP_~CS
- U501 pad 4: (no net) -> /Control/ADC_HP_MISO
- U501 pad 40: (no net) -> /Function generator/MCU_NSS
- U501 pad 41: (no net) -> /Function generator/MCU_SCLK
- U501 pad 42: (no net) -> /Function generator/MCU_MISO
- U501 pad 46: (no net) -> /MCU/TRIG_IN
- U501 pad 47: (no net) -> /MCU/TRIG_OUT
- U501 pad 48: (no net) -> /MCU/TRIG_EN
- U501 pad 5: (no net) -> /Control/ADC_HP_MOSI
- U501 pad 73: /MCU/TRIG_IN -> /Control/DAC_~CS
- U501 pad 74: /MCU/TRIG_OUT -> /Control/DAC_SCLK
- U501 pad 75: /MCU/TRIG_EN -> /Control/DAC_MISO
- U501 pad 76: (no net) -> /Control/DAC_MOSI
- U601 pad 1: (no net) -> /Connector/CXN_REL5
- U601 pad 2: (no net) -> /Connector/CXN_REL4
- U601 pad 3: (no net) -> /Connector/CXN_REL3
- U601 pad 4: (no net) -> /Connector/CXN_REL2
- U601 pad 5: (no net) -> /Connector/CXN_REL1
- U906 pad 23: (no net) -> /Control/ADC_HP_MISO
- U906 pad 24: (no net) -> /Control/ADC_HP_MOSI
- U906 pad 3: (no net) -> /Control/ADC_HP_SCLK
- U906 pad 4: (no net) -> /Control/ADC_HP_~CS
- U908 pad 12: (no net) -> /Control/DAC_SCLK
- U908 pad 13: (no net) -> /Control/DAC_~CS
- U908 pad 14: (no net) -> /Control/DAC_MOSI
- U908 pad 8: (no net) -> /Control/DAC_MISO
- U912 pad 10: (no net) -> /Control/ADC_HS_MOSI

Commit message: PCB layout
Parts:
- C1002, C1003, C1004, C1007, C1008, C1010, C1013, C1015, C1016, C1017, C1018, C1027, C1037, C1120, C1124, C1125, C1127, C1146, C1147, C1148, C1149, C1151, C301, C302, C303, C304, C305, C306, C307, C501, C502, C503, C504, C505, C506, C507, C508, C510, C512, C513, C514, C515, C516, C517, C518, C520, C522, C804, C812, D1001, FB1101, FB501, Q1002, R1019, R1022, R1029, R1036, R1050, R1127, R501, R502, R503, R505, R506, R507, R508, R509, R510, R804, Y1101: moved to B.Cu
- C1014: moved to F.Cu
- moved U1111 235.0 mm to (91.9, 181.6)
- moved C1013 230.3 mm to (192.3, 75.1), turned to 270 degrees
- moved R1034 224.1 mm to (159.3, 59.6), turned to 180 degrees
- moved C1016 223.7 mm to (189.9, 75.1), turned to 90 degrees
- moved R1025 222.7 mm to (168.4, 68.5)
- moved D1007 222.3 mm to (188.6, 69.5)
- moved D1006 221.2 mm to (184.4, 69.5)
- moved C1017 220.6 mm to (194.8, 75.1), turned to 270 degrees
- moved U1107 217.4 mm to (132.1, 99.2), turned to 90 degrees
- moved R1040 216.0 mm to (160.8, 78.0), turned to 180 degrees
- moved C1037 215.8 mm to (174.2, 55.0), turned to 180 degrees
- moved R1013 214.7 mm to (172.5, 68.5)
- moved D1001 214.5 mm to (174.2, 64.4), turned to 180 degrees
- moved C1005 213.4 mm to (165.4, 55.6), turned to 270 degrees
- moved R1029 212.6 mm to (159.3, 59.6), turned to 180 degrees
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Connections:
- J1001 pad 1: Net-(C1002-Pad2) -> (no net)
- J1001 pad 10: /Analog/AMPIN -> +15VH
- J1001 pad 15: +15VH -> /Analog/AMPIN
- J1001 pad 16: +15VH -> /Analog/AMPIN
- J1001 pad 17: OCOM -> -15V
- J1001 pad 18: OCOM -> -15V
- J1001 pad 19: -15VH -> GND
- J1001 pad 2: Net-(C1002-Pad2) -> (no net)
- J1001 pad 20: -15VH -> GND
- J1001 pad 21: (no net) -> +15V
- J1001 pad 22: (no net) -> +15V
- J1001 pad 23: (no net) -> Net-(C1002-Pad2)
- J1001 pad 24: (no net) -> Net-(C1002-Pad2)
- J1001 pad 3: +15V -> (no net)
- J1001 pad 4: +15V -> (no net)
- J1001 pad 5: GND -> -15VH
- J1001 pad 6: GND -> -15VH
- J1001 pad 7: -15V -> OCOM
- J1001 pad 8: -15V -> OCOM
- J1001 pad 9: /Analog/AMPIN -> +15VH

Commit message: PCB layout
Parts:
- added J1002: Conn_02x06, Connector_PinHeader_2.54mm:PinHeader_2x06_P2.54mm_Vertical, F.Cu at (110.0, 58.0)
- C1003: moved to F.Cu
- J1001: value Conn_02x12 -> Conn_02x02; footprint Connector_PinHeader_2.54mm:PinHeader_2x12_P2.54mm_Vertical -> Connector_PinHeader_2.54mm:PinHeader_2x02_P2.54mm_Vertical
- U901: value DG419LDY -> CPC1018N; footprint Package_SO:SOIC-8_3.9x4.9mm_P1.27mm -> Package_SO:SOP-4_3.8x4.1mm_P2.54mm
- moved D1004 178.2 mm to (129.9, 87.5), turned to 90 degrees
- moved U910 120.8 mm to (114.0, 70.6)
- moved U903 119.9 mm to (101.3, 77.7), turned to 180 degrees
- moved U901 105.8 mm to (105.9, 70.9)
- moved J1001 71.5 mm to (167.0, 83.0)
- moved U912 36.6 mm to (92.1, 87.0)
- moved U914 36.5 mm to (92.1, 93.7)
- moved U916 26.1 mm to (57.3, 84.8)
- moved U904 26.0 mm to (105.9, 63.9)
- moved U902 22.9 mm to (110.5, 94.0)
- moved U907 22.7 mm to (110.5, 87.5)
- moved U905 18.5 mm to (114.0, 63.9)
- moved U915 14.7 mm to (92.1, 70.5)
- moved U906 11.9 mm to (92.1, 78.9)
- moved U908 11.8 mm to (92.1, 63.9)
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Connections:
- J1001 pad 1: (no net) -> OCOM
- J1001 pad 2: (no net) -> -15VH
- J1001 pad 3: (no net) -> OCOM
- J1001 pad 4: (no net) -> +15VH

Commit message: PCB and schematic
Parts:
- moved U1215 105.2 mm to (49.0, 96.0)
- moved U916 26.2 mm to (83.2, 80.4)
- moved U902 12.9 mm to (101.5, 84.7)
- moved U907 9.79 mm to (101.5, 91.3)
- moved U915 9.09 mm to (83.2, 72.4)
- moved J1001 6.71 mm to (164.0, 89.0)
- moved U906 6.60 mm to (92.1, 72.3)
- moved U912 6.60 mm to (92.1, 80.4)
- moved U914 6.60 mm to (92.1, 87.1)
- moved U601 4.65 mm to (203.0, 81.4)
- moved U901 3.57 mm to (102.4, 71.1)
- moved U904 3.57 mm to (102.4, 64.1)
- moved U905 3.57 mm to (110.5, 64.1)
- moved U910 3.57 mm to (110.5, 70.9)
- moved U903 0.13 mm to (101.5, 77.7)
Connections:
- net /GPIO/MCU_10mA renamed /GPIO/GPIO_10-100mA
- J1002 pad 1: (no net) -> /Analog/10-100mA
- J1002 pad 2: (no net) -> /Analog/10-100mA
- U1201 pad 3: /Analog/10mA -> /Analog/10-100mA

Commit message: PCB layout
Parts:
- C1005, C1009, R920, R926: moved to B.Cu
- moved R926 125.5 mm to (104.9, 65.7), turned to 270 degrees
- moved R920 107.8 mm to (108.0, 69.6), turned to 270 degrees
- moved D1004 20.5 mm to (116.6, 71.9)
- moved C1009 16.7 mm to (181.2, 64.7)
- moved C1005 16.7 mm to (181.2, 60.7)
- moved C1037 1.14 mm to (173.1, 55.0)
- moved D1001 1.14 mm to (173.1, 64.4)
- moved K1001 1.14 mm to (173.1, 59.3)
- moved Q1002 1.14 mm to (173.1, 60.6)
- moved R1050 1.14 mm to (173.1, 57.3)
- moved U904 0.25 mm to (102.4, 63.9)
- moved U905 0.25 mm to (110.5, 63.9)
