File: HARDWARE/BASE/Power_Float.sch (KiCad schematic (older format))
At the start: 46 parts, among them U901 LT8330_S6, U902 LT8330_S6, U903 MC7815BD2TG, U904 MC7915BD2TG, U905 TSR1-2490, U906 TSR1-2450, U907 LM1117DTX-5.0/NOPB, U908 LM1117DTX-3.3/NOPB

Commit message: Schematic design
Parts:
- renumbered C907 to C901, C901 to C902, C909 to C904, C911 to C905, C913 to C906, C915 to C907, C918 to C908, C920 to C909, C921 to C910, C923 to C911, C905 to C912, C908 to C913, C902 to C914, C904 to C915, C910 to C916, C919 to C918, C922 to C919, C924 to C920, C912 to C921, C914 to C922, C916 to C923, C906 to C924, D902 to D901, D901 to D902, L904 to L902, L902 to L903, L903 to L904, R905 to R902, R902 to R903, R906 to R904, R903 to R905, R907 to R906, R904 to R907, U903 to U901, U907 to U902, U905 to U903, U901 to U904, U904 to U905, U908 to U906, U906 to U907, U902 to U908

Commit message: Schematic design.
Parts:
- renumbered C901 to C801, C902 to C802, C903 to C803, C904 to C804, C905 to C805, C906 to C806, C907 to C807, C908 to C808, C909 to C809, C910 to C810, C911 to C811, C912 to C812, C913 to C813, C914 to C814, C915 to C815, C916 to C816, C917 to C817, C918 to C818, C919 to C819, C920 to C820, C921 to C821, C922 to C822, C923 to C823, C924 to C824, D901 to D801, D902 to D802, L901 to L801, L902 to L802, L903 to L803, L904 to L804, R901 to R801, R902 to R802, R903 to R803, R904 to R804, R905 to R805, R906 to R806, R907 to R807, R908 to R808, U901 to U801, U902 to U802, U903 to U803, U904 to U804, U905 to U805, U906 to U806, U907 to U807, U908 to U808

Commit message: PCB and schematic design.
Parts:
- added J801: Conn_02x06_Odd_Even, Connector_PinHeader_2.54mm:PinHeader_2x06_P2.54mm_Vertical, symbol Connector_Generic:Conn_02x06_Odd_Even
Connections:
- net +24VF: now also J801.1 (Pin_1), J801.2 (Pin_2), J801.3 (Pin_3), J801.4 (Pin_4)
- net +5V: now also J801.7 (Pin_7), J801.8 (Pin_8)
- net GND: now also J801.10 (Pin_10), J801.11 (Pin_11), J801.12 (Pin_12), J801.9 (Pin_9)
- no-connect marks 0 -> 2
Changed lines of the file:
@@
 	1    0    0    -1
 $EndComp
+$Comp
+L Connector_Generic:Conn_02x06_Odd_Even J801
+U 1 1 60BE4445
+P 2100 6750
+F 0 "J801" H 2150 7167 50  0000 C CNN
+F 1 "Conn_02x06_Odd_Even" H 2150 7076 50  0000 C CNN
+F 2 "Connector_PinHeader_2.54mm:PinHeader_2x06_P2.54mm_Vertical" H 2100 6750 50  0001 C CNN
+F 3 "~" H 2100 6750 50  0001 C CNN
+	1    2100 6750
+	1    0    0    -1
+$EndComp
+$Comp
+L power:GND #PWR0825
+U 1 1 60BE7017
+P 1900 7050
+F 0 "#PWR0825" H 1900 6800 50  0001 C CNN
+F 1 "GND" V 1900 6850 50  0000 C CNN
+F 2 "" H 1900 7050 50  0001 C CNN
+F 3 "" H 1900 7050 50  0001 C CNN
+	1    1900 7050
+	0    1    1    0
+$EndComp
+$Comp
+L power:GND #PWR0823
+U 1 1 60BE8D94
+P 1900 6950
+F 0 "#PWR0823" H 1900 6700 50  0001 C CNN
+F 1 "GND" V 1900 6750 50  0000 C CNN
+F 2 "" H 1900 6950 50  0001 C CNN
+F 3 "" H 1900 6950 50  0001 C CNN
+	1    1900 6950
+	0    1    1    0
+$EndComp
+$Comp
+L power:GND #PWR0824
+U 1 1 60BF2C2E
+P 2400 6950
+F 0 "#PWR0824" H 2400 6700 50  0001 C CNN
+F 1 "GND" V 2400 6750 50  0000 C CNN
+F 2 "" H 2400 6950 50  0001 C CNN
+F 3 "" H 2400 6950 50  0001 C CNN
+	1    2400 6950
+	0    -1   -1   0
+$EndComp
+$Comp
+L power:GND #PWR0826
+U 1 1 60BF2EAA
+P 2400 7050
+F 0 "#PWR0826" H 2400 6800 50  0001 C CNN
+F 1 "GND" V 2400 6850 50  0000 C CNN
+F 2 "" H 2400 7050 50  0001 C CNN
+F 3 "" H 2400 7050 50  0001 C CNN
+	1    2400 7050
+	0    -1   -1   0
+$EndComp
+NoConn ~ 1900 6750
+NoConn ~ 2400 6750
+$Comp
+L ETH1CSMU1:+24VF #PWR0817
+U 1 1 60C10E73
+P 1900 6550
+F 0 "#PWR0817" H 1900 6400 50  0001 C CNN
+F 1 "+24VF" V 1900 6800 50  0000 C CNN
+F 2 "" H 1900 6550 50  0001 C CNN
+F 3 "" H 1900 6550 50  0001 C CNN
+	1    1900 6550
+	0    -1   -1   0
+$EndComp
+$Comp
+L ETH1CSMU1:+24VF #PWR0819
+U 1 1 60C13D26
+P 1900 6650
+F 0 "#PWR0819" H 1900 6500 50  0001 C CNN
+F 1 "+24VF" V 1900 6900 50  0000 C CNN
+F 2 "" H 1900 6650 50  0001 C CNN
+F 3 "" H 1900 6650 50  0001 C CNN
+	1    1900 6650
+	0    -1   -1   0
+$EndComp
+$Comp
+L ETH1CSMU1:+24VF #PWR0818
+U 1 1 60C13FF0
+P 2400 6550
+F 0 "#PWR0818" H 2400 6400 50  0001 C CNN
+F 1 "+24VF" V 2400 6800 50  0000 C CNN
+F 2 "" H 2400 6550 50  0001 C CNN
+F 3 "" H 2400 6550 50  0001 C CNN
+	1    2400 6550
+	0    1    1    0
+$EndComp
+$Comp
+L ETH1CSMU1:+24VF #PWR0820
+U 1 1 60C14410
+P 2400 6650
+F 0 "#PWR0820" H 2400 6500 50  0001 C CNN
+F 1 "+24VF" V 2400 6900 50  0000 C CNN
+F 2 "" H 2400 6650 50  0001 C CNN
+F 3 "" H 2400 6650 50  0001 C CNN
+	1    2400 6650
+	0    1    1    0
+$EndComp
+$Comp
+L power:+5V #PWR0821
+U 1 1 60C1600A
+P 1900 6850
+F 0 "#PWR0821" H 1900 6700 50  0001 C CNN
+F 1 "+5V" V 1900 7050 50  0000 C CNN
+F 2 "" H 1900 6850 50  0001 C CNN
+F 3 "" H 1900 6850 50  0001 C CNN
+	1    1900 6850
+	0    -1   -1   0
+$EndComp
+$Comp
+L power:+5V #PWR0822
+U 1 1 60C18A60
+P 2400 6850
+F 0 "#PWR0822" H 2400 6700 50  0001 C CNN
+F 1 "+5V" V 2400 7050 50  0000 C CNN
+F 2 "" H 2400 6850 50  0001 C CNN
+F 3 "" H 2400 6850 50  0001 C CNN
+	1    2400 6850
+	0    1    1    0
+$EndComp
 $EndSCHEMATC

Commit message: Schematic and PCB changes
Connections:
- net DGNDF is gone; now on net GND: D802.1 (K), L801.3
Changed lines of the file:
@@
 	0    -1   -1   0
-$EndComp
-$Comp
-L ETH1CSMU1:DGNDF #PWR0813
-U 1 1 5F7AA41C
-P 3300 4350
-F 0 "#PWR0813" H 3300 4100 50  0001 C CNN
-F 1 "DGNDF" H 3305 4177 50  0000 C CNN
-F 2 "" H 3300 4350 50  0001 C CNN
-F 3 "" H 3300 4350 50  0001 C CNN
-	1    3300 4350
-	1    0    0    -1
 $EndComp
 Connection ~ 3300 3950
@@
 	1    0    0    -1
 $EndComp
-$Comp
-L ETH1CSMU1:DGNDF #PWR0805
-U 1 1 5DF487C8
-P 3350 2000
-F 0 "#PWR0805" H 3350 1750 50  0001 C CNN
-F 1 "DGNDF" H 3355 1827 50  0000 C CNN
-F 2 "" H 3350 2000 50  0001 C CNN
-F 3 "" H 3350 2000 50  0001 C CNN
-	1    3350 2000
-	1    0    0    -1
-$EndComp
 Wire Wire Line
 	4100 4150 4100 4250
@@
 	0    1    1    0
 $EndComp
+$Comp
+L power:GND #PWR0101
+U 1 1 606B009B
+P 3350 2000
+F 0 "#PWR0101" H 3350 1750 50  0001 C CNN
+F 1 "GND" H 3355 1827 50  0000 C CNN
+F 2 "" H 3350 2000 50  0001 C CNN
+F 3 "" H 3350 2000 50  0001 C CNN
+	1    3350 2000
+	1    0    0    -1
+$EndComp
+$Comp
+L power:GND #PWR0102
+U 1 1 606B0F8B
+P 3300 4350
+F 0 "#PWR0102" H 3300 4100 50  0001 C CNN
+F 1 "GND" H 3305 4177 50  0000 C CNN
+F 2 "" H 3300 4350 50  0001 C CNN
+F 3 "" H 3300 4350 50  0001 C CNN
+	1    3300 4350
+	1    0    0    -1
+$EndComp
+$Comp
+L ETH1CSMU1:+24VF #PWR0805
+U 1 1 60B6AAED
+P 5600 7400
+F 0 "#PWR0805" H 5600 7250 50  0001 C CNN
+F 1 "+24VF" H 5615 7573 50  0000 C CNN
+F 2 "" H 5600 7400 50  0001 C CNN
+F 3 "" H 5600 7400 50  0001 C CNN
+	1    5600 7400
+	1    0    0    -1
+$EndComp
+$Comp
+L power:PWR_FLAG #FLG0805
+U 1 1 60B6BC5B
+P 5600 7400
+F 0 "#FLG0805" H 5600 7475 50  0001 C CNN
+F 1 "PWR_FLAG" H 5600 7573 50  0000 C CNN
+F 2 "" H 5600 7400 50  0001 C CNN
+F 3 "~" H 5600 7400 50  0001 C CNN
+	1    5600 7400
+	-1   0    0    1
+$EndComp
+$Comp
+L power:GND #PWR0813
+U 1 1 60BB7026
+P 5150 7400
+F 0 "#PWR0813" H 5150 7150 50  0001 C CNN
+F 1 "GND" H 5155 7227 50  0000 C CNN
+F 2 "" H 5150 7400 50  0001 C CNN
+F 3 "" H 5150 7400 50  0001 C CNN
+	1    5150 7400
+	-1   0    0    1
+$EndComp
+$Comp
+L power:PWR_FLAG #FLG0806
+U 1 1 60BB7A7E
+P 5150 7400
+F 0 "#FLG0806" H 5150 7475 50  0001 C CNN
+F 1 "PWR_FLAG" H 5150 7573 50  0000 C CNN
+F 2 "" H 5150 7400 50  0001 C CNN
+F 3 "~" H 5150 7400 50  0001 C CNN
+	1    5150 7400
+	-1   0    0    1
+$EndComp
 $EndSCHEMATC
