File: HARDWARE/BASE/FGEN.sch (KiCad schematic (older format))
At the start: 79 parts

Commit message: Schematic design
Parts:
- removed R?: 0, Resistor_SMD:R_0603_1608Metric_Pad1.05x0.95mm_HandSolder, symbol Device:R
- removed R? (x2): 1k, Resistor_SMD:R_0603_1608Metric_Pad1.05x0.95mm_HandSolder, symbol Device:R
- removed U?: LT1468, Package_SO:SSOP-8_3.9x5.05mm_P1.27mm, symbol ETH1CSMU1:LT1468
- added C1317, C1321: 5p, Capacitor_SMD:C_0603_1608Metric_Pad1.08x0.95mm_HandSolder, symbol Device:C
- added C1324, C1325: 8p, Capacitor_SMD:C_0603_1608Metric_Pad1.08x0.95mm_HandSolder, symbol Device:C
- added C1326: 2u2, Capacitor_SMD:C_0603_1608Metric_Pad1.08x0.95mm_HandSolder, symbol Device:C
- added C1327, C1344, C1345, C1346, C1347, C1348, C1349, C1351: 100n, Capacitor_SMD:C_0603_1608Metric_Pad1.08x0.95mm_HandSolder, symbol Device:C
- added C1350, C1352: 1u, Capacitor_SMD:C_0603_1608Metric_Pad1.08x0.95mm_HandSolder, symbol Device:C
- added FB1301: 742792031, Inductor_SMD:L_0805_2012Metric_Pad1.15x1.40mm_HandSolder, symbol Device:Ferrite_Bead
- added J1301: 20021111-00010T4LF, Connector_PinHeader_1.27mm:PinHeader_2x05_P1.27mm_Vertical, symbol Connector_Generic:Conn_02x05_Odd_Even
- added R1306: 0, Resistor_SMD:R_0603_1608Metric_Pad0.98x0.95mm_HandSolder, symbol Device:R
- added R1312, R1313, R1315: 1k/.1%, Resistor_SMD:R_0805_2012Metric_Pad1.20x1.40mm_HandSolder, symbol Device:R
- added R1316: 9k/.1%, Resistor_SMD:R_0805_2012Metric_Pad1.20x1.40mm_HandSolder, symbol Device:R
- added R1326, R1327: 10k, Resistor_SMD:R_0603_1608Metric_Pad0.98x0.95mm_HandSolder, symbol Device:R
- added R1328, R1329: 4k7, Resistor_SMD:R_0603_1608Metric_Pad0.98x0.95mm_HandSolder, symbol Device:R
- added U1302, U1303: LM318, Package_SO:SOIC-8_3.9x4.9mm_P1.27mm, symbol Amplifier_Operational:LM318M
- added U1312: STM32F413RGT6Tx, Package_QFP:LQFP-64_10x10mm_P0.5mm, symbol ETH1CSMU1:STM32F413RGT6Tx
- added U1313: 24LC08B-E/MS, Package_SO:MSOP-8_3x3mm_P0.65mm, symbol Memory_EEPROM:24LC08
- added Y1301: NX3225GD-8MHZ-STD-CRA-3, ETH1CSMU1:NX3225GD, symbol Device:Crystal
- C1301, C1302, C1303, C1304, C1305, C1307, C1309, C1310, C1311, C1312, C1313, C1314, C1315, C1316, C1318, C1319, C1320, C1322, C1323, C1328, C1329, C1330, C1331, C1333, C1334, C1335, C1336, C1337, C1338, C1339, C1340, C1341, C1342, C1343: renamed from C?; footprint Capacitor_SMD:C_0603_1608Metric_Pad1.05x0.95mm_HandSolder -> Capacitor_SMD:C_0603_1608Metric_Pad1.08x0.95mm_HandSolder
- C1306: renamed from C?; footprint Capacitor_SMD:C_1206_3216Metric_Pad1.42x1.75mm_HandSolder -> Capacitor_SMD:C_1206_3216Metric_Pad1.33x1.80mm_HandSolder
- C1308, C1332: renamed from C?; footprint Capacitor_SMD:C_0805_2012Metric_Pad1.15x1.40mm_HandSolder -> Capacitor_SMD:C_0805_2012Metric_Pad1.18x1.45mm_HandSolder
- R1301, R1302, R1303, R1304, R1305, R1307, R1308, R1309, R1310, R1311, R1314, R1317, R1318, R1319, R1320, R1321, R1322, R1323, R1324, R1325: renamed from R?; footprint Resistor_SMD:R_0603_1608Metric_Pad1.05x0.95mm_HandSolder -> Resistor_SMD:R_0603_1608Metric_Pad0.98x0.95mm_HandSolder
- gave numbers to parts that had none: 16
Connections:
- net labels added: EEPROM_SCL, EEPROM_SDA, EEPROM_WP, MCU_MISO, MCU_MOSI, MCU_NRST, MCU_NSS, MCU_SCLK, TCK_SWCLK, TMS_SWDIO, VDDA
- net labels removed: +15VF, -15VF, AGNDF, DGNDF
- wire segments 283 -> 448
- no-connect marks 7 -> 37
Other:
- moved on the sheet: C1301, C1302, C1303, C1304, C1305, C1306, C1307, C1308, C1309, C1310, C1311, C1312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

Commit message: Design
Parts:
- renumbered C1301 to C1101, C1302 to C1102, C1303 to C1103, C1304 to C1104, C1305 to C1105, C1306 to C1106, C1307 to C1107, C1308 to C1108, C1309 to C1109, C1310 to C1110, C1311 to C1111, C1312 to C1112, C1313 to C1113, C1314 to C1114, C1315 to C1115, C1316 to C1116, C1317 to C1117, C1318 to C1118, C1319 to C1119, C1320 to C1120, C1321 to C1121, C1322 to C1122, C1323 to C1123, C1324 to C1124, C1325 to C1125, C1326 to C1126, C1327 to C1127, C1328 to C1128, C1329 to C1129, C1330 to C1130, C1331 to C1131, C1332 to C1132, C1333 to C1133, C1334 to C1134, C1335 to C1135, C1336 to C1136, C1337 to C1137, C1338 to C1138, C1339 to C1139, C1340 to C1140, C1341 to C1141, C1342 to C1142, C1343 to C1143, C1344 to C1144, C1345 to C1145, C1346 to C1146, C1347 to C1147, C1348 to C1148, C1349 to C1149, C1350 to C1150, C1351 to C1151, C1352 to C1152, D1301 to D1101, D1302 to D1102, FB1301 to FB1101, J1301 to J1101, L1301 to L1101, L1302 to L1102, L1303 to L1103, R1301 to R1101, R1302 to R1102, R1303 to R1103, R1304 to R1104, R1305 to R1105, R1306 to R1106, R1307 to R1107, R1308 to R1108, R1309 to R1109, R1310 to R1110, R1311 to R1111, R1312 to R1112, R1313 to R1113, R1314 to R1114, R1315 to R1115, R1316 to R1116, R1317 to R1117, R1318 to R1118, R1319 to R1119, R1320 to R1120, R1321 to R1121, R1322 to R1122, R1323 to R1123, R1324 to R1124, R1325 to R1125, R1326 to R1126, R1327 to R1127, R1328 to R1128, R1329 to R1129, U1301 to U1101, U1302 to U1102, U1303 to U1103, U1304 to U1104, U1305 to U1105, U1306 to U1106, U1307 to U1107, U1308 to U1108, U1309 to U1109, U1310 to U1110, U1311 to U1111, U1312 to U1112, U1313 to U1113, U1314 to U1114, U1315 to U1115, Y1301 to Y1101

Commit message: PCB and schematic design.
Parts:
- removed R1128, R1129: 4k7, Resistor_SMD:R_0603_1608Metric_Pad0.98x0.95mm_HandSolder, symbol Device:R
- removed U1113: 24LC08B-E/MS, Package_SO:MSOP-8_3x3mm_P0.65mm, symbol Memory_EEPROM:24LC08
- R1110, R1111: value 1k96 -> 1k96/.1%
- R1123: value 24k9 -> 24k9/.1%
- R1124: value 100k -> 100k/.1%
- R1125: value 33k2 -> 33k2/.1%
- renumbered U1115 to U1101, U1114 to U1108

Commit message: Schematic and PCB changes
Connections:
- net +5VF is gone; now on net +5V: C1102.1, C1107.1, C1108.1, U1106.2 (Vin), U1106.3 (~Sleep~), U1107.15 (AVDD)
- net EEPROM_SCL: no longer names the net of U1112.58 (PB6,LPTIM1_ETR,TIM4_CH1,I2C1_SCL,DFSDM2_CKIN7,USART1_TX,CAN2_TX,QUADSPI_BK1_NCS,UART5_TX,SDIO_D0,EVENTOUT)
- net EEPROM_SDA: no longer names the net of U1112.59 (PB7,LPTIM1_IN2,TIM4_CH2,I2C1_SDA,DFSDM2_DATIN7,USART1_RX,FSMC_NL,EVENTOUT)
- net EEPROM_WP: no longer names the net of U1112.56 (PB4,TRST,TIM3_CH1,SPI1_MISO,SPI3_MISO,I2S3ext_SD,UART7_TX,I2C3_SDA,SAI1_SCK_A,CAN3_TX,SDIO_D0,EVENTOUT)
- no-connect marks 37 -> 40
Changed lines of the file:
@@
-	1    0    0    -1
-$EndComp
-$Comp
-L ETH1CSMU1:+5VF #PWR01107
-U 1 1 5DF82766
-P 17300 2700
-F 0 "#PWR01107" H 17300 2550 50  0001 C CNN
-F 1 "+5VF" H 17315 2873 50  0000 C CNN
-F 2 "" H 17300 2700 50  0001 C CNN
-F 3 "" H 17300 2700 50  0001 C CNN
-	1    17300 2700
 	1    0    0    -1
 $EndComp
@@
 Wire Wire Line
 	4800 2950 4750 2950
-$Comp
-L ETH1CSMU1:+5VF #PWR01111
-U 1 1 5DD2A39C
-P 4800 2950
-F 0 "#PWR01111" H 4800 2800 50  0001 C CNN
-F 1 "+5VF" V 4800 3100 50  0000 L CNN
-F 2 "" H 4800 2950 50  0001 C CNN
-F 3 "" H 4800 2950 50  0001 C CNN
-	1    4800 2950
-	0    1    1    0
-$EndComp
 Wire Wire Line
 	4450 2950 4400 2950
@@
 Wire Wire Line
 	3650 2750 3650 2700
-$Comp
-L ETH1CSMU1:+5VF #PWR01103
-U 1 1 5DD1791A
-P 3950 2650
-F 0 "#PWR01103" H 3950 2500 50  0001 C CNN
-F 1 "+5VF" H 3965 2823 50  0000 C CNN
-F 2 "" H 3950 2650 50  0001 C CNN
-F 3 "" H 3950 2650 50  0001 C CNN
-	1    3950 2650
-	1    0    0    -1
-$EndComp
 $Comp
 L Device:C C?
@@
 Wire Wire Line
 	10300 10900 10300 10950
-Wire Wire Line
-	16150 7800 16650 7800
-Text Label 16650 7800 2    50   ~ 0
-EEPROM_WP
-Text Label 16650 8000 2    50   ~ 0
-EEPROM_SCL
-Text Label 16650 8100 2    50   ~ 0
-EEPROM_SDA
-Wire Wire Line
-	16150 8100 16650 8100
-Wire Wire Line
-	16150 8000 16650 8000
 $Comp
 L Amplifier_Operational:TL072 U1108
@@
 	1    0    0    -1
 $EndComp
+NoConn ~ 16150 8100
+NoConn ~ 16150 7800
+NoConn ~ 16150 8000
+$Comp
+L power:+5V #PWR0128
+U 1 1 60DBE881
+P 3950 2650
+F 0 "#PWR0128" H 3950 2500 50  0001 C CNN
+F 1 "+5V" H 3965 2823 50  0000 C CNN
+F 2 "" H 3950 2650 50  0001 C CNN
+F 3 "" H 3950 2650 50  0001 C CNN
+	1    3950 2650
+	1    0    0    -1
+$EndComp
+$Comp
+L power:+5V #PWR0129
+U 1 1 60DC03EB
+P 4800 2950
+F 0 "#PWR0129" H 4800 2800 50  0001 C CNN
+F 1 "+5V" V 4800 3100 50  0000 L CNN
+F 2 "" H 4800 2950 50  0001 C CNN
+F 3 "" H 4800 2950 50  0001 C CNN
+	1    4800 2950
+	0    1    1    0
+$EndComp
+$Comp
+L power:+5V #PWR0130
+U 1 1 60DC868B
+P 17300 2700
+F 0 "#PWR0130" H 17300 2550 50  0001 C CNN
+F 1 "+5V" H 17315 2873 50  0000 C CNN
+F 2 "" H 17300 2700 50  0001 C CNN
+F 3 "" H 17300 2700 50  0001 C CNN
+	1    17300 2700
+	1    0    0    -1
+$EndComp

Commit message: PCB layout
Parts:
- U1105: footprint Package_SO:SSOP-8_3.9x5.05mm_P1.27mm -> Package_SO:SOIC-8_3.9x4.9mm_P1.27mm
- renumbered D1102 to D1101
Changed lines of the file:
@@
 	8200 14950 8200 14850
 $Comp
-L Diode:SD103ATW D1102
+L Diode:SD103ATW D1101
 U 3 1 5DDAE45D
 P 10250 15100
-F 0 "D1102" V 10296 15012 50  0000 R CNN
+F 0 "D1101" V 10296 15012 50  0000 R CNN
 F 1 "SD103ATW" V 10205 15012 50  0000 R CNN
 F 2 "Package_TO_SOT_SMD:SOT-363_SC-70-6" H 10250 14900 50  0001 C CNN
@@
 F 0 "U1105" H 12250 3350 50  0000 L CNN
 F 1 "LT1468" H 12250 3250 50  0000 L CNN
-F 2 "Package_SO:SSOP-8_3.9x5.05mm_P1.27mm" H 12100 3050 50  0001 C CNN
+F 2 "Package_SO:SOIC-8_3.9x4.9mm_P1.27mm" H 12100 3050 50  0001 C CNN
 F 3 "" H 12100 3050 50  0001 C CNN
 	1    12100 3050
