File: HARDWARE/BASE/Power.sch (KiCad schematic (older format))
At the start: 13 parts, among them Q201 IRFR5410, U201 MAX5902, U202 TSR 1-2433SM

Commit message: Schematic design
Parts:
- removed C201: 10u/50V, symbol Device:C
- removed C202, C204: 100n/50V, symbol Device:C
- removed C203: 10u/25V, symbol Device:C
- removed D201: SM6T30AY, symbol Device:D_Zener
- removed D202: MMSZ5249B, symbol Device:D_Zener
- removed D203: RED, symbol Device:LED
- removed F201: MF-LSMF185/33X, symbol Device:Fuse
- removed Q201: IRFR5410, symbol Device:Q_PMOS_GDS
- removed R201: 100k, symbol Device:R
- removed R202: R, symbol Device:R
- removed U201: MAX5902, symbol ETH1CSMU1:MAX5902
- removed U202: TSR 1-2433SM, symbol ETH1CSMU1:TSR1SM
- added C801, C802: 4u7/50V, Capacitor_SMD:C_1206_3216Metric_Pad1.33x1.80mm_HandSolder, symbol Device:C
- added C803, C804: 330p/2kV, Capacitor_SMD:C_1210_3225Metric_Pad1.33x2.70mm_HandSolder, symbol Device:C
- added D801: SM6T30AY, ETH1CSMU1:DO_214AA_REV, symbol Device:D_Zener
- added D802: MMSZ5249B, Diode_SMD:D_SOD-123, symbol Device:D_Zener
- added D803: RED, LED_SMD:LED_0603_1608Metric_Pad1.05x0.95mm_HandSolder, symbol Device:LED
- added F801: MF-LSMF185/33X, ETH1CSMU1:Fuse_SMD2920, symbol Device:Fuse
- added HS801: Heatsink, symbol Mechanical:Heatsink
- added L801: 7448014501, ETH1CSMU1:7448014501, symbol ETH1CSMU1:7448014501
- added Q801: IRFR5410, ETH1CSMU1:TO-252-2_Rectifier, symbol Device:Q_PMOS_GDS
- added R801: 100k, Resistor_SMD:R_0603_1608Metric_Pad0.98x0.95mm_HandSolder, symbol Device:R
- added R802: 370, Resistor_SMD:R_0603_1608Metric_Pad0.98x0.95mm_HandSolder, symbol Device:R
- added R803, R804: OPT, Resistor_SMD:R_0603_1608Metric_Pad0.98x0.95mm_HandSolder, symbol Device:R
- added U801: MAX5902, Package_TO_SOT_SMD:SOT-23-6_Handsoldering, symbol ETH1CSMU1:MAX5902
- added U802: THL15-2415WI, ETH1CSMU1:THL15, symbol ETH1CSMU1:THL15-2415WI
Connections:
- net labels added: +24VDD, +24VF, GNDPWR
- net labels removed: +3.3V
- wire segments 51 -> 63
- no-connect marks 1 -> 2

Commit message: Schematic design
Parts:
- renumbered C803 to C801, C801 to C802, C802 to C803, D802 to D801, D801 to D802, R803 to R802, R802 to R803
Changed lines of the file:
@@
 	1900 3150 1900 2600
 $Comp
-L Device:D_Zener D801
+L Device:D_Zener D802
 U 1 1 5D70DE79
 P 1900 3300
-F 0 "D801" V 1854 3379 50  0000 L CNN
+F 0 "D802" V 1854 3379 50  0000 L CNN
 F 1 "SM6T30AY" V 1945 3379 50  0000 L CNN
 F 2 "ETH1CSMU1:DO_214AA_REV" H 1900 3300 50  0001 C CNN
@@
 $EndComp
 $Comp
-L Device:D_Zener D802
+L Device:D_Zener D801
 U 1 1 5D6DFA8C
 P 4350 2750
-F 0 "D802" V 4304 2829 50  0000 L CNN
+F 0 "D801" V 4304 2829 50  0000 L CNN
 F 1 "MMSZ5249B" V 4395 2829 50  0000 L CNN
 F 2 "Diode_SMD:D_SOD-123" H 4350 2750 50  0001 C CNN
@@
 $EndComp
 $Comp
-L Device:R R802
+L Device:R R803
 U 1 1 5D6D8193
 P 4350 3100
-F 0 "R802" H 4420 3146 50  0000 L CNN
+F 0 "R803" H 4420 3146 50  0000 L CNN
 F 1 "370" H 4420 3055 50  0000 L CNN
 F 2 "Resistor_SMD:R_0603_1608Metric_Pad0.98x0.95mm_HandSolder" V 4280 3100 50  0001 C CNN
@@
 	5150 2950 5150 2600
 $Comp
-L Device:C C801
+L Device:C C802
 U 1 1 5D6CEB9C
 P 5150 3100
-F 0 "C801" H 5265 3146 50  0000 L CNN
+F 0 "C802" H 5265 3146 50  0000 L CNN
 F 1 "4u7/50V" H 5265 3055 50  0000 L CNN
 F 2 "Capacitor_SMD:C_1206_3216Metric_Pad1.33x1.80mm_HandSolder" H 5188 2950 50  0001 C CNN
@@
 $EndComp
 $Comp
-L power:+24V #PWR0802
+L power:+24V #PWR0801
 U 1 1 5D7B3705
 P 1250 2550
-F 0 "#PWR0802" H 1250 2400 50  0001 C CNN
+F 0 "#PWR0801" H 1250 2400 50  0001 C CNN
 F 1 "+24V" H 1265 2723 50  0000 C CNN
 F 2 "" H 1250 2550 50  0001 C CNN
@@
 	2400 3200 2400 3650
 $Comp
-L Device:C C802
+L Device:C C803
 U 1 1 5DA6571D
 P 5750 3100
-F 0 "C802" H 5865 3146 50  0000 L CNN
+F 0 "C803" H 5865 3146 50  0000 L CNN
 F 1 "4u7/50V" H 5865 3055 50  0000 L CNN
 F 2 "Capacitor_SMD:C_1206_3216Metric_Pad1.33x1.80mm_HandSolder" H 5788 2950 50  0001 C CNN
@@
 Connection ~ 5150 3650
 $Comp
-L power:PWR_FLAG #FLG0804
+L power:PWR_FLAG #FLG0801
 U 1 1 5E5270F4
 P 5750 2550
-F 0 "#FLG0804" H 5750 2625 50  0001 C CNN
+F 0 "#FLG0801" H 5750 2625 50  0001 C CNN
 F 1 "PWR_FLAG" H 5750 2723 50  0000 C CNN
 F 2 "" H 5750 2550 50  0001 C CNN
@@
 	5750 2550 5750 2600
 $Comp
-L power:PWR_FLAG #FLG0801
+L power:PWR_FLAG #FLG0802
 U 1 1 5DDE91B3
 P 850 7350
-F 0 "#FLG0801" H 850 7425 50  0001 C CNN
+F 0 "#FLG0802" H 850 7425 50  0001 C CNN
 F 1 "PWR_FLAG" H 850 7523 50  0000 C CNN
 F 2 "" H 850 7350 50  0001 C CNN
@@
 $EndComp
 $Comp
-L power:+24V #PWR0801
+L power:+24V #PWR0805
 U 1 1 5DDE9577
 P 850 7350
-F 0 "#PWR0801" H 850 7200 50  0001 C CNN
+F 0 "#PWR0805" H 850 7200 50  0001 C CNN
 F 1 "+24V" H 865 7523 50  0000 C CNN
 F 2 "" H 850 7350 50  0001 C CNN
@@
 $EndComp
 $Comp
-L power:PWR_FLAG #FLG0803
+L power:PWR_FLAG #FLG0804
 U 1 1 5DDFBB5F
 P 1750 7350
-F 0 "#FLG0803" H 1750 7425 50  0001 C CNN
+F 0 "#FLG0804" H 1750 7425 50  0001 C CNN
 F 1 "PWR_FLAG" H 1750 7523 50  0000 C CNN
 F 2 "" H 1750 7350 50  0001 C CNN
@@
 $EndComp
 $Comp
-L ETH1CSMU1:+24VDD #PWR0805
+L ETH1CSMU1:+24VDD #PWR0807
 U 1 1 5DDFC0E6
 P 1750 7350
-F 0 "#PWR0805" H 1750 7200 50  0001 C CNN
+F 0 "#PWR0807" H 1750 7200 50  0001 C CNN
 F 1 "+24VDD" H 1765 7523 50  0000 C CNN
 F 2 "" H 1750 7350 50  0001 C CNN
@@
 $EndComp
 $Comp
-L Device:R R803
+L Device:R R802
 U 1 1 5E464415
 P 8550 2850
-F 0 "R803" H 8620 2896 50  0000 L CNN
+F 0 "R802" H 8620 2896 50  0000 L CNN
 F 1 "OPT" H 8620 2805 50  0000 L CNN
 F 2 "Resistor_SMD:R_0603_1608Metric_Pad0.98x0.95mm_HandSolder" V 8480 2850 50  0001 C CNN
@@
 	5750 2600 6300 2600
 $Comp
-L Device:C C803
+L Device:C C801
 U 1 1 5E47CFD6
 P 7800 2200
-F 0 "C803" V 7548 2200 50  0000 C CNN
+F 0 "C801" V 7548 2200 50  0000 C CNN
 F 1 "330p/2kV" V 7639 2200 50  0000 C CNN
 F 2 "Capacitor_SMD:C_1210_3225Metric_Pad1.33x2.70mm_HandSolder" H 7838 2050 50  0001 C CNN
@@
 Connection ~ 8550 2650
 $Comp
-L ETH1CSMU1:+24VF #PWR0806
+L ETH1CSMU1:+24VF #PWR0802
 U 1 1 5E485438
 P 8850 2650
-F 0 "#PWR0806" H 8850 2500 50  0001 C CNN
+F 0 "#PWR0802" H 8850 2500 50  0001 C CNN
 F 1 "+24VF" V 8850 2800 50  0000 L CNN
 F 2 "" H 8850 2650 50  0001 C CNN
@@
 	8850 2650 8550 2650
 $Comp
-L power:GNDPWR #PWR0803
+L power:GNDPWR #PWR0804
 U 1 1 5F619953
 P 1250 3700
-F 0 "#PWR0803" H 1250 3500 50  0001 C CNN
+F 0 "#PWR0804" H 1250 3500 50  0001 C CNN
 F 1 "GNDPWR" H 1254 3546 50  0000 C CNN
 F 2 "" H 1250 3650 50  0001 C CNN
@@
 $EndComp
 $Comp
-L power:GNDPWR #PWR0804
+L power:GNDPWR #PWR0806
 U 1 1 5F61F80D
 P 1300 7350
-F 0 "#PWR0804" H 1300 7150 50  0001 C CNN
+F 0 "#PWR0806" H 1300 7150 50  0001 C CNN
 F 1 "GNDPWR" H 1305 7195 50  0000 C CNN
 F 2 "" H 1300 7300 50  0001 C CNN
@@
 $EndComp
 $Comp
-L power:PWR_FLAG #FLG0802
+L power:PWR_FLAG #FLG0803
 U 1 1 5F62072B
 P 1300 7350
-F 0 "#FLG0802" H 1300 7425 50  0001 C CNN
+F 0 "#FLG0803" H 1300 7425 50  0001 C CNN
 F 1 "PWR_FLAG" H 1300 7523 50  0000 C CNN
 F 2 "" H 1300 7350 50  0001 C CNN
@@
 	4350 2950 4350 2900
 $Comp
-L power:GND #PWR0807
+L power:GND #PWR0803
 U 1 1 6054CC9D
 P 8850 3550
-F 0 "#PWR0807" H 8850 3300 50  0001 C CNN
+F 0 "#PWR0803" H 8850 3300 50  0001 C CNN
 F 1 "GND" V 8850 3400 50  0000 R CNN
 F 2 "" H 8850 3550 50  0001 C CNN

Commit message: Schematic design.
Parts:
- renumbered C801 to C701, C802 to C702, C803 to C703, C804 to C704, D801 to D701, D802 to D702, D803 to D703, F801 to F701, HS801 to HS701, L801 to L701, Q801 to Q701, R801 to R701, R802 to R702, R803 to R703, R804 to R704, U801 to U701, U802 to U702
Changed lines of the file:
@@
 $Descr A4 11693 8268
 encoding utf-8
-Sheet 8 12
+Sheet 7 11
 Title "Power"
 Date "2020-03-07"
@@
 	1900 3150 1900 2600
 $Comp
-L Device:D_Zener D802
+L Device:D_Zener D702
 U 1 1 5D70DE79
 P 1900 3300
-F 0 "D802" V 1854 3379 50  0000 L CNN
+F 0 "D702" V 1854 3379 50  0000 L CNN
 F 1 "SM6T30AY" V 1945 3379 50  0000 L CNN
 F 2 "ETH1CSMU1:DO_214AA_REV" H 1900 3300 50  0001 C CNN
@@
 $EndComp
 $Comp
-L Device:D_Zener D801
+L Device:D_Zener D701
 U 1 1 5D6DFA8C
 P 4350 2750
-F 0 "D801" V 4304 2829 50  0000 L CNN
+F 0 "D701" V 4304 2829 50  0000 L CNN
 F 1 "MMSZ5249B" V 4395 2829 50  0000 L CNN
 F 2 "Diode_SMD:D_SOD-123" H 4350 2750 50  0001 C CNN
@@
 $EndComp
 $Comp
-L Device:R R803
+L Device:R R703
 U 1 1 5D6D8193
 P 4350 3100
-F 0 "R803" H 4420 3146 50  0000 L CNN
+F 0 "R703" H 4420 3146 50  0000 L CNN
 F 1 "370" H 4420 3055 50  0000 L CNN
 F 2 "Resistor_SMD:R_0603_1608Metric_Pad0.98x0.95mm_HandSolder" V 4280 3100 50  0001 C CNN
@@
 $EndComp
 $Comp
-L Device:LED D803
+L Device:LED D703
 U 1 1 5D6D7414
 P 4350 3450
-F 0 "D803" V 4389 3332 50  0000 R CNN
+F 0 "D703" V 4389 3332 50  0000 R CNN
 F 1 "RED" V 4298 3332 50  0000 R CNN
 F 2 "LED_SMD:LED_0603_1608Metric_Pad1.05x0.95mm_HandSolder" H 4350 3450 50  0001 C CNN
@@
 	5150 2950 5150 2600
 $Comp
-L Device:C C802
+L Device:C C702
 U 1 1 5D6CEB9C
 P 5150 3100
-F 0 "C802" H 5265 3146 50  0000 L CNN
+F 0 "C702" H 5265 3146 50  0000 L CNN
 F 1 "4u7/50V" H 5265 3055 50  0000 L CNN
 F 2 "Capacitor_SMD:C_1206_3216Metric_Pad1.33x1.80mm_HandSolder" H 5188 2950 50  0001 C CNN
@@
 	1550 2600 1250 2600
 $Comp
-L Device:Fuse F801
+L Device:Fuse F701
 U 1 1 5D5D8684
 P 1700 2600
-F 0 "F801" V 1503 2600 50  0000 C CNN
+F 0 "F701" V 1503 2600 50  0000 C CNN
 F 1 "MF-LSMF185/33X" V 1594 2600 50  0000 C CNN
 F 2 "ETH1CSMU1:Fuse_SMD2920" V 1630 2600 50  0001 C CNN
@@
 $EndComp
 $Comp
-L power:+24V #PWR0801
+L power:+24V #PWR0701
 U 1 1 5D7B3705
 P 1250 2550
-F 0 "#PWR0801" H 1250 2400 50  0001 C CNN
+F 0 "#PWR0701" H 1250 2400 50  0001 C CNN
 F 1 "+24V" H 1265 2723 50  0000 C CNN
 F 2 "" H 1250 2550 50  0001 C CNN
@@
 	1900 2600 2100 2600
 $Comp
-L ETH1CSMU1:MAX5902 U801
+L ETH1CSMU1:MAX5902 U701
 U 1 1 5D6EBA14
 P 3000 3100
-F 0 "U801" H 3000 3465 50  0000 C CNN
+F 0 "U701" H 3000 3465 50  0000 C CNN
 F 1 "MAX5902" H 3000 3374 50  0000 C CNN
 F 2 "Package_TO_SOT_SMD:SOT-23-6_Handsoldering" H 3000 3100 60  0001 C CNN
@@
 $EndComp
 $Comp
-L Device:Q_PMOS_GDS Q801
+L Device:Q_PMOS_GDS Q701
 U 1 1 5D6F32E4
 P 3600 2700
-F 0 "Q801" V 3943 2700 50  0000 C CNN
+F 0 "Q701" V 3943 2700 50  0000 C CNN
 F 1 "IRFR5410" V 3852 2700 50  0000 C CNN
 F 2 "ETH1CSMU1:TO-252-2_Rectifier" H 3800 2800 50  0001 C CNN
@@
 	2400 3000 2400 2600
 $Comp
-L Device:R R801
+L Device:R R701
 U 1 1 5D709595
 P 2100 2850
-F 0 "R801" H 2170 2896 50  0000 L CNN
+F 0 "R701" H 2170 2896 50  0000 L CNN
 F 1 "100k" H 2170 2805 50  0000 L CNN
 F 2 "Resistor_SMD:R_0603_1608Metric_Pad0.98x0.95mm_HandSolder" V 2030 2850 50  0001 C CNN
@@
 	2400 3200 2400 3650
 $Comp
-L Device:C C803
+L Device:C C703
 U 1 1 5DA6571D
 P 5750 3100
-F 0 "C803" H 5865 3146 50  0000 L CNN
+F 0 "C703" H 5865 3146 50  0000 L CNN
 F 1 "4u7/50V" H 5865 3055 50  0000 L CNN
 F 2 "Capacitor_SMD:C_1206_3216Metric_Pad1.33x1.80mm_HandSolder" H 5788 2950 50  0001 C CNN
@@
 Connection ~ 5150 3650
 $Comp
-L power:PWR_FLAG #FLG0801
+L power:PWR_FLAG #FLG0701
 U 1 1 5E5270F4
 P 5750 2550
-F 0 "#FLG0801" H 5750 2625 50  0001 C CNN
+F 0 "#FLG0701" H 5750 2625 50  0001 C CNN
 F 1 "PWR_FLAG" H 5750 2723 50  0000 C CNN
 F 2 "" H 5750 2550 50  0001 C CNN
@@
 	5750 2550 5750 2600
 $Comp
-L power:PWR_FLAG #FLG0802
+L power:PWR_FLAG #FLG0702
 U 1 1 5DDE91B3
 P 850 7350
-F 0 "#FLG0802" H 850 7425 50  0001 C CNN
+F 0 "#FLG0702" H 850 7425 50  0001 C CNN
 F 1 "PWR_FLAG" H 850 7523 50  0000 C CNN
 F 2 "" H 850 7350 50  0001 C CNN
@@
 $EndComp
 $Comp
-L power:+24V #PWR0805
+L power:+24V #PWR0705
 U 1 1 5DDE9577
 P 850 7350
-F 0 "#PWR0805" H 850 7200 50  0001 C CNN
+F 0 "#PWR0705" H 850 7200 50  0001 C CNN
 F 1 "+24V" H 865 7523 50  0000 C CNN
 F 2 "" H 850 7350 50  0001 C CNN
@@
 $EndComp
 $Comp
-L power:PWR_FLAG #FLG0804
+L power:PWR_FLAG #FLG0704
 U 1 1 5DDFBB5F
 P 1750 7350
-F 0 "#FLG0804" H 1750 7425 50  0001 C CNN
+F 0 "#FLG0704" H 1750 7425 50  0001 C CNN
 F 1 "PWR_FLAG" H 1750 7523 50  0000 C CNN
 F 2 "" H 1750 7350 50  0001 C CNN
@@
 $EndComp
 $Comp
-L ETH1CSMU1:+24VDD #PWR0807
+L ETH1CSMU1:+24VDD #PWR0707
 U 1 1 5DDFC0E6
 P 1750 7350
-F 0 "#PWR0807" H 1750 7200 50  0001 C CNN
+F 0 "#PWR0707" H 1750 7200 50  0001 C CNN
 F 1 "+24VDD" H 1765 7523 50  0000 C CNN
 F 2 "" H 1750 7350 50  0001 C CNN
@@
 Connection ~ 5150 2600
 $Comp
-L ETH1CSMU1:THL15-2415WI U802
+L ETH1CSMU1:THL15-2415WI U702
 U 1 1 5E4632D5
 P 7800 3100
-F 0 "U802" H 7800 3815 50  0000 C CNN
+F 0 "U702" H 7800 3815 50  0000 C CNN
 F 1 "THL15-2415WI" H 7800 3724 50  0000 C CNN
 F 2 "ETH1CSMU1:THL15" H 8700 3450 50  0001 C CNN
@@
 $EndComp
 $Comp
-L Device:R R802
+L Device:R R702
 U 1 1 5E464415
 P 8550 2850
-F 0 "R802" H 8620 2896 50  0000 L CNN
+F 0 "R702" H 8620 2896 50  0000 L CNN
 F 1 "OPT" H 8620 2805 50  0000 L CNN
 F 2 "Resistor_SMD:R_0603_1608Metric_Pad0.98x0.95mm_HandSolder" V 8480 2850 50  0001 C CNN
@@
 $EndComp
 $Comp
-L Device:R R804
+L Device:R R704
 U 1 1 5E464838
 P 8550 3350
-F 0 "R804" H 8620 3396 50  0000 L CNN
+F 0 "R704" H 8620 3396 50  0000 L CNN
 F 1 "OPT" H 8620 3305 50  0000 L CNN
 F 2 "Resistor_SMD:R_0603_1608Metric_Pad0.98x0.95mm_HandSolder" V 8480 3350 50  0001 C CNN
@@
 	8550 3100 8550 3200
 $Comp
-L ETH1CSMU1:7448014501 L801
+L ETH1CSMU1:7448014501 L701
 U 1 1 5E46ABAD
 P 6650 3100
-F 0 "L801" H 6650 2750 50  0000 C CNN
+F 0 "L701" H 6650 2750 50  0000 C CNN
 F 1 "7448014501" H 6650 2850 50  0000 C CNN
 F 2 "ETH1CSMU1:7448014501" H 6650 3600 50  0001 C CNN
@@
 	5750 2600 6300 2600
 $Comp
-L Device:C C801
+L Device:C C701
 U 1 1 5E47CFD6
 P 7800 2200
-F 0 "C801" V 7548 2200 50  0000 C CNN
+F 0 "C701" V 7548 2200 50  0000 C CNN
 F 1 "330p/2kV" V 7639 2200 50  0000 C CNN
 F 2 "Capacitor_SMD:C_1210_3225Metric_Pad1.33x2.70mm_HandSolder" H 7838 2050 50  0001 C CNN
@@
 $EndComp
 $Comp
-L Device:C C804
+L Device:C C704
 U 1 1 5E47E7C0
 P 7800 4000
-F 0 "C804" V 7548 4000 50  0000 C CNN
+F 0 "C704" V 7548 4000 50  0000 C CNN
 F 1 "330p/2kV" V 7639 4000 50  0000 C CNN
 F 2 "Capacitor_SMD:C_1210_3225Metric_Pad1.33x2.70mm_HandSolder" H 7838 3850 50  0001 C CNN
@@
 Connection ~ 8550 2650
 $Comp
-L ETH1CSMU1:+24VF #PWR0802
+L ETH1CSMU1:+24VF #PWR0702
 U 1 1 5E485438
 P 8850 2650
-F 0 "#PWR0802" H 8850 2500 50  0001 C CNN
+F 0 "#PWR0702" H 8850 2500 50  0001 C CNN
 F 1 "+24VF" V 8850 2800 50  0000 L CNN
 F 2 "" H 8850 2650 50  0001 C CNN
@@
 	8850 2650 8550 2650
 $Comp
-L power:GNDPWR #PWR0804
+L power:GNDPWR #PWR0704
 U 1 1 5F619953
 P 1250 3700
-F 0 "#PWR0804" H 1250 3500 50  0001 C CNN
+F 0 "#PWR0704" H 1250 3500 50  0001 C CNN
 F 1 "GNDPWR" H 1254 3546 50  0000 C CNN
 F 2 "" H 1250 3650 50  0001 C CNN
@@
 $EndComp
 $Comp
-L power:GNDPWR #PWR0806
+L power:GNDPWR #PWR0706
 U 1 1 5F61F80D
 P 1300 7350
-F 0 "#PWR0806" H 1300 7150 50  0001 C CNN
+F 0 "#PWR0706" H 1300 7150 50  0001 C CNN
 F 1 "GNDPWR" H 1305 7195 50  0000 C CNN
 F 2 "" H 1300 7300 50  0001 C CNN
@@
 $EndComp
 $Comp
-L power:PWR_FLAG #FLG0803
+L power:PWR_FLAG #FLG0703
 U 1 1 5F62072B
 P 1300 7350
-F 0 "#FLG0803" H 1300 7425 50  0001 C CNN
+F 0 "#FLG0703" H 1300 7425 50  0001 C CNN
 F 1 "PWR_FLAG" H 1300 7523 50  0000 C CNN
 F 2 "" H 1300 7350 50  0001 C CNN
@@
 	4350 2950 4350 2900
 $Comp
-L power:GND #PWR0803
+L power:GND #PWR0703
 U 1 1 6054CC9D
 P 8850 3550
-F 0 "#PWR0803" H 8850 3300 50  0001 C CNN
+F 0 "#PWR0703" H 8850 3300 50  0001 C CNN
 F 1 "GND" V 8850 3400 50  0000 R CNN
 F 2 "" H 8850 3550 50  0001 C CNN
@@
 $EndComp
 $Comp
-L Mechanical:Heatsink HS801
+L Mechanical:Heatsink HS701
 U 1 1 60910113
 P 7800 4600
-F 0 "HS801" H 7942 4721 50  0000 L CNN
+F 0 "HS701" H 7942 4721 50  0000 L CNN
 F 1 "Heatsink" H 7942 4630 50  0000 L CNN
 F 2 "" H 7812 4600 50  0001 C CNN

Commit message: PCB layout
Parts:
- removed HS701: Heatsink, symbol Mechanical:Heatsink
Changed lines of the file:
@@
 	0    -1   -1   0
 $EndComp
-$Comp
-L Mechanical:Heatsink HS701
-U 1 1 60910113
-P 7800 4600
-F 0 "HS701" H 7942 4721 50  0000 L CNN
-F 1 "Heatsink" H 7942 4630 50  0000 L CNN
-F 2 "" H 7812 4600 50  0001 C CNN
-F 3 "~" H 7812 4600 50  0001 C CNN
-	1    7800 4600
-	1    0    0    -1
-$EndComp
 $EndSCHEMATC
