File: HARDWARE/MODULE/HV_Amplifier.sch (KiCad schematic (older format))
At the start: 22 parts, among them Q201 TIP41C/D44H, Q202 MMBT3904, Q203 PZT2907A, Q204 PZT2222A, Q205 MMBT3906, Q206 TIP42C/D45H

Commit message: Schematic design.
Parts:
- HS201, HS202: value Heatsink -> HSE-B20350-NP; footprint (none) -> ETH1CSMU1:HSE-B20350-NP
- Q201, Q206: footprint Package_TO_SOT_THT:TO-220-3_Vertical -> Package_TO_SOT_THT:TO-220-3_Horizontal_TabDown
Other:
- moved on the sheet: D201, D202, D203, D204, HS201, HS202, Q201, Q202, Q203, Q204, Q205, Q206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

Commit message: PCB and schematic design.
Parts:
- added J201: Conn_02x12_Odd_Even, Connector_PinSocket_2.54mm:PinSocket_2x12_P2.54mm_Vertical, symbol Connector_Generic:Conn_02x12_Odd_Even
Connections:
- net +15V: now also J201.3 (Pin_3), J201.4 (Pin_4)
- net -15V: now also J201.7 (Pin_7), J201.8 (Pin_8)
- net AMPIN: now also J201.10 (Pin_10), J201.9 (Pin_9)
- net FLOAT_COM: now also J201.1 (Pin_1), J201.2 (Pin_2)
- new net +15VF: J201.15 (Pin_15), J201.16 (Pin_16)
- new net -15VF: J201.19 (Pin_19), J201.20 (Pin_20)
- new net GND: J201.5 (Pin_5), J201.6 (Pin_6)
- new net GNDHV: J201.17 (Pin_17), J201.18 (Pin_18)
- no-connect marks 2 -> 10
Other:
- moved on the sheet: D201, D202, D203, D204, HS201, HS202, Q201, Q202, Q203, Q204, Q205, Q206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

Commit message: PCB and schematic
Parts:
- removed J201: Conn_02x12_Odd_Even, Connector_PinSocket_2.54mm:PinSocket_2x12_P2.54mm_Vertical, symbol Connector_Generic:Conn_02x12_Odd_Even
- added J201: Conn_02x06_Odd_Even, Connector_PinSocket_2.54mm:PinSocket_2x06_P2.54mm_Vertical, symbol Connector_Generic:Conn_02x06_Odd_Even
- added Q207, Q208: 2N7002, Package_TO_SOT_SMD:SOT-23, symbol Transistor_FET:2N7002
- added R211, R212: 49k9, Resistor_SMD:R_0805_2012Metric_Pad1.20x1.40mm_HandSolder, symbol Device:R
- R204, R208: value 25/1W -> 24R9/1W
- R205: value 24R9 -> 200
- R206: value 249 -> 1k
Connections:
- net +15V: now also J201.3 (Pin_3), J201.4 (Pin_4), R211.1
- net -15V: now also J201.7 (Pin_7), J201.8 (Pin_8), R212.2
- net AMPIN: now also J201.10 (Pin_10), J201.9 (Pin_9)
- net FLOAT_COM: now also J201.1 (Pin_1), J201.2 (Pin_2), Q207.2 (S), Q208.3 (D); no longer R203.2, R207.1
- net GND: now also J201.5 (Pin_5), J201.6 (Pin_6)
- net BASE+: now reaches Q202.1 (B), R202.2
- net BASE+: now also R207.1, R211.2; no longer R203.1
- net BASE-: now reaches Q205.1 (B), R209.2
- net BASE-: now also R203.2, R212.1; no longer R207.2
- new net: Q208.2 (S), R203.1
- new net: Q207.3 (D), R207.2
- new net 100mA: J201.11 (Pin_11), J201.12 (Pin_12), Q207.1 (G), Q208.1 (G)
- no-connect marks 10 -> 2
Other:
- moved on the sheet: D201, D202, D203, D204, HS201, HS202, Q201, Q202, Q203, Q204, Q205, Q206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

Commit message: PCB layout
Parts:
- removed J201: Conn_02x06_Odd_Even, Connector_PinSocket_2.54mm:PinSocket_2x06_P2.54mm_Vertical, symbol Connector_Generic:Conn_02x06_Odd_Even
- added J201: Conn_02x08_Odd_Even, Connector_PinSocket_2.54mm:PinSocket_2x08_P2.54mm_Vertical, symbol Connector_Generic:Conn_02x08_Odd_Even
- renumbered Q207 to Q201, Q208 to Q202, Q201 to Q203, Q202 to Q204, Q203 to Q205, Q204 to Q206, Q205 to Q207, Q206 to Q208, R211 to R201, R207 to R202, R201 to R203, R203 to R204, R212 to R205, R202 to R206, R204 to R207, R205 to R208, R206 to R209, R208 to R210, R209 to R211, R210 to R212
Connections:
- net +15V: now also J201.10 (Pin_10), J201.9 (Pin_9)
- net -15V: now also J201.5 (Pin_5), J201.6 (Pin_6)
- net 100mA: now also J201.1 (Pin_1), J201.2 (Pin_2)
- net AMPIN: now also J201.3 (Pin_3), J201.4 (Pin_4)
- net FLOAT_COM: now also J201.11 (Pin_11), J201.12 (Pin_12)
- new net +15VF: J201.13 (Pin_13)
- new net -15VF: J201.15 (Pin_15)
- new net GND1: J201.7 (Pin_7), J201.8 (Pin_8)
- new net GNDHV: J201.14 (Pin_14), J201.16 (Pin_16)

Commit message: Schematic and PCB update.
Parts:
- D201, D204: value BAV99 -> BAV99LT1
Changed lines of the file:
@@
 P 7450 3050
 F 0 "D201" H 7450 3266 50  0000 C CNN
-F 1 "BAV99" H 7450 3175 50  0000 C CNN
+F 1 "BAV99LT1" H 7450 3175 50  0000 C CNN
 F 2 "Package_TO_SOT_SMD:SOT-23" H 7450 2550 50  0001 C CNN
 F 3 "https://assets.nexperia.com/documents/data-sheet/BAV99_SER.pdf" H 7450 3050 50  0001 C CNN
@@
 P 7450 5250
 F 0 "D204" H 7450 5373 50  0000 C CNN
-F 1 "BAV99" H 7450 5464 50  0000 C CNN
+F 1 "BAV99LT1" H 7450 5464 50  0000 C CNN
 F 2 "Package_TO_SOT_SMD:SOT-23" H 7450 4750 50  0001 C CNN
 F 3 "https://assets.nexperia.com/documents/data-sheet/BAV99_SER.pdf" H 7450 5250 50  0001 C CNN
