File: HARDWARE/MODULE/MODULE.kicad_pcb (KiCad board)
At the start: 2 copper layers, 160 x 100 mm, 114 parts, among them J301 Conn_02x04_Odd_Even, Q201 TIP41C/D44H, Q202 MMBT3904, Q203 PZT2907A, Q204 PZT2222A, Q205 MMBT3906, Q206 TIP42C/D45H, U301 LM317_TO-263, U302 LT8330_S6, U303 LM337_TO263, U304 LT8570_MS8E, U305 L78L15_SO8, U306 TEL10-2415, U307 SN6505BDBV, U308 L79L15_SO8

Commit message: PCB and schematic design.
Parts:
- added J201: Conn_02x12_Odd_Even, Connector_PinSocket_2.54mm:PinSocket_2x12_P2.54mm_Vertical, B.Cu at (100.0, 48.0)
- C307, C308, C320: footprint Capacitor_SMD:C_1210_3225Metric_Pad1.33x2.70mm_HandSolder -> Capacitor_SMD:C_2220_5650Metric_Pad1.97x5.40mm_HandSolder
- H101, H102, H103, H104: footprint MountingHole:MountingHole_4.3mm_M4_DIN965_Pad_TopBottom -> MountingHole:MountingHole_3.2mm_M3_DIN965_Pad
- J301: value Conn_02x04_Odd_Even -> Conn_02x06_Odd_Even; footprint Connector_PinSocket_2.54mm:PinSocket_2x04_P2.54mm_Vertical -> Connector_PinSocket_2.54mm:PinSocket_2x06_P2.54mm_Vertical; moved to B.Cu
- moved H103 389.5 mm to (221.0, 45.0)
- moved R208 379.7 mm to (220.7, 92.5), turned to 180 degrees
- moved D203 352.4 mm to (220.7, 88.5), turned to 180 degrees
- moved Q203 345.9 mm to (167.9, 89.9), turned to 180 degrees
- moved H104 337.4 mm to (167.0, 122.0)
- moved D202 319.9 mm to (187.7, 88.4)
- moved R201 318.6 mm to (167.9, 95.8)
- moved R210 314.7 mm to (200.9, 95.9), turned to 180 degrees
- moved R202 306.8 mm to (180.6, 97.5)
- moved Q202 287.5 mm to (175.8, 97.5), turned to 180 degrees
- moved H101 273.5 mm to (89.0, 135.0)
- moved H102 267.9 mm to (89.0, 45.0)
- moved L304 226.9 mm to (147.1, 98.4)
- moved C324 217.2 mm to (151.3, 64.4), turned to 180 degrees
- moved C321 204.8 mm to (142.9, 64.4)
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Connections:
- J301 pad 3: (no net) -> +24V
- J301 pad 4: (no net) -> +24V
- J301 pad 5: +5V -> (no net)
- J301 pad 6: +5V -> (no net)
- J301 pad 7: GND -> +5V
- J301 pad 8: GND -> +5V
- R205 pad 2: (no net) -> /High Voltage Amplifier/AMPIN
Other:
- outline, holes or cut-outs redrawn
- copper layers 2 -> 4

Commit message: PCB and schematic
Parts:
- added J302: Conn_02x02_Odd_Even, Connector_PinSocket_2.54mm:PinSocket_2x02_P2.54mm_Vertical, B.Cu at (164.0, 79.0)
- added Q207: 2N7002, Package_TO_SOT_SMD:SOT-23, F.Cu at (44.0, 52.4)
- added Q208: 2N7002, Package_TO_SOT_SMD:SOT-23, F.Cu at (34.5, 55.4)
- added R211: 49k9, Resistor_SMD:R_0805_2012Metric_Pad1.20x1.40mm_HandSolder, F.Cu at (34.6, 51.6)
- added R212: 49k9, Resistor_SMD:R_0805_2012Metric_Pad1.20x1.40mm_HandSolder, F.Cu at (39.4, 51.6)
- J201: value Conn_02x12_Odd_Even -> Conn_02x06_Odd_Even; footprint Connector_PinSocket_2.54mm:PinSocket_2x12_P2.54mm_Vertical -> Connector_PinSocket_2.54mm:PinSocket_2x06_P2.54mm_Vertical; moved to F.Cu
- R204, R208: value 25/1W -> 24R9/1W
- R205: value 24R9 -> 200
- R206: value 249 -> 1k
- R210: moved to B.Cu
- moved J201 70.2 mm to (30.0, 52.5), turned to 0 degrees
- moved R201 47.9 mm to (170.2, 47.9), turned to 270 degrees
- moved R208 47.6 mm to (173.5, 98.7), turned to 90 degrees
- moved D203 44.7 mm to (177.5, 99.7), turned to 90 degrees
- moved Q203 42.8 mm to (176.1, 47.9), turned to 90 degrees
- moved Q202 42.4 mm to (168.5, 55.8), turned to 90 degrees
- moved R202 38.9 mm to (168.5, 60.6), turned to 270 degrees
- moved Q201 35.6 mm to (174.6, 55.8), turned to 270 degrees
- moved Q206 34.4 mm to (174.6, 87.8), turned to 270 degrees
- moved R210 29.5 mm to (176.0, 80.0), turned to 90 degrees
- moved R204 28.3 mm to (173.7, 67.8), turned to 270 degrees
- moved Q204 26.9 mm to (176.0, 79.9), turned to 90 degrees
- moved HS201 26.3 mm to (198.8, 90.3), turned to 270 degrees
- moved D202 23.0 mm to (177.6, 67.7), turned to 270 degrees
- moved HS202 22.3 mm to (198.8, 58.3), turned to 270 degrees
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Connections:
- J201 pad 11: (no net) -> /High Voltage Amplifier/100mA
- J201 pad 12: (no net) -> /High Voltage Amplifier/100mA
- Q202 pad 1: Net-(Q202-Pad1) -> /High Voltage Amplifier/BASE+
- Q205 pad 1: Net-(Q205-Pad1) -> /High Voltage Amplifier/BASE-
- R202 pad 2: Net-(Q202-Pad1) -> /High Voltage Amplifier/BASE+
- R203 pad 1: Net-(Q202-Pad1) -> Net-(Q208-Pad2)
- R203 pad 2: /High Voltage Amplifier/FLOAT_COM -> /High Voltage Amplifier/BASE-
- R207 pad 1: /High Voltage Amplifier/FLOAT_COM -> /High Voltage Amplifier/BASE+
- R207 pad 2: Net-(Q205-Pad1) -> Net-(Q207-Pad3)
- R209 pad 2: Net-(Q205-Pad1) -> /High Voltage Amplifier/BASE-

Commit message: PCB layout
Parts:
- removed J302: Conn_02x02_Odd_Even, Connector_PinSocket_2.54mm:PinSocket_2x02_P2.54mm_Vertical
- C301, C313, C328, C331, C334, C335, C339, C340, C344, R301, R304, R308, R309, R310: moved to B.Cu
- C305, C306: value 4u7/100V -> 4u7/50V; footprint Capacitor_SMD:C_1210_3225Metric_Pad1.33x2.70mm_HandSolder -> Capacitor_SMD:C_1206_3216Metric_Pad1.33x1.80mm_HandSolder
- C326: value 470p -> 47p
- J201: value Conn_02x06_Odd_Even -> Conn_02x08_Odd_Even; footprint Connector_PinSocket_2.54mm:PinSocket_2x06_P2.54mm_Vertical -> Connector_PinSocket_2.54mm:PinSocket_2x08_P2.54mm_Vertical; moved to B.Cu
- R212: renamed from R210; moved to F.Cu
- moved R211 326.1 mm to (169.7, 94.7), turned to 180 degrees
- moved R208 324.4 mm to (165.0, 71.6), turned to 90 degrees
- moved R209 315.1 mm to (165.0, 75.7), turned to 90 degrees
- moved Q207 311.7 mm to (169.7, 89.0), turned to 180 degrees
- moved R204 291.7 mm to (165.0, 93.6), turned to 270 degrees
- moved R202 289.0 mm to (165.0, 61.3), turned to 270 degrees
- moved D204 283.0 mm to (169.7, 85.3), turned to 180 degrees
- moved D201 272.6 mm to (169.8, 53.5), turned to 180 degrees
- moved C344 198.1 mm to (145.3, 119.8), turned to 180 degrees
- moved C331 191.5 mm to (145.3, 109.6), turned to 180 degrees
- moved C318 187.7 mm to (115.7, 97.0), turned to 270 degrees
- moved C337 181.2 mm to (117.6, 114.7), turned to 270 degrees
- moved C336 175.7 mm to (120.4, 114.7), turned to 270 degrees
- moved C314 172.2 mm to (120.0, 80.0)
- moved FB302 171.0 mm to (90.0, 99.1), turned to 270 degrees
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- renumbered Q207 to Q201, Q208 to Q202, Q201 to Q203, Q202 to Q204, Q203 to Q205, Q204 to Q206, Q205 to Q207, Q206 to Q208, R211 to R201, R207 to R202, R201 to R203, R203 to R204, R212 to R205, R202 to R206, R204 to R207, R205 to R208, R206 to R209, R208 to R210, R209 to R211
Connections:
- J201 pad 1: /High Voltage Amplifier/FLOAT_COM -> /High Voltage Amplifier/100mA
- J201 pad 10: /High Voltage Amplifier/AMPIN -> +15V
- J201 pad 11: /High Voltage Amplifier/100mA -> /High Voltage Amplifier/FLOAT_COM
- J201 pad 12: /High Voltage Amplifier/100mA -> /High Voltage Amplifier/FLOAT_COM
- J201 pad 2: /High Voltage Amplifier/FLOAT_COM -> /High Voltage Amplifier/100mA
- J201 pad 3: +15V -> /High Voltage Amplifier/AMPIN
- J201 pad 4: +15V -> /High Voltage Amplifier/AMPIN
- J201 pad 5: GND -> -15V
- J201 pad 6: GND -> -15V
- J201 pad 7: -15V -> GND1
- J201 pad 8: -15V -> GND1
- J201 pad 9: /High Voltage Amplifier/AMPIN -> +15V
Routing:
- net /High Voltage Amplifier/FLOAT_COM: track 0.00 -> 175.7 mm, vias 0 -> 6
- net -15V: track 0.00 -> 138.7 mm, vias 0 -> 4
- net +15V: track 0.00 -> 136.4 mm, vias 0 -> 4
- net GNDHV: track 0.00 -> 116.7 mm, vias 0 -> 65
- net /High Voltage Amplifier/100mA: track 0.00 -> 96.3 mm, vias 0 -> 2
- net +15VF: track 0.00 -> 95.5 mm, vias 0 -> 1
- net -15VF: track 0.00 -> 94.6 mm, vias 0 -> 1
- net +HV: track 0.00 -> 72.8 mm, vias 0 -> 10
- net /High Voltage Amplifier/AMPIN: track 0.00 -> 66.7 mm
- net -HV: track 0.00 -> 61.2 mm, vias 0 -> 15
- net Net-(Q205-Pad1): track 0.00 -> 51.3 mm, vias 0 -> 3
- net +5V: track 0.00 -> 34.6 mm
- net Net-(C318-Pad1): track 0.00 -> 33.9 mm, vias 0 -> 1
- net VDD: track 0.00 -> 29.3 mm, vias 0 -> 3
- net Net-(C330-Pad2): track 0.00 -> 27.4 mm
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- added copper zone on B.Cu, net +24V
- added copper zone on F.Cu, net +24V
- added copper zone on In2.Cu, net +24V
- added copper zone on B.Cu, net +24V_HV
- added copper zone on F.Cu, net +24V_HV
- added copper zone on In2.Cu, net +24V_HV
- added copper zone on B.Cu, net +HV
- added copper zone on F.Cu, net +HV
- added copper zone on In2.Cu, net +HV
- added copper zone on B.Cu, net -HV
- added copper zone on F.Cu, net -HV
- added copper zone on In2.Cu, net -HV
- added copper zone on B.Cu, net GND
- added copper zone on F.Cu, net GND
- added copper zone on In1.Cu, net GND
- added copper zone on B.Cu, net GNDHV
- added copper zone on F.Cu, net GNDHV
- added copper zone on In1.Cu, net GNDHV
- added copper zone on F.Cu, net Net-(C301-Pad1)
- added copper zone on B.Cu, net Net-(C304-Pad1)
- added copper zone on F.Cu, net Net-(C304-Pad1)
- added copper zone on B.Cu, net Net-(C317-Pad1)
- added copper zone on F.Cu, net Net-(C317-Pad1)
- added copper zone on F.Cu, net Net-(C318-Pad1)
- added copper zone on B.Cu, net Net-(C331-Pad2)
- added copper zone on F.Cu, net Net-(C331-Pad2)
- added copper zone on B.Cu, net Net-(C344-Pad2)
- added copper zone on F.Cu, net Net-(C344-Pad2)
- added copper zone on B.Cu, net Net-(D301-Pad2)
- added copper zone on F.Cu, net Net-(D301-Pad2)
- added copper zone on F.Cu, net Net-(R301-Pad2)
- added copper zone on F.Cu, net Net-(R308-Pad2)
Other:
- net class Default: trace_width 0.25 -> 0.254; via_dia 0.8 -> 0.5; via_drill 0.4 -> 0.2
- rule via_min_drill: 0.3 -> 0.2

Commit message: PCB layout
Parts:
- moved J301 1.00 mm to (110.0, 133.0)
Routing:
- net +5V: track 34.6 -> 24.6 mm
- net +24V_HV: track 7.40 -> 0.00 mm
- net GNDHV: track 116.7 -> 109.9 mm, vias 65 -> 74
- net VDD: track 29.3 -> 25.6 mm
- net Net-(Q205-Pad1): track 51.3 -> 49.2 mm
- net Net-(C332-Pad2): track 17.9 -> 19.1 mm
- net /High Voltage Amplifier/100mA: track 96.3 -> 97.4 mm
- net /High Voltage Amplifier/FLOAT_COM: track 175.7 -> 174.8 mm
- net Net-(C330-Pad2): track 27.4 -> 26.6 mm

Commit message: Schematic and PCB update.
Parts:
- D201, D204: value BAV99 -> BAV99LT1

Commit message: PCB changes
Routing:
- net GNDHV: track 109.9 -> 146.0 mm, vias 74 -> 86

Commit message: PCB changes
Parts:
- moved H101 15.0 mm to (74.0, 135.0)
Changed lines of the file:
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@@
     (tags "mounting hole 3.2mm m3 din965")
     (attr virtual)
-    (fp_text reference H104 (at 0 -3.8) (layer F.SilkS)
+    (fp_text reference H104 (at 0 -3.8) (layer Dwgs.User)
       (effects (font (size 0.6 0.6) (thickness 0.12)))
     )
@@
     (tags "mounting hole 3.2mm m3 din965")
     (attr virtual)
-    (fp_text reference H103 (at 0 3.514) (layer F.SilkS)
+    (fp_text reference H103 (at 0 3.514) (layer Dwgs.User)
       (effects (font (size 0.6 0.6) (thickness 0.12)))
     )
@@
     (tags "mounting hole 3.2mm m3 din965")
     (attr virtual)
-    (fp_text reference H102 (at 0 3.514) (layer F.SilkS)
+    (fp_text reference H102 (at 0 3.514) (layer Dwgs.User)
       (effects (font (size 0.6 0.6) (thickness 0.12)))
     )
@@
   )
   (module MountingHole:MountingHole_3.2mm_M3_DIN965_Pad (layer F.Cu)
-    (at 89 135)
+    (at 74 135)
     (descr "Mounting Hole 3.2mm, M3, DIN965")
     (tags "mounting hole 3.2mm m3 din965")
     (attr virtual)
-    (fp_text reference H101 (at 0 -3.8) (layer F.SilkS)
+    (fp_text reference H101 (at 0 -3.8) (layer Dwgs.User)
       (effects (font (size 0.6 0.6) (thickness 0.12)))
     )
