File: HARDWARE/MODULE/HV_Power.sch (KiCad schematic (older format))
At the start: 88 parts, among them J301 Conn_02x04_Odd_Even, U301 LM317_TO-263, U302 LM337_TO263, U303 LT8330_S6, U304 LT8570_MS8E, U305 TEL10-2415, U306 L78L15_SO8, U307 SN6505BDBV, U308 L79L15_SO8

Commit message: Schematic design.
Parts:
- removed C344: 470p, Capacitor_SMD:C_0603_1608Metric_Pad1.08x0.95mm_HandSolder, symbol Device:C
- added C326: 470p, Capacitor_SMD:C_0603_1608Metric_Pad1.08x0.95mm_HandSolder, symbol Device:C
- J301: footprint (none) -> Connector_PinSocket_2.54mm:PinSocket_2x04_P2.54mm_Vertical
- L302: renamed from L301; value 7438335068 -> 74438335068; footprint (none) -> ETH1CSMU1:74438335068
- L304: renamed from L305; footprint (none) -> ETH1CSMU1:MSD7342
- U304: footprint (none) -> Package_SO:MSOP-8-1EP_3x3mm_P0.65mm_EP1.68x1.88mm_ThermalVias
- renumbered C302 to C301, C301 to C302, C306 to C305, C307 to C306, C308 to C307, C309 to C308, C305 to C309, C317 to C310, C336 to C311, C337 to C312, C316 to C313, C343 to C314, C310 to C315, C338 to C316, C311 to C317, C312 to C318, C313 to C319, C314 to C320, C315 to C321, C339 to C322, C340 to C323, C341 to C324, C342 to C325, C345 to C327, C346 to C328, C321 to C329, C323 to C330, C318 to C331, C324 to C332, C325 to C333, C326 to C334, C327 to C335, C319 to C336, C320 to C337, C328 to C338, C329 to C339, C330 to C340, C331 to C341, C332 to C342, C333 to C343, C322 to C344, C334 to C345, C335 to C346, L302 to L301, L306 to L303, L303 to L305, L304 to L306, R303 to R302, R304 to R303, R307 to R304, R309 to R305, R311 to R306, R305 to R307, R302 to R308, R306 to R309, R308 to R310, R310 to R311, U303 to U302, U302 to U303, U306 to U305, U305 to U306
Connections:
- net GNDHV: now also C326.2
- net at R311.1, U304.2 (VC): now also C326.1
Other:
- moved on the sheet: C301, C302, C303, C304, C305, C306, C307, C308, C309, C310, C311, C312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

Commit message: PCB and schematic design.
Parts:
- removed J301: Conn_02x04_Odd_Even, Connector_PinSocket_2.54mm:PinSocket_2x04_P2.54mm_Vertical, symbol Connector_Generic:Conn_02x04_Odd_Even
- added J301: Conn_02x06_Odd_Even, Connector_PinSocket_2.54mm:PinSocket_2x06_P2.54mm_Vertical, symbol Connector_Generic:Conn_02x06_Odd_Even
- C307, C308, C320: footprint Capacitor_SMD:C_1210_3225Metric_Pad1.33x2.70mm_HandSolder -> Capacitor_SMD:C_2220_5650Metric_Pad1.97x5.40mm_HandSolder
Connections:
- net +24V: now also J301.1 (Pin_1), J301.2 (Pin_2), J301.3 (Pin_3), J301.4 (Pin_4)
- net +5V: now also J301.7 (Pin_7), J301.8 (Pin_8)
- net GND: now also J301.10 (Pin_10), J301.11 (Pin_11), J301.12 (Pin_12), J301.9 (Pin_9)
Changed lines of the file:
@@
 L power:+24V #PWR0324
 U 1 1 6068368D
-P 4800 10500
-F 0 "#PWR0324" H 4800 10350 50  0001 C CNN
-F 1 "+24V" V 4800 10650 50  0000 L CNN
-F 2 "" H 4800 10500 50  0001 C CNN
-F 3 "" H 4800 10500 50  0001 C CNN
-	1    4800 10500
+P 4500 10300
+F 0 "#PWR0324" H 4500 10150 50  0001 C CNN
+F 1 "+24V" V 4500 10450 50  0000 L CNN
+F 2 "" H 4500 10300 50  0001 C CNN
+F 3 "" H 4500 10300 50  0001 C CNN
+	1    4500 10300
 	0    1    1    0
 $EndComp
@@
 L power:+24V #PWR0323
 U 1 1 60683E2D
-P 4300 10500
-F 0 "#PWR0323" H 4300 10350 50  0001 C CNN
-F 1 "+24V" V 4300 10650 50  0000 L CNN
-F 2 "" H 4300 10500 50  0001 C CNN
-F 3 "" H 4300 10500 50  0001 C CNN
-	1    4300 10500
+P 4000 10300
+F 0 "#PWR0323" H 4000 10150 50  0001 C CNN
+F 1 "+24V" V 4000 10450 50  0000 L CNN
+F 2 "" H 4000 10300 50  0001 C CNN
+F 3 "" H 4000 10300 50  0001 C CNN
+	1    4000 10300
 	0    -1   -1   0
 $EndComp
-NoConn ~ 4800 10600
-NoConn ~ 4300 10600
 $Comp
 L power:+5V #PWR?
 U 1 1 606AB97E
-P 4800 10700
+P 4500 10600
 AR Path="/6067C9FD/606AB97E" Ref="#PWR?"  Part="1"
 AR Path="/60626568/606AB97E" Ref="#PWR?"  Part="1"
 AR Path="/6063ACFE/606AB97E" Ref="#PWR0327"  Part="1"
-F 0 "#PWR0327" H 4800 10550 50  0001 C CNN
-F 1 "+5V" V 4800 10900 50  0000 C CNN
-F 2 "" H 4800 10700 50  0001 C CNN
-F 3 "" H 4800 10700 50  0001 C CNN
-	1    4800 10700
+F 0 "#PWR0327" H 4500 10450 50  0001 C CNN
+F 1 "+5V" V 4500 10800 50  0000 C CNN
+F 2 "" H 4500 10600 50  0001 C CNN
+F 3 "" H 4500 10600 50  0001 C CNN
+	1    4500 10600
 	0    1    1    0
 $EndComp
@@
 L power:+5V #PWR?
 U 1 1 606ACC3F
-P 4300 10700
+P 4000 10600
 AR Path="/6067C9FD/606ACC3F" Ref="#PWR?"  Part="1"
 AR Path="/60626568/606ACC3F" Ref="#PWR?"  Part="1"
 AR Path="/6063ACFE/606ACC3F" Ref="#PWR0326"  Part="1"
-F 0 "#PWR0326" H 4300 10550 50  0001 C CNN
-F 1 "+5V" V 4300 10900 50  0000 C CNN
-F 2 "" H 4300 10700 50  0001 C CNN
-F 3 "" H 4300 10700 50  0001 C CNN
-	1    4300 10700
+F 0 "#PWR0326" H 4000 10450 50  0001 C CNN
+F 1 "+5V" V 4000 10800 50  0000 C CNN
+F 2 "" H 4000 10600 50  0001 C CNN
+F 3 "" H 4000 10600 50  0001 C CNN
+	1    4000 10600
 	0    -1   -1   0
-$EndComp
-$Comp
-L Connector_Generic:Conn_02x04_Odd_Even J301
-U 1 1 606AD9D0
-P 4500 10600
-F 0 "J301" H 4550 10917 50  0000 C CNN
-F 1 "Conn_02x04_Odd_Even" H 4550 10826 50  0000 C CNN
-F 2 "Connector_PinSocket_2.54mm:PinSocket_2x04_P2.54mm_Vertical" H 4500 10600 50  0001 C CNN
-F 3 "~" H 4500 10600 50  0001 C CNN
-	1    4500 10600
-	1    0    0    -1
 $EndComp
 $Comp
 L power:GND #PWR?
 U 1 1 606AE5C7
-P 4800 10800
+P 4500 10800
 AR Path="/6067C9FD/606AE5C7" Ref="#PWR?"  Part="1"
 AR Path="/60626568/606AE5C7" Ref="#PWR?"  Part="1"
 AR Path="/6063ACFE/606AE5C7" Ref="#PWR0329"  Part="1"
-F 0 "#PWR0329" H 4800 10550 50  0001 C CNN
-F 1 "GND" V 4800 10600 50  0000 C CNN
-F 2 "" H 4800 10800 50  0001 C CNN
-F 3 "" H 4800 10800 50  0001 C CNN
-	1    4800 10800
+F 0 "#PWR0329" H 4500 10550 50  0001 C CNN
+F 1 "GND" V 4500 10600 50  0000 C CNN
+F 2 "" H 4500 10800 50  0001 C CNN
+F 3 "" H 4500 10800 50  0001 C CNN
+	1    4500 10800
 	0    -1   -1   0
 $EndComp
@@
 L power:GND #PWR?
 U 1 1 606AF089
-P 4300 10800
+P 4000 10800
 AR Path="/6067C9FD/606AF089" Ref="#PWR?"  Part="1"
 AR Path="/60626568/606AF089" Ref="#PWR?"  Part="1"
 AR Path="/6063ACFE/606AF089" Ref="#PWR0328"  Part="1"
-F 0 "#PWR0328" H 4300 10550 50  0001 C CNN
-F 1 "GND" V 4300 10600 50  0000 C CNN
-F 2 "" H 4300 10800 50  0001 C CNN
-F 3 "" H 4300 10800 50  0001 C CNN
-	1    4300 10800
+F 0 "#PWR0328" H 4000 10550 50  0001 C CNN
+F 1 "GND" V 4000 10600 50  0000 C CNN
+F 2 "" H 4000 10800 50  0001 C CNN
+F 3 "" H 4000 10800 50  0001 C CNN
+	1    4000 10800
 	0    1    1    0
 $EndComp
@@
 F 0 "C307" H 9815 1796 50  0000 L CNN
 F 1 "4u7/100V" H 9815 1705 50  0000 L CNN
-F 2 "Capacitor_SMD:C_1210_3225Metric_Pad1.33x2.70mm_HandSolder" H 9738 1600 50  0001 C CNN
+F 2 "Capacitor_SMD:C_2220_5650Metric_Pad1.97x5.40mm_HandSolder" H 9738 1600 50  0001 C CNN
 F 3 "~" H 9700 1750 50  0001 C CNN
 	1    9700 1750
@@
 F 0 "C308" H 10465 1796 50  0000 L CNN
 F 1 "22u/100V" H 10465 1705 50  0000 L CNN
-F 2 "Capacitor_SMD:C_1210_3225Metric_Pad1.33x2.70mm_HandSolder" H 10388 1600 50  0001 C CNN
+F 2 "Capacitor_SMD:C_2220_5650Metric_Pad1.97x5.40mm_HandSolder" H 10388 1600 50  0001 C CNN
 F 3 "~" H 10350 1750 50  0001 C CNN
 	1    10350 1750
@@
 F 0 "C320" H 9765 4296 50  0000 L CNN
 F 1 "4u7/100V" H 9765 4205 50  0000 L CNN
-F 2 "Capacitor_SMD:C_1210_3225Metric_Pad1.33x2.70mm_HandSolder" H 9688 4100 50  0001 C CNN
+F 2 "Capacitor_SMD:C_2220_5650Metric_Pad1.97x5.40mm_HandSolder" H 9688 4100 50  0001 C CNN
 F 3 "~" H 9650 4250 50  0001 C CNN
 	1    9650 4250
@@
 	1    0    0    -1
 $EndComp
+$Comp
+L Connector_Generic:Conn_02x06_Odd_Even J301
+U 1 1 6063FBDA
+P 4200 10500
+F 0 "J301" H 4250 10917 50  0000 C CNN
+F 1 "Conn_02x06_Odd_Even" H 4250 10826 50  0000 C CNN
+F 2 "Connector_PinSocket_2.54mm:PinSocket_2x06_P2.54mm_Vertical" H 4200 10500 50  0001 C CNN
+F 3 "~" H 4200 10500 50  0001 C CNN
+	1    4200 10500
+	1    0    0    -1
+$EndComp
+$Comp
+L power:+24V #PWR0101
+U 1 1 606426C9
+P 4000 10400
+F 0 "#PWR0101" H 4000 10250 50  0001 C CNN
+F 1 "+24V" V 4000 10550 50  0000 L CNN
+F 2 "" H 4000 10400 50  0001 C CNN
+F 3 "" H 4000 10400 50  0001 C CNN
+	1    4000 10400
+	0    -1   -1   0
+$EndComp
+$Comp
+L power:+24V #PWR0102
+U 1 1 606429BA
+P 4500 10400
+F 0 "#PWR0102" H 4500 10250 50  0001 C CNN
+F 1 "+24V" V 4500 10550 50  0000 L CNN
+F 2 "" H 4500 10400 50  0001 C CNN
+F 3 "" H 4500 10400 50  0001 C CNN
+	1    4500 10400
+	0    1    1    0
+$EndComp
+NoConn ~ 4000 10500
+NoConn ~ 4500 10500
+$Comp
+L power:GND #PWR?
+U 1 1 6067E7C6
+P 4000 10700
+AR Path="/6067C9FD/6067E7C6" Ref="#PWR?"  Part="1"
+AR Path="/60626568/6067E7C6" Ref="#PWR?"  Part="1"
+AR Path="/6063ACFE/6067E7C6" Ref="#PWR0103"  Part="1"
+F 0 "#PWR0103" H 4000 10450 50  0001 C CNN
+F 1 "GND" V 4000 10500 50  0000 C CNN
+F 2 "" H 4000 10700 50  0001 C CNN
+F 3 "" H 4000 10700 50  0001 C CNN
+	1    4000 10700
+	0    1    1    0
+$EndComp
+$Comp
+L power:GND #PWR?
+U 1 1 6067EA6C
+P 4500 10700
+AR Path="/6067C9FD/6067EA6C" Ref="#PWR?"  Part="1"
+AR Path="/60626568/6067EA6C" Ref="#PWR?"  Part="1"
+AR Path="/6063ACFE/6067EA6C" Ref="#PWR0104"  Part="1"
+F 0 "#PWR0104" H 4500 10450 50  0001 C CNN
+F 1 "GND" V 4500 10500 50  0000 C CNN
+F 2 "" H 4500 10700 50  0001 C CNN
+F 3 "" H 4500 10700 50  0001 C CNN
+	1    4500 10700
+	0    -1   -1   0
+$EndComp
 $EndSCHEMATC

Commit message: PCB and schematic
Parts:
- added J302: Conn_02x02_Odd_Even, Connector_PinSocket_2.54mm:PinSocket_2x02_P2.54mm_Vertical, symbol Connector_Generic:Conn_02x02_Odd_Even
Connections:
- net +15VF: now also J302.4 (Pin_4)
- net -15VF: now also J302.2 (Pin_2)
- net GNDHV: now also J302.1 (Pin_1), J302.3 (Pin_3)
Changed lines of the file:
@@
 	0    -1   -1   0
 $EndComp
+$Comp
+L Connector_Generic:Conn_02x02_Odd_Even J302
+U 1 1 6071ED7D
+P 5100 10600
+F 0 "J302" V 5196 10412 50  0000 R CNN
+F 1 "Conn_02x02_Odd_Even" V 5105 10412 50  0000 R CNN
+F 2 "Connector_PinSocket_2.54mm:PinSocket_2x02_P2.54mm_Vertical" H 5100 10600 50  0001 C CNN
+F 3 "~" H 5100 10600 50  0001 C CNN
+	1    5100 10600
+	0    -1   -1   0
+$EndComp
+$Comp
+L ETH1CSMU1:GNDHV #PWR0337
+U 1 1 60722D34
+P 5200 10900
+F 0 "#PWR0337" H 5200 10650 50  0001 C CNN
+F 1 "GNDHV" H 5205 10727 50  0000 C CNN
+F 2 "" H 5200 10900 50  0001 C CNN
+F 3 "" H 5200 10900 50  0001 C CNN
+	1    5200 10900
+	1    0    0    -1
+$EndComp
+Wire Wire Line
+	5200 10800 5200 10850
+Wire Wire Line
+	5200 10850 5100 10850
+Wire Wire Line
+	5100 10850 5100 10800
+Wire Wire Line
+	5200 10900 5200 10850
+Connection ~ 5200 10850
+$Comp
+L ETH1CSMU1:-15VF #PWR0335
+U 1 1 6076485E
+P 5100 10300
+F 0 "#PWR0335" H 5100 10150 50  0001 C CNN
+F 1 "-15VF" V 5100 10450 50  0000 L CNN
+F 2 "" H 5100 10300 50  0001 C CNN
+F 3 "" H 5100 10300 50  0001 C CNN
+	1    5100 10300
+	1    0    0    -1
+$EndComp
+$Comp
+L ETH1CSMU1:+15VF #PWR0336
+U 1 1 60769C55
+P 5200 10300
+F 0 "#PWR0336" H 5200 10150 50  0001 C CNN
+F 1 "+15VF" V 5200 10450 50  0000 L CNN
+F 2 "" H 5200 10300 50  0001 C CNN
+F 3 "" H 5200 10300 50  0001 C CNN
+	1    5200 10300
+	1    0    0    -1
+$EndComp
 $EndSCHEMATC

Commit message: PCB layout
Parts:
- removed J302: Conn_02x02_Odd_Even, Connector_PinSocket_2.54mm:PinSocket_2x02_P2.54mm_Vertical, symbol Connector_Generic:Conn_02x02_Odd_Even
- C305, C306: value 4u7/100V -> 4u7/50V; footprint Capacitor_SMD:C_1210_3225Metric_Pad1.33x2.70mm_HandSolder -> Capacitor_SMD:C_1206_3216Metric_Pad1.33x1.80mm_HandSolder
- C326: value 470p -> 47p
Other:
- moved on the sheet: C320, C321, C327

Commit message: Created active BOM list with Kicad plugin. Created first code for MCU1 and MCU2.
Parts:
- R309: value 481k -> 487k
Changed lines of the file:
@@
 P 7250 4250
 F 0 "R309" V 7043 4250 50  0000 C CNN
-F 1 "481k" V 7134 4250 50  0000 C CNN
+F 1 "487k" V 7134 4250 50  0000 C CNN
 F 2 "Resistor_SMD:R_0603_1608Metric_Pad0.98x0.95mm_HandSolder" V 7180 4250 50  0001 C CNN
 F 3 "~" H 7250 4250 50  0001 C CNN
